File: Input_PP.kicad_sch (KiCad schematic)
At the start: 19 parts, among them IC1 LM74502HDDFR, Q1 PSMN8R5-40MSDX

Commit message: 2nd
Parts:
- R13: value 9k -> 10k
- R28: value 135k -> 200k
Other:
- note added: "Overvoltage Protection: 29.03V Vovr = (R2 * Vov)/(R1 + R2) Vov = Vovr * (R1 + R2) / R2 18.125 = 1.25 * (200k + 10k) / 10k Vovr = 1.25V (datasheet)"
- note removed: "Overvoltage Protection: 29.03V Vovr = (R2 * Vov)/(R1 + R2) Vov = Vovr * (R1 + R2) / R2 20 = 1.25 * (200k + 9k) / 9k Vovr = 1.25V"
