File: Output_PP.kicad_sch (KiCad schematic)
At the start: 19 parts, among them IC3 LM74502HDDFR, Q2 PSMN8R5-40MSDX

Commit message: 2nd
Parts:
- R2: value 200k -> 100k
- R3: value 9k -> 4.3k
Other:
- note added: "Overvoltage Protection: 29.03V Vovr = (R2 * Vov)/(R1 + R2) Vov = Vovr * (R1 + R2) / R2 30.319 = 1.25 ((100k+4.3k)/4.3k)"
- note removed: "Overvoltage Protection: 29.03V Vovr = (R2 * Vov)/(R1 + R2) Vov = Vovr * (R1 + R2) / R2 29.03 = 1.25 * (200k + 9k) / 9k"
Changed lines of the file:
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@@
 	(generator_version "9.0")
 	(paper "A4")
-	(text "Overvoltage Protection: 29.03V\nVovr = (R2 * Vov)/(R1 + R2)\nVov = Vovr * (R1 + R2) / R2\n29.03 = 1.25 * (200k + 9k) / 9k"
-		(exclude_from_sim no)
-		(at 166.37 80.01 0)
+	(text "Overvoltage Protection: 29.03V\nVovr = (R2 * Vov)/(R1 + R2)\nVov = Vovr * (R1 + R2) / R2\n30.319 = 1.25 ((100k+4.3k)/4.3k)"
+		(exclude_from_sim no)
+		(at 146.812 97.282 0)
 		(effects
 			(font
@@
 		(fields_autoplaced yes)
 		(property "Reference" "R2"
-			(at 132.715 74.9299 0)
+			(at 133.35 74.9299 0)
 			(effects
 				(font
@@
 			)
 		)
-		(property "Value" "200k"
-			(at 132.715 77.4699 0)
+		(property "Value" "100k"
+			(at 133.35 77.4699 0)
 			(effects
 				(font
@@
 			)
 		)
-		(property "Value" "9k"
+		(property "Value" "4.3k"
 			(at 140.97 78.74 90)
 			(effects
