File: PS-ChargerInterfacePCB.kicad_sch (KiCad schematic)
At the start: 0 parts

Commit message: Initial PCB files for RevA
Parts:
- added BZ1: Buzzer, symbol Device:Buzzer
- added C19, C26, C31: 4u7, symbol Device:C
- added C22, C23, C24, C25, C27, C28, C29, C30, C32, C33: 100n, symbol Device:C
- added D1, D2, D3, D4: LED, LED_SMD:LED_0402_1005Metric, symbol Device:LED
- added DS1: EA_DIP205B-4NLW, EADIP205B4NLW, symbol EA DIP205B-4NLW:EA_DIP205B-4NLW
- added J2: LV_Elcon_Connector, symbol Connector:Conn_01x04_Pin
- added J3: ~, symbol utsvt_connectors2:LSOM_DaughterConn
- added J4: PeripheralCAN, UTSVT_Connectors:Molex_Nano-Fit_105309-xx04_1x04_P2.50mm_Vertical, symbol utsvt_connectors2:PeripheralCANConnector
- added J5: EStop_Conn, symbol Connector:Conn_01x02_Pin
- added K1: Fujitsu_FTR-LYCA005x, Relay_THT:Relay_SPDT_Fujitsu_FTR-LYCA005x_FormC_Vertical, symbol Relay:Fujitsu_FTR-LYCA005x
- added R14, R6: 10k, symbol Device:R
- added R15, R16, R17: 11k, Resistor_SMD:R_0402_1005Metric, symbol Device:R
- added R19: 10k, Resistor_SMD:R_0402_1005Metric, symbol Device:R
- added R5: 220R, Resistor_SMD:R_0402_1005Metric, symbol Device:R
Connections:
- new net: D2.2 (A), J3.33 (ADC1_IN3)
- new net: D3.2 (A), J3.40 (ADC1_IN11)
- new net: D4.2 (A), J3.45 (ADC1_IN12)
- new net: J5.1 (Pin_1), K1.A2
- new net: D2.1 (K), R15.2
- new net: D3.1 (K), R16.2
- new net: DS1.3 (VEE), R14.2, R6.1
- new net: D1.2 (A), DS1.17 (A)
- new net +3.3V: BZ1.1 (+), C19.1, C22.1, C23.1, C24.1, C25.1, C31.1, C32.1, DS1.2 (VDD), J3.1 (+3.3V), J3.2 (+3.3V), J3.3 (+3.3V), J3.4 (+3.3V), R19.1, R6.2
- new net 12V_IN: J2.1 (Pin_1), K1.11, K1.12
- new net 24V_OUT: C26.1, C27.1, C28.1, C29.1, C30.1, J3.21 (24VExt), J3.22 (24VExt), J3.23 (24VExt), J3.24 (24VExt), J4.1 (24V)
- new net CarCAN_H: J3.32 (CarCAN_L), J4.3 (CAN_H)
- new net CarCAN_L: J3.30 (CarCAN_H), J4.4 (CAN_L)
- new net Display_MISO: DS1.7 (D0_(SOD)), J3.44 (SPI2_MISO)
- new net Display_MOSI: DS1.5 (R/W_(SID)), J3.42 (SPI2_MOSI)
- new net Display_NSS: DS1.4 (RS_(CS)), J3.48 (SPI2_NSS)
- new net Display_SCLK: DS1.6 (E_(SCLK)), J3.46 (SPI2_SCK)
- new net Elcon_CAN_H: J2.2 (Pin_2), J3.8 (IntCAN_L)
- new net Elcon_CAN_L: J2.3 (Pin_3), J3.6 (IntCAN_H)
- new net GND: BZ1.2 (-), C19.2, C22.2, C23.2, C24.2, C25.2, C26.2, C27.2, C28.2, C29.2, C30.2, C31.2, C32.2, C33.2, DS1.1 (VSS), DS1.18 (C), J2.4 (Pin_4), J3.25 (GND), J3.26 (GND), J3.27 (GND), J3.28 (GND), J3.29 (GND), J4.2 (GND), J5.2 (Pin_2), K1.14, R14.1, R15.1, R16.1, R17.1, R5.1
- new net LED_A: D1.1 (K), D4.1 (K), R17.2, R5.2
- new net RES: C33.1, DS1.16 (RES), R19.2
- no-connect marks 0 -> 32
Other:
- added sheet 12V-24V Boost Converter (12V-24VBoostConverter.kicad_sch)
- added sheet Input_PP (Input_PP.kicad_sch)
- added sheet Output_PP (Output_PP.kicad_sch)
- note added: "BPS Connector"
- note added: "Decoupling Capacitors"
- note added: "EStop"
- note added: "LSOM"
- note added: "SPI Display"

Commit message: 2nd
Parts:
- removed BZ1: Buzzer, symbol Device:Buzzer
- removed C31: 4u7, symbol Device:C
- removed C32, C33: 100n, symbol Device:C
- removed D1, D2, D3, D4: LED, LED_SMD:LED_0402_1005Metric, symbol Device:LED
- removed DS1: EA_DIP205B-4NLW, EADIP205B4NLW, symbol EA DIP205B-4NLW:EA_DIP205B-4NLW
- removed J5: EStop_Conn, symbol Connector:Conn_01x02_Pin
- removed K1: Fujitsu_FTR-LYCA005x, Relay_THT:Relay_SPDT_Fujitsu_FTR-LYCA005x_FormC_Vertical, symbol Relay:Fujitsu_FTR-LYCA005x
- removed R14, R6: 10k, symbol Device:R
- removed R15, R16, R17: 11k, Resistor_SMD:R_0402_1005Metric, symbol Device:R
- removed R19: 10k, Resistor_SMD:R_0402_1005Metric, symbol Device:R
- removed R5: 220R, Resistor_SMD:R_0402_1005Metric, symbol Device:R
- added C39: 4u7, symbol Device:C
- added C40: 100n, symbol Device:C
- added TP1, TP11, TP12, TP13, TP2, TP3, TP4, TP7, TP8, TP9: TestPoint, symbol Connector:TestPoint
Connections:
- net +3.3V: now also TP2.1
- net 12V_IN: now also TP4.1
- net 24V_IN: now also TP8.1
- net 24V_OUT: now also TP1.1
- net CarCAN_H: now also J3.30 (CarCAN_H), TP12.1; no longer J3.32 (CarCAN_L)
- net CarCAN_L: now also J3.32 (CarCAN_L), TP13.1; no longer J3.30 (CarCAN_H)
- net Elcon_CAN_H: now also J3.6 (IntCAN_H), TP11.1; no longer J3.8 (IntCAN_L)
- net Elcon_CAN_L: now also J3.8 (IntCAN_L), TP9.1; no longer J3.6 (IntCAN_H)
- net GND: now also C39.2, C40.2
- net LED_HV: now reaches J3.33 (ADC1_IN3)
- net LED_FAULT: now reaches J3.35 (ADC1_IN2)
- net +3.3VA: now reaches J3.37 (+3.3VA)
- net +3.3VA: now also C39.1, C40.1, TP3.1
- net GNDA: now reaches J3.38 (GNDA)
- net LED_CHARGE: now reaches J3.39 (ADC1_IN1)
- new net 12V_IN_BC: TP7.1
- no-connect marks 32 -> 18
Other:
- added sheet EStop (Estop.kicad_sch)
- added sheet LEDIndicator (LEDIndicator.kicad_sch)
- added sheet SPI_display (SPI_display.kicad_sch)
- added sheet SpeakerAmp (SpeakerAmp.kicad_sch)
- sheet 12V-24V Boost Converter ports: added none; removed 12V_IN, 24V_OUT
- note added: "Change Amp to PWM"
- note added: "TO DOS: - new buzzer/speaker - estop design (Estop1 IN and ESTOP 1 OUT are in series) - pwm speaker tone"
- note added: "Test Points"
- note added: "Wire Estop with rest of circuit"
- note removed: "Decoupling Capacitors"
- note removed: "EStop"
- note removed: "LSOM"
- note removed: "SPI Display"
- moved on the sheet: C19, C22, C23, C24, C25, C26, C27, C28, C29, C30, J4

Commit message: rev3
Parts:
- removed C19, C26, C39: 4u7, symbol Device:C
- removed C22, C23, C24, C25, C27, C28, C29, C30, C40: 100n, symbol Device:C
- added J5: Estop 2, symbol Connector_Generic:Conn_01x02
- added J6: Estop 3, symbol Connector_Generic:Conn_01x02
- added R26: 0, symbol Device:R_Small_US
- added TP14: TestPoint, symbol Connector:TestPoint
Connections:
- net +3.3VA: no longer J3.37 (+3.3VA)
- net 24V_OUT: no longer J3.21 (24VExt), J3.22 (24VExt), J3.23 (24VExt), J3.24 (24VExt)
- net GND: now also TP14.1
- net LED_HEART: now reaches J3.40 (ADC1_IN11)
- net Display_RES: now reaches J3.41 (ADC1_IN8)
- net BuzzPWM: now reaches J3.10 (ADC1_IN7)
- net 12V_IN_BC renamed 12V_OUT
- net 24V_IN renamed 24V
- net GNDA: no longer names the net of J3.38 (GNDA)
- new net +24V: J3.21 (24VExt), J3.22 (24VExt), J3.23 (24VExt), J3.24 (24VExt)
- new net EStop2: J5.1 (Pin_1), J5.2 (Pin_2), R26.1, R26.2
- new net EStopConn: J6.1 (Pin_1), J6.2 (Pin_2)
- no-connect marks 18 -> 17
Other:
- removed sheet EStop
- removed sheet SpeakerAmp
- added sheet Buzzer (Buzzer.kicad_sch)
- sheet 12V-24V Boost Converter: file 12V-24VBoostConverter.kicad_sch -> External Sch/12V-24VBoostConverter.kicad_sch
- sheet 12V-24V Boost Converter ports: added 12V_IN_BC, 24V_OUT_BC; removed none
- sheet Input_PP: file Input_PP.kicad_sch -> External Sch/Input_PP.kicad_sch
- sheet Input_PP ports: added 12V_IN, 12V_OUT; removed none
- sheet LEDIndicator ports: added LED_CHARGE, LED_FAULT, LED_HEART, LED_HV; removed none
- sheet Output_PP ports: added 24V_IN, 24V_OUT; removed none
- sheet SPI_display ports: added Display_MISO, Display_MOSI, Display_NSS, Display_RES, Display_SCLK; removed none
- note added: "EStop"
- note added: "Notes: - PWM to sirens - MOSFET - 24V speaker"
- note removed: "Change Amp to PWM"
- note removed: "Wire Estop with rest of circuit"
- moved on the sheet: TP2, TP3

Commit message: small rev3 changes
Other:
- sheet 12V-24V Boost Converter: file External Sch/12V-24VBoostConverter.kicad_sch -> 12V-24VBoostConverter.kicad_sch
- sheet Input_PP: file External Sch/Input_PP.kicad_sch -> Input_PP.kicad_sch
- note removed: "Notes: - PWM to sirens - MOSFET - 24V speaker"
- note removed: "TO DOS: - new buzzer/speaker - estop design (Estop1 IN and ESTOP 1 OUT are in series) - pwm speaker tone"
Changed lines of the file:
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@@
 		)
 	)
-	(text "Notes:\n- PWM to sirens\n- MOSFET\n- 24V speaker"
-		(exclude_from_sim no)
-		(at 82.55 191.262 0)
-		(effects
-			(font
-				(size 1.27 1.27)
-			)
-			(justify left)
-		)
-	)
 	(text "BPS Connector"
 		(exclude_from_sim no)
@@
 		)
 	)
-	(text "TO DOS:\n- new buzzer/speaker\n- estop design (Estop1 IN and ESTOP 1 OUT are in series)\n- pwm speaker tone\n"
-		(exclude_from_sim no)
-		(at 14.224 190.246 0)
-		(effects
-			(font
-				(size 1.27 1.27)
-			)
-			(justify left)
-		)
-	)
 	(text "EStop\n"
 		(exclude_from_sim no)
@@
 	(wire
 		(pts
-			(xy 194.31 73.66) (xy 201.93 73.66)
+			(xy 194.31 81.28) (xy 201.93 81.28)
 		)
 		(stroke
@@
 	)
 	(label "BuzzPWM"
-		(at 194.31 73.66 0)
+		(at 194.31 81.28 0)
 		(effects
 			(font
@@
 			)
 		)
-		(property "Sheetfile" "External Sch/Input_PP.kicad_sch"
+		(property "Sheetfile" "Input_PP.kicad_sch"
 			(at 62.23 49.022 0)
 			(effects
@@
 	)
 	(sheet
-		(at 201.93 68.58)
+		(at 201.93 76.2)
 		(size 20.32 19.05)
 		(exclude_from_sim no)
@@
 		)
 		(property "Sheetname" "Buzzer"
-			(at 201.93 67.8684 0)
+			(at 201.93 75.4884 0)
 			(effects
 				(font
@@
 		)
 		(property "Sheetfile" "Buzzer.kicad_sch"
-			(at 201.93 88.2146 0)
+			(at 201.93 95.8346 0)
 			(effects
 				(font
@@
 		)
 		(pin "BuzzPWM" input
-			(at 201.93 73.66 180)
+			(at 201.93 81.28 180)
 			(effects
 				(font
@@
 			)
 		)
-		(property "Sheetfile" "External Sch/12V-24VBoostConverter.kicad_sch"
+		(property "Sheetfile" "12V-24VBoostConverter.kicad_sch"
 			(at 106.934 49.022 0)
 			(effects

Commit message: revA4
Parts:
- removed R26: 0, symbol Device:R_Small_US
- added K2: Relay_SPST-NC, symbol Relay:Relay_SPST-NC
- added R14: 100k, Resistor_SMD:R_0603_1608Metric, symbol Device:R_US
- added R19: 47k, Resistor_SMD:R_0603_1608Metric, symbol Device:R_US
- added R2: 0, symbol Device:R_US
- added R20, R25: 4.3k, Resistor_SMD:R_0603_1608Metric, symbol Device:R_US
- added TP10, TP15, TP16, TP17, TP5, TP6: TestPoint, symbol Connector:TestPoint
- added Z5, Z6: SMAF4751A-TP, UTSVT_Passives:SODFL5026X125N, symbol UTSVT_Power:SMAF4749A-TP
- added Z7, Z8: SMAF4744A, UTSVT_Passives:SODFL5026X125N, symbol UTSVT_Power:SMAF4749A-TP
- J4: value PeripheralCAN -> BPSConn
Connections:
- net 12V_OUT is gone; now on net Display_RES: TP7.1
- net 24V is gone; now on net Display_MOSI: TP8.1
- net +24V: now also J6.1 (Pin_1), TP4.1, K2.11
- net 12V_IN: now also R19.1, Z8.1 (K); no longer TP4.1
- net 24V_OUT: now also R14.1, Z6.1 (K); no longer TP1.1
- net Display_MISO: now also TP1.1
- net Display_NSS: now also TP6.1
- net Display_SCLK: now also TP5.1
- net GND: now also K2.A2, R20.2, R25.2, Z5.2 (A), Z6.2 (A), Z7.2 (A), Z8.2 (A)
- net LED_CHARGE: now also TP16.1
- net LED_FAULT: now also TP15.1
- net LED_HEART: now also TP17.1
- net LED_HV: now also TP10.1
- net +3.3VA renamed +12V
- net +12V: now also K2.12
- net EStop2 renamed EStop2_OUT
- net EStop2_OUT: now also R2.1; no longer J5.2 (Pin_2)
- net EStopConn renamed EStop3_RET
- net EStop3_RET: now also K2.A1; no longer J6.1 (Pin_1)
- new net EStop2_RET: J5.2 (Pin_2), R2.2
- new net Power12V/OV: R19.2, R20.1
- new net Power24V/OV: R14.2, R25.1
- new net RPP_EN12: Z7.1 (K)
- new net RPP_EN24: Z5.1 (K)
Other:
- removed sheet Input_PP
- removed sheet Output_PP
- added sheet Power12V (Power.kicad_sch)
- added sheet Power24V (Power.kicad_sch)
- note added: "Boost Converter"
- note added: "Bzz Bzz"
- note added: "Connectors"
- note added: "Display"
- note added: "LEDs"
- note added: "LSOM"
- note added: "Power Protection"
- note removed: "BPS Connector"
- moved on the sheet: J2, J4, J5, J6, TP1, TP11, TP12, TP13, TP14, TP2, TP3, TP4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

Commit message: RevA4 small changes
Connections:
- no-connect marks 17 -> 21
Changed lines of the file:
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@@
 	)
 	(junction
+		(at 83.82 44.45)
+		(diameter 0)
+		(color 0 0 0 0)
+	)
+	(junction
 		(at 48.26 100.33)
 		(diameter 0)
@@
 		(color 0 0 0 0)
 	)
+	(junction
+		(at 48.26 93.98)
+		(diameter 0)
+		(color 0 0 0 0)
+	)
 	(no_connect
 		(at 152.4 86.36)
@@
 	)
 	(no_connect
+		(at 95.25 106.68)
+	)
+	(no_connect
 		(at 114.3 72.39)
 	)
 	(no_connect
+		(at 95.25 114.3)
+	)
+	(no_connect
 		(at 114.3 93.98)
 	)
@@
 	)
 	(no_connect
+		(at 95.25 109.22)
+	)
+	(no_connect
 		(at 95.25 80.01)
 	)
@@
 	)
 	(no_connect
+		(at 95.25 111.76)
+	)
+	(no_connect
 		(at 152.4 97.79)
 	)
@@
 	(wire
 		(pts
-			(xy 48.26 92.71) (xy 48.26 95.25)
+			(xy 48.26 92.71) (xy 48.26 93.98)
 		)
 		(stroke
@@
 	(wire
 		(pts
+			(xy 48.26 93.98) (xy 48.26 95.25)
+		)
+		(stroke
+			(width 0)
+			(type default)
+		)
+	)
+	(wire
+		(pts
 			(xy 274.32 27.94) (xy 274.32 30.48)
 		)
@@
 	(wire
 		(pts
+			(xy 83.82 44.45) (xy 90.17 44.45)
+		)
+		(stroke
+			(width 0)
+			(type default)
+		)
+	)
+	(wire
+		(pts
 			(xy 152.4 81.28) (xy 158.75 81.28)
 		)
@@
 	(wire
 		(pts
-			(xy 82.55 44.45) (xy 90.17 44.45)
+			(xy 82.55 44.45) (xy 83.82 44.45)
 		)
 		(stroke
@@
 	)
 	(symbol
+		(lib_id "power:PWR_FLAG")
+		(at 83.82 44.45 0)
+		(unit 1)
+		(exclude_from_sim no)
+		(in_bom yes)
+		(on_board yes)
+		(dnp no)
+		(fields_autoplaced yes)
+		(property "Reference" "#FLG02"
+			(at 83.82 42.545 0)
+			(effects
+				(font
+					(size 1.27 1.27)
+				)
+				(hide yes)
+			)
+		)
+		(property "Value" "PWR_FLAG"
+			(at 83.82 39.37 0)
+			(effects
+				(font
+					(size 1.27 1.27)
+				)
+			)
+		)
+		(property "Footprint" ""
+			(at 83.82 44.45 0)
+			(effects
+				(font
+					(size 1.27 1.27)
+				)
+				(hide yes)
+			)
+		)
+		(property "Datasheet" "~"
+			(at 83.82 44.45 0)
+			(effects
+				(font
+					(size 1.27 1.27)
+				)
+				(hide yes)
+			)
+		)
+		(property "Description" "Special symbol for telling ERC where power comes from"
+			(at 83.82 44.45 0)
+			(effects
+				(font
+					(size 1.27 1.27)
+				)
+				(hide yes)
+			)
+		)
+		(pin "1"
+		)
+		(instances
+			(project "PS-ChargerInterfacePCB"
+				(path "/d45494af-ff47-4110-bed2-dd613b557244"
+					(reference "#FLG02")
+					(unit 1)
+				)
+			)
+		)
+	)
+	(symbol
 		(lib_id "UTSVT_Power:SMAF4749A-TP")
 		(at 222.25 27.94 270)
@@
 					(unit 1)
 				)
+			)
+		)
+	)
+	(symbol
+		(lib_id "power:PWR_FLAG")
+		(at 48.26 93.98 90)
+		(unit 1)
+		(exclude_from_sim no)
+		(in_bom yes)
+		(on_board yes)
+		(dnp no)
+		(property "Reference" "#FLG01"
+			(at 46.355 93.98 0)
+			(effects
+				(font
+					(size 1.27 1.27)
+				)
+				(hide yes)
+			)
+		)
+		(property "Value" "PWR_FLAG"
+			(at 44.45 94.996 90)
+			(effects
+				(font
+					(size 1.27 1.27)
+				)
+				(justify left)
+				(hide yes)
+			)
+		)
+		(property "Footprint" ""
+			(at 48.26 93.98 0)
+			(effects
+				(font
+					(size 1.27 1.27)
+				)
+				(hide yes)
+			)
+		)
+		(property "Datasheet" "~"
+			(at 48.26 93.98 0)
+			(effects
+				(font
+					(size 1.27 1.27)
+				)
+				(hide yes)
+			)
+		)
+		(property "Description" "Special symbol for telling ERC where power comes from"
+			(at 48.26 93.98 0)
+			(effects
+				(font
+					(size 1.27 1.27)
+				)
+				(hide yes)
+			)
+		)
+		(pin "1"
+		)
+		(instances
+			(project ""
+				(path "/d45494af-ff47-4110-bed2-dd613b557244"
+					(reference "#FLG01")
+					(unit 1)
+				)

Commit message: RevA5
Parts:
- removed J5: Estop 2, symbol Connector_Generic:Conn_01x02
- removed K2: Relay_SPST-NC, symbol Relay:Relay_SPST-NC
- removed TP1, TP10, TP11, TP12, TP13, TP15, TP16, TP17, TP5, TP6, TP7, TP8, TP9: TestPoint, symbol Connector:TestPoint
- added J1: Bread Board Testing Points, SSW-107-21-G-D:SAMTEC_SSW-107-21-G-D, symbol SSW-107-21-G-D:SSW-107-21-G-D
- R2: footprint (none) -> Resistor_SMD:R_0402_1005Metric; now not fitted
- TP14, TP2, TP3, TP4: footprint (none) -> UTSVT_Special:TestPoint_HEX_3mmID
Connections:
- net EStop2_OUT is gone; now on net +3.3V: R2.1
- net EStop2_RET is gone; now on net Estop: R2.2
- net EStop3_RET is gone; now on net Estop: J6.2 (Pin_2)
- net +24V: no longer J6.1 (Pin_1)
- net +3.3V: now also J6.1 (Pin_1)
- net CarCAN_H: now also J1.02
- net CarCAN_L: now also J1.04
- net Display_MISO: now also J1.05
- net Display_MOSI: now also J1.03
- net Display_NSS: now also J1.09
- net Display_RES: now also J1.01
- net Display_SCLK: now also J1.07
- net Elcon_CAN_H: now also J1.13
- net Elcon_CAN_L: now also J1.11
- net LED_CHARGE: now also J1.10
- net LED_FAULT: now also J1.08
- net LED_HEART: now also J1.12
- net LED_HV: now also J1.06
- net Estop: now reaches J3.12 (ADC1_IN6)
- net Estop: now also J1.14
- no-connect marks 21 -> 20
Other:
- moved on the sheet: J2, J4, J6, TP14, TP2, TP3, TP4

Commit message: RevA6
Parts:
- J2: footprint (none) -> 0334722006
- J6: footprint (none) -> 1053091202
Connections:
- net +24V: now also J4.1 (24V)
- net 24V_OUT: no longer J4.1 (24V)
Changed lines of the file:
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@@
 	)
 	(junction
-		(at 64.77 39.37)
-		(diameter 0)
-		(color 0 0 0 0)
-	)
-	(junction
 		(at 27.94 93.98)
 		(diameter 0)
@@
 	(wire
 		(pts
-			(xy 125.73 30.48) (xy 130.81 30.48)
+			(xy 125.73 30.48) (xy 133.35 30.48)
 		)
 		(stroke
@@
 	(wire
 		(pts
-			(xy 130.81 30.48) (xy 130.81 29.21)
-		)
-		(stroke
-			(width 0)
-			(type default)
-		)
-	)
-	(wire
-		(pts
 			(xy 218.44 39.37) (xy 219.71 39.37)
 		)
@@
 	(wire
 		(pts
-			(xy 64.77 39.37) (xy 71.12 39.37)
+			(xy 63.5 39.37) (xy 68.58 39.37)
 		)
 		(stroke
@@
 	(wire
 		(pts
-			(xy 63.5 39.37) (xy 64.77 39.37)
-		)
-		(stroke
-			(width 0)
-			(type default)
-		)
-	)
-	(wire
-		(pts
 			(xy 271.78 57.15) (xy 271.78 54.61)
 		)
@@
 		)
 	)
+	(label "24V_OUT"
+		(at 133.35 30.48 180)
+		(effects
+			(font
+				(size 0.889 0.889)
+			)
+			(justify right bottom)
+		)
+	)
 	(label "Display_SCLK"
 		(at 38.1 142.24 0)
@@
 		)
 	)
-	(label "24V_OUT"
-		(at 71.12 39.37 180)
-		(effects
-			(font
-				(size 0.889 0.889)
-			)
-			(justify right bottom)
-		)
-	)
 	(label "Display_NSS"
 		(at 229.87 124.46 0)
@@
 	)
 	(symbol
-		(lib_id "power:PWR_FLAG")
-		(at 64.77 39.37 0)
+		(lib_id "power:+24V")
+		(at 68.58 39.37 0)
 		(unit 1)
 		(exclude_from_sim no)
@@
 		(on_board yes)
 		(dnp no)
-		(fields_autoplaced yes)
-		(property "Reference" "#FLG02"
-			(at 64.77 37.465 0)
+		(property "Reference" "#PWR016"
+			(at 68.58 43.18 0)
 			(effects
 				(font
@@
 			)
 		)
-		(property "Value" "PWR_FLAG"
-			(at 64.77 34.29 0)
+		(property "Value" "+24V"
+			(at 68.58 35.56 0)
 			(effects
 				(font
@@
 		)
 		(property "Footprint" ""
-			(at 64.77 39.37 0)
+			(at 68.58 39.37 0)
 			(effects
 				(font
@@
 			)
 		)
-		(property "Datasheet" "~"
-			(at 64.77 39.37 0)
+		(property "Datasheet" ""
+			(at 68.58 39.37 0)
 			(effects
 				(font
@@
 			)
 		)
-		(property "Description" "Special symbol for telling ERC where power comes from"
-			(at 64.77 39.37 0)
+		(property "Description" "Power symbol creates a global label with name \"+24V\""
+			(at 68.58 39.37 0)
 			(effects
 				(font
@@
 		)
 		(instances
-			(project "PS-ChargerInterfacePCB"
+			(project ""
 				(path "/d45494af-ff47-4110-bed2-dd613b557244"
-					(reference "#FLG02")
+					(reference "#PWR016")
 					(unit 1)
 				)
@@
 		(dnp no)
 		(property "Reference" "J2"
-			(at 25.4 34.544 0)
+			(at 24.892 33.274 0)
 			(effects
 				(font
@@
 		)
 		(property "Value" "LV_Elcon_Connector"
-			(at 34.544 36.576 0)
+			(at 34.29 35.306 0)
 			(effects
 				(font
@@
 			)
 		)
-		(property "Footprint" ""
+		(property "Footprint" "0334722006"
 			(at 25.4 41.91 0)
 			(effects
@@
 			)
 		)
-		(property "Datasheet" "~"
+		(property "Datasheet" "https://tools.molex.com/pdm_docs/as/AS-33611-001.pdf"
 			(at 25.4 41.91 0)
 			(effects
@@
 	)
 	(symbol
-		(lib_id "power:+24V")
-		(at 130.81 29.21 0)
-		(unit 1)
-		(exclude_from_sim no)
-		(in_bom yes)
-		(on_board yes)
-		(dnp no)
-		(fields_autoplaced yes)
-		(property "Reference" "#PWR062"
-			(at 130.81 33.02 0)
-			(effects
-				(font
-					(size 1.27 1.27)
-				)
-				(hide yes)
-			)
-		)
-		(property "Value" "+24V"
-			(at 130.81 24.13 0)
-			(effects
-				(font
-					(size 1.27 1.27)
-				)
-			)
-		)
-		(property "Footprint" ""
-			(at 130.81 29.21 0)
-			(effects
-				(font
-					(size 1.27 1.27)
-				)
-				(hide yes)
-			)
-		)
-		(property "Datasheet" ""
-			(at 130.81 29.21 0)
-			(effects
-				(font
-					(size 1.27 1.27)
-				)
-				(hide yes)
-			)
-		)
-		(property "Description" "Power symbol creates a global label with name \"+24V\""
-			(at 130.81 29.21 0)
-			(effects
-				(font
-					(size 1.27 1.27)
-				)
-				(hide yes)
-			)
-		)
-		(pin "1"
-		)
-		(instances
-			(project ""
-				(path "/d45494af-ff47-4110-bed2-dd613b557244"
-					(reference "#PWR062")
-					(unit 1)
-				)
-			)
-		)
-	)
-	(symbol
 		(lib_id "Device:R_US")
 		(at 261.62 33.02 0)
@@
 			)
 		)
-		(property "Footprint" ""
+		(property "Footprint" "1053091202"
 			(at 274.32 82.55 0)
 			(effects
@@
 			)
 		)
-		(property "Datasheet" "~"
+		(property "Datasheet" "https://www.molex.com/en-us/products/part-detail/1053091202?display=pdf"
 			(at 274.32 82.55 0)
 			(effects
