File: PS-ChargerInterfacePCB.kicad_sch (KiCad schematic)
At the start: 18 parts, among them J1 Bread Board Testing Points, J2 LV_Elcon_Connector, J4 BPSConn, J6 Estop 3

Commit message: RevA6 footprint updates
Parts:
- J1: footprint SSW-107-21-G-D:SAMTEC_SSW-107-21-G-D -> SSW-107-21-G-D:CON14_2X7_TU_SSQ
- J2: footprint 0334722006 -> 334722006:Molex-33472-2006-MFG
- J3: footprint (none) -> UTSVT_Special:LeaderSOM
- J6: footprint 1053091202 -> 153091202:1053091202
Changed lines of the file:
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@@
 			)
 		)
-		(property "Footprint" ""
+		(property "Footprint" "UTSVT_Special:LeaderSOM"
 			(at 113.03 49.53 0)
 			(effects
@@
 			)
 		)
-		(property "Footprint" "0334722006"
+		(property "Footprint" "334722006:Molex-33472-2006-MFG"
 			(at 25.4 41.91 0)
 			(effects
@@
 			)
 		)
-		(property "Footprint" "SSW-107-21-G-D:SAMTEC_SSW-107-21-G-D"
+		(property "Footprint" "SSW-107-21-G-D:CON14_2X7_TU_SSQ"
 			(at 58.42 142.24 0)
 			(effects
@@
 			)
 		)
-		(property "Footprint" ""
+		(property "Footprint" "UTSVT_Special:LeaderSOM"
 			(at 55.88 49.53 0)
 			(effects
@@
 			)
 		)
-		(property "Footprint" "1053091202"
+		(property "Footprint" "153091202:1053091202"
 			(at 274.32 82.55 0)
 			(effects

Commit message: RevA7 layout
Parts:
- removed J1: Bread Board Testing Points, SSW-107-21-G-D:CON14_2X7_TU_SSQ, symbol SSW-107-21-G-D:SSW-107-21-G-D
- added J1: Conn_02x07_Top_Bottom, Connector_PinHeader_2.54mm:PinHeader_2x07_P2.54mm_Vertical, symbol Connector_Generic:Conn_02x07_Top_Bottom
- J2: footprint 334722006:Molex-33472-2006-MFG -> Conn_1x4_1053091304:CONN_SD-105309-100_04_MOL
Connections:
- net 12V_IN: now also J2.4 (Pin_4); no longer J2.1 (Pin_1)
- net Display_MISO: now also J1.7 (Pin_7)
- net Display_MOSI: now also J1.9 (Pin_9)
- net Display_NSS: now also J1.6 (Pin_6)
- net Display_RES: now also J1.5 (Pin_5)
- net Display_SCLK: now also J1.2 (Pin_2)
- net Estop: now also J1.4 (Pin_4)
- net GND: now also J2.1 (Pin_1); no longer J2.4 (Pin_4)
- net LED_CHARGE: now also J1.12 (Pin_12)
- net LED_FAULT: now also J1.14 (Pin_14)
- net LED_HEART: now also J1.8 (Pin_8)
- net LED_HV: now also J1.10 (Pin_10)
- net CAN_H_Car renamed CAN_Car_+
- net CAN_Car_+: now also J1.11 (Pin_11)
- net CAN_H_Elcon renamed CAN_Elcon_+
- net CAN_Elcon_+: now also J2.3 (Pin_3), J1.3 (Pin_3); no longer J2.2 (Pin_2)
- net CAN_L_Car renamed CAN_Car_-
- net CAN_Car_-: now also J1.13 (Pin_13)
- net CAN_L_Elcon renamed CAN_Elcon_-
- net CAN_Elcon_-: now also J2.2 (Pin_2), J1.1 (Pin_1); no longer J2.3 (Pin_3)
Other:
- note added: "Net Class for Diff Pair: CAN_H_Elcon = CAN_Elcon_+ CAN_L_Elcon = CAN_Elcon_- CAN_H_Car = CAN_Car_+ CAN_L_Car = CAN_Car_-"

Commit message: RevA7 updates, dont review
Connections:
- net 12V_IN: now also J2.1 (Pin_1); no longer J2.4 (Pin_4)
- net CAN_Elcon_+: now also J2.2 (Pin_2); no longer J2.3 (Pin_3)
- net CAN_Elcon_-: now also J2.3 (Pin_3); no longer J2.2 (Pin_2)
- net GND: now also J2.4 (Pin_4); no longer J2.1 (Pin_1)
Changed lines of the file:
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@@
-		)
-	)
-	(label "CAN_Elcon_-"
-		(at 39.37 41.91 180)
-		(effects
-			(font
-				(size 0.889 0.889)
-			)
-			(justify right bottom)
 		)
 	)
@@
 	)
 	(label "12V_IN"
-		(at 33.02 48.26 0)
-		(effects
-			(font
-				(size 0.889 0.889)
-			)
-			(justify left bottom)
+		(at 38.1 39.37 180)
+		(effects
+			(font
+				(size 0.889 0.889)
+			)
+			(justify right bottom)
 		)
 	)
@@
 	)
 	(label "CAN_Elcon_+"
-		(at 39.37 44.45 180)
+		(at 39.37 41.91 180)
 		(effects
 			(font
@@
 			)
 			(justify left bottom)
+		)
+	)
+	(label "CAN_Elcon_-"
+		(at 39.37 44.45 180)
+		(effects
+			(font
+				(size 0.889 0.889)
+			)
+			(justify right bottom)
 		)
 	)
@@
 	(symbol
 		(lib_id "power:GND")
-		(at 38.1 39.37 180)
+		(at 33.02 48.26 0)
 		(unit 1)
 		(exclude_from_sim no)
@@
 		(fields_autoplaced yes)
 		(property "Reference" "#PWR06"
-			(at 38.1 33.02 0)
+			(at 33.02 54.61 0)
 			(effects
 				(font
@@
 		)
 		(property "Value" "GND"
-			(at 38.1 34.29 0)
+			(at 33.02 53.34 0)
 			(effects
 				(font
@@
 		)
 		(property "Footprint" ""
-			(at 38.1 39.37 0)
+			(at 33.02 48.26 0)
 			(effects
 				(font
@@
 		)
 		(property "Datasheet" ""
-			(at 38.1 39.37 0)
+			(at 33.02 48.26 0)
 			(effects
 				(font
@@
 		)
 		(property "Description" "Power symbol creates a global label with name \"GND\" , ground"
-			(at 38.1 39.37 0)
-			(effects
-				(font
+			(at 33.02 48.26 0)
+			(effects
+				(font

Commit message: RevA7 saving changes
Connections:
- net CAN_Car_+: now also J1.2 (Pin_2); no longer J1.11 (Pin_11)
- net CAN_Car_-: now also J1.4 (Pin_4); no longer J1.13 (Pin_13)
- net Display_MISO: now also J1.9 (Pin_9), J3.14 (SPI3_MISO); no longer J1.7 (Pin_7), J3.44 (SPI2_MISO)
- net Display_MOSI: now also J1.5 (Pin_5), J3.18 (SPI3_MOSI); no longer J1.9 (Pin_9), J3.42 (SPI2_MOSI)
- net Display_NSS: now also J1.13 (Pin_13), J3.16 (SPI3_NSS); no longer J1.6 (Pin_6), J3.48 (SPI2_NSS)
- net Display_RES: now also J1.11 (Pin_11), J3.12 (ADC1_IN6); no longer J1.5 (Pin_5), J3.41 (ADC1_IN8)
- net Display_SCLK: now also J1.7 (Pin_7), J3.20 (SPI3_SCK); no longer J1.2 (Pin_2), J3.46 (SPI2_SCK)
- net Estop: now also J1.6 (Pin_6), J3.41 (ADC1_IN8); no longer J1.4 (Pin_4), J3.12 (ADC1_IN6)
Changed lines of the file:
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@@
 	)
 	(no_connect
-		(at 132.08 80.01)
+		(at 132.08 105.41)
 	)
 	(no_connect
-		(at 74.93 92.71)
+		(at 132.08 80.01)
 	)
 	(no_connect
-		(at 74.93 100.33)
+		(at 74.93 92.71)
 	)
 	(no_connect
@@
 	)
 	(no_connect
-		(at 74.93 107.95)
+		(at 132.08 100.33)
 	)
 	(no_connect
@@
 	)
 	(no_connect
-		(at 74.93 102.87)
-	)
-	(no_connect
 		(at 74.93 73.66)
 	)
@@
 	)
 	(no_connect
-		(at 74.93 105.41)
+		(at 132.08 102.87)
+	)
+	(no_connect
+		(at 132.08 107.95)
 	)
 	(no_connect
@@
 	(wire
 		(pts
-			(xy 132.08 105.41) (xy 142.24 105.41)
-		)
-		(stroke
-			(width 0)
-			(type default)
-		)
-	)
-	(wire
-		(pts
 			(xy 67.31 46.99) (xy 67.31 48.26)
 		)
@@
 	(wire
 		(pts
-			(xy 132.08 100.33) (xy 142.24 100.33)
-		)
-		(stroke
-			(width 0)
-			(type default)
-		)
-	)
-	(wire
-		(pts
 			(xy 86.36 72.39) (xy 93.98 72.39)
 		)
@@
 	(wire
 		(pts
-			(xy 91.44 96.52) (xy 93.98 96.52)
+			(xy 74.93 107.95) (xy 85.09 107.95)
 		)
 		(stroke
@@
 	(wire
 		(pts
-			(xy 29.21 123.19) (xy 29.21 127)
+			(xy 74.93 100.33) (xy 85.09 100.33)
 		)
 		(stroke
@@
 	(wire
 		(pts
-			(xy 38.1 149.86) (xy 45.72 149.86)
+			(xy 91.44 96.52) (xy 93.98 96.52)
 		)
 		(stroke
@@
 	(wire
 		(pts
-			(xy 38.1 147.32) (xy 45.72 147.32)
+			(xy 29.21 123.19) (xy 29.21 127)
 		)
 		(stroke
@@
 	(wire
 		(pts
-			(xy 132.08 77.47) (xy 138.43 77.47)
+			(xy 38.1 149.86) (xy 45.72 149.86)
 		)
 		(stroke
@@
 	(wire
 		(pts
-			(xy 200.66 39.37) (xy 209.55 39.37)
+			(xy 38.1 147.32) (xy 45.72 147.32)
 		)
 		(stroke
@@
 	(wire
 		(pts
-			(xy 38.1 139.7) (xy 45.72 139.7)
+			(xy 132.08 77.47) (xy 138.43 77.47)
 		)
 		(stroke
@@
 	(wire
 		(pts
-			(xy 219.71 54.61) (xy 219.71 39.37)
+			(xy 200.66 39.37) (xy 209.55 39.37)
 		)
 		(stroke
@@
 	(wire
 		(pts
-			(xy 132.08 102.87) (xy 142.24 102.87)
+			(xy 38.1 139.7) (xy 45.72 139.7)
+		)
+		(stroke
+			(width 0)
+			(type default)
+		)
+	)
+	(wire
+		(pts
+			(xy 219.71 54.61) (xy 219.71 39.37)
 		)
 		(stroke
@@
 	(wire
 		(pts
+			(xy 74.93 102.87) (xy 85.09 102.87)
+		)
+		(stroke
+			(width 0)
+			(type default)
+		)
+	)
+	(wire
+		(pts
 			(xy 252.73 27.94) (xy 261.62 27.94)
 		)
@@
 	(wire
 		(pts
-			(xy 58.42 142.24) (xy 66.04 142.24)
+			(xy 58.42 142.24) (xy 67.31 142.24)
 		)
 		(stroke
@@
 	(wire
 		(pts
-			(xy 132.08 107.95) (xy 142.24 107.95)
-		)
-		(stroke
-			(width 0)
-			(type default)
-		)
-	)
-	(wire
-		(pts
 			(xy 35.56 127) (xy 35.56 123.19)
 		)
@@
 	(wire
 		(pts
+			(xy 74.93 105.41) (xy 85.09 105.41)
+		)
+		(stroke
+			(width 0)
+			(type default)
+		)
+	)
+	(wire
+		(pts
 			(xy 261.62 54.61) (xy 271.78 54.61)
 		)
@@
 	)
 	(label "Estop"
-		(at 82.55 68.58 180)
+		(at 138.43 77.47 180)
 		(effects
 			(font
@@
 	)
 	(label "Display_RES"
-		(at 138.43 77.47 180)
+		(at 82.55 68.58 180)
 		(effects
 			(font
@@
 	)
 	(label "Display_NSS"
-		(at 38.1 147.32 0)
+		(at 66.04 147.32 180)
 		(effects
 			(font
 				(size 0.889 0.889)
 			)
-			(justify left bottom)
+			(justify right bottom)
 		)
 	)
@@
 	)
 	(label "Display_RES"
-		(at 38.1 144.78 0)
+		(at 67.31 142.24 180)
 		(effects
 			(font
 				(size 0.889 0.889)
 			)
-			(justify left bottom)
+			(justify right bottom)
 		)
 	)
 	(label "CAN_Car_-"
-		(at 66.04 147.32 180)
+		(at 38.1 142.24 0)
 		(effects
 			(font
 				(size 0.889 0.889)
 			)
-			(justify right bottom)
+			(justify left bottom)
 		)
 	)
@@
 	)
 	(label "Display_NSS"
-		(at 142.24 107.95 180)
+		(at 85.09 102.87 180)
 		(effects
 			(font
@@
 	)
 	(label "Display_SCLK"
-		(at 38.1 137.16 0)
+		(at 38.1 149.86 0)
 		(effects
 			(font
@@
 	)
 	(label "Display_MISO"
-		(at 142.24 102.87 180)
+		(at 85.09 100.33 180)
 		(effects
 			(font
@@
 	)
 	(label "CAN_Car_+"
-		(at 66.04 142.24 180)
+		(at 38.1 137.16 0)
 		(effects
 			(font
 				(size 0.889 0.889)
 			)
-			(justify right bottom)
+			(justify left bottom)
 		)
 	)
@@
 	)
 	(label "Estop"
-		(at 38.1 142.24 0)
+		(at 38.1 147.32 0)
 		(effects
 			(font
@@
 	)
 	(label "Display_MOSI"
-		(at 142.24 100.33 180)
+		(at 85.09 105.41 180)
 		(effects
 			(font
@@
 	)
 	(label "Display_MOSI"
-		(at 66.04 137.16 180)
+		(at 38.1 144.78 0)
 		(effects
 			(font
 				(size 0.889 0.889)
 			)
-			(justify right bottom)
+			(justify left bottom)
 		)
 	)
@@
 	)
 	(label "Display_SCLK"
-		(at 142.24 105.41 180)
+		(at 85.09 107.95 180)
 		(effects
 			(font
@@
 	)
 	(label "Display_MISO"
-		(at 38.1 149.86 0)
+		(at 66.04 137.16 180)
 		(effects
 			(font
 				(size 0.889 0.889)
 			)
-			(justify left bottom)
+			(justify right bottom)
 		)
 	)

Commit message: RevA8 layout changes
Parts:
- removed Z5: SMAF4751A-TP, UTSVT_Passives:SODFL5026X125N, symbol UTSVT_Power:SMAF4749A-TP
- removed Z7: SMAF4744A, UTSVT_Passives:SODFL5026X125N, symbol UTSVT_Power:SMAF4749A-TP
Connections:
- net LED_CHARGE: now also J1.8 (Pin_8); no longer J1.12 (Pin_12)
- net LED_FAULT: now also J1.10 (Pin_10); no longer J1.14 (Pin_14)
- net LED_HEART: now also J1.14 (Pin_14); no longer J1.8 (Pin_8)
- net LED_HV: now also J1.12 (Pin_12); no longer J1.10 (Pin_10)
Other:
- sheet Power12V ports: added none; removed RPP_EN
- sheet Power24V ports: added none; removed RPP_EN

Commit message: RevA9 for review
Parts:
- removed J1: Conn_02x07_Top_Bottom, Connector_PinHeader_2.54mm:PinHeader_2x07_P2.54mm_Vertical, symbol Connector_Generic:Conn_02x07_Top_Bottom
- removed J3: ~, UTSVT_Special:LeaderSOM, symbol utsvt_connectors2:LSOM_DaughterConn
- added J3, J5: SFH11-PBPC-D05-ST-BK, UTSVT_Connectors:CONN_SFH11-xxxC-D05-ST-XX_SUL, symbol utsvt_connectors2:SFH11-PBPC-D05-ST-BK
- added U1: LeaderSOM, UTSVT_Special:LeaderSOM, symbol utsvt_connectors2:LeaderSOMConnector
- renumbered TP3 to TP_12V, TP4 to TP_24V, TP2 to TP_3V3, TP14 to TP_GND
Connections:
- net +24V: now also U1.21 (24VExt), U1.22 (24VExt), U1.23 (24VExt), U1.24 (24VExt)
- net +3.3V: now also U1.1 (+3.3V), U1.2 (+3.3V), U1.3 (+3.3V), U1.4 (+3.3V)
- net BuzzPWM: now also U1.10 (ADC2_IN12)
- net CAN_Car_+: now also J5.10 (CH0), U1.30 (CarCAN_H)
- net CAN_Car_-: now also J5.8 (CH2), U1.32 (CarCAN_L)
- net CAN_Elcon_+: now also J5.7 (CH3), U1.6 (IntCAN_H)
- net CAN_Elcon_-: now also J5.9 (CH1), U1.8 (IntCAN_L)
- net Display_MISO: now also J3.6 (CH4), U1.14 (SPI2_MISO)
- net Display_MOSI: now also J3.3 (CH7), U1.18 (SPI2_MOSI)
- net Display_NSS: now also J3.10 (CH0), U1.16 (SPI2_NSS)
- net Display_RES: now also J3.8 (CH2), U1.12 (ADC1_IN11)
- net Display_SCLK: now also J3.4 (CH6), U1.20 (SPI2_SCK)
- net Estop: now also J3.5 (CH5), U1.41 (ADC1_IN2)
- net GND: now also J3.1 (GND), J3.2 (GND), J5.1 (GND), J5.2 (GND), U1.25 (GND), U1.26 (GND), U1.27 (GND), U1.28 (GND), U1.29 (GND)
- net LED_CHARGE: now also J5.6 (CH4), U1.46 (SPI3_MOSI)
- net LED_FAULT: now also J5.3 (CH7), U1.44 (SPI3_NSS)
- net LED_HEART: now also J5.5 (CH5), U1.48 (SPI3_SCK)
- net LED_HV: now also J5.4 (CH6), U1.42 (SPI3_MISO)
- no-connect marks 20 -> 22
Other:
- note added: "To dos: - move 12Vs and PPs closer - Update testing points to logic analyzer in kicad sharepoint - move LEDs"

Commit message: RevA9 small changes
Parts:
- renumbered J2 to J1, J3 to J2, J4 to J3, J5 to J4, J6 to J5, R14 to R1, R25 to R2, R2 to R3, R19 to R4, R20 to R5, TP_12V to TP_12V1, TP_24V to TP_24V1, TP_3V3 to TP_3V1, TP_GND to TP_GND1, Z6 to Z1, Z8 to Z2
Changed lines of the file:
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@@
 		(on_board yes)
 		(dnp no)
-		(property "Reference" "#PWR016"
+		(property "Reference" "#PWR08"
 			(at 68.58 43.18 0)
 			(effects
@@
 			(project ""
 				(path "/d45494af-ff47-4110-bed2-dd613b557244"
-					(reference "#PWR016")
+					(reference "#PWR08")
 					(unit 1)
 				)
@@
 		(on_board yes)
 		(dnp no)
-		(property "Reference" "Z6"
+		(property "Reference" "Z1"
 			(at 223.012 28.448 90)
 			(effects
@@
 			(project "PS-ChargerInterfacePCB"
 				(path "/d45494af-ff47-4110-bed2-dd613b557244"
-					(reference "Z6")
+					(reference "Z1")
 					(unit 1)
 				)
@@
 		(on_board yes)
 		(dnp no)
-		(property "Reference" "TP_24V"
+		(property "Reference" "TP_24V1"
 			(at 84.328 132.08 0)
 			(effects
@@
 			(project "PS-ChargerInterfacePCB"
 				(path "/d45494af-ff47-4110-bed2-dd613b557244"
-					(reference "TP_24V")
+					(reference "TP_24V1")
 					(unit 1)
 				)
@@
 		(dnp no)
 		(fields_autoplaced yes)
-		(property "Reference" "#PWR021"
+		(property "Reference" "#PWR06"
 			(at 57.15 162.56 0)
 			(effects
@@
 			(project ""
 				(path "/d45494af-ff47-4110-bed2-dd613b557244"
-					(reference "#PWR021")
+					(reference "#PWR06")
 					(unit 1)
 				)
@@
 		(dnp no)
 		(fields_autoplaced yes)
-		(property "Reference" "#PWR06"
+		(property "Reference" "#PWR04"
 			(at 33.02 54.61 0)
 			(effects
@@
 			(project "PS-ChargerInterfacePCB"
 				(path "/d45494af-ff47-4110-bed2-dd613b557244"
-					(reference "#PWR06")
+					(reference "#PWR04")
 					(unit 1)
 				)
@@
 		(on_board yes)
 		(dnp no)
-		(property "Reference" "#PWR033"
+		(property "Reference" "#PWR012"
 			(at 88.9 116.84 0)
 			(effects
@@
 			(project ""
 				(path "/d45494af-ff47-4110-bed2-dd613b557244"
-					(reference "#PWR033")
+					(reference "#PWR012")
 					(unit 1)
 				)
@@
 		(dnp no)
 		(fields_autoplaced yes)
-		(property "Reference" "#PWR022"
+		(property "Reference" "#PWR011"
 			(at 88.9 162.56 0)
 			(effects
@@
 			(project ""
 				(path "/d45494af-ff47-4110-bed2-dd613b557244"
-					(reference "#PWR022")
+					(reference "#PWR011")
 					(unit 1)
 				)
@@
 		(on_board yes)
 		(dnp no)
-		(property "Reference" "#PWR08"
+		(property "Reference" "#PWR010"
 			(at 82.55 127 0)
 			(effects
@@
 			(project ""
 				(path "/d45494af-ff47-4110-bed2-dd613b557244"
-					(reference "#PWR08")
+					(reference "#PWR010")
 					(unit 1)
 				)
@@
 		(on_board yes)
 		(dnp no)
-		(property "Reference" "J2"
+		(property "Reference" "J1"
 			(at 24.892 33.274 0)
 			(effects
@@
 			(project ""
 				(path "/d45494af-ff47-4110-bed2-dd613b557244"
-					(reference "J2")
+					(reference "J1")
 					(unit 1)
 				)
@@
 		(on_board yes)
 		(dnp no)
-		(property "Reference" "#PWR01"
+		(property "Reference" "#PWR03"
 			(at 29.21 127 0)
 			(effects
@@
 			(project ""
 				(path "/d45494af-ff47-4110-bed2-dd613b557244"
-					(reference "#PWR01")
+					(reference "#PWR03")
 					(unit 1)
 				)
@@
 		(dnp no)
 		(fields_autoplaced yes)
-		(property "Reference" "#PWR02"
+		(property "Reference" "#PWR013"
 			(at 91.44 119.38 0)
 			(effects
@@
 			(project ""
 				(path "/d45494af-ff47-4110-bed2-dd613b557244"
-					(reference "#PWR02")
+					(reference "#PWR013")
 					(unit 1)
 				)
@@
 		(on_board yes)
 		(dnp yes)
-		(property "Reference" "R2"
+		(property "Reference" "R3"
 			(at 242.062 82.042 0)
 			(effects
@@
 			(project ""
 				(path "/d45494af-ff47-4110-bed2-dd613b557244"
-					(reference "R2")
+					(reference "R3")
 					(unit 1)
 				)
@@
 		(dnp no)
 		(fields_autoplaced yes)
-		(property "Reference" "#PWR039"
+		(property "Reference" "#PWR01"
 			(at 26.67 69.85 0)
 			(effects
@@
 			(project ""
 				(path "/d45494af-ff47-4110-bed2-dd613b557244"
-					(reference "#PWR039")
+					(reference "#PWR01")
 					(unit 1)
 				)
@@
 		(on_board yes)
 		(dnp no)
-		(property "Reference" "TP_GND"
+		(property "Reference" "TP_GND1"
 			(at 90.17 134.62 0)
 			(effects
@@
 			(project "PS-ChargerInterfacePCB"
 				(path "/d45494af-ff47-4110-bed2-dd613b557244"
-					(reference "TP_GND")
+					(reference "TP_GND1")
 					(unit 1)
 				)
@@
 		(on_board yes)
 		(dnp no)
-		(property "Reference" "#PWR03"
+		(property "Reference" "#PWR02"
 			(at 27.94 90.17 0)
 			(effects
@@
 			(project ""
 				(path "/d45494af-ff47-4110-bed2-dd613b557244"
-					(reference "#PWR03")
+					(reference "#PWR02")
 					(unit 1)
 				)
@@
 		(on_board yes)
 		(dnp no)
-		(property "Reference" "R20"
+		(property "Reference" "R5"
 			(at 266.7 42.418 90)
 			(effects
@@
 			(project "PS-ChargerInterfacePCB"
 				(path "/d45494af-ff47-4110-bed2-dd613b557244"
-					(reference "R20")
+					(reference "R5")
 					(unit 1)
 				)
@@
 		(dnp no)
 		(fields_autoplaced yes)
-		(property "Reference" "#PWR031"
+		(property "Reference" "#PWR015"
 			(at 219.71 63.5 0)
 			(effects
@@
 			(project "PS-ChargerInterfacePCB"
 				(path "/d45494af-ff47-4110-bed2-dd613b557244"
-					(reference "#PWR031")
+					(reference "#PWR015")
 					(unit 1)
 				)
@@
 		(on_board yes)
 		(dnp no)
-		(property "Reference" "#PWR027"
+		(property "Reference" "#PWR014"
 			(at 204.47 27.94 0)
 			(effects
@@
 			(project "PS-ChargerInterfacePCB"
 				(path "/d45494af-ff47-4110-bed2-dd613b557244"
-					(reference "#PWR027")
+					(reference "#PWR014")
 					(unit 1)
 				)
@@
 		(dnp no)
 		(fields_autoplaced yes)
-		(property "Reference" "#PWR044"
+		(property "Reference" "#PWR018"
 			(at 271.78 63.5 0)
 			(effects
@@
 			(project "PS-ChargerInterfacePCB"
 				(path "/d45494af-ff47-4110-bed2-dd613b557244"
-					(reference "#PWR044")
+					(reference "#PWR018")
 					(unit 1)
 				)
@@
 		(dnp no)
 		(fields_autoplaced yes)
-		(property "Reference" "#PWR061"
+		(property "Reference" "#PWR09"
 			(at 81.28 33.02 0)
 			(effects
@@
 			(project ""
 				(path "/d45494af-ff47-4110-bed2-dd613b557244"
-					(reference "#PWR061")
+					(reference "#PWR09")
 					(unit 1)
 				)
@@
 		(on_board yes)
 		(dnp no)
-		(property "Reference" "TP_12V"
+		(property "Reference" "TP_12V1"
 			(at 32.258 133.35 0)
 			(effects
@@
 			(project "PS-ChargerInterfacePCB"
 				(path "/d45494af-ff47-4110-bed2-dd613b557244"
-					(reference "TP_12V")
+					(reference "TP_12V1")
 					(unit 1)
 				)
@@
 		(on_board yes)
 		(dnp no)
-		(property "Reference" "#PWR040"
+		(property "Reference" "#PWR05"
 			(at 35.56 127 0)
 			(effects
@@
 			(project "PS-ChargerInterfacePCB"
 				(path "/d45494af-ff47-4110-bed2-dd613b557244"
-					(reference "#PWR040")
+					(reference "#PWR05")
 					(unit 1)
 				)
@@
 		(on_board yes)
 		(dnp no)
-		(property "Reference" "#PWR05"
+		(property "Reference" "#PWR016"
 			(at 246.38 80.01 0)
 			(effects
@@
 			(project ""
 				(path "/d45494af-ff47-4110-bed2-dd613b557244"
-					(reference "#PWR05")
+					(reference "#PWR016")
 					(unit 1)
 				)
@@
 		(on_board yes)
 		(dnp no)
-		(property "Reference" "TP_3V3"
+		(property "Reference" "TP_3V1"
 			(at 41.656 132.588 0)
 			(effects
@@
 			(project "PS-ChargerInterfacePCB"
 				(path "/d45494af-ff47-4110-bed2-dd613b557244"
-					(reference "TP_3V3")
+					(reference "TP_3V1")
 					(unit 1)
 				)
@@
 		(on_board yes)
 		(dnp no)
-		(property "Reference" "R25"
+		(property "Reference" "R2"
 			(at 214.63 42.418 90)
 			(effects
@@
 			(project "PS-ChargerInterfacePCB"
 				(path "/d45494af-ff47-4110-bed2-dd613b557244"
-					(reference "R25")
+					(reference "R2")
 					(unit 1)
 				)
@@
 		(on_board yes)
 		(dnp no)
-		(property "Reference" "J4"
+		(property "Reference" "J3"
 			(at 50.292 34.544 0)
 			(effects
@@
 			(project ""
 				(path "/d45494af-ff47-4110-bed2-dd613b557244"
-					(reference "J4")
+					(reference "J3")
 					(unit 1)
 				)
@@
 		(on_board yes)
 		(dnp no)
-		(property "Reference" "R19"
+		(property "Reference" "R4"
 			(at 263.652 32.004 0)
 			(effects
@@
 			(project "PS-ChargerInterfacePCB"
 				(path "/d45494af-ff47-4110-bed2-dd613b557244"
-					(reference "R19")
+					(reference "R4")
 					(unit 1)
 				)
@@
 		(on_board yes)
 		(dnp no)
-		(property "Reference" "J6"
+		(property "Reference" "J5"
 			(at 274.32 76.2 0)
 			(effects
@@
 			(project "PS-ChargerInterfacePCB"
 				(path "/d45494af-ff47-4110-bed2-dd613b557244"
-					(reference "J6")
+					(reference "J5")
 					(unit 1)
 				)
@@
 		(on_board yes)
 		(dnp no)
-		(property "Reference" "J3"
+		(property "Reference" "J2"
 			(at 36.068 162.814 0)
 			(effects
@@
 			(project ""
 				(path "/d45494af-ff47-4110-bed2-dd613b557244"
-					(reference "J3")
+					(reference "J2")
 					(unit 1)
 				)
@@
 		(dnp no)
 		(fields_autoplaced yes)
-		(property "Reference" "R14"
+		(property "Reference" "R1"
 			(at 212.09 31.7499 0)
 			(effects
@@
 			(project "PS-ChargerInterfacePCB"
 				(path "/d45494af-ff47-4110-bed2-dd613b557244"
-					(reference "R14")
+					(reference "R1")
 					(unit 1)
 				)
@@
 		(on_board yes)
 		(dnp no)
-		(property "Reference" "J5"
+		(property "Reference" "J4"
 			(at 67.818 162.814 0)
 			(effects
@@
 			(project "PS-ChargerInterfacePCB"
 				(path "/d45494af-ff47-4110-bed2-dd613b557244"
-					(reference "J5")
+					(reference "J4")
 					(unit 1)
 				)
@@
 		(on_board yes)
 		(dnp no)
-		(property "Reference" "Z8"
+		(property "Reference" "Z2"
 			(at 275.59 27.94 90)
 			(effects
@@
 			(project "PS-ChargerInterfacePCB"
 				(path "/d45494af-ff47-4110-bed2-dd613b557244"
-					(reference "Z8")
+					(reference "Z2")
 					(unit 1)
 				)
@@
 		(on_board yes)
 		(dnp no)
-		(property "Reference" "#PWR043"
+		(property "Reference" "#PWR017"
 			(at 256.54 27.94 0)
 			(effects
@@
 			(project "PS-ChargerInterfacePCB"
 				(path "/d45494af-ff47-4110-bed2-dd613b557244"
-					(reference "#PWR043")
+					(reference "#PWR017")
 					(unit 1)
 				)
