File: PS-ChargerInterfacePCB.kicad_sch (KiCad schematic)
At the start: 17 parts, among them J1 LV_Elcon_Connector, J2 SFH11-PBPC-D05-ST-BK, J3 BPSConn, J4 SFH11-PBPC-D05-ST-BK, J5 Estop 3, U1 LeaderSOM

Commit message: RevA10 for review
Parts:
- J1: footprint Conn_1x4_1053091304:CONN_SD-105309-100_04_MOL -> UTSVT_Connectors:Molex_Nano-Fit_105309-xx04_1x04_P2.50mm_Vertical; Distrbutor Link (none) -> https://www.mouser.com/ProductDetail/Molex/105309-1304?qs=P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; Manufacturer (none) -> Molex; Manufacturer_Part_Number (none) -> 105309-1304
- J2, J4: Distrbutor Link (none) -> https://www.digikey.com/en/products/detail/sullins-connecto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; Manufacturer (none) -> Sullins Connector Solutions; Manufacturer_Part_Number (none) -> SFH11-PBPC-D05-ST-BK
- J3: Distrbutor Link (none) -> https://www.mouser.com/ProductDetail/Molex/105309-1304?qs=P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; Manufacturer (none) -> Molex; Manufacturer_Part_Number (none) -> 105309-1304
- J5: Distrbutor Link (none) -> https://www.digikey.com/en/products/detail/molex/1053091202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; Manufacturer (none) -> Molex; Manufacturer_Part_Number (none) -> 1053091202
- R1: Distrbutor Link (none) -> https://www.mouser.com/ProductDetail/Vishay/CRCW0603100KFKE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; Manufacturer (none) -> Vishay; Manufacturer_Part_Number (none) -> CRCW0603100KFKEE
- R2, R5: Distrbutor Link (none) -> https://www.mouser.com/ProductDetail/Vishay/CRCW06034K30FKE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; Manufacturer (none) -> Vishay; Manufacturer_Part_Number (none) -> CRCW06034K30FKEA
- R3: Distrbutor Link (none) -> https://www.mouser.com/ProductDetail/Vishay-Beyschlag/MCS04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; Manufacturer (none) -> Vishay / Beyschlag; Manufacturer_Part_Number (none) -> MCS0402MZ0000ZE000
- R4: Distrbutor Link (none) -> https://www.mouser.com/ProductDetail/Vishay/CRCW060347K0FKE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; Manufacturer (none) -> Vishay; Manufacturer_Part_Number (none) -> CRCW060347K0FKECC
- TP_12V1, TP_24V1, TP_3V1, TP_GND1: now left out of the parts list
- Z1: Distrbutor Link (none) -> https://www.mouser.com/ProductDetail/Micro-Commercial-Compo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; Manufacturer (none) -> Micro Commercial Components (MCC)
- Z2: Distrbutor Link (none) -> https://www.mccsemi.com/products/diodes/zener-diodes/SMAF47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; Manufacturer (none) -> Micro Commercial Components (MCC); Manufacturer_Part_Number SMAF4749A-TP -> SMAF4744A
