File: Buzzer.kicad_sch (KiCad schematic)
At the start: 5 parts, among them J1 BuzzConn, Q3 AO3400A

Commit message: revA4
Parts:
- removed C19: 10u, symbol Device:C
- removed J1: BuzzConn, symbol Connector_Generic:Conn_01x02
- removed Q3: AO3400A, Package_TO_SOT_SMD:SOT-23, symbol Transistor_FET:AO3400A
- removed R5: 100, symbol Device:R
- removed R6: 100k, symbol Device:R
- added C1: 0u1, symbol Device:C
- added C2: 10u, symbol Device:C
- added D1: 1N5819, Diode_THT:D_DO-41_SOD81_P10.16mm_Horizontal, symbol Diode:1N5819
- added J7: BuzzConn, symbol Connector_Generic:Conn_01x02
- added Q1: PSMN8R5-40MSDX, BUK7M1780EX, symbol utsvt_power:PSMN8R5-40MSDX
- added R1: 100k, symbol Device:R
Connections:
- net +12V: now also C1.1, C2.1, D1.1 (K), J7.1 (Pin_1)
- net BuzzPWM: now also Q1.4 (G), R1.2
- net GND: now also C1.2, C2.2, Q1.1 (S_1), R1.1
- new net: D1.2 (A), J7.2 (Pin_2), Q1.5 (D_1)
- no-connect marks 0 -> 8
Other:
- note added: "Bzz Bzz"
- note removed: "D"
- note removed: "G"
- note removed: "S"

Commit message: RevA5
Parts:
- C1: footprint (none) -> Capacitor_SMD:C_0603_1608Metric
- C2: footprint (none) -> Capacitor_SMD:C_0805_2012Metric
- R1: footprint (none) -> Resistor_SMD:R_0603_1608Metric
Changed lines of the file:
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@@
 			)
 		)
-		(property "Footprint" ""
+		(property "Footprint" "Resistor_SMD:R_0603_1608Metric"
 			(at 51.562 67.31 90)
 			(effects
@@
 			)
 		)
-		(property "Footprint" ""
+		(property "Footprint" "Capacitor_SMD:C_0805_2012Metric"
 			(at 91.7448 39.37 0)
 			(effects
@@
 			)
 		)
-		(property "Footprint" ""
+		(property "Footprint" "Capacitor_SMD:C_0603_1608Metric"
 			(at 104.4448 39.37 0)
 			(effects

Commit message: RevA6
Parts:
- J7: footprint (none) -> 1053091202
Changed lines of the file:
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@@
 			)
 		)
-		(property "Footprint" ""
+		(property "Footprint" "1053091202"
 			(at 135.89 49.53 0)
 			(effects
@@
 			)
 		)
-		(property "Datasheet" "https://www.amazon.com/Stemedu-Decibel-Sounder-Electronic-Continuous/dp/B096P5K9W1"
+		(property "Datasheet" "https://www.molex.com/en-us/products/part-detail/1053091202?display=pdf"
 			(at 135.89 49.53 0)
 			(effects

Commit message: RevA6 footprint updates
Parts:
- J7: footprint 1053091202 -> 153091202:1053091202
- Q1: footprint BUK7M1780EX -> UTSVT_Power:PSMN8R5-40MSDX
Changed lines of the file:
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@@
 			)
 		)
-		(property "Footprint" "1053091202"
+		(property "Footprint" "153091202:1053091202"
 			(at 135.89 49.53 0)
 			(effects
@@
 			)
 		)
-		(property "Footprint" "BUK7M1780EX"
+		(property "Footprint" "UTSVT_Power:PSMN8R5-40MSDX"
 			(at 93.98 146.99 0)
 			(effects

Commit message: RevA7 updates, dont review
Connections:
- net GND: now also Q1.2 (S_2), Q1.3 (S_3)
- net at D1.2 (A), J7.2 (Pin_2), Q1.5 (D_1): now also Q1.10 (D_6), Q1.11 (D_7), Q1.6 (D_2), Q1.7 (D_3), Q1.8 (D_4), Q1.9 (D_5)
- no-connect marks 8 -> 0
Changed lines of the file:
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@@
+	)
+	(junction
+		(at 67.31 54.61)
+		(diameter 0)
+		(color 0 0 0 0)
 	)
 	(junction
@@
 	)
 	(junction
+		(at 100.33 62.23)
+		(diameter 0)
+		(color 0 0 0 0)
+	)
+	(junction
+		(at 100.33 57.15)
+		(diameter 0)
+		(color 0 0 0 0)
+	)
+	(junction
 		(at 121.92 45.72)
 		(diameter 0)
@@
 	)
 	(junction
+		(at 67.31 52.07)
+		(diameter 0)
+		(color 0 0 0 0)
+	)
+	(junction
+		(at 100.33 59.69)
+		(diameter 0)
+		(color 0 0 0 0)
+	)
+	(junction
 		(at 92.71 31.75)
 		(diameter 0)
@@
 	)
 	(junction
+		(at 100.33 64.77)
+		(diameter 0)
+		(color 0 0 0 0)
+	)
+	(junction
+		(at 100.33 52.07)
+		(diameter 0)
+		(color 0 0 0 0)
+	)
+	(junction
 		(at 92.71 39.37)
 		(diameter 0)
 		(color 0 0 0 0)
 	)
-	(no_connect
-		(at 97.79 67.31)
-	)
-	(no_connect
-		(at 97.79 59.69)
-	)
-	(no_connect
-		(at 97.79 57.15)
-	)
-	(no_connect
-		(at 97.79 64.77)
-	)
-	(no_connect
-		(at 72.39 57.15)
-	)
-	(no_connect
-		(at 97.79 54.61)
-	)
-	(no_connect
-		(at 72.39 54.61)
-	)
-	(no_connect
-		(at 97.79 62.23)
+	(junction
+		(at 100.33 54.61)
+		(diameter 0)
+		(color 0 0 0 0)
+	)
+	(wire
+		(pts
+			(xy 97.79 59.69) (xy 100.33 59.69)
+		)
+		(stroke
+			(width 0)
+			(type default)
+		)
+	)
+	(wire
+		(pts
+			(xy 100.33 52.07) (xy 118.11 52.07)
+		)
+		(stroke
+			(width 0)
+			(type default)
+		)
+	)
+	(wire
+		(pts
+			(xy 97.79 62.23) (xy 100.33 62.23)
+		)
+		(stroke
+			(width 0)
+			(type default)
+		)
 	)
 	(wire
@@
 	(wire
 		(pts
-			(xy 97.79 52.07) (xy 118.11 52.07)
+			(xy 67.31 57.15) (xy 72.39 57.15)
+		)
+		(stroke
+			(width 0)
+			(type default)
+		)
+	)
+	(wire
+		(pts
+			(xy 97.79 64.77) (xy 100.33 64.77)
+		)
+		(stroke
+			(width 0)
+			(type default)
+		)
+	)
+	(wire
+		(pts
+			(xy 97.79 52.07) (xy 100.33 52.07)
+		)
+		(stroke
+			(width 0)
+			(type default)
+		)
+	)
+	(wire
+		(pts
+			(xy 100.33 59.69) (xy 100.33 57.15)
 		)
 		(stroke
@@
 	(wire
 		(pts
+			(xy 67.31 54.61) (xy 67.31 57.15)
+		)
+		(stroke
+			(width 0)
+			(type default)
+		)
+	)
+	(wire
+		(pts
 			(xy 121.92 45.72) (xy 125.73 45.72)
 		)
@@
 	(wire
 		(pts
+			(xy 97.79 57.15) (xy 100.33 57.15)
+		)
+		(stroke
+			(width 0)
+			(type default)
+		)
+	)
+	(wire
+		(pts
+			(xy 100.33 67.31) (xy 100.33 64.77)
+		)
+		(stroke
+			(width 0)
+			(type default)
+		)
+	)
+	(wire
+		(pts
+			(xy 100.33 62.23) (xy 100.33 59.69)
+		)
+		(stroke
+			(width 0)
+			(type default)
+		)
+	)
+	(wire
+		(pts
 			(xy 118.11 53.34) (xy 121.92 53.34)
 		)
@@
 	(wire
 		(pts
+			(xy 67.31 52.07) (xy 67.31 54.61)
+		)
+		(stroke
+			(width 0)
+			(type default)
+		)
+	)
+	(wire
+		(pts
 			(xy 53.34 59.69) (xy 72.39 59.69)
 		)
@@
 	(wire
 		(pts
+			(xy 67.31 54.61) (xy 72.39 54.61)
+		)
+		(stroke
+			(width 0)
+			(type default)
+		)
+	)
+	(wire
+		(pts
 			(xy 125.73 52.07) (xy 130.81 52.07)
 		)
@@
 	(wire
 		(pts
-			(xy 67.31 53.34) (xy 67.31 52.07)
+			(xy 67.31 48.26) (xy 67.31 52.07)
+		)
+		(stroke
+			(width 0)
+			(type default)
+		)
+	)
+	(wire
+		(pts
+			(xy 97.79 54.61) (xy 100.33 54.61)
+		)
+		(stroke
+			(width 0)
+			(type default)
+		)
+	)
+	(wire
+		(pts
+			(xy 97.79 67.31) (xy 100.33 67.31)
 		)
 		(stroke
@@
 		(pts
 			(xy 92.71 39.37) (xy 92.71 40.64)
+		)
+		(stroke
+			(width 0)
+			(type default)
+		)
+	)
+	(wire
+		(pts
+			(xy 100.33 64.77) (xy 100.33 62.23)
+		)
+		(stroke
+			(width 0)
+			(type default)
+		)
+	)
+	(wire
+		(pts
+			(xy 100.33 52.07) (xy 100.33 54.61)
+		)
+		(stroke
+			(width 0)
+			(type default)
+		)
+	)
+	(wire
+		(pts
+			(xy 100.33 57.15) (xy 100.33 54.61)
 		)
 		(stroke
@@
 	(symbol
 		(lib_id "power:GND")
-		(at 67.31 53.34 0)
+		(at 67.31 48.26 180)
 		(unit 1)
 		(exclude_from_sim no)
@@
 		(fields_autoplaced yes)
 		(property "Reference" "#PWR018"
-			(at 67.31 59.69 0)
+			(at 67.31 41.91 0)
 			(effects
 				(font
@@
 		)
 		(property "Value" "GND"
-			(at 67.31 58.42 0)
+			(at 67.31 43.18 0)
 			(effects
 				(font
@@
 		)
 		(property "Footprint" ""
-			(at 67.31 53.34 0)
+			(at 67.31 48.26 0)
 			(effects
 				(font
@@
 		)
 		(property "Datasheet" ""
-			(at 67.31 53.34 0)
+			(at 67.31 48.26 0)
 			(effects
 				(font
@@
 		)
 		(property "Description" "Power symbol creates a global label with name \"GND\" , ground"
-			(at 67.31 53.34 0)
-			(effects
-				(font
+			(at 67.31 48.26 0)
+			(effects
+				(font

Commit message: RevA9 for review
Parts:
- removed Q1: PSMN8R5-40MSDX, UTSVT_Power:PSMN8R5-40MSDX, symbol utsvt_power:PSMN8R5-40MSDX
- added Q4: PSMN8R5-40MSDX, UTSVT_Power:PSMN8R5-40MSDX, symbol utsvt_power:PSMN8R5-40MSDX
Connections:
- net BuzzPWM: now also Q4.2 (G)
- net GND: now also Q4.1 (S)
- net Buzz_Post_Diodes: now reaches D1.2 (A), J7.2 (Pin_2)
- net Buzz_Post_Diodes: now also Q4.3 (D)

Commit message: RevA9 small changes
Parts:
- renumbered C2 to C22, C1 to C23, D1 to D2, J7 to J6, Q4 to Q3, R1 to R14
Changed lines of the file:
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@@
 		(dnp no)
 		(fields_autoplaced yes)
-		(property "Reference" "Q4"
+		(property "Reference" "Q3"
 			(at 84.455 48.895 0)
 			(effects
@@
 			(project ""
 				(path "/d45494af-ff47-4110-bed2-dd613b557244/5a3494bd-2769-4cc7-96c1-4c8c29abb5e6"
-					(reference "Q4")
+					(reference "Q3")
 					(unit 1)
 				)
@@
 		(on_board yes)
 		(dnp no)
-		(property "Reference" "R1"
+		(property "Reference" "R14"
 			(at 50.292 66.548 0)
 			(effects
@@
 			(project "PS-ChargerInterfacePCB"
 				(path "/d45494af-ff47-4110-bed2-dd613b557244/5a3494bd-2769-4cc7-96c1-4c8c29abb5e6"
-					(reference "R1")
+					(reference "R14")
 					(unit 1)
 				)
@@
 		(on_board yes)
 		(dnp no)
-		(property "Reference" "D1"
+		(property "Reference" "D2"
 			(at 121.666 54.864 90)
 			(effects
@@
 			(project "PS-ChargerInterfacePCB"
 				(path "/d45494af-ff47-4110-bed2-dd613b557244/5a3494bd-2769-4cc7-96c1-4c8c29abb5e6"
-					(reference "D1")
+					(reference "D2")
 					(unit 1)
 				)
@@
 		(dnp no)
 		(fields_autoplaced yes)
-		(property "Reference" "#PWR020"
+		(property "Reference" "#PWR040"
 			(at 92.71 33.02 0)
 			(effects
@@
 			(project "PS-ChargerInterfacePCB"
 				(path "/d45494af-ff47-4110-bed2-dd613b557244/5a3494bd-2769-4cc7-96c1-4c8c29abb5e6"
-					(reference "#PWR020")
+					(reference "#PWR040")
 					(unit 1)
 				)
@@
 		(on_board yes)
 		(dnp no)
-		(property "Reference" "C2"
+		(property "Reference" "C22"
 			(at 89.408 34.29 0)
 			(effects
@@
 			(project "PS-ChargerInterfacePCB"
 				(path "/d45494af-ff47-4110-bed2-dd613b557244/5a3494bd-2769-4cc7-96c1-4c8c29abb5e6"
-					(reference "C2")
+					(reference "C22")
 					(unit 1)
 				)
@@
 		(on_board yes)
 		(dnp no)
-		(property "Reference" "C1"
+		(property "Reference" "C23"
 			(at 102.108 34.29 0)
 			(effects
@@
 			(project "PS-ChargerInterfacePCB"
 				(path "/d45494af-ff47-4110-bed2-dd613b557244/5a3494bd-2769-4cc7-96c1-4c8c29abb5e6"
-					(reference "C1")
+					(reference "C23")
 					(unit 1)
 				)
@@
 		(on_board yes)
 		(dnp no)
-		(property "Reference" "J7"
+		(property "Reference" "J6"
 			(at 135.89 43.18 0)
 			(effects
@@
 			(project "PS-ChargerInterfacePCB"
 				(path "/d45494af-ff47-4110-bed2-dd613b557244/5a3494bd-2769-4cc7-96c1-4c8c29abb5e6"
-					(reference "J7")
+					(reference "J6")
 					(unit 1)
 				)
@@
 		(dnp no)
 		(fields_autoplaced yes)
-		(property "Reference" "#PWR015"
+		(property "Reference" "#PWR038"
 			(at 53.34 80.01 0)
 			(effects
@@
 			(project "PS-ChargerInterfacePCB"
 				(path "/d45494af-ff47-4110-bed2-dd613b557244/5a3494bd-2769-4cc7-96c1-4c8c29abb5e6"
-					(reference "#PWR015")
+					(reference "#PWR038")
 					(unit 1)
 				)
@@
 		(dnp no)
 		(fields_autoplaced yes)
-		(property "Reference" "#PWR018"
+		(property "Reference" "#PWR039"
 			(at 67.31 41.91 0)
 			(effects
@@
 			(project "PS-ChargerInterfacePCB"
 				(path "/d45494af-ff47-4110-bed2-dd613b557244/5a3494bd-2769-4cc7-96c1-4c8c29abb5e6"
-					(reference "#PWR018")
+					(reference "#PWR039")
 					(unit 1)
 				)
@@
 		(dnp no)
 		(fields_autoplaced yes)
-		(property "Reference" "#PWR04"
+		(property "Reference" "#PWR041"
 			(at 92.71 46.99 0)
 			(effects
@@
 			(project ""
 				(path "/d45494af-ff47-4110-bed2-dd613b557244/5a3494bd-2769-4cc7-96c1-4c8c29abb5e6"
-					(reference "#PWR04")
-					(unit 1)
-				)
+					(reference "#PWR041")
+					(unit 1)
+				)

Commit message: RevA10 for review
Parts:
- removed D2: 1N5819, Diode_THT:D_DO-41_SOD81_P10.16mm_Horizontal, symbol Diode:1N5819
- added D2: D_Schottky, SK32A_LTP:SDO_DO-214AC-SMA_MCE, symbol Device:D_Schottky
- C22: Distrbutor Link (none) -> https://www.mouser.com/ProductDetail/Murata-Electronics/GRM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; Manufacturer (none) -> Murata Electronics; Manufacturer_Part_Number (none) -> GRM21BR61H106KE43K
- C23: value 0u1 -> 0.1u; Distrbutor Link (none) -> https://www.mouser.com/ProductDetail/TAIYO-YUDEN/MLASH168SB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; Manufacturer (none) -> TAIYO YUDEN; Manufacturer_Part_Number (none) -> MLASH168SB7104KTNA01
- J6: Distrbutor Link (none) -> https://www.digikey.com/en/products/detail/molex/1053091202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; Manufacturer (none) -> Molex; Manufacturer_Part_Number (none) -> 1053091202
- Q3: Distrbutor Link (none) -> https://www.mouser.com/ProductDetail/Nexperia/PSMN8R5-40MSD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; Manufacturer (none) -> Nexperia
- R14: Distrbutor Link (none) -> https://www.mouser.com/ProductDetail/Vishay/CRCW0603100KFKE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; Manufacturer (none) -> Vishay; Manufacturer_Part_Number (none) -> CRCW0603100KFKEE
Connections:
- net +12V: now also D2.1 (K)
- net Buzz_Post_Diodes: now also D2.2 (A)
Changed lines of the file:
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@@
+	)
+	(junction
+		(at 105.41 31.75)
+		(diameter 0)
+		(color 0 0 0 0)
+	)
+	(junction
+		(at 92.71 31.75)
+		(diameter 0)
+		(color 0 0 0 0)
 	)
 	(junction
@@
 	)
 	(junction
-		(at 105.41 31.75)
-		(diameter 0)
-		(color 0 0 0 0)
-	)
-	(junction
-		(at 92.71 31.75)
-		(diameter 0)
-		(color 0 0 0 0)
-	)
-	(junction
 		(at 92.71 39.37)
 		(diameter 0)
@@
 	(wire
 		(pts
+			(xy 121.92 53.34) (xy 125.73 53.34)
+		)
+		(stroke
+			(width 0)
+			(type default)
+		)
+	)
+	(wire
+		(pts
 			(xy 125.73 45.72) (xy 125.73 49.53)
 		)
@@
 	(wire
 		(pts
-			(xy 125.73 53.34) (xy 121.92 53.34)
-		)
-		(stroke
-			(width 0)
-			(type default)
-		)
-	)
-	(wire
-		(pts
 			(xy 53.34 63.5) (xy 53.34 59.69)
 		)
@@
 	(wire
 		(pts
+			(xy 76.2 62.865) (xy 84.455 62.865)
+		)
+		(stroke
+			(width 0)
+			(type default)
+		)
+	)
+	(wire
+		(pts
 			(xy 121.92 45.72) (xy 125.73 45.72)
-		)
-		(stroke
-			(width 0)
-			(type default)
-		)
-	)
-	(wire
-		(pts
-			(xy 76.2 62.865) (xy 84.455 62.865)
 		)
 		(stroke
@@
 			)
 		)
+		(property "Distrbutor Link" "https://www.mouser.com/ProductDetail/Nexperia/PSMN8R5-40MSDX?qs=vHuUswq2%252BswjdnYdBdHaPw%3D%3D&srsltid=AfmBOoqfk8rzjvl6Boo70jTxvjxp_5zF02h80jXmt8EqD9mSqXKDmpWA"
+			(at 84.455 56.515 0)
+			(effects
+				(font
+					(size 1.27 1.27)
+				)
+				(hide yes)
+			)
+		)
+		(property "Manufacturer" "Nexperia"
+			(at 84.455 56.515 0)
+			(effects
+				(font
+					(size 1.27 1.27)
+				)
+				(hide yes)
+			)
+		)
 		(pin "2"
 		)
@@
 			)
 		)
+		(property "Distrbutor Link" "https://www.mouser.com/ProductDetail/Vishay/CRCW0603100KFKEE?qs=%252B6g0mu59x7I1D%252BO0qMg%252Bjg%3D%3D&srsltid=AfmBOopUoX5SRH4kgw3t3NsysWvdNpHKSQXbyiBR5Kri4fiJTbfEazFl"
+			(at 53.34 67.31 0)
+			(effects
+				(font
+					(size 1.27 1.27)
+				)
+				(hide yes)
+			)
+		)
+		(property "Manufacturer" "Vishay"
+			(at 53.34 67.31 0)
+			(effects
+				(font
+					(size 1.27 1.27)
+				)
+				(hide yes)
+			)
+		)
+		(property "Manufacturer_Part_Number" "CRCW0603100KFKEE"
+			(at 53.34 67.31 0)
+			(effects
+				(font
+					(size 1.27 1.27)
+				)
+				(hide yes)
+			)
+		)
 		(pin "1"
 		)
@@
 				(path "/d45494af-ff47-4110-bed2-dd613b557244/5a3494bd-2769-4cc7-96c1-4c8c29abb5e6"
 					(reference "R14")
-					(unit 1)
-				)
-			)
-		)
-	)
-	(symbol
-		(lib_id "Diode:1N5819")
-		(at 121.92 49.53 270)
-		(unit 1)
-		(exclude_from_sim no)
-		(in_bom yes)
-		(on_board yes)
-		(dnp no)
-		(property "Reference" "D2"
-			(at 121.666 54.864 90)
-			(effects
-				(font
-					(size 1.27 1.27)
-				)
-			)
-		)
-		(property "Value" "1N5819"
-			(at 122.428 57.912 90)
-			(effects
-				(font
-					(size 1.27 1.27)
-				)
-			)
-		)
-		(property "Footprint" "Diode_THT:D_DO-41_SOD81_P10.16mm_Horizontal"
-			(at 117.475 49.53 0)
-			(effects
-				(font
-					(size 1.27 1.27)
-				)
-				(hide yes)
-			)
-		)
-		(property "Datasheet" "http://www.vishay.com/docs/88525/1n5817.pdf"
-			(at 121.92 49.53 0)
-			(effects
-				(font
-					(size 1.27 1.27)
-				)
-				(hide yes)
-			)
-		)
-		(property "Description" "40V 1A Schottky Barrier Rectifier Diode, DO-41"
-			(at 121.92 49.53 0)
-			(effects
-				(font
-					(size 1.27 1.27)
-				)
-				(hide yes)
-			)
-		)
-		(property "MANUFACTURER" ""
-			(at 121.92 49.53 90)
-			(effects
-				(font
-					(size 1.27 1.27)
-				)
-				(hide yes)
-			)
-		)
-		(property "PARTREV" ""
-			(at 121.92 49.53 90)
-			(effects
-				(font
-					(size 1.27 1.27)
-				)
-				(hide yes)
-			)
-		)
-		(property "STANDARD" ""
-			(at 121.92 49.53 90)
-			(effects
-				(font
-					(size 1.27 1.27)
-				)
-				(hide yes)
-			)
-		)
-		(pin "2"
-		)
-		(pin "1"
-		)
-		(instances
-			(project "PS-ChargerInterfacePCB"
-				(path "/d45494af-ff47-4110-bed2-dd613b557244/5a3494bd-2769-4cc7-96c1-4c8c29abb5e6"
-					(reference "D2")
 					(unit 1)
 				)
@@
 			)
 		)
+		(property "Distrbutor Link" "https://www.mouser.com/ProductDetail/Murata-Electronics/GRM21BR61H106KE43K?qs=xZ%2FP%252Ba9zWqbh3%252B96jyTKxw%3D%3D&srsltid=AfmBOooOWPD4zTBWFOdsFTWSEfQ5tcdFt57vSozifhtwlehrhxhA2k6m"
+			(at 92.71 35.56 0)
+			(effects
+				(font
+					(size 1.27 1.27)
+				)
+				(hide yes)
+			)
+		)
+		(property "Manufacturer" "Murata Electronics"
+			(at 92.71 35.56 0)
+			(effects
+				(font
+					(size 1.27 1.27)
+				)
+				(hide yes)
+			)
+		)
+		(property "Manufacturer_Part_Number" "GRM21BR61H106KE43K"
+			(at 92.71 35.56 0)
+			(effects
+				(font
+					(size 1.27 1.27)
+				)
+				(hide yes)
+			)
+		)
 		(pin "2"
 		)
@@
 			)
 		)
-		(property "Value" "0u1"
+		(property "Value" "0.1u"
 			(at 102.616 36.83 0)
 			(effects
@@
 		)
 		(property "STANDARD" ""
+			(at 105.41 35.56 0)
+			(effects
+				(font
+					(size 1.27 1.27)
+				)
+				(hide yes)
+			)
+		)
+		(property "Distrbutor Link" "https://www.mouser.com/ProductDetail/TAIYO-YUDEN/MLASH168SB7104KTNA01?qs=tlsG%2FOw5FFi7JK68L1DgIQ%3D%3D&srsltid=AfmBOorVpJ3mcbZ5tis8ztDksE2XqfTExs2YzjOUm6_fYjixjAtIEVC5"
+			(at 105.41 35.56 0)
+			(effects
+				(font
+					(size 1.27 1.27)
+				)
+				(hide yes)
+			)
+		)
+		(property "Manufacturer" "TAIYO YUDEN"
+			(at 105.41 35.56 0)
+			(effects
+				(font
+					(size 1.27 1.27)
+				)
+				(hide yes)
+			)
+		)
+		(property "Manufacturer_Part_Number" "MLASH168SB7104KTNA01"
 			(at 105.41 35.56 0)
 			(effects
@@
 				(path "/d45494af-ff47-4110-bed2-dd613b557244/5a3494bd-2769-4cc7-96c1-4c8c29abb5e6"
 					(reference "C23")
+					(unit 1)
+				)
+			)
+		)
+	)
+	(symbol
+		(lib_id "Device:D_Schottky")
+		(at 121.92 49.53 90)
+		(mirror x)
+		(unit 1)
+		(exclude_from_sim no)
+		(in_bom yes)
+		(on_board yes)
+		(dnp no)
+		(property "Reference" "D2"
+			(at 121.92 41.91 90)
+			(effects
+				(font
+					(size 1.27 1.27)
+				)
+			)
+		)
+		(property "Value" "D_Schottky"
+			(at 121.92 43.688 90)
+			(effects
+				(font
+					(size 1.27 1.27)
+				)
+			)
+		)
+		(property "Footprint" "SK32A_LTP:SDO_DO-214AC-SMA_MCE"
+			(at 121.92 49.53 0)
+			(effects
+				(font
+					(size 1.27 1.27)
+				)
+				(hide yes)
+			)
+		)
+		(property "Datasheet" "https://www.mouser.com/datasheet/3/225/1/SK32A-L-SK310A-L(SMA).pdf"
+			(at 121.92 49.53 0)
+			(effects
+				(font
+					(size 1.27 1.27)
+				)
+				(hide yes)
+			)
+		)
+		(property "Description" "Schottky diode"
+			(at 121.92 49.53 0)
+			(effects
+				(font
+					(size 1.27 1.27)
+				)
+				(hide yes)
+			)
+		)
+		(property "MANUFACTURER" ""
+			(at 121.92 49.53 0)
+			(effects
+				(font
+					(size 1.27 1.27)
+				)
+				(hide yes)
+			)
+		)
+		(property "PARTREV" ""
+			(at 121.92 49.53 0)
+			(effects
+				(font
+					(size 1.27 1.27)
+				)
+				(hide yes)
+			)
+		)
+		(property "STANDARD" ""
+			(at 121.92 49.53 0)
+			(effects
+				(font
+					(size 1.27 1.27)
+				)
+				(hide yes)
+			)
+		)
+		(property "Distrbutor Link" "https://www.mouser.com/ProductDetail/Micro-Commercial-Components-MCC/SK32A-LTP?qs=JeAkOuORR2U5XhGW5SLK2g%3D%3D&srsltid=AfmBOoqFiyx6irMBt28Q3Vo65pAmn7yAO98wOsjACKNj2Ab_fSU83u8p"
+			(at 121.92 49.53 90)
+			(effects
+				(font
+					(size 1.27 1.27)
+				)
+				(hide yes)
+			)
+		)
+		(property "Manufacturer" "Micro Commercial Components (MCC)"
+			(at 121.92 49.53 90)
+			(effects
+				(font
+					(size 1.27 1.27)
+				)
+				(hide yes)
+			)
+		)
+		(property "Manufacturer_Part_Number" "SK32A-LTP"
+			(at 121.92 49.53 90)
+			(effects
+				(font
+					(size 1.27 1.27)
+				)
+				(hide yes)
+			)
+		)
+		(pin "1"
+		)
+		(pin "2"
+		)
+		(instances
+			(project "PS-ChargerInterfacePCB"
+				(path "/d45494af-ff47-4110-bed2-dd613b557244/5a3494bd-2769-4cc7-96c1-4c8c29abb5e6"
+					(reference "D2")
 					(unit 1)
 				)
@@
 			(at 135.89 49.53 0)
 			(effects
+				(font
+					(size 1.27 1.27)
+				)
+				(hide yes)
+			)
+		)
+		(property "Distrbutor Link" "https://www.digikey.com/en/products/detail/molex/1053091202/6131607"
+			(at 135.89 49.53 0)
+			(effects
+				(font
+					(size 1.27 1.27)
+				)
+				(hide yes)
+			)
+		)
+		(property "Manufacturer" "Molex"
+			(at 135.89 49.53 0)
+			(effects
+				(font
+					(size 1.27 1.27)
+				)
+				(hide yes)
+			)
+		)
+		(property "Manufacturer_Part_Number" "1053091202"
+			(at 135.89 49.53 0)
+			(effects
