File: Buzzer.kicad_sch (KiCad schematic)
At the start: 5 parts, among them Q9 IRLML0030TRPBF

Commit message: implemented some of new comments
Parts:
- renumbered C70 to C31, C71 to C32, Q9 to Q1, R57 to R35
Other:
- moved on the sheet: C31, C32, Q1

Commit message: new orginization
Changed lines of the file:
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@@
-		)
-	)
-	(hierarchical_label "Buzz_Drain"
-		(shape input)
-		(at 58.42 45.72 0)
-		(effects
-			(font
-				(size 1.27 1.27)
-			)
-			(justify left)
 		)
 	)

Commit message: org stuf
Connections:
- net GND renamed BUZ_GND
Other:
- moved on the sheet: D1, Q1, R35

Commit message: final schem is done
Parts:
- C31: footprint Capacitor_SMD:C_0805_2012Metric -> Capacitor_SMD:C_0805_2012Metric_Pad1.18x1.45mm_HandSolder; Distrbutor Link https://www.mouser.com/ProductDetail/Murata-Electronics/GRM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 -> (none); Manufacturer Murata Electronics -> (none)
- C32: footprint Capacitor_SMD:C_0603_1608Metric -> Capacitor_SMD:C_0603_1608Metric_Pad1.08x0.95mm_HandSolder; Distrbutor Link https://www.mouser.com/ProductDetail/TAIYO-YUDEN/MLASH168SB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 -> (none); Manufacturer TAIYO YUDEN -> (none)
- D1: footprint (none) -> LHRS_Passives:SODFL5226X100N
- Q1: Height 1.12 -> (none); Manufacturer_Name Infineon -> (none); Manufacturer_Part_Number IRLML0030TRPBF -> (none); Mouser Part Number 942-IRLML0030TRPBF -> (none); Mouser Price/Stock https://www.mouser.co.uk/ProductDetail/Infineon-Technologie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 -> (none)
- R35: Distrbutor Link https://www.mouser.com/ProductDetail/Vishay/CRCW0603100KFKE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 -> (none); Manufacturer Vishay -> (none)

Commit message: shoupu review done
Changed lines of the file:
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@@
 	(text "BUZZZZZZZZZZZZZZZZ\n"
 		(exclude_from_sim no)
-		(at 24.892 14.224 0)
+		(at 25.4 13.97 0)
 		(effects
 			(font
@@
 		(color 0 0 0 0)
 	)
-	(bus_entry
-		(at 129.54 69.85)
-		(size 2.54 2.54)
-		(stroke
-			(width 0)
-			(type default)
-		)
-	)
 	(wire

Commit message: review council
Changed lines of the file:
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@@
+	)
+	(junction
+		(at 52.07 26.67)
+		(diameter 0)
+		(color 0 0 0 0)
 	)
 	(junction
@@
 	(wire
 		(pts
-			(xy 45.72 27.94) (xy 52.07 27.94)
+			(xy 45.72 26.67) (xy 52.07 26.67)
 		)
 		(stroke
@@
 	(hierarchical_label "BUZ_DRAIN"
 		(shape output)
-		(at 45.72 27.94 180)
-		(effects
-			(font
+		(at 45.72 26.67 180)
+		(effects
+			(font
