File: LEDIndicator.kicad_sch (KiCad schematic)
At the start: 8 parts

Commit message: small rev3 changes
Other:
- note removed: "add heartbeat leds"
Changed lines of the file:
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@@
 	(generator_version "9.0")
 	(paper "A4")
-	(text "add heartbeat leds"
-		(exclude_from_sim no)
-		(at 71.628 37.846 0)
-		(effects
-			(font
-				(size 1.27 1.27)
-			)
-		)
-	)
 	(text "R = (3.3V- Vf)/I\n590 = (3.3V - 2.12)/0.002\nI = 2mA (port limit?)\n\nVf = 2.2V (red leds?)\n"
 		(exclude_from_sim no)

Commit message: revA4
Changed lines of the file:
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@@
 	(generator_version "9.0")
 	(paper "A4")
+	(rectangle
+		(start 15.24 15.24)
+		(end 81.28 50.8)
+		(stroke
+			(width 0)
+			(type default)
+		)
+		(fill
+			(type none)
+		)
+	)
 	(text "R = (3.3V- Vf)/I\n590 = (3.3V - 2.12)/0.002\nI = 2mA (port limit?)\n\nVf = 2.2V (red leds?)\n"
 		(exclude_from_sim no)

Commit message: RevA9 small changes
Parts:
- renumbered D2 to D3, D3 to D4, D4 to D5, D5 to D6, R23 to R18
Changed lines of the file:
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@@
 		(on_board yes)
 		(dnp no)
-		(property "Reference" "#PWR041"
+		(property "Reference" "#PWR051"
 			(at 59.69 52.07 0)
 			(effects
@@
 			(project "PS-ChargerInterfacePCB"
 				(path "/d45494af-ff47-4110-bed2-dd613b557244/bb9f496a-74d6-44ce-af81-3e80cd51536d"
-					(reference "#PWR041")
+					(reference "#PWR051")
 					(unit 1)
 				)
@@
 		(on_board yes)
 		(dnp no)
-		(property "Reference" "R23"
+		(property "Reference" "R18"
 			(at 50.8 41.656 90)
 			(effects
@@
 			(project "PS-ChargerInterfacePCB"
 				(path "/d45494af-ff47-4110-bed2-dd613b557244/bb9f496a-74d6-44ce-af81-3e80cd51536d"
-					(reference "R23")
+					(reference "R18")
 					(unit 1)
 				)
@@
 		(on_board yes)
 		(dnp no)
-		(property "Reference" "#PWR029"
+		(property "Reference" "#PWR050"
 			(at 59.69 44.45 0)
 			(effects
@@
 			(project "PS-ChargerInterfacePCB"
 				(path "/d45494af-ff47-4110-bed2-dd613b557244/bb9f496a-74d6-44ce-af81-3e80cd51536d"
-					(reference "#PWR029")
+					(reference "#PWR050")
 					(unit 1)
 				)
@@
 		(on_board yes)
 		(dnp no)
-		(property "Reference" "D2"
+		(property "Reference" "D3"
 			(at 42.672 20.066 0)
 			(effects
@@
 			(project "PS-ChargerInterfacePCB"
 				(path "/d45494af-ff47-4110-bed2-dd613b557244/bb9f496a-74d6-44ce-af81-3e80cd51536d"
-					(reference "D2")
+					(reference "D3")
 					(unit 1)
 				)
@@
 		(on_board yes)
 		(dnp no)
-		(property "Reference" "D4"
+		(property "Reference" "D5"
 			(at 42.672 35.56 0)
 			(effects
@@
 			(project "PS-ChargerInterfacePCB"
 				(path "/d45494af-ff47-4110-bed2-dd613b557244/bb9f496a-74d6-44ce-af81-3e80cd51536d"
-					(reference "D4")
+					(reference "D5")
 					(unit 1)
 				)
@@
 		(on_board yes)
 		(dnp no)
-		(property "Reference" "#PWR017"
+		(property "Reference" "#PWR048"
 			(at 59.69 29.21 0)
 			(effects
@@
 			(project "PS-ChargerInterfacePCB"
 				(path "/d45494af-ff47-4110-bed2-dd613b557244/bb9f496a-74d6-44ce-af81-3e80cd51536d"
-					(reference "#PWR017")
+					(reference "#PWR048")
 					(unit 1)
 				)
@@
 		(on_board yes)
 		(dnp no)
-		(property "Reference" "D5"
+		(property "Reference" "D6"
 			(at 42.672 43.18 0)
 			(effects
@@
 			(project "PS-ChargerInterfacePCB"
 				(path "/d45494af-ff47-4110-bed2-dd613b557244/bb9f496a-74d6-44ce-af81-3e80cd51536d"
-					(reference "D5")
+					(reference "D6")
 					(unit 1)
 				)
@@
 		(on_board yes)
 		(dnp no)
-		(property "Reference" "#PWR019"
+		(property "Reference" "#PWR049"
 			(at 59.69 36.83 0)
 			(effects
@@
 			(project "PS-ChargerInterfacePCB"
 				(path "/d45494af-ff47-4110-bed2-dd613b557244/bb9f496a-74d6-44ce-af81-3e80cd51536d"
-					(reference "#PWR019")
+					(reference "#PWR049")
 					(unit 1)
 				)
@@
 		(on_board yes)
 		(dnp no)
-		(property "Reference" "D3"
+		(property "Reference" "D4"
 			(at 42.672 27.94 0)
 			(effects
@@
 			(project "PS-ChargerInterfacePCB"
 				(path "/d45494af-ff47-4110-bed2-dd613b557244/bb9f496a-74d6-44ce-af81-3e80cd51536d"
-					(reference "D3")
+					(reference "D4")
 					(unit 1)
 				)

Commit message: RevA10 for review
Parts:
- D3, D4, D5, D6: footprint LED_SMD:LED_0402_1005Metric -> LED_SMD:LED_0201_0603Metric; Distrbutor Link https://www.mouser.com/ProductDetail/Wurth-Elektronik/15004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 -> https://jlcpcb.com/partdetail/85432-NCD0603R1/C84263; Manufacturer Wurth Elektronik -> Foshan NationStar Optoelectronics; Manufacturer_Part_Number (none) -> NCD0603R1
- R15, R16, R17, R18: Distrbutor Link https://www.mouser.com/ProductDetail/YAGEO/RC0402FR-0722RL?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 -> https://www.mouser.com/ProductDetail/Vishay/CRCW0402590RFKE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; Manufacturer YAGEO -> Vishay; Manufacturer_Part_Number (none) -> CRCW0402590RFKED
Changed lines of the file:
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@@
 			)
 		)
-		(property "Distrbutor Link" "https://www.mouser.com/ProductDetail/YAGEO/RC0402FR-0722RL?qs=V1yeUXFNrkkRg6zf08ADKQ%3D%3D&srsltid=AfmBOor2cctyaIBQ_jqcS6bpD20PEk7e4pkUfEXfcnBnOJxoQq0CeGeb"
+		(property "Distrbutor Link" "https://www.mouser.com/ProductDetail/Vishay/CRCW0402590RFKED?qs=sGAEpiMZZMvdGkrng054txEw7b1YnvGup5OXobtv2Yw%3D"
 			(at 50.8 45.72 90)
 			(effects
@@
 			)
 		)
-		(property "Manufacturer" "YAGEO"
+		(property "Manufacturer" "Vishay"
 			(at 50.8 45.72 90)
 			(effects
@@
 		)
 		(property "STANDARD" ""
+			(at 50.8 45.72 90)
+			(effects
+				(font
+					(size 1.27 1.27)
+				)
+				(hide yes)
+			)
+		)
+		(property "Manufacturer_Part_Number" "CRCW0402590RFKED"
 			(at 50.8 45.72 90)
 			(effects
@@
 			)
 		)
-		(property "Footprint" "LED_SMD:LED_0402_1005Metric"
+		(property "Footprint" "LED_SMD:LED_0201_0603Metric"
 			(at 43.18 22.86 0)
 			(effects
@@
 			)
 		)
-		(property "Distrbutor Link" "https://www.mouser.com/ProductDetail/Wurth-Elektronik/150040RS73240?qs=sGAEpiMZZMv0DJfhVcWlKzXaUAZs%252BSGNmIzZWRrMt9JQwN0vgp7biA%3D%3D"
+		(property "Distrbutor Link" "https://jlcpcb.com/partdetail/85432-NCD0603R1/C84263"
 			(at 43.18 22.86 0)
 			(effects
@@
 			)
 		)
-		(property "Manufacturer" "Wurth Elektronik"
+		(property "Manufacturer" "Foshan NationStar Optoelectronics"
 			(at 43.18 22.86 0)
 			(effects
@@
 		)
 		(property "STANDARD" ""
+			(at 43.18 22.86 0)
+			(effects
+				(font
+					(size 1.27 1.27)
+				)
+				(hide yes)
+			)
+		)
+		(property "Manufacturer_Part_Number" "NCD0603R1"
 			(at 43.18 22.86 0)
 			(effects
@@
 			)
 		)
-		(property "Distrbutor Link" "https://www.mouser.com/ProductDetail/YAGEO/RC0402FR-0722RL?qs=V1yeUXFNrkkRg6zf08ADKQ%3D%3D&srsltid=AfmBOor2cctyaIBQ_jqcS6bpD20PEk7e4pkUfEXfcnBnOJxoQq0CeGeb"
+		(property "Distrbutor Link" "https://www.mouser.com/ProductDetail/Vishay/CRCW0402590RFKED?qs=sGAEpiMZZMvdGkrng054txEw7b1YnvGup5OXobtv2Yw%3D"
 			(at 50.8 30.48 90)
 			(effects
@@
 			)
 		)
-		(property "Manufacturer" "YAGEO"
+		(property "Manufacturer" "Vishay"
 			(at 50.8 30.48 90)
 			(effects
@@
 		)
 		(property "STANDARD" ""
+			(at 50.8 30.48 90)
+			(effects
+				(font
+					(size 1.27 1.27)
+				)
+				(hide yes)
+			)
+		)
+		(property "Manufacturer_Part_Number" "CRCW0402590RFKED"
 			(at 50.8 30.48 90)
 			(effects
@@
 			)
 		)
-		(property "Footprint" "LED_SMD:LED_0402_1005Metric"
+		(property "Footprint" "LED_SMD:LED_0201_0603Metric"
 			(at 43.18 38.1 0)
 			(effects
@@
 			)
 		)
-		(property "Distrbutor Link" "https://www.mouser.com/ProductDetail/Wurth-Elektronik/150040RS73240?qs=sGAEpiMZZMv0DJfhVcWlKzXaUAZs%252BSGNmIzZWRrMt9JQwN0vgp7biA%3D%3D"
+		(property "Distrbutor Link" "https://jlcpcb.com/partdetail/85432-NCD0603R1/C84263"
 			(at 43.18 38.1 0)
 			(effects
@@
 			)
 		)
-		(property "Manufacturer" "Wurth Elektronik"
+		(property "Manufacturer" "Foshan NationStar Optoelectronics"
 			(at 43.18 38.1 0)
 			(effects
@@
 		)
 		(property "STANDARD" ""
+			(at 43.18 38.1 0)
+			(effects
+				(font
+					(size 1.27 1.27)
+				)
+				(hide yes)
+			)
+		)
+		(property "Manufacturer_Part_Number" "NCD0603R1"
 			(at 43.18 38.1 0)
 			(effects
@@
 			)
 		)
-		(property "Footprint" "LED_SMD:LED_0402_1005Metric"
+		(property "Footprint" "LED_SMD:LED_0201_0603Metric"
 			(at 43.18 45.72 0)
 			(effects
@@
 			)
 		)
-		(property "Distrbutor Link" "https://www.mouser.com/ProductDetail/Wurth-Elektronik/150040RS73240?qs=sGAEpiMZZMv0DJfhVcWlKzXaUAZs%252BSGNmIzZWRrMt9JQwN0vgp7biA%3D%3D"
+		(property "Distrbutor Link" "https://jlcpcb.com/partdetail/85432-NCD0603R1/C84263"
 			(at 43.18 45.72 0)
 			(effects
@@
 			)
 		)
-		(property "Manufacturer" "Wurth Elektronik"
+		(property "Manufacturer" "Foshan NationStar Optoelectronics"
 			(at 43.18 45.72 0)
 			(effects
@@
 		)
 		(property "STANDARD" ""
+			(at 43.18 45.72 0)
+			(effects
+				(font
+					(size 1.27 1.27)
+				)
+				(hide yes)
+			)
+		)
+		(property "Manufacturer_Part_Number" "NCD0603R1"
 			(at 43.18 45.72 0)
 			(effects
@@
 			)
 		)
-		(property "Distrbutor Link" "https://www.mouser.com/ProductDetail/YAGEO/RC0402FR-0722RL?qs=V1yeUXFNrkkRg6zf08ADKQ%3D%3D&srsltid=AfmBOor2cctyaIBQ_jqcS6bpD20PEk7e4pkUfEXfcnBnOJxoQq0CeGeb"
+		(property "Distrbutor Link" "https://www.mouser.com/ProductDetail/Vishay/CRCW0402590RFKED?qs=sGAEpiMZZMvdGkrng054txEw7b1YnvGup5OXobtv2Yw%3D"
 			(at 50.8 22.86 90)
 			(effects
@@
 			)
 		)
-		(property "Manufacturer" "YAGEO"
+		(property "Manufacturer" "Vishay"
 			(at 50.8 22.86 90)
 			(effects
@@
 		)
 		(property "STANDARD" ""
+			(at 50.8 22.86 90)
+			(effects
+				(font
+					(size 1.27 1.27)
+				)
+				(hide yes)
+			)
+		)
+		(property "Manufacturer_Part_Number" "CRCW0402590RFKED"
 			(at 50.8 22.86 90)
 			(effects
@@
 			)
 		)
-		(property "Distrbutor Link" "https://www.mouser.com/ProductDetail/YAGEO/RC0402FR-0722RL?qs=V1yeUXFNrkkRg6zf08ADKQ%3D%3D&srsltid=AfmBOor2cctyaIBQ_jqcS6bpD20PEk7e4pkUfEXfcnBnOJxoQq0CeGeb"
+		(property "Distrbutor Link" "https://www.mouser.com/ProductDetail/Vishay/CRCW0402590RFKED?qs=sGAEpiMZZMvdGkrng054txEw7b1YnvGup5OXobtv2Yw%3D"
 			(at 50.8 38.1 90)
 			(effects
@@
 			)
 		)
-		(property "Manufacturer" "YAGEO"
+		(property "Manufacturer" "Vishay"
 			(at 50.8 38.1 90)
 			(effects
@@
 		)
 		(property "STANDARD" ""
+			(at 50.8 38.1 90)
+			(effects
+				(font
+					(size 1.27 1.27)
+				)
+				(hide yes)
+			)
+		)
+		(property "Manufacturer_Part_Number" "CRCW0402590RFKED"
 			(at 50.8 38.1 90)
 			(effects
@@
 			)
 		)
-		(property "Footprint" "LED_SMD:LED_0402_1005Metric"
+		(property "Footprint" "LED_SMD:LED_0201_0603Metric"
 			(at 43.18 30.48 0)
 			(effects
@@
 			)
 		)
-		(property "Distrbutor Link" "https://www.mouser.com/ProductDetail/Wurth-Elektronik/150040RS73240?qs=sGAEpiMZZMv0DJfhVcWlKzXaUAZs%252BSGNmIzZWRrMt9JQwN0vgp7biA%3D%3D"
+		(property "Distrbutor Link" "https://jlcpcb.com/partdetail/85432-NCD0603R1/C84263"
 			(at 43.18 30.48 0)
 			(effects
@@
 			)
 		)
-		(property "Manufacturer" "Wurth Elektronik"
+		(property "Manufacturer" "Foshan NationStar Optoelectronics"
 			(at 43.18 30.48 0)
 			(effects
@@
 			(at 43.18 30.48 0)
 			(effects
+				(font
+					(size 1.27 1.27)
+				)
+				(hide yes)
+			)
+		)
+		(property "Manufacturer_Part_Number" "NCD0603R1"
+			(at 43.18 30.48 0)
+			(effects

Commit message: Final Push
Parts:
- D3, D4, D5, D6: footprint LED_SMD:LED_0201_0603Metric -> LED_SMD:LED_0603_1608Metric
- R15, R16, R17, R18: footprint Resistor_SMD:R_0402_1005Metric -> Resistor_SMD:R_0603_1608Metric
Changed lines of the file:
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@@
 			)
 		)
-		(property "Footprint" "Resistor_SMD:R_0402_1005Metric"
+		(property "Footprint" "Resistor_SMD:R_0603_1608Metric"
 			(at 50.8 47.498 90)
 			(effects
@@
 			)
 		)
-		(property "Footprint" "LED_SMD:LED_0201_0603Metric"
+		(property "Footprint" "LED_SMD:LED_0603_1608Metric"
 			(at 43.18 22.86 0)
 			(effects
@@
 			)
 		)
-		(property "Footprint" "Resistor_SMD:R_0402_1005Metric"
+		(property "Footprint" "Resistor_SMD:R_0603_1608Metric"
 			(at 50.8 32.258 90)
 			(effects
@@
 			)
 		)
-		(property "Footprint" "LED_SMD:LED_0201_0603Metric"
+		(property "Footprint" "LED_SMD:LED_0603_1608Metric"
 			(at 43.18 38.1 0)
 			(effects
@@
 			)
 		)
-		(property "Footprint" "LED_SMD:LED_0201_0603Metric"
+		(property "Footprint" "LED_SMD:LED_0603_1608Metric"
 			(at 43.18 45.72 0)
 			(effects
@@
 			)
 		)
-		(property "Footprint" "Resistor_SMD:R_0402_1005Metric"
+		(property "Footprint" "Resistor_SMD:R_0603_1608Metric"
 			(at 50.8 24.638 90)
 			(effects
@@
 			)
 		)
-		(property "Footprint" "Resistor_SMD:R_0402_1005Metric"
+		(property "Footprint" "Resistor_SMD:R_0603_1608Metric"
 			(at 50.8 39.878 90)
 			(effects
@@
 			)
 		)
-		(property "Footprint" "LED_SMD:LED_0201_0603Metric"
+		(property "Footprint" "LED_SMD:LED_0603_1608Metric"
 			(at 43.18 30.48 0)
 			(effects
