File: SPI_display.kicad_sch (KiCad schematic)
At the start: 13 parts

Commit message: small rev3 changes
Other:
- moved on the sheet: C42, C43, C44, C45, C46, C47, C48, C49, C50, C51, C52, C53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

Commit message: revA4
Other:
- note added: "SPI Display"
- moved on the sheet: C44, C45, C52, C53
Changed lines of the file:
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@@
 	(generator_version "9.0")
 	(paper "A4")
+	(rectangle
+		(start 21.59 17.78)
+		(end 158.75 80.01)
+		(stroke
+			(width 0)
+			(type default)
+		)
+		(fill
+			(type none)
+		)
+	)
+	(text "SPI Display"
+		(exclude_from_sim no)
+		(at 22.098 19.812 0)
+		(effects
+			(font
+				(size 1.27 1.27)
+			)
+			(justify left)
+		)
+	)
 	(junction
 		(at 137.16 72.39)
@@
 	)
 	(junction
-		(at 58.42 68.58)
+		(at 30.48 49.53)
 		(diameter 0)
 		(color 0 0 0 0)
 	)
 	(junction
-		(at 71.12 68.58)
+		(at 43.18 49.53)
 		(diameter 0)
 		(color 0 0 0 0)
 	)
 	(junction
-		(at 58.42 82.55)
+		(at 30.48 63.5)
 		(diameter 0)
 		(color 0 0 0 0)
@@
 	)
 	(junction
-		(at 71.12 82.55)
+		(at 43.18 63.5)
 		(diameter 0)
 		(color 0 0 0 0)
@@
 	(wire
 		(pts
-			(xy 71.12 76.2) (xy 58.42 76.2)
-		)
-		(stroke
-			(width 0)
-			(type default)
-		)
-	)
-	(wire
-		(pts
-			(xy 58.42 68.58) (xy 71.12 68.58)
+			(xy 43.18 57.15) (xy 30.48 57.15)
+		)
+		(stroke
+			(width 0)
+			(type default)
+		)
+	)
+	(wire
+		(pts
+			(xy 30.48 49.53) (xy 43.18 49.53)
 		)
 		(stroke
@@
 	(wire
 		(pts
-			(xy 71.12 68.58) (xy 85.09 68.58)
+			(xy 43.18 49.53) (xy 57.15 49.53)
 		)
 		(stroke
@@
 	(wire
 		(pts
-			(xy 71.12 82.55) (xy 86.36 82.55)
+			(xy 43.18 63.5) (xy 58.42 63.5)
 		)
 		(stroke
@@
 	(wire
 		(pts
-			(xy 71.12 90.17) (xy 58.42 90.17)
-		)
-		(stroke
-			(width 0)
-			(type default)
-		)
-	)
-	(wire
-		(pts
-			(xy 58.42 82.55) (xy 71.12 82.55)
+			(xy 43.18 71.12) (xy 30.48 71.12)
+		)
+		(stroke
+			(width 0)
+			(type default)
+		)
+	)
+	(wire
+		(pts
+			(xy 30.48 63.5) (xy 43.18 63.5)
 		)
 		(stroke
@@
 	(wire
 		(pts
-			(xy 58.42 81.28) (xy 58.42 82.55)
+			(xy 30.48 62.23) (xy 30.48 63.5)
 		)
 		(stroke
@@
 	(wire
 		(pts
-			(xy 58.42 67.31) (xy 58.42 68.58)
+			(xy 30.48 48.26) (xy 30.48 49.53)
 		)
 		(stroke
@@
 	)
 	(label "Backlight_PWR"
-		(at 85.09 68.58 180)
+		(at 57.15 49.53 180)
 		(effects
 			(font
@@
 	)
 	(label "DisplayVDD"
-		(at 86.36 82.55 180)
+		(at 58.42 63.5 180)
 		(effects
 			(font
@@
 	(symbol
 		(lib_id "Device:C")
-		(at 71.12 86.36 0)
+		(at 43.18 67.31 0)
 		(unit 1)
 		(exclude_from_sim no)
@@
 		(dnp no)
 		(property "Reference" "C53"
-			(at 72.644 84.328 0)
+			(at 44.704 65.278 0)
 			(effects
 				(font
@@
 		)
 		(property "Value" "100n"
-			(at 73.914 86.36 0)
+			(at 45.974 67.31 0)
 			(effects
 				(font
@@
 		)
 		(property "Footprint" ""
-			(at 72.0852 90.17 0)
+			(at 44.1452 71.12 0)
 			(effects
 				(font
@@
 		)
 		(property "Datasheet" "~"
-			(at 71.12 86.36 0)
+			(at 43.18 67.31 0)
 			(effects
 				(font
@@
 		)
 		(property "Description" "Unpolarized capacitor"
-			(at 71.12 86.36 0)
+			(at 43.18 67.31 0)
 			(effects
 				(font
@@
 	(symbol
 		(lib_id "Device:C")
-		(at 71.12 72.39 0)
+		(at 43.18 53.34 0)
 		(unit 1)
 		(exclude_from_sim no)
@@
 		(dnp no)
 		(property "Reference" "C45"
-			(at 72.644 70.358 0)
+			(at 44.704 51.308 0)
 			(effects
 				(font
@@
 		)
 		(property "Value" "100n"
-			(at 73.914 72.39 0)
+			(at 45.974 53.34 0)
 			(effects
 				(font
@@
 		)
 		(property "Footprint" ""
-			(at 72.0852 76.2 0)
+			(at 44.1452 57.15 0)
 			(effects
 				(font
@@
 		)
 		(property "Datasheet" "~"
-			(at 71.12 72.39 0)
+			(at 43.18 53.34 0)
 			(effects
 				(font
@@
 		)
 		(property "Description" "Unpolarized capacitor"
-			(at 71.12 72.39 0)
+			(at 43.18 53.34 0)
 			(effects
 				(font
@@
 	(symbol
 		(lib_id "Device:C")
-		(at 58.42 86.36 0)
+		(at 30.48 67.31 0)
 		(unit 1)
 		(exclude_from_sim no)
@@
 		(dnp no)
 		(property "Reference" "C52"
-			(at 52.324 84.582 0)
+			(at 24.384 65.532 0)
 			(effects
 				(font
@@
 		)
 		(property "Value" "4u7"
-			(at 51.816 86.868 0)
+			(at 23.876 67.818 0)
 			(effects
 				(font
@@
 		)
 		(property "Footprint" ""
-			(at 59.3852 90.17 0)
+			(at 31.4452 71.12 0)
 			(effects
 				(font
@@
 		)
 		(property "Datasheet" "~"
-			(at 58.42 86.36 0)
+			(at 30.48 67.31 0)
 			(effects
 				(font
@@
 		)
 		(property "Description" "Unpolarized capacitor"
-			(at 58.42 86.36 0)
+			(at 30.48 67.31 0)
 			(effects
 				(font
@@
 	(symbol
 		(lib_id "power:+3.3V")
-		(at 58.42 81.28 0)
+		(at 30.48 62.23 0)
 		(mirror y)
 		(unit 1)
@@
 		(dnp no)
 		(property "Reference" "#PWR048"
-			(at 58.42 85.09 0)
+			(at 30.48 66.04 0)
 			(effects
 				(font
@@
 		)
 		(property "Value" "+3.3V"
-			(at 61.722 81.026 0)
+			(at 33.782 61.976 0)
 			(effects
 				(font
@@
 		)
 		(property "Footprint" ""
-			(at 58.42 81.28 0)
+			(at 30.48 62.23 0)
 			(effects
 				(font
@@
 		)
 		(property "Datasheet" ""
-			(at 58.42 81.28 0)
+			(at 30.48 62.23 0)
 			(effects
 				(font
@@
 		)
 		(property "Description" "Power symbol creates a global label with name \"+3.3V\""
-			(at 58.42 81.28 0)
+			(at 30.48 62.23 0)
 			(effects
 				(font
@@
 	(symbol
 		(lib_id "power:+3.3V")
-		(at 58.42 67.31 0)
+		(at 30.48 48.26 0)
 		(mirror y)
 		(unit 1)
@@
 		(dnp no)
 		(property "Reference" "#PWR047"
-			(at 58.42 71.12 0)
+			(at 30.48 52.07 0)
 			(effects
 				(font
@@
 		)
 		(property "Value" "+3.3V"
-			(at 61.722 67.056 0)
+			(at 33.782 48.006 0)
 			(effects
 				(font
@@
 		)
 		(property "Footprint" ""
-			(at 58.42 67.31 0)
+			(at 30.48 48.26 0)
 			(effects
 				(font
@@
 		)
 		(property "Datasheet" ""
-			(at 58.42 67.31 0)
+			(at 30.48 48.26 0)
 			(effects
 				(font
@@
 		)
 		(property "Description" "Power symbol creates a global label with name \"+3.3V\""
-			(at 58.42 67.31 0)
+			(at 30.48 48.26 0)
 			(effects
 				(font
@@
 	(symbol
 		(lib_id "Device:C")
-		(at 58.42 72.39 0)
+		(at 30.48 53.34 0)
 		(unit 1)
 		(exclude_from_sim no)
@@
 		(dnp no)
 		(property "Reference" "C44"
-			(at 52.324 70.612 0)
+			(at 24.384 51.562 0)
 			(effects
 				(font
@@
 		)
 		(property "Value" "4u7"
-			(at 51.816 72.898 0)
+			(at 23.876 53.848 0)
 			(effects
 				(font
@@
 		)
 		(property "Footprint" ""
-			(at 59.3852 76.2 0)
+			(at 31.4452 57.15 0)
 			(effects
 				(font
@@
 		)
 		(property "Datasheet" "~"
-			(at 58.42 72.39 0)
+			(at 30.48 53.34 0)
 			(effects
 				(font
@@
 		)
 		(property "Description" "Unpolarized capacitor"
-			(at 58.42 72.39 0)
-			(effects
-				(font
+			(at 30.48 53.34 0)
+			(effects
+				(font

Commit message: RevA5
Parts:
- C42, C43, C44, C51, C52: footprint (none) -> Capacitor_SMD:C_0805_2012Metric
- C45, C46, C47, C48, C49, C50, C53: footprint (none) -> Capacitor_SMD:C_0603_1608Metric
Connections:
- net GND: now also C44.2, C45.2, C52.2, C53.2
Other:
- moved on the sheet: C44, C45, C52, C53

Commit message: RevA6 footprint updates
Parts:
- DS2: footprint NHDC12832A1ZFSBFBW3V3 -> NHD-C12832A1Z-FSB-FBW-3V3:NHDC12832A1ZFSBFBW3V3
Changed lines of the file:
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@@
 			)
 		)
-		(property "Footprint" "NHDC12832A1ZFSBFBW3V3"
+		(property "Footprint" "NHD-C12832A1Z-FSB-FBW-3V3:NHDC12832A1ZFSBFBW3V3"
 			(at 95.25 124.13 0)
 			(effects

Commit message: RevA9 small changes
Parts:
- renumbered C44 to C24, C45 to C25, C52 to C26, C53 to C27, C42 to C28, C43 to C29, C51 to C30, C50 to C31, C49 to C32, C48 to C33, C47 to C34, C46 to C35, DS2 to DS1
Changed lines of the file:
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@@
 		(on_board yes)
 		(dnp no)
-		(property "Reference" "C47"
+		(property "Reference" "C34"
 			(at 146.812 33.782 0)
 			(effects
@@
 			(project "PS-ChargerInterfacePCB"
 				(path "/d45494af-ff47-4110-bed2-dd613b557244/eaa01ebb-42bc-4c5b-a5da-d0a713cda722"
-					(reference "C47")
+					(reference "C34")
 					(unit 1)
 				)
@@
 		(on_board yes)
 		(dnp no)
-		(property "Reference" "C49"
+		(property "Reference" "C32"
 			(at 138.938 44.196 0)
 			(effects
@@
 			(project "PS-ChargerInterfacePCB"
 				(path "/d45494af-ff47-4110-bed2-dd613b557244/eaa01ebb-42bc-4c5b-a5da-d0a713cda722"
-					(reference "C49")
+					(reference "C32")
 					(unit 1)
 				)
@@
 		(on_board yes)
 		(dnp no)
-		(property "Reference" "C42"
+		(property "Reference" "C28"
 			(at 128.524 43.18 90)
 			(effects
@@
 			(project ""
 				(path "/d45494af-ff47-4110-bed2-dd613b557244/eaa01ebb-42bc-4c5b-a5da-d0a713cda722"
-					(reference "C42")
+					(reference "C28")
 					(unit 1)
 				)
@@
 		(on_board yes)
 		(dnp no)
-		(property "Reference" "C48"
+		(property "Reference" "C33"
 			(at 143.002 38.862 0)
 			(effects
@@
 			(project "PS-ChargerInterfacePCB"
 				(path "/d45494af-ff47-4110-bed2-dd613b557244/eaa01ebb-42bc-4c5b-a5da-d0a713cda722"
-					(reference "C48")
+					(reference "C33")
 					(unit 1)
 				)
@@
 		(on_board yes)
 		(dnp no)
-		(property "Reference" "C53"
+		(property "Reference" "C27"
 			(at 77.724 66.548 0)
 			(effects
@@
 			(project "PS-ChargerInterfacePCB"
 				(path "/d45494af-ff47-4110-bed2-dd613b557244/eaa01ebb-42bc-4c5b-a5da-d0a713cda722"
-					(reference "C53")
+					(reference "C27")
 					(unit 1)
 				)
@@
 		(on_board yes)
 		(dnp no)
-		(property "Reference" "C45"
+		(property "Reference" "C25"
 			(at 43.434 66.548 0)
 			(effects
@@
 			(project "PS-ChargerInterfacePCB"
 				(path "/d45494af-ff47-4110-bed2-dd613b557244/eaa01ebb-42bc-4c5b-a5da-d0a713cda722"
-					(reference "C45")
+					(reference "C25")
 					(unit 1)
 				)
@@
 		(on_board yes)
 		(dnp no)
-		(property "Reference" "C52"
+		(property "Reference" "C26"
 			(at 57.404 66.802 0)
 			(effects
@@
 			(project "PS-ChargerInterfacePCB"
 				(path "/d45494af-ff47-4110-bed2-dd613b557244/eaa01ebb-42bc-4c5b-a5da-d0a713cda722"
-					(reference "C52")
+					(reference "C26")
 					(unit 1)
 				)
@@
 		(on_board yes)
 		(dnp no)
-		(property "Reference" "C46"
+		(property "Reference" "C35"
 			(at 152.146 27.94 0)
 			(effects
@@
 			(project "PS-ChargerInterfacePCB"
 				(path "/d45494af-ff47-4110-bed2-dd613b557244/eaa01ebb-42bc-4c5b-a5da-d0a713cda722"
-					(reference "C46")
+					(reference "C35")
 					(unit 1)
 				)
@@
 		(dnp no)
 		(fields_autoplaced yes)
-		(property "Reference" "#PWR024"
+		(property "Reference" "#PWR043"
 			(at 29.21 81.28 0)
 			(effects
@@
 			(project ""
 				(path "/d45494af-ff47-4110-bed2-dd613b557244/eaa01ebb-42bc-4c5b-a5da-d0a713cda722"
-					(reference "#PWR024")
+					(reference "#PWR043")
 					(unit 1)
 				)
@@
 		(on_board yes)
 		(dnp no)
-		(property "Reference" "C50"
+		(property "Reference" "C31"
 			(at 135.382 49.276 0)
 			(effects
@@
 			(project "PS-ChargerInterfacePCB"
 				(path "/d45494af-ff47-4110-bed2-dd613b557244/eaa01ebb-42bc-4c5b-a5da-d0a713cda722"
-					(reference "C50")
+					(reference "C31")
 					(unit 1)
 				)
@@
 		(on_board yes)
 		(dnp no)
-		(property "Reference" "C43"
+		(property "Reference" "C29"
 			(at 128.27 48.26 90)
 			(effects
@@
 			(project "PS-ChargerInterfacePCB"
 				(path "/d45494af-ff47-4110-bed2-dd613b557244/eaa01ebb-42bc-4c5b-a5da-d0a713cda722"
-					(reference "C43")
+					(reference "C29")
 					(unit 1)
 				)
@@
 		(on_board yes)
 		(dnp no)
-		(property "Reference" "#PWR048"
+		(property "Reference" "#PWR044"
 			(at 63.5 67.31 0)
 			(effects
@@
 			(project "PS-ChargerInterfacePCB"
 				(path "/d45494af-ff47-4110-bed2-dd613b557244/eaa01ebb-42bc-4c5b-a5da-d0a713cda722"
-					(reference "#PWR048")
+					(reference "#PWR044")
 					(unit 1)
 				)
@@
 		(on_board yes)
 		(dnp no)
-		(property "Reference" "DS2"
+		(property "Reference" "DS1"
 			(at 103.124 21.082 0)
 			(effects
@@
 			(project ""
 				(path "/d45494af-ff47-4110-bed2-dd613b557244/eaa01ebb-42bc-4c5b-a5da-d0a713cda722"
-					(reference "DS2")
+					(reference "DS1")
 					(unit 1)
 				)
@@
 		(dnp no)
 		(fields_autoplaced yes)
-		(property "Reference" "#PWR049"
+		(property "Reference" "#PWR047"
 			(at 125.73 82.55 0)
 			(effects
@@
 			(project ""
 				(path "/d45494af-ff47-4110-bed2-dd613b557244/eaa01ebb-42bc-4c5b-a5da-d0a713cda722"
-					(reference "#PWR049")
+					(reference "#PWR047")
 					(unit 1)
 				)
@@
 		(on_board yes)
 		(dnp no)
-		(property "Reference" "#PWR047"
+		(property "Reference" "#PWR042"
 			(at 29.21 67.31 0)
 			(effects
@@
 			(project "PS-ChargerInterfacePCB"
 				(path "/d45494af-ff47-4110-bed2-dd613b557244/eaa01ebb-42bc-4c5b-a5da-d0a713cda722"
-					(reference "#PWR047")
+					(reference "#PWR042")
 					(unit 1)
 				)
@@
 		(on_board yes)
 		(dnp no)
-		(property "Reference" "C44"
+		(property "Reference" "C24"
 			(at 23.114 66.802 0)
 			(effects
@@
 			(project "PS-ChargerInterfacePCB"
 				(path "/d45494af-ff47-4110-bed2-dd613b557244/eaa01ebb-42bc-4c5b-a5da-d0a713cda722"
-					(reference "C44")
+					(reference "C24")
 					(unit 1)
 				)
@@
 		(dnp no)
 		(fields_autoplaced yes)
-		(property "Reference" "#PWR023"
+		(property "Reference" "#PWR045"
 			(at 63.5 81.28 0)
 			(effects
@@
 			(project ""
 				(path "/d45494af-ff47-4110-bed2-dd613b557244/eaa01ebb-42bc-4c5b-a5da-d0a713cda722"
-					(reference "#PWR023")
+					(reference "#PWR045")
 					(unit 1)
 				)
@@
 		(on_board yes)
 		(dnp no)
-		(property "Reference" "C51"
+		(property "Reference" "C30"
 			(at 129.794 54.356 0)
 			(effects
@@
 			(project "PS-ChargerInterfacePCB"
 				(path "/d45494af-ff47-4110-bed2-dd613b557244/eaa01ebb-42bc-4c5b-a5da-d0a713cda722"
-					(reference "C51")
-					(unit 1)
-				)
+					(reference "C30")
+					(unit 1)
+				)

Commit message: RevA10 for review
Parts:
- C24, C26: Distrbutor Link (none) -> https://www.mouser.com/ProductDetail/KYOCERA-AVX/08055D475K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; Manufacturer (none) -> KYOCERA AVX; Manufacturer_Part_Number (none) -> 08055D475KAT4A
- C25, C27: value 100n -> 0.1u; Distrbutor Link (none) -> https://www.mouser.com/ProductDetail/TAIYO-YUDEN/MLASH168SB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; Manufacturer (none) -> TAIYO YUDEN; Manufacturer_Part_Number (none) -> MLASH168SB7104KTNA01
- C28, C29, C30: Distrbutor Link (none) -> https://www.mouser.com/ProductDetail/TAIYO-YUDEN/MCJCT21GCB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; Manufacturer (none) -> TAIYO YUDEN; Manufacturer_Part_Number (none) -> MCJCT21GCB7225MTPA1J
- C31, C32, C33, C34, C35: Distrbutor Link (none) -> https://www.mouser.com/ProductDetail/TAIYO-YUDEN/MLASU168SB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; Manufacturer (none) -> TAIYO YUDEN; Manufacturer_Part_Number (none) -> MLASU168SB5105KTNA01
- DS1: Distrbutor Link (none) -> https://www.mouser.com/ProductDetail/Newhaven-Display/NHD-C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; Manufacturer (none) -> Newhaven Display

Commit message: Added BOM, CPL
Parts:
- C24, C26: Manufacturer_Part_Number 08055D475KAT4A -> (none); P/N (none) -> 08055D475KAT4A
- C25, C27: Manufacturer_Part_Number MLASH168SB7104KTNA01 -> (none); P/N (none) -> MLASH168SB7104KTNA01
- C28, C29, C30: Manufacturer_Part_Number MCJCT21GCB7225MTPA1J -> (none); P/N (none) -> MCJCT21GCB7225MTPA1J
- C31, C32, C33, C34, C35: Manufacturer_Part_Number MLASU168SB5105KTNA01 -> (none); P/N (none) -> MLASU168SB5105KTNA01
- DS1: Manufacturer_Part_Number NHD-C12832A1Z-FSB-FBW-3V3 -> (none); P/N (none) -> NHD-C12832A1Z-FSB-FBW-3V3
Changed lines of the file:
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@@
 			)
 		)
-		(property "Manufacturer_Part_Number" "MLASU168SB5105KTNA01"
+		(property "P/N" "MLASU168SB5105KTNA01"
 			(at 148.59 38.1 0)
 			(effects
@@
 			)
 		)
-		(property "Manufacturer_Part_Number" "MLASU168SB5105KTNA01"
+		(property "P/N" "MLASU168SB5105KTNA01"
 			(at 140.97 48.26 0)
 			(effects
@@
 			)
 		)
-		(property "Manufacturer_Part_Number" "MCJCT21GCB7225MTPA1J"
+		(property "P/N" "MCJCT21GCB7225MTPA1J"
 			(at 124.46 41.91 90)
 			(effects
@@
 			)
 		)
-		(property "Manufacturer_Part_Number" "MLASU168SB5105KTNA01"
+		(property "P/N" "MLASU168SB5105KTNA01"
 			(at 144.78 43.18 0)
 			(effects
@@
 			)
 		)
-		(property "Manufacturer_Part_Number" "MLASH168SB7104KTNA01"
+		(property "P/N" "MLASH168SB7104KTNA01"
 			(at 76.2 68.58 0)
 			(effects
@@
 			)
 		)
-		(property "Manufacturer_Part_Number" "MLASH168SB7104KTNA01"
+		(property "P/N" "MLASH168SB7104KTNA01"
 			(at 41.91 68.58 0)
 			(effects
@@
 			)
 		)
-		(property "Manufacturer_Part_Number" "08055D475KAT4A"
+		(property "P/N" "08055D475KAT4A"
 			(at 63.5 68.58 0)
 			(effects
@@
 			)
 		)
-		(property "Manufacturer_Part_Number" "MLASU168SB5105KTNA01"
+		(property "P/N" "MLASU168SB5105KTNA01"
 			(at 153.67 33.02 0)
 			(effects
@@
 			)
 		)
-		(property "Manufacturer_Part_Number" "MLASU168SB5105KTNA01"
+		(property "P/N" "MLASU168SB5105KTNA01"
 			(at 137.16 53.34 0)
 			(effects
@@
 			)
 		)
-		(property "Manufacturer_Part_Number" "MCJCT21GCB7225MTPA1J"
+		(property "P/N" "MCJCT21GCB7225MTPA1J"
 			(at 124.46 49.53 90)
 			(effects
@@
 			)
 		)
-		(property "Manufacturer_Part_Number" "NHD-C12832A1Z-FSB-FBW-3V3"
-			(at 95.25 824.13 0)
-			(effects
-				(font
-					(size 1.27 1.27)
-				)
-				(justify left top)
-				(hide yes)
-			)
-		)
 		(property "MANUFACTURER" ""
 			(at 119.38 29.21 0)
@@
 		)
 		(property "Manufacturer" "Newhaven Display"
+			(at 119.38 29.21 0)
+			(effects
+				(font
+					(size 1.27 1.27)
+				)
+				(hide yes)
+			)
+		)
+		(property "P/N" "NHD-C12832A1Z-FSB-FBW-3V3"
 			(at 119.38 29.21 0)
 			(effects
@@
 			)
 		)
-		(property "Manufacturer_Part_Number" "08055D475KAT4A"
+		(property "P/N" "08055D475KAT4A"
 			(at 29.21 68.58 0)
 			(effects
@@
 			)
 		)
-		(property "Manufacturer_Part_Number" "MCJCT21GCB7225MTPA1J"
+		(property "P/N" "MCJCT21GCB7225MTPA1J"
 			(at 132.08 58.42 0)
 			(effects
