File: Power.kicad_sch (KiCad schematic)
At the start: 11 parts, among them IC5 LM74502HDDFR, Q5 PSMN8R5-40MSDX

Commit message: RevA5 small changes
Other:
- note added: "Bypass Cap"
- note removed: "24 Input Bypass Cap"
Changed lines of the file:
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@@
 		)
 	)
-	(text "24 Input\nBypass Cap"
+	(text "Bypass Cap"
 		(exclude_from_sim no)
-		(at 117.094 59.436 0)
+		(at 117.094 58.674 0)
 		(effects
 			(font

Commit message: RevA8 layout changes
Parts:
- removed C33: 22n, Capacitor_SMD:C_0603_1608Metric, symbol Device:C
- removed Q5: PSMN8R5-40MSDX, UTSVT_Power:PSMN8R5-40MSDX, symbol UTSVT_Power:PSMN8R5-40MSDX
- added Q2: PSMN8R5-40MSDX, UTSVT_Power:PSMN8R5-40MSDX, symbol utsvt_power:PSMN8R5-40MSDX
Connections:
- net VIN: now also Q2.3 (D)
- net V_OUT: now also Q2.1 (S)
- net at IC5.6 (GATE): now also Q2.2 (G)

Commit message: RevA9 for review
Parts:
- removed 12V_TP3: TestPoint, UTSVT_Special:TestPoint_HEX_3mmID, symbol Connector:TestPoint
Other:
- note added: "Overvoltage Protection: 14.91V Vovr = (R2 * Vov)/(R1 + R2) Vov = Vovr * (R1 + R2) / R2 14.91 = 1.25 * (47k + 4.3k) / 4.3k Vovr = 1.25V (datasheet)"
- note removed: "Overvoltage Protection: 14.91V Vovr = (R2 * Vov)/(R1 + R2) Vov = Vovr * (R1 + R2) / R2 18.125 = 1.25 * (47k + 4.3k) / 4.3k Vovr = 1.25V (datasheet)"

Commit message: RevA9 small changes
Parts:
- renumbered C31 to C10, C32 to C11, C34 to C12, C35 to C13, C36 to C14, C37 to C15, IC5 to IC2, Q2 to Q1, R22 to R12
Changed lines of the file:
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@@
 		(dnp no)
 		(fields_autoplaced yes)
-		(property "Reference" "#PWR058"
+		(property "Reference" "#PWR029"
 			(at 114.3 55.88 0)
 			(effects
@@
 			(project "PS-ChargerInterfacePCB"
 				(path "/d45494af-ff47-4110-bed2-dd613b557244/ac7656e7-8ca1-4189-8850-b703de13aef3"
-					(reference "#PWR052")
-					(unit 1)
-				)
-				(path "/d45494af-ff47-4110-bed2-dd613b557244/f4ec1410-3a5f-45f2-a31b-30d8be6fbeab"
-					(reference "#PWR058")
+					(reference "#PWR035")
+					(unit 1)
+				)
+				(path "/d45494af-ff47-4110-bed2-dd613b557244/f4ec1410-3a5f-45f2-a31b-30d8be6fbeab"
+					(reference "#PWR029")
 					(unit 1)
 				)
@@
 		(dnp no)
 		(fields_autoplaced yes)
-		(property "Reference" "#PWR056"
+		(property "Reference" "#PWR027"
 			(at 67.31 90.17 0)
 			(effects
@@
 			(project "PS-ChargerInterfacePCB"
 				(path "/d45494af-ff47-4110-bed2-dd613b557244/ac7656e7-8ca1-4189-8850-b703de13aef3"
-					(reference "#PWR050")
-					(unit 1)
-				)
-				(path "/d45494af-ff47-4110-bed2-dd613b557244/f4ec1410-3a5f-45f2-a31b-30d8be6fbeab"
-					(reference "#PWR056")
+					(reference "#PWR033")
+					(unit 1)
+				)
+				(path "/d45494af-ff47-4110-bed2-dd613b557244/f4ec1410-3a5f-45f2-a31b-30d8be6fbeab"
+					(reference "#PWR027")
 					(unit 1)
 				)
@@
 		(dnp no)
 		(fields_autoplaced yes)
-		(property "Reference" "C36"
+		(property "Reference" "C14"
 			(at 130.175 35.5599 0)
 			(effects
@@
 			(project "PS-ChargerInterfacePCB"
 				(path "/d45494af-ff47-4110-bed2-dd613b557244/ac7656e7-8ca1-4189-8850-b703de13aef3"
-					(reference "C29")
-					(unit 1)
-				)
-				(path "/d45494af-ff47-4110-bed2-dd613b557244/f4ec1410-3a5f-45f2-a31b-30d8be6fbeab"
-					(reference "C36")
+					(reference "C20")
+					(unit 1)
+				)
+				(path "/d45494af-ff47-4110-bed2-dd613b557244/f4ec1410-3a5f-45f2-a31b-30d8be6fbeab"
+					(reference "C14")
 					(unit 1)
 				)
@@
 		(dnp no)
 		(fields_autoplaced yes)
-		(property "Reference" "R22"
+		(property "Reference" "R12"
 			(at 44.45 46.9899 0)
 			(effects
@@
 			(project "PS-ChargerInterfacePCB"
 				(path "/d45494af-ff47-4110-bed2-dd613b557244/ac7656e7-8ca1-4189-8850-b703de13aef3"
-					(reference "R21")
-					(unit 1)
-				)
-				(path "/d45494af-ff47-4110-bed2-dd613b557244/f4ec1410-3a5f-45f2-a31b-30d8be6fbeab"
-					(reference "R22")
+					(reference "R13")
+					(unit 1)
+				)
+				(path "/d45494af-ff47-4110-bed2-dd613b557244/f4ec1410-3a5f-45f2-a31b-30d8be6fbeab"
+					(reference "R12")
 					(unit 1)
 				)
@@
 		(dnp no)
 		(fields_autoplaced yes)
-		(property "Reference" "C31"
+		(property "Reference" "C10"
 			(at 30.48 67.3099 0)
 			(effects
@@
 			(project "PS-ChargerInterfacePCB"
 				(path "/d45494af-ff47-4110-bed2-dd613b557244/ac7656e7-8ca1-4189-8850-b703de13aef3"
-					(reference "C24")
-					(unit 1)
-				)
-				(path "/d45494af-ff47-4110-bed2-dd613b557244/f4ec1410-3a5f-45f2-a31b-30d8be6fbeab"
-					(reference "C31")
+					(reference "C16")
+					(unit 1)
+				)
+				(path "/d45494af-ff47-4110-bed2-dd613b557244/f4ec1410-3a5f-45f2-a31b-30d8be6fbeab"
+					(reference "C10")
 					(unit 1)
 				)
@@
 		(on_board yes)
 		(dnp no)
-		(property "Reference" "IC5"
+		(property "Reference" "IC2"
 			(at 67.31 57.785 0)
 			(effects
@@
 			(project "PS-ChargerInterfacePCB"
 				(path "/d45494af-ff47-4110-bed2-dd613b557244/ac7656e7-8ca1-4189-8850-b703de13aef3"
-					(reference "IC4")
-					(unit 1)
-				)
-				(path "/d45494af-ff47-4110-bed2-dd613b557244/f4ec1410-3a5f-45f2-a31b-30d8be6fbeab"
-					(reference "IC5")
+					(reference "IC3")
+					(unit 1)
+				)
+				(path "/d45494af-ff47-4110-bed2-dd613b557244/f4ec1410-3a5f-45f2-a31b-30d8be6fbeab"
+					(reference "IC2")
 					(unit 1)
 				)
@@
 		(on_board yes)
 		(dnp no)
-		(property "Reference" "Q2"
+		(property "Reference" "Q1"
 			(at 67.945 20.955 0)
 			(effects
@@
 			(project ""
 				(path "/d45494af-ff47-4110-bed2-dd613b557244/ac7656e7-8ca1-4189-8850-b703de13aef3"
-					(reference "Q3")
-					(unit 1)
-				)
-				(path "/d45494af-ff47-4110-bed2-dd613b557244/f4ec1410-3a5f-45f2-a31b-30d8be6fbeab"
 					(reference "Q2")
+					(unit 1)
+				)
+				(path "/d45494af-ff47-4110-bed2-dd613b557244/f4ec1410-3a5f-45f2-a31b-30d8be6fbeab"
+					(reference "Q1")
 					(unit 1)
 				)
@@
 		(dnp no)
 		(fields_autoplaced yes)
-		(property "Reference" "C37"
+		(property "Reference" "C15"
 			(at 140.335 35.5599 0)
 			(effects
@@
 			(project "PS-ChargerInterfacePCB"
 				(path "/d45494af-ff47-4110-bed2-dd613b557244/ac7656e7-8ca1-4189-8850-b703de13aef3"
-					(reference "C30")
-					(unit 1)
-				)
-				(path "/d45494af-ff47-4110-bed2-dd613b557244/f4ec1410-3a5f-45f2-a31b-30d8be6fbeab"
-					(reference "C37")
+					(reference "C21")
+					(unit 1)
+				)
+				(path "/d45494af-ff47-4110-bed2-dd613b557244/f4ec1410-3a5f-45f2-a31b-30d8be6fbeab"
+					(reference "C15")
 					(unit 1)
 				)
@@
 		(dnp no)
 		(fields_autoplaced yes)
-		(property "Reference" "#PWR057"
+		(property "Reference" "#PWR028"
 			(at 88.9 53.34 0)
 			(effects
@@
 			(project "PS-ChargerInterfacePCB"
 				(path "/d45494af-ff47-4110-bed2-dd613b557244/ac7656e7-8ca1-4189-8850-b703de13aef3"
-					(reference "#PWR051")
-					(unit 1)
-				)
-				(path "/d45494af-ff47-4110-bed2-dd613b557244/f4ec1410-3a5f-45f2-a31b-30d8be6fbeab"
-					(reference "#PWR057")
+					(reference "#PWR034")
+					(unit 1)
+				)
+				(path "/d45494af-ff47-4110-bed2-dd613b557244/f4ec1410-3a5f-45f2-a31b-30d8be6fbeab"
+					(reference "#PWR028")
 					(unit 1)
 				)
@@
 		(dnp no)
 		(fields_autoplaced yes)
-		(property "Reference" "#PWR060"
+		(property "Reference" "#PWR031"
 			(at 137.16 55.88 0)
 			(effects
@@
 			(project "PS-ChargerInterfacePCB"
 				(path "/d45494af-ff47-4110-bed2-dd613b557244/ac7656e7-8ca1-4189-8850-b703de13aef3"
-					(reference "#PWR054")
-					(unit 1)
-				)
-				(path "/d45494af-ff47-4110-bed2-dd613b557244/f4ec1410-3a5f-45f2-a31b-30d8be6fbeab"
-					(reference "#PWR060")
+					(reference "#PWR037")
+					(unit 1)
+				)
+				(path "/d45494af-ff47-4110-bed2-dd613b557244/f4ec1410-3a5f-45f2-a31b-30d8be6fbeab"
+					(reference "#PWR031")
 					(unit 1)
 				)
@@
 		(dnp no)
 		(fields_autoplaced yes)
-		(property "Reference" "C34"
+		(property "Reference" "C12"
 			(at 92.075 41.9099 0)
 			(effects
@@
 			(project "PS-ChargerInterfacePCB"
 				(path "/d45494af-ff47-4110-bed2-dd613b557244/ac7656e7-8ca1-4189-8850-b703de13aef3"
-					(reference "C27")
-					(unit 1)
-				)
-				(path "/d45494af-ff47-4110-bed2-dd613b557244/f4ec1410-3a5f-45f2-a31b-30d8be6fbeab"
-					(reference "C34")
+					(reference "C18")
+					(unit 1)
+				)
+				(path "/d45494af-ff47-4110-bed2-dd613b557244/f4ec1410-3a5f-45f2-a31b-30d8be6fbeab"
+					(reference "C12")
 					(unit 1)
 				)
@@
 		(dnp no)
 		(fields_autoplaced yes)
-		(property "Reference" "#PWR059"
+		(property "Reference" "#PWR030"
 			(at 127 55.88 0)
 			(effects
@@
 			(project "PS-ChargerInterfacePCB"
 				(path "/d45494af-ff47-4110-bed2-dd613b557244/ac7656e7-8ca1-4189-8850-b703de13aef3"
-					(reference "#PWR053")
-					(unit 1)
-				)
-				(path "/d45494af-ff47-4110-bed2-dd613b557244/f4ec1410-3a5f-45f2-a31b-30d8be6fbeab"
-					(reference "#PWR059")
+					(reference "#PWR036")
+					(unit 1)
+				)
+				(path "/d45494af-ff47-4110-bed2-dd613b557244/f4ec1410-3a5f-45f2-a31b-30d8be6fbeab"
+					(reference "#PWR030")
 					(unit 1)
 				)
@@
 		(dnp no)
 		(fields_autoplaced yes)
-		(property "Reference" "C32"
+		(property "Reference" "C11"
 			(at 45.085 67.3099 0)
 			(effects
@@
 			(project "PS-ChargerInterfacePCB"
 				(path "/d45494af-ff47-4110-bed2-dd613b557244/ac7656e7-8ca1-4189-8850-b703de13aef3"
-					(reference "C25")
-					(unit 1)
-				)
-				(path "/d45494af-ff47-4110-bed2-dd613b557244/f4ec1410-3a5f-45f2-a31b-30d8be6fbeab"
-					(reference "C32")
+					(reference "C17")
+					(unit 1)
+				)
+				(path "/d45494af-ff47-4110-bed2-dd613b557244/f4ec1410-3a5f-45f2-a31b-30d8be6fbeab"
+					(reference "C11")
 					(unit 1)
 				)
@@
 		(dnp no)
 		(fields_autoplaced yes)
-		(property "Reference" "#PWR055"
+		(property "Reference" "#PWR026"
 			(at 34.29 80.01 0)
 			(effects
@@
 			(project "PS-ChargerInterfacePCB"
 				(path "/d45494af-ff47-4110-bed2-dd613b557244/ac7656e7-8ca1-4189-8850-b703de13aef3"
-					(reference "#PWR045")
-					(unit 1)
-				)
-				(path "/d45494af-ff47-4110-bed2-dd613b557244/f4ec1410-3a5f-45f2-a31b-30d8be6fbeab"
-					(reference "#PWR055")
+					(reference "#PWR032")
+					(unit 1)
+				)
+				(path "/d45494af-ff47-4110-bed2-dd613b557244/f4ec1410-3a5f-45f2-a31b-30d8be6fbeab"
+					(reference "#PWR026")
 					(unit 1)
 				)
@@
 		(dnp no)
 		(fields_autoplaced yes)
-		(property "Reference" "C35"
+		(property "Reference" "C13"
 			(at 118.11 35.5599 0)
 			(effects
@@
 			(project "PS-ChargerInterfacePCB"
 				(path "/d45494af-ff47-4110-bed2-dd613b557244/ac7656e7-8ca1-4189-8850-b703de13aef3"
-					(reference "C28")
-					(unit 1)
-				)
-				(path "/d45494af-ff47-4110-bed2-dd613b557244/f4ec1410-3a5f-45f2-a31b-30d8be6fbeab"
-					(reference "C35")
+					(reference "C19")
+					(unit 1)
+				)
+				(path "/d45494af-ff47-4110-bed2-dd613b557244/f4ec1410-3a5f-45f2-a31b-30d8be6fbeab"
+					(reference "C13")
 					(unit 1)
 				)
@@
 		(dnp no)
 		(fields_autoplaced yes)
-		(property "Reference" "#FLG06"
+		(property "Reference" "#FLG02"
 			(at 95.25 36.195 0)
 			(effects
@@
 			(project "PS-ChargerInterfacePCB"
 				(path "/d45494af-ff47-4110-bed2-dd613b557244/ac7656e7-8ca1-4189-8850-b703de13aef3"
-					(reference "#FLG05")
-					(unit 1)
-				)
-				(path "/d45494af-ff47-4110-bed2-dd613b557244/f4ec1410-3a5f-45f2-a31b-30d8be6fbeab"
-					(reference "#FLG06")
-					(unit 1)
-				)
+					(reference "#FLG03")
+					(unit 1)
+				)
+				(path "/d45494af-ff47-4110-bed2-dd613b557244/f4ec1410-3a5f-45f2-a31b-30d8be6fbeab"
+					(reference "#FLG02")
+					(unit 1)
+				)

Commit message: RevA10 for review
Parts:
- C10: Distrbutor Link (none) -> https://www.mouser.com/ProductDetail/TAIYO-YUDEN/MLASU168SB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; Manufacturer (none) -> TAIYO YUDEN; Manufacturer_Part_Number (none) -> MLASU168SB5105KTNA01
- C11: value 220n -> 0.22u; Distrbutor Link (none) -> https://www.mouser.com/ProductDetail/TAIYO-YUDEN/MSASU168SB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; Manufacturer (none) -> TAIYO YUDEN; Manufacturer_Part_Number (none) -> MSASU168SB7224KTNB25
- C12, C13: Distrbutor Link (none) -> https://www.mouser.com/ProductDetail/Murata-Electronics/GRM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; Manufacturer (none) -> Murata Electronics; Manufacturer_Part_Number (none) -> GRM21BR61H106KE43K
- C14, C15: Distrbutor Link (none) -> https://www.mouser.com/ProductDetail/TAIYO-YUDEN/MLASH168SB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; Manufacturer (none) -> TAIYO YUDEN; Manufacturer_Part_Number (none) -> MLASH168SB7104KTNA01
- IC2: Distrbutor Link (none) -> https://www.mouser.com/ProductDetail/Texas-Instruments/LM74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; Manufacturer (none) -> Texas Instruments
- Q1: Distrbutor Link (none) -> https://www.mouser.com/ProductDetail/Nexperia/PSMN8R5-40MSD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; Manufacturer (none) -> Nexperia
- R12: Distrbutor Link (none) -> https://www.mouser.com/ProductDetail/Vishay/CRCW060310K0FKE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; Manufacturer (none) -> Vishay; Manufacturer_Part_Number (none) -> CRCW060310K0FKEI
Changed lines of the file:
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@@
+			)
+		)
+		(property "Distrbutor Link" "https://www.mouser.com/ProductDetail/TAIYO-YUDEN/MLASH168SB7104KTNA01?qs=tlsG%2FOw5FFi7JK68L1DgIQ%3D%3D&srsltid=AfmBOorVpJ3mcbZ5tis8ztDksE2XqfTExs2YzjOUm6_fYjixjAtIEVC5"
+			(at 127 36.83 0)
+			(effects
+				(font
+					(size 1.27 1.27)
+				)
+				(hide yes)
+			)
+		)
+		(property "Manufacturer" "TAIYO YUDEN"
+			(at 127 36.83 0)
+			(effects
+				(font
+					(size 1.27 1.27)
+				)
+				(hide yes)
+			)
+		)
+		(property "Manufacturer_Part_Number" "MLASH168SB7104KTNA01"
+			(at 127 36.83 0)
+			(effects
+				(font
+					(size 1.27 1.27)
+				)
+				(hide yes)
 			)
 		)
@@
 		)
 		(property "STANDARD" ""
+			(at 41.91 48.26 0)
+			(effects
+				(font
+					(size 1.27 1.27)
+				)
+				(hide yes)
+			)
+		)
+		(property "Distrbutor Link" "https://www.mouser.com/ProductDetail/Vishay/CRCW060310K0FKEI?qs=3qWEzBg5KnKofE%252B8acPBRA%3D%3D&srsltid=AfmBOopeC-KWud4lBTFtge_WyCoVbALtqYG1UPN_QCfpWzcG6F3pAdmo"
+			(at 41.91 48.26 0)
+			(effects
+				(font
+					(size 1.27 1.27)
+				)
+				(hide yes)
+			)
+		)
+		(property "Manufacturer" "Vishay"
+			(at 41.91 48.26 0)
+			(effects
+				(font
+					(size 1.27 1.27)
+				)
+				(hide yes)
+			)
+		)
+		(property "Manufacturer_Part_Number" "CRCW060310K0FKEI"
 			(at 41.91 48.26 0)
 			(effects
@@
 			)
 		)
+		(property "Distrbutor Link" "https://www.mouser.com/ProductDetail/TAIYO-YUDEN/MLASU168SB5105KTNA01?qs=tlsG%2FOw5FFhPjKzzJZMnOQ%3D%3D&srsltid=AfmBOorcMlsFle3SkG0XtJIKbOuFrpMRrEVUmZYMN7uFvSiB2BlKWNRY"
+			(at 34.29 68.58 0)
+			(effects
+				(font
+					(size 1.27 1.27)
+				)
+				(hide yes)
+			)
+		)
+		(property "Manufacturer" "TAIYO YUDEN"
+			(at 34.29 68.58 0)
+			(effects
+				(font
+					(size 1.27 1.27)
+				)
+				(hide yes)
+			)
+		)
+		(property "Manufacturer_Part_Number" "MLASU168SB5105KTNA01"
+			(at 34.29 68.58 0)
+			(effects
+				(font
+					(size 1.27 1.27)
+				)
+				(hide yes)
+			)
+		)
 		(pin "2"
 		)
@@
 		)
 		(property "STANDARD" ""
+			(at 50.8 64.77 0)
+			(effects
+				(font
+					(size 1.27 1.27)
+				)
+				(hide yes)
+			)
+		)
+		(property "Distrbutor Link" "https://www.mouser.com/ProductDetail/Texas-Instruments/LM74502HDDFR?qs=t7xnP681wgWDbfat8Yg%252B%2Fg%3D%3D&srsltid=AfmBOoq5cFNpUh1QodJ1dkyZnwnLQl8oMFYa9SuI8ZaVdKUNzEMaYa5s"
+			(at 50.8 64.77 0)
+			(effects
+				(font
+					(size 1.27 1.27)
+				)
+				(hide yes)
+			)
+		)
+		(property "Manufacturer" "Texas Instruments"
 			(at 50.8 64.77 0)
 			(effects
@@
 			)
 		)
+		(property "Distrbutor Link" "https://www.mouser.com/ProductDetail/Nexperia/PSMN8R5-40MSDX?qs=vHuUswq2%252BswjdnYdBdHaPw%3D%3D&srsltid=AfmBOoqfk8rzjvl6Boo70jTxvjxp_5zF02h80jXmt8EqD9mSqXKDmpWA"
+			(at 67.945 28.575 0)
+			(effects
+				(font
+					(size 1.27 1.27)
+				)
+				(hide yes)
+			)
+		)
+		(property "Manufacturer" "Nexperia"
+			(at 67.945 28.575 0)
+			(effects
+				(font
+					(size 1.27 1.27)
+				)
+				(hide yes)
+			)
+		)
 		(pin "2"
 		)
@@
 			)
 		)
+		(property "Distrbutor Link" "https://www.mouser.com/ProductDetail/TAIYO-YUDEN/MLASH168SB7104KTNA01?qs=tlsG%2FOw5FFi7JK68L1DgIQ%3D%3D&srsltid=AfmBOorVpJ3mcbZ5tis8ztDksE2XqfTExs2YzjOUm6_fYjixjAtIEVC5"
+			(at 137.16 36.83 0)
+			(effects
+				(font
+					(size 1.27 1.27)
+				)
+				(hide yes)
+			)
+		)
+		(property "Manufacturer" "TAIYO YUDEN"
+			(at 137.16 36.83 0)
+			(effects
+				(font
+					(size 1.27 1.27)
+				)
+				(hide yes)
+			)
+		)
+		(property "Manufacturer_Part_Number" "MLASH168SB7104KTNA01"
+			(at 137.16 36.83 0)
+			(effects
+				(font
+					(size 1.27 1.27)
+				)
+				(hide yes)
+			)
+		)
 		(pin "1"
 		)
@@
 		)
 		(property "STANDARD" ""
+			(at 88.9 43.18 0)
+			(effects
+				(font
+					(size 1.27 1.27)
+				)
+				(hide yes)
+			)
+		)
+		(property "Distrbutor Link" "https://www.mouser.com/ProductDetail/Murata-Electronics/GRM21BR61H106KE43K?qs=xZ%2FP%252Ba9zWqbh3%252B96jyTKxw%3D%3D&srsltid=AfmBOooOWPD4zTBWFOdsFTWSEfQ5tcdFt57vSozifhtwlehrhxhA2k6m"
+			(at 88.9 43.18 0)
+			(effects
+				(font
+					(size 1.27 1.27)
+				)
+				(hide yes)
+			)
+		)
+		(property "Manufacturer" "Murata Electronics"
+			(at 88.9 43.18 0)
+			(effects
+				(font
+					(size 1.27 1.27)
+				)
+				(hide yes)
+			)
+		)
+		(property "Manufacturer_Part_Number" "GRM21BR61H106KE43K"
 			(at 88.9 43.18 0)
 			(effects
@@
 			)
 		)
-		(property "Value" "220n"
+		(property "Value" "0.22u"
 			(at 45.085 69.8499 0)
 			(effects
@@
 		)
 		(property "STANDARD" ""
+			(at 41.91 68.58 0)
+			(effects
+				(font
+					(size 1.27 1.27)
+				)
+				(hide yes)
+			)
+		)
+		(property "Distrbutor Link" "https://www.mouser.com/ProductDetail/TAIYO-YUDEN/MSASU168SB7224KTNB25?qs=tlsG%2FOw5FFipzD362lh8GQ%3D%3D&srsltid=AfmBOopGYOC_my1aArrkkcgEqwtzTM9VZgH8ll-X52QaBFHxMr3S4Jt4"
+			(at 41.91 68.58 0)
+			(effects
+				(font
+					(size 1.27 1.27)
+				)
+				(hide yes)
+			)
+		)
+		(property "Manufacturer" "TAIYO YUDEN"
+			(at 41.91 68.58 0)
+			(effects
+				(font
+					(size 1.27 1.27)
+				)
+				(hide yes)
+			)
+		)
+		(property "Manufacturer_Part_Number" "MSASU168SB7224KTNB25"
 			(at 41.91 68.58 0)
 			(effects
@@
 			(at 114.3 36.83 0)
 			(effects
+				(font
+					(size 1.27 1.27)
+				)
+				(hide yes)
+			)
+		)
+		(property "Distrbutor Link" "https://www.mouser.com/ProductDetail/Murata-Electronics/GRM21BR61H106KE43K?qs=xZ%2FP%252Ba9zWqbh3%252B96jyTKxw%3D%3D&srsltid=AfmBOooOWPD4zTBWFOdsFTWSEfQ5tcdFt57vSozifhtwlehrhxhA2k6m"
+			(at 114.3 36.83 0)
+			(effects
+				(font
+					(size 1.27 1.27)
+				)
+				(hide yes)
+			)
+		)
+		(property "Manufacturer" "Murata Electronics"
+			(at 114.3 36.83 0)
+			(effects
+				(font
+					(size 1.27 1.27)
+				)
+				(hide yes)
+			)
+		)
+		(property "Manufacturer_Part_Number" "GRM21BR61H106KE43K"
+			(at 114.3 36.83 0)
+			(effects

Commit message: Added BOM, CPL
Parts:
- C10: Manufacturer_Part_Number MLASU168SB5105KTNA01 -> (none); P/N (none) -> MLASU168SB5105KTNA01
- C11: Manufacturer_Part_Number MSASU168SB7224KTNB25 -> (none); P/N (none) -> MSASU168SB7224KTNB25
- C12, C13: Manufacturer_Part_Number GRM21BR61H106KE43K -> (none); P/N (none) -> GRM21BR61H106KE43K
- C14, C15: Manufacturer_Part_Number MLASH168SB7104KTNA01 -> (none); P/N (none) -> MLASH168SB7104KTNA01
- IC2: Manufacturer_Part_Number LM74502HDDFR -> (none); P/N (none) -> LM74502HDDFR
- Q1: Manufacturer_Part_Number PSMN8R5-40MSDX -> (none); P/N (none) -> PSMN8R5-40MSDX
- R12: Manufacturer_Part_Number CRCW060310K0FKEI -> (none); P/N (none) -> CRCW060310K0FKEI
Changed lines of the file:
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@@
 			)
 		)
-		(property "Manufacturer_Part_Number" "MLASH168SB7104KTNA01"
+		(property "P/N" "MLASH168SB7104KTNA01"
 			(at 127 36.83 0)
 			(effects
@@
 			)
 		)
-		(property "Manufacturer_Part_Number" "CRCW060310K0FKEI"
+		(property "P/N" "CRCW060310K0FKEI"
 			(at 41.91 48.26 0)
 			(effects
@@
 			)
 		)
-		(property "Manufacturer_Part_Number" "MLASU168SB5105KTNA01"
+		(property "P/N" "MLASU168SB5105KTNA01"
 			(at 34.29 68.58 0)
 			(effects
@@
 			)
 		)
-		(property "Manufacturer_Part_Number" "LM74502HDDFR"
-			(at 80.01 859.69 0)
-			(effects
-				(font
-					(size 1.27 1.27)
-				)
-				(justify left top)
-				(hide yes)
-			)
-		)
 		(property "MANUFACTURER" ""
 			(at 50.8 64.77 0)
@@
 		)
 		(property "Manufacturer" "Texas Instruments"
+			(at 50.8 64.77 0)
+			(effects
+				(font
+					(size 1.27 1.27)
+				)
+				(hide yes)
+			)
+		)
+		(property "P/N" "LM74502HDDFR"
 			(at 50.8 64.77 0)
 			(effects
@@
 			)
 		)
-		(property "Manufacturer_Part_Number" "PSMN8R5-40MSDX"
-			(at 46.355 823.495 0)
-			(effects
-				(font
-					(size 1.27 1.27)
-				)
-				(justify left top)
-				(hide yes)
-			)
-		)
 		(property "MANUFACTURER" ""
 			(at 67.945 28.575 0)
@@
 		)
 		(property "Manufacturer" "Nexperia"
+			(at 67.945 28.575 0)
+			(effects
+				(font
+					(size 1.27 1.27)
+				)
+				(hide yes)
+			)
+		)
+		(property "P/N" "PSMN8R5-40MSDX"
 			(at 67.945 28.575 0)
 			(effects
@@
 			)
 		)
-		(property "Manufacturer_Part_Number" "MLASH168SB7104KTNA01"
+		(property "P/N" "MLASH168SB7104KTNA01"
 			(at 137.16 36.83 0)
 			(effects
@@
 			)
 		)
-		(property "Manufacturer_Part_Number" "GRM21BR61H106KE43K"
+		(property "P/N" "GRM21BR61H106KE43K"
 			(at 88.9 43.18 0)
 			(effects
@@
 			)
 		)
-		(property "Manufacturer_Part_Number" "MSASU168SB7224KTNB25"
+		(property "P/N" "MSASU168SB7224KTNB25"
 			(at 41.91 68.58 0)
 			(effects
@@
 			)
 		)
-		(property "Manufacturer_Part_Number" "GRM21BR61H106KE43K"
+		(property "P/N" "GRM21BR61H106KE43K"
 			(at 114.3 36.83 0)
 			(effects

Commit message: RevB1
Parts:
- added TP_Drain1, TP_Gate1, TP_OV, TP_Source1, TP_VS, TP_Vcap: TestPoint, UTSVT_Special:TestPoint_HEX_3mmID, symbol Connector:TestPoint
Connections:
- net OV: now also TP_OV.1
- net RPP_EN: now also TP_VS.1
- net VIN: now also TP_Drain1.1
- net V_OUT: now also TP_Source1.1
- net Vcap: now reaches C11.2, IC2.4 (VCAP)
- net Vcap: now also TP_Vcap.1
- net OV/RPP Gate: now reaches IC2.6 (GATE), Q1.2 (G)
- net OV/RPP Gate: now also TP_Gate1.1
Other:
- note added: "Overvoltage Protection: 14.91V Vovr = (R2 * Vov)/(R1 + R2) Vov = Vovr * (R1 + R2) / R2 14.91 = 1.25 * (47k + 4.3k) / 4.3k Vovr = 1.25V (datasheet) LOL"
- note added: "Overvoltage Protection: 29.5V Vovr = (R2 * Vov)/(R1 + R2) Vov = Vovr * (R1 + R2) / R2 29.5 = 1.25 ((45.3k+2k)/2k)"
- note removed: "Overvoltage Protection: 14.91V Vovr = (R2 * Vov)/(R1 + R2) Vov = Vovr * (R1 + R2) / R2 14.91 = 1.25 * (47k + 4.3k) / 4.3k Vovr = 1.25V (datasheet)"
- note removed: "Overvoltage Protection: 30.319V Vovr = (R2 * Vov)/(R1 + R2) Vov = Vovr * (R1 + R2) / R2 30.319 = 1.25 ((100k+4.3k)/4.3k)"
