File: stm32.kicad_sch (KiCad schematic)
At the start: 0 parts

Commit message: basic arch
Parts:
- added C10, C28, C29, C30, C31, C33, C35, C36, C37: 0.1uF, Capacitor_SMD:C_0603_1608Metric_Pad1.08x0.95mm_HandSolder, symbol Device:C
- added C11: 10uF, Capacitor_SMD:C_0805_2012Metric, symbol Device:C
- added C32, C34: 1uF, Capacitor_SMD:C_0603_1608Metric_Pad1.08x0.95mm_HandSolder, symbol Device:C
- added C38: 100nF, Capacitor_SMD:C_0603_1608Metric_Pad1.08x0.95mm_HandSolder, symbol Device:C
- added C8, C9: 26p, Capacitor_SMD:C_0603_1608Metric_Pad1.08x0.95mm_HandSolder, symbol Device:C
- added D3: RGB_LED, LHRS_Special:RGB_LED, symbol lhrs_special:RGB_LED
- added D4: TVS, Diode_SMD:D_SOD-323, symbol lhrs_misc:Boot_TVS
- added D5: LED, LED_SMD:LED_0603_1608Metric, symbol lhrs_misc:Blue_LED
- added FB1, FB2: FerriteBead, Capacitor_SMD:C_0603_1608Metric_Pad1.08x0.95mm_HandSolder, symbol Device:FerriteBead
- added J1: SWD_Header, LHRS_Connectors:SWD_Conn, symbol 100PinMCU:SWD_Header_02x02
- added J2: SWD, Connector_PinHeader_2.54mm:PinHeader_1x04_P2.54mm_Vertical, symbol Connector_Generic:Conn_01x04
- added R10, R14, R7, R9: 1k, Resistor_SMD:R_0603_1608Metric_Pad0.98x0.95mm_HandSolder, symbol Device:R
- added R11, R12: 22, Resistor_SMD:R_0603_1608Metric_Pad0.98x0.95mm_HandSolder, symbol Device:R
- added R13, R8: 10k, Resistor_SMD:R_0603_1608Metric_Pad0.98x0.95mm_HandSolder, symbol Device:R
- added SW1: Reset, LHRS_Special:TL3365AF180QG, symbol Switch:SW_Push
- added SW2: SW_SPDT, LHRS_Special:BootSW, symbol Switch:SW_SPDT
- added U1: STM32G473CETx, LHRS_Special:48PinMCU, symbol lhrs_special:STM32G473CET6
- added Y1: Crystal, LHRS_Passives:Crystal_SMD_Abracon_ABM3-2Pin_5.0x3.2mm, symbol Device:Crystal
Connections:
- new net: D3.4, R9.1
- new net: C8.2, U1.5 (PF0-OSC_IN), Y1.1
- new net: C9.1, U1.6 (PF1-OSC_OUT), Y1.2
- new net: D4.2 (A2), D5.2 (A), R13.2, SW2.2 (B)
- new net: J1.3 (Pin_3), J2.3 (Pin_3), R11.2
- new net: J1.4 (Pin_4), J2.4 (Pin_4), R12.2
- new net: D3.2, R7.1
- new net: D3.6, R10.1
- new net: D5.1 (K), R14.1
- new net +3V3: C11.1, C29.1, C31.1, C33.1, C35.1, C36.1, C37.1, FB2.1, J1.1 (Pin_1), J2.1 (Pin_1), R8.2, SW2.1 (A), U1.1 (VBAT), U1.24 (VDD), U1.36 (VDD), U1.48 (VDD)
- new net BOOT0: R13.1, U1.45 (PB8-BOOT0)
- new net GND: C11.2, C28.2, C29.2, C31.2, C33.2, C35.2, C36.2, C37.2, C8.1, C9.2, D4.1 (A1), FB1.2, J1.2 (Pin_2), J2.2 (Pin_2), R10.2, R14.2, R7.2, R9.2, SW1.2, SW2.3 (C), U1.23 (VSS), U1.35 (VSS), U1.47 (VSS)
- new net GNDA: C10.2, C30.2, C32.2, C34.2, C38.2, FB1.1, U1.19 (VSSA)
- new net NRST: C28.1, R8.1, SW1.1, U1.7 (PG10-NRST)
- new net PA0: D3.5, U1.8 (PA0-GPIO_BLUE)
- new net PA1: D3.3, U1.9 (PA1_GPIO_RED)
- new net PA10: U1.32 (PA10)
- new net PA15: U1.39 (PA15)
- new net PA2: D3.1, U1.10 (PA2-GPIO_GREEN)
- new net PA3: U1.11 (PA3)
- new net PA4: U1.12 (PA4)
- new net PA5: U1.13 (PA5)
- new net PA6: U1.14 (PA6)
- new net PA7: U1.15 (PA7)
- new net PA8: U1.30 (PA8)
- new net PA9: U1.31 (PA9)
- new net PB0: U1.16 (PB0)
- new net PB1: U1.17 (PB1)
- new net PB10: U1.22 (PB10)
- new net PB11: U1.25 (PB11)
- new net PB12: U1.26 (PB12)
- new net PB13: U1.27 (PB13)
- new net PB14: U1.28 (PB14)
- new net PB15: U1.29 (PB15)
- new net PB2: U1.18 (PB2)
- new net PB3: U1.40 (PB3)
- new net PB4: U1.41 (PB4)
- new net PB5: U1.42 (PB5)
- new net PB6: U1.43 (PB6)
- new net PB7: U1.44 (PB7)
- new net PB9: U1.46 (PB9)
- new net PC13: U1.2 (PC13)
- new net PC14: U1.3 (PC14-OSC32_IN)
- new net PC15: U1.4 (PC15-OSC32_OUT)
- new net SWCLK: R11.1, U1.38 (PA14)
- new net SWDIO: R12.1, U1.37 (PA13)
- new net USB_DM: U1.33 (PA11)
- new net USB_DP: U1.34 (PA12)
- new net VDDA: C10.1, C30.1, C32.1, C34.1, C38.1, FB2.2, U1.20 (VREF+), U1.21 (VDDA)
Other:
- note added: "*Place oscillator circuitry close to MCU"
- note added: "48 Pin MCU"
- note added: "BLUE"
- note added: "BOOT0 low -> Load into app BOOT0 high -> Load into bootloader"
- note added: "Beware, using PC13 - 15 as GPIOs ..."
- note added: "CLK"
- note added: "Conn"
- note added: "GREEN"
- note added: "IO"
- note added: "Main Flash (user code)"
- note added: "Pin Headers"
- note added: "Place these decoupling caps as close as possible to their respective leads."
- note added: "Power Source Filtering/Isolation"
- note added: "RED"
- note added: "RGB LED"
- note added: "Reset BTN + Boot SW"
- note added: "Serial Wire Communication"
- note added: "Sys Memory (bootloader)"
- note added: "Use PA0, PA1, PA2 to PWM RGB LED (TIM2_CH1, TIM2_CH2, TIM2_CH3)"
- note added: "VBAT Decoupling Cap"
- note added: "VDD Decoupling Caps"
- note added: "VDDA Decoupling Caps"
- note added: "VDDA Seperation"
