File: 48PinMCU.kicad_sch (KiCad schematic)
At the start: 34 parts, among them J1 SWD_Header, J2 SWD, SW1 Reset, SW2 SW_SPDT, U1 STM32G473CETx, Y1 Crystal

Commit message: basic arch
Parts:
- renumbered C3 to C10, C4 to C11, C5 to C28, C6 to C29, C7 to C30, C8 to C31, C9 to C32, C10 to C33, C11 to C34, C12 to C35, C13 to C36, C14 to C37, C15 to C38, C1 to C8, C2 to C9, D1 to D3, D2 to D4, D3 to D5, R4 to R10, R5 to R11, R6 to R12, R7 to R13, R8 to R14, R1 to R7, R2 to R8, R3 to R9
