File: 48PinMCU.kicad_sch (KiCad schematic)
At the start: 34 parts, among them J12 SWD_Header, J13 SWD, SW3 Reset, SW4 SW_SPDT, U6 STM32G473CETx, Y2 Crystal

Commit message: updated from review
Parts:
- C10: renamed from C60; Mouser Part Number MLASH168SB7104KTNA01 -> (none)
- C11: renamed from C61; Mouser Part Number MLASH168SB7104KTNA01 -> (none)
- C12: renamed from C62; Mouser Part Number MLASH168SB7104KTNA01 -> (none)
- C13: renamed from C63; Mouser Part Number MLASH168SB7104KTNA01 -> (none)
- C14: renamed from C64; Mouser Part Number MLASH168SB7104KTNA01 -> (none)
- C15: renamed from C65; Mouser Part Number MLASH168SB7104KTNA01 -> (none)
- C16: renamed from C66; Mouser Part Number MLASH168SB7104KTNA01 -> (none)
- C17: renamed from C67; Mouser Part Number MLASH168SB7104KTNA01 -> (none)
- C18: renamed from C68; Mouser Part Number MLASH168SB7104KTNA01 -> (none)
- C7: renamed from C57; Mouser Part Number MLASH168SB7104KTNA01 -> (none)
- C8: renamed from C58; Mouser Part Number 08055D475KAT4A -> (none)
- C9: renamed from C59; Mouser Part Number MLASH168SB7104KTNA01 -> (none)
- D6: renamed from D14; MANUFACTURER Everlight -> (none)
- D7: renamed from D15; Color Blue -> (none); Mouser P/N 771-PESD15VL1BA-T/R -> (none)
- J8: renamed from J12; LSCS P/N C17492485 -> (none)
- R14: renamed from R40; Mouser Part Number CRCW060310K0FKEI -> (none)
- R19: renamed from R45; Mouser Part Number CRCW060310K0FKEI -> (none)
- SW1: renamed from SW3; Mouser Part Number 612-TL3365AF180QG -> (none)
- renumbered C69 to C19, C55 to C5, C56 to C6, D16 to D8, FB3 to FB1, FB4 to FB2, J13 to J12, R39 to R13, R41 to R15, R42 to R16, R43 to R17, R44 to R18, R55 to R20, SW4 to SW2, U6 to U2, Y2 to Y1
Other:
- moved on the sheet: C10, C11, C12, C13, C14, C15, C16, C17, C18, C19, C5, C6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
