File: CAN_Transceiver.kicad_sch (KiCad schematic)
At the start: 9 parts, among them IC2 TCAN3413DR

Commit message: idk wtf im doingggggggggggg
Parts:
- renumbered C20 to C24, C21 to C25, C22 to C26, C23 to C27, D9 to D10, IC2 to IC3, JP1 to JP2, R17 to R19, R18 to R20
Changed lines of the file:
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@@
 		(in_pos_files yes)
 		(dnp no)
-		(property "Reference" "C21"
+		(property "Reference" "C25"
 			(at 76.2 73.66 0)
 			(show_name no)
@@
 		)
 		(instances
+			(project "PS-ChargerInterfacePCB"
+				(path "/24809a72-9525-4be8-be3e-46bc27cfe8fb/ba69df00-9c22-4c65-92b6-b1bd518e51cc/28c8bb30-5aee-42e2-a184-4f9c3cc306ab"
+					(reference "C25")
+					(unit 1)
+				)
+				(path "/24809a72-9525-4be8-be3e-46bc27cfe8fb/ba69df00-9c22-4c65-92b6-b1bd518e51cc/f3193b22-5837-4bd9-9023-4143db12e377"
+					(reference "C25")
+					(unit 1)
+				)
+			)
 			(project ""
 				(path "/69b823fd-c065-40ff-9bb9-c5835555f3eb/9d9eae1e-c713-4323-9845-a569cff8d5d3"
 					(reference "C6")
-					(unit 1)
-				)
-			)
-			(project "PS-ChargerInterfacePCB"
-				(path "/76be3fbd-da4b-465f-ad8f-cf483283a19d/28c8bb30-5aee-42e2-a184-4f9c3cc306ab"
-					(reference "C25")
-					(unit 1)
-				)
-				(path "/76be3fbd-da4b-465f-ad8f-cf483283a19d/f3193b22-5837-4bd9-9023-4143db12e377"
-					(reference "C21")
 					(unit 1)
 				)
@@
 		(in_pos_files yes)
 		(dnp no)
-		(property "Reference" "C23"
+		(property "Reference" "C27"
 			(at 194.564 88.646 0)
 			(show_name no)
@@
 		)
 		(instances
+			(project "PS-ChargerInterfacePCB"
+				(path "/24809a72-9525-4be8-be3e-46bc27cfe8fb/ba69df00-9c22-4c65-92b6-b1bd518e51cc/28c8bb30-5aee-42e2-a184-4f9c3cc306ab"
+					(reference "C27")
+					(unit 1)
+				)
+				(path "/24809a72-9525-4be8-be3e-46bc27cfe8fb/ba69df00-9c22-4c65-92b6-b1bd518e51cc/f3193b22-5837-4bd9-9023-4143db12e377"
+					(reference "C27")
+					(unit 1)
+				)
+			)
 			(project ""
 				(path "/69b823fd-c065-40ff-9bb9-c5835555f3eb/9d9eae1e-c713-4323-9845-a569cff8d5d3"
 					(reference "C8")
-					(unit 1)
-				)
-			)
-			(project "PS-ChargerInterfacePCB"
-				(path "/76be3fbd-da4b-465f-ad8f-cf483283a19d/28c8bb30-5aee-42e2-a184-4f9c3cc306ab"
-					(reference "C27")
-					(unit 1)
-				)
-				(path "/76be3fbd-da4b-465f-ad8f-cf483283a19d/f3193b22-5837-4bd9-9023-4143db12e377"
-					(reference "C23")
 					(unit 1)
 				)
@@
 		(dnp no)
 		(fields_autoplaced yes)
-		(property "Reference" "JP1"
+		(property "Reference" "JP2"
 			(at 215.9 78.74 0)
 			(show_name no)
@@
 		)
 		(instances
+			(project "PS-ChargerInterfacePCB"
+				(path "/24809a72-9525-4be8-be3e-46bc27cfe8fb/ba69df00-9c22-4c65-92b6-b1bd518e51cc/28c8bb30-5aee-42e2-a184-4f9c3cc306ab"
+					(reference "JP2")
+					(unit 1)
+				)
+				(path "/24809a72-9525-4be8-be3e-46bc27cfe8fb/ba69df00-9c22-4c65-92b6-b1bd518e51cc/f3193b22-5837-4bd9-9023-4143db12e377"
+					(reference "JP2")
+					(unit 1)
+				)
+			)
 			(project ""
 				(path "/69b823fd-c065-40ff-9bb9-c5835555f3eb/9d9eae1e-c713-4323-9845-a569cff8d5d3"
 					(reference "JP2")
-					(unit 1)
-				)
-			)
-			(project "PS-ChargerInterfacePCB"
-				(path "/76be3fbd-da4b-465f-ad8f-cf483283a19d/28c8bb30-5aee-42e2-a184-4f9c3cc306ab"
-					(reference "JP2")
-					(unit 1)
-				)
-				(path "/76be3fbd-da4b-465f-ad8f-cf483283a19d/f3193b22-5837-4bd9-9023-4143db12e377"
-					(reference "JP1")
 					(unit 1)
 				)
@@
 		(in_pos_files yes)
 		(dnp no)
-		(property "Reference" "C22"
+		(property "Reference" "C26"
 			(at 88.138 73.66 0)
 			(show_name no)
@@
 		)
 		(instances
+			(project "PS-ChargerInterfacePCB"
+				(path "/24809a72-9525-4be8-be3e-46bc27cfe8fb/ba69df00-9c22-4c65-92b6-b1bd518e51cc/28c8bb30-5aee-42e2-a184-4f9c3cc306ab"
+					(reference "C26")
+					(unit 1)
+				)
+				(path "/24809a72-9525-4be8-be3e-46bc27cfe8fb/ba69df00-9c22-4c65-92b6-b1bd518e51cc/f3193b22-5837-4bd9-9023-4143db12e377"
+					(reference "C26")
+					(unit 1)
+				)
+			)
 			(project ""
 				(path "/69b823fd-c065-40ff-9bb9-c5835555f3eb/9d9eae1e-c713-4323-9845-a569cff8d5d3"
 					(reference "C7")
-					(unit 1)
-				)
-			)
-			(project "PS-ChargerInterfacePCB"
-				(path "/76be3fbd-da4b-465f-ad8f-cf483283a19d/28c8bb30-5aee-42e2-a184-4f9c3cc306ab"
-					(reference "C26")
-					(unit 1)
-				)
-				(path "/76be3fbd-da4b-465f-ad8f-cf483283a19d/f3193b22-5837-4bd9-9023-4143db12e377"
-					(reference "C22")
 					(unit 1)
 				)
@@
 		(in_pos_files yes)
 		(dnp no)
-		(property "Reference" "C20"
+		(property "Reference" "C24"
 			(at 65.278 73.66 0)
 			(show_name no)
@@
 		)
 		(instances
+			(project "PS-ChargerInterfacePCB"
+				(path "/24809a72-9525-4be8-be3e-46bc27cfe8fb/ba69df00-9c22-4c65-92b6-b1bd518e51cc/28c8bb30-5aee-42e2-a184-4f9c3cc306ab"
+					(reference "C24")
+					(unit 1)
+				)
+				(path "/24809a72-9525-4be8-be3e-46bc27cfe8fb/ba69df00-9c22-4c65-92b6-b1bd518e51cc/f3193b22-5837-4bd9-9023-4143db12e377"
+					(reference "C24")
+					(unit 1)
+				)
+			)
 			(project ""
 				(path "/69b823fd-c065-40ff-9bb9-c5835555f3eb/9d9eae1e-c713-4323-9845-a569cff8d5d3"
 					(reference "C5")
-					(unit 1)
-				)
-			)
-			(project "PS-ChargerInterfacePCB"
-				(path "/76be3fbd-da4b-465f-ad8f-cf483283a19d/28c8bb30-5aee-42e2-a184-4f9c3cc306ab"
-					(reference "C24")
-					(unit 1)
-				)
-				(path "/76be3fbd-da4b-465f-ad8f-cf483283a19d/f3193b22-5837-4bd9-9023-4143db12e377"
-					(reference "C20")
 					(unit 1)
 				)
@@
 		(in_pos_files yes)
 		(dnp no)
-		(property "Reference" "R18"
+		(property "Reference" "R20"
 			(at 201.93 80.01 90)
 			(show_name no)
@@
 		)
 		(instances
+			(project "PS-ChargerInterfacePCB"
+				(path "/24809a72-9525-4be8-be3e-46bc27cfe8fb/ba69df00-9c22-4c65-92b6-b1bd518e51cc/28c8bb30-5aee-42e2-a184-4f9c3cc306ab"
+					(reference "R20")
+					(unit 1)
+				)
+				(path "/24809a72-9525-4be8-be3e-46bc27cfe8fb/ba69df00-9c22-4c65-92b6-b1bd518e51cc/f3193b22-5837-4bd9-9023-4143db12e377"
+					(reference "R20")
+					(unit 1)
+				)
+			)
 			(project "kk36984"
 				(path "/69b823fd-c065-40ff-9bb9-c5835555f3eb/9d9eae1e-c713-4323-9845-a569cff8d5d3"
 					(reference "R23")
-					(unit 1)
-				)
-			)
-			(project "PS-ChargerInterfacePCB"
-				(path "/76be3fbd-da4b-465f-ad8f-cf483283a19d/28c8bb30-5aee-42e2-a184-4f9c3cc306ab"
-					(reference "R20")
-					(unit 1)
-				)
-				(path "/76be3fbd-da4b-465f-ad8f-cf483283a19d/f3193b22-5837-4bd9-9023-4143db12e377"
-					(reference "R18")
 					(unit 1)
 				)
@@
 		(dnp no)
 		(fields_autoplaced yes)
-		(property "Reference" "D9"
+		(property "Reference" "D10"
 			(at 196.85 46.99 0)
 			(show_name no)
@@
 		)
 		(instances
+			(project "PS-ChargerInterfacePCB"
+				(path "/24809a72-9525-4be8-be3e-46bc27cfe8fb/ba69df00-9c22-4c65-92b6-b1bd518e51cc/28c8bb30-5aee-42e2-a184-4f9c3cc306ab"
+					(reference "D10")
+					(unit 1)
+				)
+				(path "/24809a72-9525-4be8-be3e-46bc27cfe8fb/ba69df00-9c22-4c65-92b6-b1bd518e51cc/f3193b22-5837-4bd9-9023-4143db12e377"
+					(reference "D10")
+					(unit 1)
+				)
+			)
 			(project ""
 				(path "/69b823fd-c065-40ff-9bb9-c5835555f3eb/9d9eae1e-c713-4323-9845-a569cff8d5d3"
 					(reference "D8")
-					(unit 1)
-				)
-			)
-			(project "PS-ChargerInterfacePCB"
-				(path "/76be3fbd-da4b-465f-ad8f-cf483283a19d/28c8bb30-5aee-42e2-a184-4f9c3cc306ab"
-					(reference "D10")
-					(unit 1)
-				)
-				(path "/76be3fbd-da4b-465f-ad8f-cf483283a19d/f3193b22-5837-4bd9-9023-4143db12e377"
-					(reference "D9")
 					(unit 1)
 				)
@@
 		(dnp no)
 		(fields_autoplaced yes)
-		(property "Reference" "IC2"
+		(property "Reference" "IC3"
 			(at 128.27 63.5 0)
 			(show_name no)
@@
 		)
 		(instances
+			(project "PS-ChargerInterfacePCB"
+				(path "/24809a72-9525-4be8-be3e-46bc27cfe8fb/ba69df00-9c22-4c65-92b6-b1bd518e51cc/28c8bb30-5aee-42e2-a184-4f9c3cc306ab"
+					(reference "IC3")
+					(unit 1)
+				)
+				(path "/24809a72-9525-4be8-be3e-46bc27cfe8fb/ba69df00-9c22-4c65-92b6-b1bd518e51cc/f3193b22-5837-4bd9-9023-4143db12e377"
+					(reference "IC3")
+					(unit 1)
+				)
+			)
 			(project ""
 				(path "/69b823fd-c065-40ff-9bb9-c5835555f3eb/9d9eae1e-c713-4323-9845-a569cff8d5d3"
 					(reference "IC1")
-					(unit 1)
-				)
-			)
-			(project "PS-ChargerInterfacePCB"
-				(path "/76be3fbd-da4b-465f-ad8f-cf483283a19d/28c8bb30-5aee-42e2-a184-4f9c3cc306ab"
-					(reference "IC3")
-					(unit 1)
-				)
-				(path "/76be3fbd-da4b-465f-ad8f-cf483283a19d/f3193b22-5837-4bd9-9023-4143db12e377"
-					(reference "IC2")
 					(unit 1)
 				)
@@
 		(in_pos_files yes)
 		(dnp no)
-		(property "Reference" "R17"
+		(property "Reference" "R19"
 			(at 176.53 80.01 90)
 			(show_name no)
@@
 		)
 		(instances
+			(project "PS-ChargerInterfacePCB"
+				(path "/24809a72-9525-4be8-be3e-46bc27cfe8fb/ba69df00-9c22-4c65-92b6-b1bd518e51cc/28c8bb30-5aee-42e2-a184-4f9c3cc306ab"
+					(reference "R19")
+					(unit 1)
+				)
+				(path "/24809a72-9525-4be8-be3e-46bc27cfe8fb/ba69df00-9c22-4c65-92b6-b1bd518e51cc/f3193b22-5837-4bd9-9023-4143db12e377"
+					(reference "R19")
+					(unit 1)
+				)
+			)
 			(project ""
 				(path "/69b823fd-c065-40ff-9bb9-c5835555f3eb/9d9eae1e-c713-4323-9845-a569cff8d5d3"
@@
 					(unit 1)
 				)
-			)
-			(project "PS-ChargerInterfacePCB"
-				(path "/76be3fbd-da4b-465f-ad8f-cf483283a19d/28c8bb30-5aee-42e2-a184-4f9c3cc306ab"
-					(reference "R19")
-					(unit 1)
-				)
-				(path "/76be3fbd-da4b-465f-ad8f-cf483283a19d/f3193b22-5837-4bd9-9023-4143db12e377"
-					(reference "R17")
-					(unit 1)
-				)
