File: mcu.kicad_sch (KiCad schematic)
At the start: 0 parts

Commit message: nothing useful
Other:
- sheet 48PinMCU ports: added USB_DM, USB_DP; removed none
Changed lines of the file:
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@@
 		)
 		(pin "CC1" bidirectional
-			(at 67.31 31.75 0)
+			(at 67.31 35.56 0)
 			(effects
 				(font
@@
 		)
 		(pin "CC2" bidirectional
-			(at 67.31 34.29 0)
+			(at 67.31 38.1 0)
 			(effects
 				(font
@@
 		)
 		(pin "GND" input
-			(at 24.13 45.72 180)
+			(at 24.13 35.56 180)
 			(effects
 				(font
@@
 		)
 		(pin "USB_5V" output
-			(at 24.13 49.53 180)
+			(at 24.13 41.91 180)
 			(effects
 				(font
@@
 		)
 		(pin "USB_DM" bidirectional
-			(at 67.31 41.91 0)
+			(at 67.31 45.72 0)
 			(effects
 				(font
@@
 		)
 		(pin "USB_DP" bidirectional
-			(at 67.31 39.37 0)
+			(at 67.31 43.18 0)
 			(effects
 				(font
@@
 	)
 	(sheet
-		(at 99.06 27.94)
+		(at 92.71 27.94)
 		(size 43.18 24.13)
 		(exclude_from_sim no)
@@
 		)
 		(property "Sheetname" "48PinMCU"
-			(at 99.06 27.2284 0)
+			(at 92.71 27.2284 0)
 			(show_name no)
 			(do_not_autoplace no)
@@
 		)
 		(property "Sheetfile" "48PinMCU.kicad_sch"
-			(at 99.06 52.6546 0)
+			(at 92.71 52.6546 0)
 			(show_name no)
 			(do_not_autoplace no)
@@
 		)
 		(property "Date Modified" "5/3/2026"
-			(at -63.5 -13.97 0)
+			(at 68.58 0 0)
 			(hide yes)
 			(show_name no)
@@
 		)
 		(property "Author" "Sathvik Yechuri"
-			(at -63.5 -13.97 0)
+			(at 68.58 0 0)
 			(hide yes)
 			(show_name no)
@@
 			)
 		)
+		(pin "USB_DM" bidirectional
+			(at 92.71 35.56 180)
+			(effects
+				(font
+					(size 1.27 1.27)
+				)
+				(justify left)
+			)
+		)
+		(pin "USB_DP" bidirectional
+			(at 92.71 38.1 180)
+			(effects
+				(font
+					(size 1.27 1.27)
+				)
+				(justify left)
+			)
+		)

Commit message: idk wtf im doingggggggggggg
Other:
- sheet USB-C_Connector ports: added none; removed CC1, CC2
Changed lines of the file:
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@@
 	(generator_version "10.0")
 	(paper "A4")
+	(wire
+		(pts
+			(xy 67.31 40.64) (xy 73.66 40.64)
+		)
+		(stroke
+			(width 0)
+			(type default)
+		)
+	)
+	(wire
+		(pts
+			(xy 86.36 34.29) (xy 92.71 34.29)
+		)
+		(stroke
+			(width 0)
+			(type default)
+		)
+	)
+	(wire
+		(pts
+			(xy 67.31 34.29) (xy 73.66 34.29)
+		)
+		(stroke
+			(width 0)
+			(type default)
+		)
+	)
+	(wire
+		(pts
+			(xy 86.36 40.64) (xy 92.71 40.64)
+		)
+		(stroke
+			(width 0)
+			(type default)
+		)
+	)
+	(label "USB_M"
+		(at 73.66 40.64 180)
+		(effects
+			(font
+				(size 1.27 1.27)
+			)
+			(justify right bottom)
+		)
+	)
+	(label "USB_M"
+		(at 86.36 40.64 0)
+		(effects
+			(font
+				(size 1.27 1.27)
+			)
+			(justify left bottom)
+		)
+	)
+	(label "USB_P"
+		(at 73.66 34.29 180)
+		(effects
+			(font
+				(size 1.27 1.27)
+			)
+			(justify right bottom)
+		)
+	)
+	(label "USB_P"
+		(at 86.36 34.29 0)
+		(effects
+			(font
+				(size 1.27 1.27)
+			)
+			(justify left bottom)
+		)
+	)
 	(sheet
 		(at 24.13 27.94)
@@
 			)
 		)
-		(pin "CC1" bidirectional
-			(at 67.31 35.56 0)
-			(effects
-				(font
-					(size 1.27 1.27)
-				)
-				(justify right)
-			)
-		)
-		(pin "CC2" bidirectional
-			(at 67.31 38.1 0)
-			(effects
-				(font
-					(size 1.27 1.27)
-				)
-				(justify right)
-			)
-		)
 		(pin "GND" input
 			(at 24.13 35.56 180)
@@
 		)
 		(pin "USB_DM" bidirectional
-			(at 67.31 45.72 0)
+			(at 67.31 40.64 0)
 			(effects
 				(font
@@
 		)
 		(pin "USB_DP" bidirectional
-			(at 67.31 43.18 0)
+			(at 67.31 34.29 0)
 			(effects
 				(font
@@
 		(instances
 			(project "PS-ChargerInterfacePCB"
-				(path "/b7e42da5-6f2f-462d-9722-f11b3aabae29"
-					(page "8")
+				(path "/24809a72-9525-4be8-be3e-46bc27cfe8fb/84410e9c-5d36-47d4-a265-5b9dbc512cd8"
+					(page "18")
 				)
 			)
@@
 		)
 		(pin "USB_DM" bidirectional
-			(at 92.71 35.56 180)
+			(at 92.71 40.64 180)
 			(effects
 				(font
@@
 		)
 		(pin "USB_DP" bidirectional
-			(at 92.71 38.1 180)
+			(at 92.71 34.29 180)
 			(effects
 				(font
@@
 		(instances
 			(project "PS-ChargerInterfacePCB"
-				(path "/b7e42da5-6f2f-462d-9722-f11b3aabae29"
-					(page "7")
-				)
-			)
+				(path "/24809a72-9525-4be8-be3e-46bc27cfe8fb/84410e9c-5d36-47d4-a265-5b9dbc512cd8"
+					(page "19")
+				)
+			)
