File: power_system.kicad_sch (KiCad schematic)
At the start: 0 parts

Commit message: idk wtf im doingggggggggggg
Changed lines of the file:
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@@
 	(wire
 		(pts
-			(xy 180.34 35.56) (xy 185.42 35.56)
-		)
-		(stroke
-			(width 0)
-			(type default)
-		)
-	)
-	(wire
-		(pts
-			(xy 180.34 48.26) (xy 185.42 48.26)
-		)
-		(stroke
-			(width 0)
-			(type default)
-		)
-	)
-	(wire
-		(pts
-			(xy 113.03 46.99) (xy 118.11 46.99)
+			(xy 194.31 35.56) (xy 199.39 35.56)
+		)
+		(stroke
+			(width 0)
+			(type default)
+		)
+	)
+	(wire
+		(pts
+			(xy 194.31 48.26) (xy 199.39 48.26)
+		)
+		(stroke
+			(width 0)
+			(type default)
+		)
+	)
+	(wire
+		(pts
+			(xy 120.65 46.99) (xy 125.73 46.99)
 		)
 		(stroke
@@
 	(wire
 		(pts
-			(xy 163.83 34.29) (xy 168.91 34.29)
-		)
-		(stroke
-			(width 0)
-			(type default)
-		)
-	)
-	(wire
-		(pts
-			(xy 231.14 35.56) (xy 236.22 35.56)
+			(xy 171.45 34.29) (xy 176.53 34.29)
+		)
+		(stroke
+			(width 0)
+			(type default)
+		)
+	)
+	(wire
+		(pts
+			(xy 245.11 35.56) (xy 250.19 35.56)
 		)
 		(stroke
@@
 	(wire
 		(pts
-			(xy 113.03 34.29) (xy 118.11 34.29)
+			(xy 120.65 34.29) (xy 125.73 34.29)
 		)
 		(stroke
@@
 	)
 	(label "GND"
-		(at 180.34 48.26 180)
+		(at 194.31 48.26 180)
 		(effects
 			(font
@@
 	)
 	(label "LV_PROTECTED"
-		(at 113.03 34.29 180)
+		(at 120.65 34.29 180)
 		(effects
 			(font
@@
 	)
 	(label "GND"
-		(at 113.03 46.99 180)
+		(at 120.65 46.99 180)
 		(effects
 			(font
@@
 	)
 	(label "+5V"
-		(at 180.34 35.56 180)
+		(at 194.31 35.56 180)
 		(effects
 			(font
@@
 	(hierarchical_label "+3V3"
 		(shape output)
-		(at 236.22 35.56 0)
+		(at 250.19 35.56 0)
 		(effects
 			(font
@@
 	(hierarchical_label "+5V"
 		(shape output)
-		(at 168.91 34.29 0)
+		(at 176.53 34.29 0)
 		(effects
 			(font
@@
 	)
 	(sheet
-		(at 185.42 27.94)
+		(at 199.39 27.94)
 		(size 45.72 27.94)
 		(exclude_from_sim no)
@@
 		)
 		(property "Sheetname" "3V3_Regulator"
-			(at 185.42 27.2284 0)
+			(at 199.39 27.2284 0)
 			(show_name no)
 			(do_not_autoplace no)
@@
 		)
 		(property "Sheetfile" "LDO.kicad_sch"
-			(at 185.42 56.4646 0)
+			(at 199.39 56.4646 0)
 			(show_name no)
 			(do_not_autoplace no)
@@
 		)
 		(pin "+5V" input
-			(at 185.42 35.56 180)
+			(at 199.39 35.56 180)
 			(effects
 				(font
@@
 		)
 		(pin "+3V3" output
-			(at 231.14 35.56 0)
+			(at 245.11 35.56 0)
 			(effects
 				(font
@@
 		)
 		(pin "GND" input
-			(at 185.42 48.26 180)
+			(at 199.39 48.26 180)
 			(effects
 				(font
@@
 	)
 	(sheet
-		(at 118.11 26.67)
+		(at 125.73 26.67)
 		(size 45.72 27.94)
 		(exclude_from_sim no)
@@
 		)
 		(property "Sheetname" "5V_Buck"
-			(at 118.11 25.9584 0)
+			(at 125.73 25.9584 0)
 			(show_name no)
 			(do_not_autoplace no)
@@
 		)
 		(property "Sheetfile" "12VBuck.kicad_sch"
-			(at 118.11 55.1946 0)
+			(at 125.73 55.1946 0)
 			(show_name no)
 			(do_not_autoplace no)
@@
 		)
 		(pin "LV_PROTECTED" input
-			(at 118.11 34.29 180)
+			(at 125.73 34.29 180)
 			(effects
 				(font
@@
 		)
 		(pin "+5V" output
-			(at 163.83 34.29 0)
+			(at 171.45 34.29 0)
 			(effects
 				(font
@@
 		)
 		(pin "GND" bidirectional
-			(at 118.11 46.99 180)
-			(effects
-				(font
+			(at 125.73 46.99 180)
+			(effects
+				(font
