File: shutdown.kicad_sch (KiCad schematic)
At the start: 0 parts

Commit message: idk wtf im doingggggggggggg
Parts:
- added C20, C21: 100n, symbol Device:C
- added J4: E_STOP, UTSVT_Connectors:Molex_Nano-Fit_105309-xx02_1x02_P2.50mm_Vertical, symbol Connector_Generic:Conn_01x02
- added J5: SOFT_SHUTDOWN, UTSVT_Connectors:Molex_Nano-Fit_105309-xx02_1x02_P2.50mm_Vertical, symbol Connector_Generic:Conn_01x02
- added R23, R24: 10k, symbol Device:R
Connections:
- new net +3.3V: R23.1, R24.1
- new net ESTOP_SENSE: C20.1, J4.1 (Pin_1), R23.2
- new net GND: C20.2, C21.2, J4.2 (Pin_2), J5.2 (Pin_2)
- new net SOFT_SHUTDOWN: C21.1, J5.1 (Pin_1), R24.2
Other:
- note added: "GPIO inputs are 3.3 V only. E-stop sensing does not replace the independent hardware shutdown path."
- note added: "Normally-closed E-stop: normal = LOW; pressed, broken wire, or unplugged = HIGH (FAULT)"
- note added: "Normally-open soft-shutdown button: released = HIGH; pressed = LOW"
