File: ui.kicad_sch (KiCad schematic)
At the start: 0 parts

Commit message: idk wtf im doingggggggggggg
Parts:
- added D10, D6, D7, D9: LED, LED_SMD:LED_0603_1608Metric, symbol Device:LED
- added Panel_LED801: 105314-1110, charger_parts:105314-1110, symbol 105314-1110:105314-1110
- added Q13, Q4, Q5, Q6, Q7: IRLML0030TRPBF, charger_parts:IRLML0030TRPBF, symbol IRLML0030TRPBF:IRLML0030TRPBF
- added R15, R16, R17, R18, R19: 100k, Resistor_SMD:R_0603_1608Metric, symbol Device:R_US
- added R32, R33, R35, R36: 470, Resistor_SMD:R_0603_1608Metric, symbol Device:R_US
Connections:
- new net: D6.2 (A), R32.2
- new net: D7.2 (A), R33.2
- new net: D10.2 (A), R36.2
- new net: D9.2 (A), R35.2
- new net +14V: Panel_LED801.10, Panel_LED801.6, Panel_LED801.7, Panel_LED801.8, Panel_LED801.9
- new net CHARGE-: Panel_LED801.2, Q5.3 (D)
- new net EVSE-: Panel_LED801.1, Q13.3 (D)
- new net FAULT-: Panel_LED801.4, Q4.3 (D)
- new net GND: D10.1 (K), D6.1 (K), D7.1 (K), D9.1 (K), Q13.2 (S), Q4.2 (S), Q5.2 (S), Q6.2 (S), Q7.2 (S), R15.2, R16.2, R17.2, R18.2, R19.2
- new net HEART-: Panel_LED801.3, Q6.3 (D)
- new net HV-: Panel_LED801.5, Q7.3 (D)
- new net LED_CHARGE: Q5.1 (G), R18.1, R35.1
- new net LED_EVSE: Q13.1 (G), R19.1, R36.1
- new net LED_FAULT: Q4.1 (G), R16.1
- new net LED_HEART: Q6.1 (G), R17.1, R33.1
- new net LED_HV: Q7.1 (G), R15.1, R32.1
Other:
- note added: "LEDS: https://www.amazon.com/Gebildet-12-24V-Indicator-Waterproof-Directional/dp/B088D1M47R 12-24V, 0.02 amps"
- note added: "LED_HV = HV active or not LED_FAULT = external siren / beacon on FAULT+ and FAULT- LED_Heart = power up for 14v/24v LED_Charge = Charging Active or Not LED_EVSE = EVSE detected + pilot ready"
