File: 12VBuck.kicad_sch (KiCad schematic)
At the start: 14 parts, among them U3 LMR51635XDDCR

Commit message: YOOO KICAD IS KICADDING IT MAKES SENSEEEEEEEEEEEEEE
Parts:
- renumbered C14 to C45, C15 to C46, C16 to C47, C17 to C48, C18 to C49, C19 to C50, L1 to L2, R15 to R31, R16 to R34, TP1 to TP5, TP2 to TP6, TP3 to TP7, TP4 to TP8, U3 to U4
Changed lines of the file:
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@@
 		(dnp no)
 		(fields_autoplaced yes)
-		(property "Reference" "#FLG02"
+		(property "Reference" "#FLG07"
 			(at 149.86 79.375 0)
 			(hide yes)
@@
 				(path "/331f457b-ed4e-4d4a-ad6d-c8acb2febfed/9243f342-8d42-4433-b049-031be1288812"
 					(reference "#FLG013")
+					(unit 1)
+				)
+			)
+			(project "PS-ChargerInterfacePCB"
+				(path "/894adbd2-6316-426a-afb4-88808e8ec51a/8fb4e0f4-a81e-4963-ba02-cb881e23146d"
+					(reference "#FLG07")
 					(unit 1)
 				)
@@
 		(dnp no)
 		(fields_autoplaced yes)
-		(property "Reference" "C14"
+		(property "Reference" "C45"
 			(at 96.52 85.0962 0)
 			(show_name no)
@@
 				(path "/331f457b-ed4e-4d4a-ad6d-c8acb2febfed/9243f342-8d42-4433-b049-031be1288812"
 					(reference "C11")
+					(unit 1)
+				)
+			)
+			(project "PS-ChargerInterfacePCB"
+				(path "/894adbd2-6316-426a-afb4-88808e8ec51a/8fb4e0f4-a81e-4963-ba02-cb881e23146d"
+					(reference "C45")
 					(unit 1)
 				)
@@
 		(in_pos_files yes)
 		(dnp no)
-		(property "Reference" "TP1"
+		(property "Reference" "TP5"
 			(at 229.87 123.6979 0)
 			(hide yes)
@@
 				(path "/24809a72-9525-4be8-be3e-46bc27cfe8fb/cd4ac576-e1cf-46c0-a1b5-c681437cfde8/eaf4dc2b-ad73-4e1e-8bba-aa12f0e48269"
 					(reference "TP1")
+					(unit 1)
+				)
+			)
+			(project "PS-ChargerInterfacePCB"
+				(path "/894adbd2-6316-426a-afb4-88808e8ec51a/8fb4e0f4-a81e-4963-ba02-cb881e23146d"
+					(reference "TP5")
 					(unit 1)
 				)
@@
 		(in_pos_files yes)
 		(dnp no)
-		(property "Reference" "L1"
+		(property "Reference" "L2"
 			(at 161.29 87.884 90)
 			(show_name no)
@@
 				(path "/331f457b-ed4e-4d4a-ad6d-c8acb2febfed/9243f342-8d42-4433-b049-031be1288812"
 					(reference "L3")
+					(unit 1)
+				)
+			)
+			(project "PS-ChargerInterfacePCB"
+				(path "/894adbd2-6316-426a-afb4-88808e8ec51a/8fb4e0f4-a81e-4963-ba02-cb881e23146d"
+					(reference "L2")
 					(unit 1)
 				)
@@
 		(in_pos_files yes)
 		(dnp no)
-		(property "Reference" "TP3"
+		(property "Reference" "TP7"
 			(at 242.57 123.6979 0)
 			(hide yes)
@@
 				(path "/24809a72-9525-4be8-be3e-46bc27cfe8fb/cd4ac576-e1cf-46c0-a1b5-c681437cfde8/eaf4dc2b-ad73-4e1e-8bba-aa12f0e48269"
 					(reference "TP3")
+					(unit 1)
+				)
+			)
+			(project "PS-ChargerInterfacePCB"
+				(path "/894adbd2-6316-426a-afb4-88808e8ec51a/8fb4e0f4-a81e-4963-ba02-cb881e23146d"
+					(reference "TP7")
 					(unit 1)
 				)
@@
 		(in_pos_files yes)
 		(dnp no)
-		(property "Reference" "TP2"
+		(property "Reference" "TP6"
 			(at 229.87 136.3979 0)
 			(hide yes)
@@
 				(path "/24809a72-9525-4be8-be3e-46bc27cfe8fb/cd4ac576-e1cf-46c0-a1b5-c681437cfde8/eaf4dc2b-ad73-4e1e-8bba-aa12f0e48269"
 					(reference "TP2")
+					(unit 1)
+				)
+			)
+			(project "PS-ChargerInterfacePCB"
+				(path "/894adbd2-6316-426a-afb4-88808e8ec51a/8fb4e0f4-a81e-4963-ba02-cb881e23146d"
+					(reference "TP6")
 					(unit 1)
 				)
@@
 		(dnp no)
 		(fields_autoplaced yes)
-		(property "Reference" "U3"
+		(property "Reference" "U4"
 			(at 129.54 71.12 0)
 			(show_name no)
@@
 				(path "/331f457b-ed4e-4d4a-ad6d-c8acb2febfed/9243f342-8d42-4433-b049-031be1288812"
 					(reference "U3")
+					(unit 1)
+				)
+			)
+			(project "PS-ChargerInterfacePCB"
+				(path "/894adbd2-6316-426a-afb4-88808e8ec51a/8fb4e0f4-a81e-4963-ba02-cb881e23146d"
+					(reference "U4")
 					(unit 1)
 				)
@@
 		(in_pos_files yes)
 		(dnp no)
-		(property "Reference" "TP4"
+		(property "Reference" "TP8"
 			(at 242.57 136.3979 0)
 			(hide yes)
@@
 				(path "/24809a72-9525-4be8-be3e-46bc27cfe8fb/cd4ac576-e1cf-46c0-a1b5-c681437cfde8/eaf4dc2b-ad73-4e1e-8bba-aa12f0e48269"
 					(reference "TP4")
+					(unit 1)
+				)
+			)
+			(project "PS-ChargerInterfacePCB"
+				(path "/894adbd2-6316-426a-afb4-88808e8ec51a/8fb4e0f4-a81e-4963-ba02-cb881e23146d"
+					(reference "TP8")
 					(unit 1)
 				)
@@
 		(dnp no)
 		(fields_autoplaced yes)
-		(property "Reference" "#FLG04"
+		(property "Reference" "#FLG09"
 			(at 179.07 84.455 0)
 			(hide yes)
@@
 				(path "/331f457b-ed4e-4d4a-ad6d-c8acb2febfed/9243f342-8d42-4433-b049-031be1288812"
 					(reference "#FLG015")
+					(unit 1)
+				)
+			)
+			(project "PS-ChargerInterfacePCB"
+				(path "/894adbd2-6316-426a-afb4-88808e8ec51a/8fb4e0f4-a81e-4963-ba02-cb881e23146d"
+					(reference "#FLG09")
 					(unit 1)
 				)
@@
 		(dnp no)
 		(fields_autoplaced yes)
-		(property "Reference" "#FLG01"
+		(property "Reference" "#FLG06"
 			(at 88.9 79.375 0)
 			(hide yes)
@@
 				(path "/331f457b-ed4e-4d4a-ad6d-c8acb2febfed/9243f342-8d42-4433-b049-031be1288812"
 					(reference "#FLG011")
+					(unit 1)
+				)
+			)
+			(project "PS-ChargerInterfacePCB"
+				(path "/894adbd2-6316-426a-afb4-88808e8ec51a/8fb4e0f4-a81e-4963-ba02-cb881e23146d"
+					(reference "#FLG06")
 					(unit 1)
 				)
@@
 		(in_pos_files yes)
 		(dnp no)
-		(property "Reference" "C17"
+		(property "Reference" "C48"
 			(at 164.084 93.98 0)
 			(show_name no)
@@
 				(path "/24809a72-9525-4be8-be3e-46bc27cfe8fb/cd4ac576-e1cf-46c0-a1b5-c681437cfde8/eaf4dc2b-ad73-4e1e-8bba-aa12f0e48269"
 					(reference "C17")
+					(unit 1)
+				)
+			)
+			(project "PS-ChargerInterfacePCB"
+				(path "/894adbd2-6316-426a-afb4-88808e8ec51a/8fb4e0f4-a81e-4963-ba02-cb881e23146d"
+					(reference "C48")
 					(unit 1)
 				)
@@
 		(in_pos_files yes)
 		(dnp no)
-		(property "Reference" "C19"
+		(property "Reference" "C50"
 			(at 189.992 93.98 0)
 			(show_name no)
@@
 				(path "/24809a72-9525-4be8-be3e-46bc27cfe8fb/cd4ac576-e1cf-46c0-a1b5-c681437cfde8/eaf4dc2b-ad73-4e1e-8bba-aa12f0e48269"
 					(reference "C19")
+					(unit 1)
+				)
+			)
+			(project "PS-ChargerInterfacePCB"
+				(path "/894adbd2-6316-426a-afb4-88808e8ec51a/8fb4e0f4-a81e-4963-ba02-cb881e23146d"
+					(reference "C50")
 					(unit 1)
 				)
@@
 		(in_pos_files yes)
 		(dnp no)
-		(property "Reference" "C16"
+		(property "Reference" "C47"
 			(at 156.718 80.01 0)
 			(show_name no)
@@
 				(path "/331f457b-ed4e-4d4a-ad6d-c8acb2febfed/9243f342-8d42-4433-b049-031be1288812"
 					(reference "C12")
+					(unit 1)
+				)
+			)
+			(project "PS-ChargerInterfacePCB"
+				(path "/894adbd2-6316-426a-afb4-88808e8ec51a/8fb4e0f4-a81e-4963-ba02-cb881e23146d"
+					(reference "C47")
 					(unit 1)
 				)
@@
 		(in_pos_files yes)
 		(dnp no)
-		(property "Reference" "#FLG03"
+		(property "Reference" "#FLG08"
 			(at 149.86 84.455 0)
 			(hide yes)
@@
 				(path "/331f457b-ed4e-4d4a-ad6d-c8acb2febfed/9243f342-8d42-4433-b049-031be1288812"
 					(reference "#FLG014")
+					(unit 1)
+				)
+			)
+			(project "PS-ChargerInterfacePCB"
+				(path "/894adbd2-6316-426a-afb4-88808e8ec51a/8fb4e0f4-a81e-4963-ba02-cb881e23146d"
+					(reference "#FLG08")
 					(unit 1)
 				)
@@
 		(dnp no)
 		(fields_autoplaced yes)
-		(property "Reference" "R15"
+		(property "Reference" "R31"
 			(at 227.33 85.0899 0)
 			(show_name no)
@@
 				(path "/331f457b-ed4e-4d4a-ad6d-c8acb2febfed/9243f342-8d42-4433-b049-031be1288812"
 					(reference "R1")
+					(unit 1)
+				)
+			)
+			(project "PS-ChargerInterfacePCB"
+				(path "/894adbd2-6316-426a-afb4-88808e8ec51a/8fb4e0f4-a81e-4963-ba02-cb881e23146d"
+					(reference "R31")
 					(unit 1)
 				)
@@
 		(dnp no)
 		(fields_autoplaced yes)
-		(property "Reference" "C15"
+		(property "Reference" "C46"
 			(at 105.41 87.6362 0)
 			(show_name no)
@@
 				(path "/24809a72-9525-4be8-be3e-46bc27cfe8fb/cd4ac576-e1cf-46c0-a1b5-c681437cfde8/eaf4dc2b-ad73-4e1e-8bba-aa12f0e48269"
 					(reference "C15")
+					(unit 1)
+				)
+			)
+			(project "PS-ChargerInterfacePCB"
+				(path "/894adbd2-6316-426a-afb4-88808e8ec51a/8fb4e0f4-a81e-4963-ba02-cb881e23146d"
+					(reference "C46")
 					(unit 1)
 				)
@@
 		(dnp no)
 		(fields_autoplaced yes)
-		(property "Reference" "R16"
+		(property "Reference" "R34"
 			(at 227.33 92.7099 0)
 			(show_name no)
@@
 				(path "/331f457b-ed4e-4d4a-ad6d-c8acb2febfed/9243f342-8d42-4433-b049-031be1288812"
 					(reference "R4")
+					(unit 1)
+				)
+			)
+			(project "PS-ChargerInterfacePCB"
+				(path "/894adbd2-6316-426a-afb4-88808e8ec51a/8fb4e0f4-a81e-4963-ba02-cb881e23146d"
+					(reference "R34")
 					(unit 1)
 				)
@@
 		(in_pos_files yes)
 		(dnp no)
-		(property "Reference" "C18"
+		(property "Reference" "C49"
 			(at 173.482 94.234 0)
 			(show_name no)
@@
 					(unit 1)
 				)
+			)
+			(project "PS-ChargerInterfacePCB"
+				(path "/894adbd2-6316-426a-afb4-88808e8ec51a/8fb4e0f4-a81e-4963-ba02-cb881e23146d"
+					(reference "C49")
+					(unit 1)
+				)
