File: PowerProtection.kicad_sch (KiCad schematic)
At the start: 18 parts, among them IC1 LM74502DDFR, Q1 PSMN012-100YS, Q2 PSMN012-100YS

Commit message: YOOO KICAD IS KICADDING IT MAKES SENSEEEEEEEEEEEEEE
Parts:
- renumbered C1 to C22, C2 to C23, C3 to C40, C4 to C41, C5 to C42, C6 to C43, C7 to C44, D1 to D11, D2 to D12, IC1 to IC2, Q1 to Q3, Q2 to Q8, R1 to R25, R2 to R26, R3 to R27, R4 to R28, R5 to R29, R6 to R30
Changed lines of the file:
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@@
 		(in_pos_files yes)
 		(dnp no)
-		(property "Reference" "D2"
+		(property "Reference" "D12"
 			(at 40.64 82.296 0)
 			(show_name no)
@@
 				(path "/24809a72-9525-4be8-be3e-46bc27cfe8fb/cd4ac576-e1cf-46c0-a1b5-c681437cfde8/8c26e1fb-a8ae-4852-ae6e-03a0af74066d"
 					(reference "D2")
+					(unit 1)
+				)
+			)
+			(project "PS-ChargerInterfacePCB"
+				(path "/894adbd2-6316-426a-afb4-88808e8ec51a/734086b2-1e51-47d3-b0a3-7759e9e847f1"
+					(reference "D12")
 					(unit 1)
 				)
@@
 		(dnp no)
 		(fields_autoplaced yes)
-		(property "Reference" "C3"
+		(property "Reference" "C40"
 			(at 57.785 80.0099 0)
 			(show_name no)
@@
 				(path "/24809a72-9525-4be8-be3e-46bc27cfe8fb/cd4ac576-e1cf-46c0-a1b5-c681437cfde8/8c26e1fb-a8ae-4852-ae6e-03a0af74066d"
 					(reference "C3")
+					(unit 1)
+				)
+			)
+			(project "PS-ChargerInterfacePCB"
+				(path "/894adbd2-6316-426a-afb4-88808e8ec51a/734086b2-1e51-47d3-b0a3-7759e9e847f1"
+					(reference "C40")
 					(unit 1)
 				)
@@
 		(in_pos_files yes)
 		(dnp no)
-		(property "Reference" "D1"
+		(property "Reference" "D11"
 			(at 22.606 49.276 0)
 			(show_name no)
@@
 				(path "/24809a72-9525-4be8-be3e-46bc27cfe8fb/cd4ac576-e1cf-46c0-a1b5-c681437cfde8/8c26e1fb-a8ae-4852-ae6e-03a0af74066d"
 					(reference "D1")
+					(unit 1)
+				)
+			)
+			(project "PS-ChargerInterfacePCB"
+				(path "/894adbd2-6316-426a-afb4-88808e8ec51a/734086b2-1e51-47d3-b0a3-7759e9e847f1"
+					(reference "D11")
 					(unit 1)
 				)
@@
 		(dnp no)
 		(fields_autoplaced yes)
-		(property "Reference" "R1"
+		(property "Reference" "R25"
 			(at 45.72 60.9599 0)
 			(show_name no)
@@
 				(path "/24809a72-9525-4be8-be3e-46bc27cfe8fb/cd4ac576-e1cf-46c0-a1b5-c681437cfde8/8c26e1fb-a8ae-4852-ae6e-03a0af74066d"
 					(reference "R1")
+					(unit 1)
+				)
+			)
+			(project "PS-ChargerInterfacePCB"
+				(path "/894adbd2-6316-426a-afb4-88808e8ec51a/734086b2-1e51-47d3-b0a3-7759e9e847f1"
+					(reference "R25")
 					(unit 1)
 				)
@@
 		(in_pos_files yes)
 		(dnp no)
-		(property "Reference" "R6"
+		(property "Reference" "R30"
 			(at 137.668 90.17 90)
 			(show_name no)
@@
 				(path "/24809a72-9525-4be8-be3e-46bc27cfe8fb/cd4ac576-e1cf-46c0-a1b5-c681437cfde8/8c26e1fb-a8ae-4852-ae6e-03a0af74066d"
 					(reference "R6")
+					(unit 1)
+				)
+			)
+			(project "PS-ChargerInterfacePCB"
+				(path "/894adbd2-6316-426a-afb4-88808e8ec51a/734086b2-1e51-47d3-b0a3-7759e9e847f1"
+					(reference "R30")
 					(unit 1)
 				)
@@
 		(in_pos_files yes)
 		(dnp no)
-		(property "Reference" "C1"
+		(property "Reference" "C22"
 			(at 38.1 49.5299 0)
 			(show_name no)
@@
 				(path "/24809a72-9525-4be8-be3e-46bc27cfe8fb/cd4ac576-e1cf-46c0-a1b5-c681437cfde8/8c26e1fb-a8ae-4852-ae6e-03a0af74066d"
 					(reference "C1")
+					(unit 1)
+				)
+			)
+			(project "PS-ChargerInterfacePCB"
+				(path "/894adbd2-6316-426a-afb4-88808e8ec51a/734086b2-1e51-47d3-b0a3-7759e9e847f1"
+					(reference "C22")
 					(unit 1)
 				)
@@
 		(in_pos_files yes)
 		(dnp no)
-		(property "Reference" "R2"
+		(property "Reference" "R26"
 			(at 67.31 54.61 90)
 			(show_name no)
@@
 				(path "/24809a72-9525-4be8-be3e-46bc27cfe8fb/cd4ac576-e1cf-46c0-a1b5-c681437cfde8/8c26e1fb-a8ae-4852-ae6e-03a0af74066d"
 					(reference "R2")
+					(unit 1)
+				)
+			)
+			(project "PS-ChargerInterfacePCB"
+				(path "/894adbd2-6316-426a-afb4-88808e8ec51a/734086b2-1e51-47d3-b0a3-7759e9e847f1"
+					(reference "R26")
 					(unit 1)
 				)
@@
 		(in_pos_files yes)
 		(dnp no)
-		(property "Reference" "IC1"
+		(property "Reference" "IC2"
 			(at 75.184 73.66 0)
 			(show_name no)
@@
 				(path "/24809a72-9525-4be8-be3e-46bc27cfe8fb/cd4ac576-e1cf-46c0-a1b5-c681437cfde8/8c26e1fb-a8ae-4852-ae6e-03a0af74066d"
 					(reference "IC1")
+					(unit 1)
+				)
+			)
+			(project "PS-ChargerInterfacePCB"
+				(path "/894adbd2-6316-426a-afb4-88808e8ec51a/734086b2-1e51-47d3-b0a3-7759e9e847f1"
+					(reference "IC2")
 					(unit 1)
 				)
@@
 		(in_pos_files yes)
 		(dnp no)
-		(property "Reference" "Q1"
+		(property "Reference" "Q3"
 			(at 52.578 38.862 90)
 			(show_name no)
@@
 				(path "/24809a72-9525-4be8-be3e-46bc27cfe8fb/cd4ac576-e1cf-46c0-a1b5-c681437cfde8/8c26e1fb-a8ae-4852-ae6e-03a0af74066d"
 					(reference "Q1")
+					(unit 1)
+				)
+			)
+			(project "PS-ChargerInterfacePCB"
+				(path "/894adbd2-6316-426a-afb4-88808e8ec51a/734086b2-1e51-47d3-b0a3-7759e9e847f1"
+					(reference "Q3")
 					(unit 1)
 				)
@@
 		(in_pos_files yes)
 		(dnp no)
-		(property "Reference" "C6"
+		(property "Reference" "C43"
 			(at 113.284 89.154 0)
 			(show_name no)
@@
 				(path "/24809a72-9525-4be8-be3e-46bc27cfe8fb/cd4ac576-e1cf-46c0-a1b5-c681437cfde8/8c26e1fb-a8ae-4852-ae6e-03a0af74066d"
 					(reference "C6")
+					(unit 1)
+				)
+			)
+			(project "PS-ChargerInterfacePCB"
+				(path "/894adbd2-6316-426a-afb4-88808e8ec51a/734086b2-1e51-47d3-b0a3-7759e9e847f1"
+					(reference "C43")
 					(unit 1)
 				)
@@
 		(in_pos_files yes)
 		(dnp no)
-		(property "Reference" "C4"
+		(property "Reference" "C41"
 			(at 54.864 62.23 0)
 			(show_name no)
@@
 				(path "/24809a72-9525-4be8-be3e-46bc27cfe8fb/cd4ac576-e1cf-46c0-a1b5-c681437cfde8/8c26e1fb-a8ae-4852-ae6e-03a0af74066d"
 					(reference "C4")
+					(unit 1)
+				)
+			)
+			(project "PS-ChargerInterfacePCB"
+				(path "/894adbd2-6316-426a-afb4-88808e8ec51a/734086b2-1e51-47d3-b0a3-7759e9e847f1"
+					(reference "C41")
 					(unit 1)
 				)
@@
 		(in_pos_files yes)
 		(dnp no)
-		(property "Reference" "C5"
+		(property "Reference" "C42"
 			(at 112.395 49.5299 0)
 			(show_name no)
@@
 				(path "/24809a72-9525-4be8-be3e-46bc27cfe8fb/cd4ac576-e1cf-46c0-a1b5-c681437cfde8/8c26e1fb-a8ae-4852-ae6e-03a0af74066d"
 					(reference "C5")
+					(unit 1)
+				)
+			)
+			(project "PS-ChargerInterfacePCB"
+				(path "/894adbd2-6316-426a-afb4-88808e8ec51a/734086b2-1e51-47d3-b0a3-7759e9e847f1"
+					(reference "C42")
 					(unit 1)
 				)
@@
 		(in_pos_files yes)
 		(dnp no)
-		(property "Reference" "Q2"
+		(property "Reference" "Q8"
 			(at 100.584 38.608 90)
 			(show_name no)
@@
 				(path "/24809a72-9525-4be8-be3e-46bc27cfe8fb/cd4ac576-e1cf-46c0-a1b5-c681437cfde8/8c26e1fb-a8ae-4852-ae6e-03a0af74066d"
 					(reference "Q2")
+					(unit 1)
+				)
+			)
+			(project "PS-ChargerInterfacePCB"
+				(path "/894adbd2-6316-426a-afb4-88808e8ec51a/734086b2-1e51-47d3-b0a3-7759e9e847f1"
+					(reference "Q8")
 					(unit 1)
 				)
@@
 		(in_pos_files yes)
 		(dnp no)
-		(property "Reference" "R4"
+		(property "Reference" "R28"
 			(at 118.618 90.424 90)
 			(show_name no)
@@
 				(path "/24809a72-9525-4be8-be3e-46bc27cfe8fb/cd4ac576-e1cf-46c0-a1b5-c681437cfde8/8c26e1fb-a8ae-4852-ae6e-03a0af74066d"
 					(reference "R4")
+					(unit 1)
+				)
+			)
+			(project "PS-ChargerInterfacePCB"
+				(path "/894adbd2-6316-426a-afb4-88808e8ec51a/734086b2-1e51-47d3-b0a3-7759e9e847f1"
+					(reference "R28")
 					(unit 1)
 				)
@@
 		(in_pos_files yes)
 		(dnp no)
-		(property "Reference" "C2"
+		(property "Reference" "C23"
 			(at 31.75 82.5499 0)
 			(show_name no)
@@
 				(path "/24809a72-9525-4be8-be3e-46bc27cfe8fb/cd4ac576-e1cf-46c0-a1b5-c681437cfde8/8c26e1fb-a8ae-4852-ae6e-03a0af74066d"
 					(reference "C2")
+					(unit 1)
+				)
+			)
+			(project "PS-ChargerInterfacePCB"
+				(path "/894adbd2-6316-426a-afb4-88808e8ec51a/734086b2-1e51-47d3-b0a3-7759e9e847f1"
+					(reference "C23")
 					(unit 1)
 				)
@@
 		(in_pos_files yes)
 		(dnp no)
-		(property "Reference" "C7"
+		(property "Reference" "C44"
 			(at 132.08 88.9 0)
 			(show_name no)
@@
 				(path "/24809a72-9525-4be8-be3e-46bc27cfe8fb/cd4ac576-e1cf-46c0-a1b5-c681437cfde8/8c26e1fb-a8ae-4852-ae6e-03a0af74066d"
 					(reference "C7")
+					(unit 1)
+				)
+			)
+			(project "PS-ChargerInterfacePCB"
+				(path "/894adbd2-6316-426a-afb4-88808e8ec51a/734086b2-1e51-47d3-b0a3-7759e9e847f1"
+					(reference "C44")
 					(unit 1)
 				)
@@
 		(in_pos_files yes)
 		(dnp no)
-		(property "Reference" "R3"
+		(property "Reference" "R27"
 			(at 118.11 78.74 90)
 			(show_name no)
@@
 				(path "/24809a72-9525-4be8-be3e-46bc27cfe8fb/cd4ac576-e1cf-46c0-a1b5-c681437cfde8/8c26e1fb-a8ae-4852-ae6e-03a0af74066d"
 					(reference "R3")
+					(unit 1)
+				)
+			)
+			(project "PS-ChargerInterfacePCB"
+				(path "/894adbd2-6316-426a-afb4-88808e8ec51a/734086b2-1e51-47d3-b0a3-7759e9e847f1"
+					(reference "R27")
 					(unit 1)
 				)
@@
 		(in_pos_files yes)
 		(dnp no)
-		(property "Reference" "R5"
+		(property "Reference" "R29"
 			(at 137.16 77.47 90)
 			(show_name no)
@@
 					(unit 1)
 				)
+			)
+			(project "PS-ChargerInterfacePCB"
+				(path "/894adbd2-6316-426a-afb4-88808e8ec51a/734086b2-1e51-47d3-b0a3-7759e9e847f1"
+					(reference "R29")
+					(unit 1)
+				)
