File: PowerProtection.kicad_sch (KiCad schematic)
At the start: 18 parts, among them IC2 LM74502DDFR, Q3 PSMN012-100YS, Q8 PSMN012-100YS

Commit message: updated from review
Parts:
- IC2: Manufacturer_Name Texas Instruments -> (none); Manufacturer_Part_Number LM74502DDFR -> (none); Mouser Part Number 595-LM74502DDFR -> (none); Mouser Price/Stock https://www.mouser.co.uk/ProductDetail/Texas-Instruments/LM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 -> (none)
- R25, R27, R28, R29, R30: symbol Device:R_US -> Device:R
- R26: symbol Device:R_US -> Device:R; Mouser Part Number 594-MCT06030C3309FP5 -> (none)
- renumbered C40 to C34, C41 to C35, C42 to C36, C43 to C37, C44 to C38, Q8 to Q4
Connections:
- net LV_INPUT renamed Vin
- net LV_PROTECTED renamed Vout
Other:
- note added: "Supp Battery Range: 10V-14.7V"

Commit message: final schem is done
Parts:
- IC2: Height 1.1 -> (none)
- R28: value 7.32k -> 7.5k
- R30: value 15.8k -> 16k
Changed lines of the file:
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@@
 			)
 		)
-		(property "Value" "15.8k"
+		(property "Value" "16k"
 			(at 142.1766 90.6279 90)
 			(show_name no)
@@
 					(size 1.27 1.27)
 				)
-			)
-		)
-		(property "Height" "1.1"
-			(at 87.8206 472.8479 0)
-			(hide yes)
-			(show_name no)
-			(do_not_autoplace no)
-			(effects
-				(font
-					(size 1.27 1.27)
-				)
-				(justify left top)
 			)
 		)
@@
 			)
 		)
-		(property "Value" "7.32k"
+		(property "Value" "7.5k"
 			(at 123.3806 90.6279 90)
 			(show_name no)
@@
 		)
 	)
-	(group "PowerProtection"
-		(lib_id "LHRS_Design_Blocks:PowerProtection")
-		(members "0157c5b9-1d12-4516-850c-df565267155d" "028d7e33-5495-41d6-951d-e09212ed3103"
-			"03fbb6c3-15d6-4535-82c3-c84cadec759c" "042b9804-47b9-407a-87bf-5006a6aed699"
-			"0532c7ef-c8b3-4369-b510-030cbcdb8621" "059216cd-1ded-4c32-9f18-13b3db375266"
-			"0aa69882-de1c-4b10-8454-c23ce2acdd91" "0b30506d-1261-4f6a-9a3e-4c30c82a78fa"
-			"0cfad45b-7b2d-40f5-aa4f-d2214414e9a0" "0fa2286c-1be4-48ff-9c31-fcb86345438d"
-			"14f2588b-629f-40c0-a55f-d15f2922381c" "15394460-0b64-47c5-be51-1e4fcfa417d4"
-			"1842124c-90fe-4fba-9347-6a7260ba0eca" "199aa610-9666-48a9-b1cc-4d7400331b7d"
-			"1bf284e5-4120-42a9-8010-d59a01609411" "1df926d3-e014-409c-a713-f3cb5e429ba0"
-			"2740b1f3-b2f5-419e-b651-a6b35e5f1ddf" "27bb416f-21f7-4e22-bc56-e869d50905e8"
-			"2a291319-3f12-4c65-aded-7d3a127b1252" "2bbb7cb1-8cce-48ea-96aa-93d2882b58c5"
-			"2c45fc8a-bcc4-4313-aeca-374a3cb5e0de" "2c76a0cc-58b1-4c06-b0d9-ee9e63c15e57"
-			"30175d18-769c-4cf5-98fe-c1abd5d1092e" "3042d6a4-c126-4ba0-8ab9-c162ceb99787"
-			"31ae8354-1bd7-40a1-86ef-acc8f08023be" "31d51f2a-243b-4f91-82d5-c2cd00048be3"
-			"337eba05-736d-45d9-b0f8-e60a04f8013c" "34033bf7-70d3-41fc-80b6-c0602c302ef3"
-			"35d0e42a-8cfa-43f0-9e71-9eb0ec5ead55" "37b56203-4752-4bdb-bb86-efe7fa80cf3e"
-			"3801b2eb-c26d-4923-b07e-bb6a16c9d9dc" "382ad997-2959-49b6-8ab7-83c23a463de1"
-			"40c8c654-4b92-454b-a551-60c222526fbc" "40d80543-15a9-4e01-a3fa-784f61793bf4"
-			"4388180a-b57a-4cc6-be50-953f71979e49" "43e6aa5a-b8c1-4ab4-afc3-a7efaaca1b67"
-			"44f24f69-2ebf-48c9-8feb-7d7ea03996d8" "48062dd8-60d4-4c44-80a1-928bb08f13b0"
-			"4bf2de47-0582-4482-b8ca-6c9a319ed0da" "4fe2900d-664e-42fc-863b-e732cb8dc69d"
-			"51544d6f-e376-4a23-9c06-49f513e0d5c3" "531a336d-51aa-4c26-976d-7a821624a89d"
-			"5548a6b6-c8db-4fc6-a165-38341904b29b" "554c6273-4c35-418e-b9d9-5d7b3feeab64"
-			"565f1b0c-8d57-4fec-bd87-e5f22db5587d" "5753d70c-6755-432a-8c59-3c71c675263b"
-			"57559998-a595-4153-b68e-1335bb4fac8d" "598575bc-3048-42fa-a1e1-914413ea14b9"
-			"59c254e2-8f4e-431c-91ae-2b5f150727f9" "5a1edcc6-e02b-4a70-a838-d5cd3df2c5e5"
-			"5c984d6a-b70e-4989-a490-4d2b48765eda" "5cab5f5b-0835-4fce-b37f-add97d1d6188"
-			"5f18d0a5-2501-46ec-b092-fdc9000bfef1" "5f5d4641-114a-492c-8314-f76781a829e7"
-			"5f8c95be-4bec-4715-b67b-6a9afc6a3131" "65f4a0d1-5d21-4425-a99d-6227947d25b9"
-			"6a21298e-67e8-4795-9c87-4e04e75f29db" "6a2ff7b5-2f3a-4ada-af27-acf146ad2ad8"
-			"6d11c85c-4365-434d-a995-ca1ab2b98a96" "6f61fa7b-fa77-470a-a21c-aa81b96025ad"
-			"727bf9c3-1734-4672-b662-92fe1024f40d" "72cb8fba-a330-4160-b789-ddddf7b5a89c"
-			"73dcf30c-1114-4b7f-9b6d-e8e575b19d22" "73f1f844-30cb-409c-930e-4e260e176e8c"
-			"790db299-76a0-434a-80c5-01995928d894" "7aff0b31-24d0-44b7-8e25-f1e4d07b7170"
-			"7b638785-7db1-4c9a-aa60-2218ea513bd0" "7bc694e4-819e-483a-90c2-22587174c927"
-			"7d25a8b7-ef74-4c9e-9f8f-32b3f27d3cc3" "7ef6a9c6-6dfc-4d5d-9283-e70d8c20270f"
-			"7f642bd0-3679-4f40-b67e-20f9329162fe" "82c09f50-9749-4d1f-bf8a-45afddd9ca33"
-			"831575bb-49e0-4cdb-93b8-525333b308ac" "863a57f8-9727-4506-9f01-2bdfd54f8dc7"
-			"8b737fda-6574-4690-9394-92383143474c" "8d007b28-9816-472b-b6c4-43ca10aad6f5"
-			"8e0823b6-e6ac-43d8-9953-fe455cb21e99" "919fdca5-2912-4f1c-a885-7e3a3ebfcb90"
-			"91a7aaf4-8965-47be-900f-cb00d29ddd84" "98a46178-137c-4697-845c-5d56c9be7f60"
-			"9a0d61c7-7560-4484-b50d-b84161d849f5" "9a374655-09c5-4637-97f7-32388f92fc1f"
-			"9ad8d2ea-210c-4b9b-a887-7ae5ea15f9b5" "9b1ddc4f-24aa-46be-8d1e-e07bf585137f"
-			"9ca2f5d2-8fba-42ee-b899-b582337ac0c5" "9ecdc88e-62ed-4bbf-95d3-eb0f8a62dccf"
-			"9f1318a2-0d2e-4c0a-a1d7-6dc5345f06f4" "a0dc4068-8e72-44ac-ab37-6e2f6d52b340"
-			"a320d627-67b8-4194-99a1-8bbac51b6563" "a434ae9d-2945-490b-a49b-a3f3f0acb338"
-			"a4deae88-7df1-4411-8ab3-b2332c17194a" "a54230e9-d804-4c90-912c-5b4f0c59f243"
-			"a643014a-f928-43c7-bf94-eec8ea1e787f" "a65db99e-b6d1-461d-9c1d-6a77bda00c65"
-			"a7b1ba28-2bb6-4437-805c-05a5a100cb4b" "a7b3dbed-73ff-4e87-8084-24d293d6789b"
-			"a7dbae91-56e6-4952-a182-78002621aba1" "b04a0a47-0a87-4e18-a9be-a2503cc77592"
-			"b0c78084-6d90-4b63-a054-6d5dc55d9fa2" "b95bdb84-4318-4c45-880f-e78847cceddb"
-			"ba30a29a-dfdd-4ab7-a41f-d3ef9360a0f6" "bb691a7d-ab90-4d7c-8a58-08500182539f"
-			"bcfc2c39-37c9-4a25-84f6-09f2b66c751d" "bd1a9720-fb99-4847-bca2-7d59f7ee436d"
-			"bdaef940-3615-4156-9afa-ac1ba9c8a896" "be94d869-90f2-4669-bef8-7f9b9e85a653"
-			"bfe7bf24-16b5-45b8-8a2c-083d1914e08a" "c2dd4931-d5fc-46ac-aa80-da145d727bd3"
-			"c8a78fcb-d744-4655-a3db-07f6c7ef3c33" "c99346f3-cf25-4b2b-b50c-e7e063bd40c1"
-			"ce515302-37c1-46f4-9605-324717ada18d" "d0931abc-1d63-495a-a11e-cefecba35ff8"
-			"d1ed36c6-e316-437e-8836-007106c2baca" "d2886056-b0d4-4197-9281-c8007cdcb4fd"
-			"d3dbe8c4-0167-43f1-91ab-5e760928b53f" "d4b220b6-0bfb-4e81-a6a0-7446c58193d0"
-			"d82c2d9c-5f25-43a3-bd89-29d34615c72c" "dc50b215-6e88-4055-b18d-dec3d913aa62"
-			"e113135d-12a9-4987-b998-7e6f28eb3824" "e206ab59-1ae1-491c-b1fb-63358e7fa2aa"
-			"e2bdff8b-4fb3-40ca-8820-b2efc8b45b22" "e4d69209-f38e-4f7d-b217-7636e4c3ef67"
-			"e6323ddc-dd3b-428a-a630-75f00c295f4e" "e924a9bb-b010-4265-8293-2b0fb47251d4"
-			"eaa9b6e8-df89-4094-b71d-a7cbdcccd5e6" "eaec819f-fce9-4599-9b78-2432217b750b"
-			"ebd9efad-b1ae-437b-8a4f-c139746881ed" "eed295d2-d863-41b8-8f82-f58eb00d6d72"
-			"ef3248e5-e1a4-4434-b8bf-c43907dff49b" "f071ec24-e472-4003-9896-c8d9a2aadeeb"
-			"f07653c5-8d88-4702-88df-582da9d44e81" "f663a02e-90fd-430f-a693-e67fe2b4fdbf"
-			"f8dd055b-d303-4a1d-8308-7974c919c9c5" "fac22fc4-7e9e-4207-bfc0-c7591103cd8f"
-			"fbfaecd8-c9de-4f4d-b582-c1b58168393f" "fd950331-3579-4221-8212-897c11e97a5d"
-			"fecacf80-cf0b-411b-9c59-69530ade4a30" "fef0aad0-107f-4307-9fc2-a0cc47dcf58f"
-		)
-	)

Commit message: review council
Parts:
- IC2: Height (none) -> 1.1
- R28: value 7.5k -> 7.32k
- R30: value 16k -> 15.8k
- renumbered C34 to C33, C35 to C34, C36 to C35, C37 to C36, C38 to C37
Other:
- moved on the sheet: C22, C23, C33, C34, C35, C36, C37, D11, D12, IC2, Q3, Q4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
