File: untitled.kicad_sch (KiCad schematic)
At the start: 20 parts, among them Q10 IRLML0030TRPBF, Q11 IRLML0030TRPBF, Q12 IRLML0030TRPBF, Q14 IRLML0030TRPBF, Q9 IRLML0030TRPBF

Commit message: documentation is better than gpt tony was right
Parts:
- renumbered D14 to D18, D15 to D19, D16 to D20, D17 to D21, D22 to D23, Q9 to Q15, Q10 to Q16, Q11 to Q17, Q12 to Q18, Q14 to Q19, R37 to R46, R38 to R47, R39 to R48, R40 to R49, R41 to R50, R42 to R51, R43 to R52, R44 to R53, R45 to R54, R55 to R56
Other:
- note added: "Drain/MCU"
