File: untitled.kicad_sch (KiCad schematic)
At the start: 20 parts, among them Q15 IRLML0030TRPBF, Q16 IRLML0030TRPBF, Q17 IRLML0030TRPBF, Q18 IRLML0030TRPBF, Q19 IRLML0030TRPBF

Commit message: half ish done with review fixes
Parts:
- R47, R49, R52, R54, R56: value 470 -> 1k
Other:
- note removed: "Drain/MCU"
- moved on the sheet: D18, D21, Q15, Q19, R46, R47, R53, R54

Commit message: updated from review
Parts:
- removed D21: LED, LED_SMD:LED_0603_1608Metric, symbol Device:LED
- removed Q19: IRLML0030TRPBF, charger_parts:IRLML0030TRPBF, symbol IRLML0030TRPBF:IRLML0030TRPBF
- removed R53: 100k, Resistor_SMD:R_0603_1608Metric, symbol Device:R_US
- removed R54: 1k, Resistor_SMD:R_0603_1608Metric, symbol Device:R_US
- added D21: LED_RGBA, LED_SMD:LED_Cree-XHP50_3V_HighDensity, symbol Device:LED_RGBA
- added R42, R43: 100, symbol Device:R
- added R44: 330, symbol Device:R
Connections:
- new net: D21.1 (RK), R44.1
- new net: D21.2 (GK), R43.1
- new net: D21.3 (BK), R42.1
- new net ANODE_IN: D21.4 (A)
- new net MCU_B: R42.2
- new net MCU_G: R43.2
- new net MCU_R: R44.2
