File: atempt_2.kicad_sch (KiCad schematic)
At the start: 4 parts, among them J6 Elcon Connector, J7 BPSL Connector, J8 CAN_NANO_01x03, J9 Conn_02x05_Counter_Clockwise

Commit message: documentation is better than gpt tony was right
Parts:
- added J10, J11: Conn_01x02, Package_DIP:DIP-20_W7.62mm, symbol Connector_Generic:Conn_01x02
Connections:
- net +14V: now also J9.1 (Pin_1), J9.2 (Pin_2), J9.3 (Pin_3), J9.4 (Pin_4), J9.5 (Pin_5)
- net GND: now also J10.2 (Pin_2), J11.2 (Pin_2)
- net HV-: now reaches J9.10 (Pin_10)
- net EVSE-: now reaches J9.6 (Pin_6)
- net CHARGE-: now reaches J9.7 (Pin_7)
- net HEART-: now reaches J9.8 (Pin_8)
- net FAULT-: now reaches J9.9 (Pin_9)
- new net ESTOP_BUT: J10.1 (Pin_1)
- new net SHUTDOWN_BUT: J11.1 (Pin_1)
Other:
- removed sheet MCU
- sheet BigRedButtons ports: added ESTOP, ESTOP_SENSE, SOFT_SHUT, SOFT_SHUTDOWN; removed none
- sheet LEDS ports: added CHARGE-, EVSE-, FAULT-, HEART-, HV-, LED_CHARGE, LED_EVSE, LED_FAULT, LED_HEART, LED_HV; removed none
- moved on the sheet: J6, J7, J8, J9

Commit message: I THIHK I GET IT NOW
Other:
- added sheet 48PinMCU (48PinMCU.kicad_sch)
- sheet Buzzer ports: added BUZ+, BUZ-, BuzzPWM; removed none
- sheet Display ports: added BLK, CS, DC, GND, RES, SCL, SDA, VCC; removed none
- note added: "Buzzer"
- note added: "Display SPI"
- note added: "Interface"
- moved on the sheet: J10, J11, J6, J7, J8, J9

Commit message: mcuuuuuuuu
Parts:
- removed J6: Elcon Connector, LHRS_Connectors:Molex_Nano-Fit_105309-xx04_1x04_P2.50mm_Vertical, symbol lhrs_connectors:PeripheralCANConnector
- removed J7: BPSL Connector, LHRS_Connectors:Molex_Nano-Fit_105309-xx04_1x04_P2.50mm_Vertical, symbol lhrs_connectors:PeripheralCANConnector
- added J15: Buzzer, Package_DIP:DIP-20_W7.62mm, symbol Connector_Generic:Conn_01x02
- added J16: ELCON_CAN, LHRS_Connectors:Molex_Nano-Fit_105309-xx05_1x04_P2.50mm_Vertical, symbol lhrs_connectors:CAN_DEBUG_NANO_01x04
- added J17: BPS_CAN, LHRS_Connectors:Molex_Nano-Fit_105309-xx05_1x04_P2.50mm_Vertical, symbol lhrs_connectors:CAN_DEBUG_NANO_01x04
- added J18: ELCON_CAN_DEBUG, Package_DIP:DIP-20_W7.62mm, symbol Connector_Generic:Conn_01x02
- J10: value Conn_01x02 -> ESTOP
- J11: value Conn_01x02 -> SHUTDOWN
- J9: value Conn_02x05_Counter_Clockwise -> LEDS
Connections:
- net Car_CAN_H: now also J17.2 (CAN_H)
- net Car_CAN_L: now also J17.3 (CAN_L)
- net Elcon_CAN_H: now also J16.2 (CAN_H), J18.1 (Pin_1)
- net Elcon_CAN_L: now also J16.3 (CAN_L), J18.2 (Pin_2)
- net GND: now also J16.4 (GND), J17.4 (GND)
- net Vin: now also J16.1 (14V)
- new net BUZ+: J15.1 (Pin_1)
- new net BUZ-: J15.2 (Pin_2)

Commit message: need to do mcu now
Other:
- added sheet EVSE (EVSE.kicad_sch)
- sheet 48PinMCU ports: added +3V3, BOOT0, GND, GNDA, NRST, PA10, PA15, PA3, PA4, PA5, PA6, PA7, PA8, PA9, PB0, PB1, PB10, PB11, PB12, PB13, PB14, PB15, PB2, PB3, PB4, PB5, PB6, PB7, PB9, PC13, PC14, PC15, USB_DM, USB_DP, VDDA; removed none
- note added: "ELCON GND"
- note added: "EVSE"

Commit message: mcu working maybe????????????
Other:
- added sheet BPS_CAN (BPS_CAN.kicad_sch)
- added sheet ELCON_CAN (ELCON_CAN.kicad_sch)
- added sheet USB-C_Connector (USB-C_Connector.kicad_sch)
- sheet 48PinMCU ports: added none; removed +3V3, BOOT0, GNDA, NRST, PA10, PA15, PA6, PA8, PA9, PC13, PC14, PC15, VDDA
- note added: "CAN"
- note added: "USB-C"
