File: LDO.kicad_sch (KiCad schematic)
At the start: 5 parts, among them U2 MCP1826S

Commit message: deleted the bs
Parts:
- renumbered C12 to C51, C13 to C52, D8 to D13, TP_3.3V1 to TP_3.3V2, U2 to U5
Changed lines of the file:
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@@
 		(dnp no)
 		(fields_autoplaced yes)
-		(property "Reference" "C13"
+		(property "Reference" "C52"
 			(at 168.275 68.5735 0)
 			(show_name no)
@@
 		(in_pos_files yes)
 		(dnp no)
-		(property "Reference" "TP_3.3V1"
+		(property "Reference" "TP_3.3V2"
 			(at 166.624 54.356 90)
 			(show_name no)
@@
 		(dnp no)
 		(fields_autoplaced yes)
-		(property "Reference" "U2"
+		(property "Reference" "U5"
 			(at 152.4 56.515 0)
 			(show_name no)
@@
 		(dnp no)
 		(fields_autoplaced yes)
-		(property "Reference" "D8"
+		(property "Reference" "D13"
 			(at 133.604 57.15 0)
 			(show_name no)
@@
 		(dnp no)
 		(fields_autoplaced yes)
-		(property "Reference" "C12"
+		(property "Reference" "C51"
 			(at 142.875 68.5735 0)
 			(show_name no)
