File: LDO.kicad_sch (KiCad schematic)
At the start: 5 parts, among them U5 MCP1826S

Commit message: final schem is done
Parts:
- C51, C52: Mouser P/N GRM21BR61H106KE43K -> (none)
- D13: Old LCSC P/N C124187 -> (none); Old P/N BAT760-7 -> (none)
- U5: Datasheet Embed kicad-embed://22057B.pdf -> (none); LCSC MFG P/N LM39100S-3.3 -> (none)
Changed lines of the file:
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@@
-			)
-		)
-		(property "Mouser P/N" "GRM21BR61H106KE43K"
-			(at 165.1 69.85 0)
-			(hide yes)
-			(show_name no)
-			(do_not_autoplace no)
-			(effects
-				(font
-					(size 1.27 1.27)
-				)
 			)
 		)
@@
 			(at 165.1 63.5 0)
 			(hide yes)
-			(show_name no)
-			(do_not_autoplace no)
-			(effects
-				(font
-					(size 1.27 1.27)
-				)
-			)
-		)
-		(property "Color" ""
-			(at 165.1 63.5 0)
-			(show_name no)
-			(do_not_autoplace no)
-			(effects
-				(font
-					(size 1.27 1.27)
-				)
-			)
-		)
-		(property "If" ""
-			(at 165.1 63.5 0)
-			(show_name no)
-			(do_not_autoplace no)
-			(effects
-				(font
-					(size 1.27 1.27)
-				)
-			)
-		)
-		(property "Mfg" ""
-			(at 165.1 63.5 0)
-			(show_name no)
-			(do_not_autoplace no)
-			(effects
-				(font
-					(size 1.27 1.27)
-				)
-			)
-		)
-		(property "Vf" ""
-			(at 165.1 63.5 0)
 			(show_name no)
 			(do_not_autoplace no)
@@
 			)
 		)
-		(property "Datasheet Embed" "kicad-embed://22057B.pdf"
-			(at 152.4 63.5 0)
-			(hide yes)
-			(show_name no)
-			(do_not_autoplace no)
-			(effects
-				(font
-					(size 1.27 1.27)
-				)
-			)
-		)
 		(property "P/N" "MCP1826S-3302E/DB"
 			(at 152.4 63.5 0)
@@
 		)
 		(property "LCSC P/N" "C126055"
-			(at 152.4 63.5 0)
-			(hide yes)
-			(show_name no)
-			(do_not_autoplace no)
-			(effects
-				(font
-					(size 1.27 1.27)
-				)
-			)
-		)
-		(property "LCSC MFG P/N" "LM39100S-3.3"
 			(at 152.4 63.5 0)
 			(hide yes)
@@
 			)
 		)
-		(property "Old P/N" "BAT760-7"
-			(at 133.35 63.5 0)
-			(hide yes)
-			(show_name no)
-			(do_not_autoplace no)
-			(effects
-				(font
-					(size 1.27 1.27)
-				)
-			)
-		)
-		(property "Old LCSC P/N" "C124187"
-			(at 133.35 63.5 0)
-			(hide yes)
-			(show_name no)
-			(do_not_autoplace no)
-			(effects
-				(font
-					(size 1.27 1.27)
-				)
-			)
-		)
 		(pin "1"
 		)
@@
 			(at 139.7 69.85 0)
 			(hide yes)
-			(show_name no)
-			(do_not_autoplace no)
-			(effects
-				(font
-					(size 1.27 1.27)
-				)
-			)
-		)
-		(property "Mouser P/N" "GRM21BR61H106KE43K"
-			(at 139.7 69.85 0)
-			(hide yes)

Commit message: shoupu review done
Changed lines of the file:
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@@
 	(text "5V Nominal"
 		(exclude_from_sim no)
-		(at 127 66.675 0)
+		(at 127 67.31 0)
 		(effects
 			(font
@@
 	(text "Input Nominal: 5V\nDiode Forward Voltage: 500-600 mV\nLDO Dropout Voltage Max: 400 mV\n-> ~0.7V headroom on input"
 		(exclude_from_sim no)
-		(at 172.72 116.205 0)
+		(at 172.72 116.84 0)
 		(effects
 			(font
@@
 	(text "VR=regulated output voltage=3.3V"
 		(exclude_from_sim no)
-		(at 261.62 102.235 0)
+		(at 261.62 102.87 0)
 		(effects
 			(font
@@
 	(text "3.3V Nominal"
 		(exclude_from_sim no)
-		(at 173.355 60.96 0)
+		(at 173.99 60.96 0)
 		(effects
 			(font
