File: BPS_CAN.kicad_sch (KiCad schematic)
At the start: 9 parts, among them IC4 TCAN3413DR

Commit message: updated from review
Parts:
- removed C74: 10u, Capacitor_SMD:C_0805_2012Metric_Pad1.18x1.45mm_HandSolder, symbol Device:C
- removed C75, C76: 0.1u, Capacitor_SMD:C_0603_1608Metric_Pad1.08x0.95mm_HandSolder, symbol Device:C
- removed C77: 0.1u, Capacitor_SMD:C_0603_1608Metric_Pad1.08x0.95mm_HandSolder, symbol ECE319K:C
- removed D26: CDSOT23-T24CAN, LHRS_Passives:CDSOT23-T24CAN, symbol CDSOT23-T24CAN:CDSOT23-T24CAN
- removed IC4: TCAN3413DR, LHRS_Passives:TCAN3413DR, symbol TCAN3413DR:TCAN3413DR
- removed R68, R69: 60, Resistor_SMD:R_0603_1608Metric_Pad0.98x0.95mm_HandSolder, symbol Device:R
- added C21: 10u, Capacitor_SMD:C_0805_2012Metric_Pad1.18x1.45mm_HandSolder, symbol Device:C
- added C24, C25: 0.1u, Capacitor_SMD:C_0603_1608Metric_Pad1.08x0.95mm_HandSolder, symbol Device:C
- added C26: 0.1u, Capacitor_SMD:C_0603_1608Metric_Pad1.08x0.95mm_HandSolder, symbol ECE319K:C
- added D14: CDSOT23-T24CAN, LHRS_Passives:CDSOT23-T24CAN, symbol CDSOT23-T24CAN:CDSOT23-T24CAN
- added IC1: TCAN3413DR, LHRS_Passives:TCAN3413DR, symbol TCAN3413DR:TCAN3413DR
- added R23, R24: 60, Resistor_SMD:R_0603_1608Metric_Pad0.98x0.95mm_HandSolder, symbol Device:R
Connections:
- net CAN_H: now also D14.1 (CAN_H), IC1.7 (CANH), R23.1
- net CAN_L: now also D14.2 (CAN_L), IC1.6 (CANL)
- net CAN_RX: now also IC1.4 (RXD)
- net CAN_TX: now also IC1.1 (TXD)
- net GND: now also C21.2, C24.2, C25.2, C26.1, D14.3 (GND), IC1.2 (GND), IC1.8 (STB)
- net at JP1.1 (A): now also R24.2
- new net: C26.2, R23.2, R24.1
- new net 3V3: C21.1, C24.1, C25.1, IC1.3 (VCC), IC1.5 (SHDNV_IO)
