File: Power_Mux.kicad_sch (KiCad schematic)
At the start: 6 parts, among them U1 TPS2117DRLR

Commit message: test points? never heard of her
Parts:
- added R2: 16k, Package_DIP:DIP-8_W7.62mm, symbol Device:R
- added R3: 4.7k, symbol Device:R
Connections:
- net MX_GND: now also R3.2
- net PR1: now also R2.2, R3.1
- net VIN_1: now also R2.1
Other:
- note removed: "R1"
- note removed: "R2"
Changed lines of the file:
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@@
-	)
-	(rectangle
-		(start 30.48 58.42)
-		(end 33.02 63.5)
-		(stroke
-			(width 0)
-			(type default)
-		)
-		(fill
-			(type none)
-		)
-	)
-	(rectangle
-		(start 30.48 66.04)
-		(end 33.02 71.12)
-		(stroke
-			(width 0)
-			(type default)
-		)
-		(fill
-			(type none)
-		)
 	)
 	(rectangle
@@
 			(font
 				(size 2.54 2.54)
-			)
-		)
-	)
-	(text "R2"
-		(exclude_from_sim no)
-		(at 31.75 68.834 0)
-		(effects
-			(font
-				(size 1.27 1.27)
-			)
-		)
-	)
-	(text "R1"
-		(exclude_from_sim no)
-		(at 31.75 61.214 0)
-		(effects
-			(font
-				(size 1.27 1.27)
 			)
 		)
@@
 	)
 	(junction
+		(at 31.75 64.77)
+		(diameter 0)
+		(color 0 0 0 0)
+	)
+	(junction
 		(at 88.9 54.61)
 		(diameter 0)
@@
 	)
 	(junction
+		(at 31.75 72.39)
+		(diameter 0)
+		(color 0 0 0 0)
+	)
+	(junction
 		(at 31.75 57.15)
 		(diameter 0)
@@
 	(wire
 		(pts
-			(xy 30.48 64.77) (xy 39.37 64.77)
+			(xy 30.48 64.77) (xy 31.75 64.77)
 		)
 		(stroke
@@
 	(wire
 		(pts
+			(xy 31.75 64.77) (xy 39.37 64.77)
+		)
+		(stroke
+			(width 0)
+			(type default)
+		)
+	)
+	(wire
+		(pts
 			(xy 80.01 54.61) (xy 88.9 54.61)
 		)
@@
 	(wire
 		(pts
+			(xy 31.75 72.39) (xy 39.37 72.39)
+		)
+		(stroke
+			(width 0)
+			(type default)
+		)
+	)
+	(wire
+		(pts
 			(xy 31.75 57.15) (xy 39.37 57.15)
 		)
@@
 	(wire
 		(pts
-			(xy 30.48 72.39) (xy 39.37 72.39)
+			(xy 30.48 72.39) (xy 31.75 72.39)
 		)
 		(stroke
@@
 		)
 		(instances
+			(project "atempt_2"
+				(path "/86244622-fc6f-4400-a6c8-ba7d84e5ad42/81e1c9b9-1f16-4620-9331-536fea3807a2"
+					(reference "C4")
+					(unit 1)
+				)
+			)
 			(project "PS-ChargerInterfacePCB"
 				(path "/894adbd2-6316-426a-afb4-88808e8ec51a/81e1c9b9-1f16-4620-9331-536fea3807a2"
@@
 				(path "/c8207045-8aef-4538-bcc4-1e380c549c2c"
 					(reference "C4")
+					(unit 1)
+				)
+			)
+		)
+	)
+	(symbol
+		(lib_id "Device:R")
+		(at 31.75 60.96 0)
+		(unit 1)
+		(body_style 1)
+		(exclude_from_sim no)
+		(in_bom yes)
+		(on_board yes)
+		(in_pos_files yes)
+		(dnp no)
+		(property "Reference" "R2"
+			(at 33.02 59.69 0)
+			(show_name no)
+			(do_not_autoplace no)
+			(effects
+				(font
+					(size 1.27 1.27)
+				)
+				(justify left)
+			)
+		)
+		(property "Value" "16k"
+			(at 33.02 62.23 0)
+			(show_name no)
+			(do_not_autoplace no)
+			(effects
+				(font
+					(size 1.27 1.27)
+				)
+				(justify left)
+			)
+		)
+		(property "Footprint" "Package_DIP:DIP-8_W7.62mm"
+			(at 29.972 60.96 90)
+			(hide yes)
+			(show_name no)
+			(do_not_autoplace no)
+			(effects
+				(font
+					(size 1.27 1.27)
+				)
+			)
+		)
+		(property "Datasheet" ""
+			(at 31.75 60.96 0)
+			(hide yes)
+			(show_name no)
+			(do_not_autoplace no)
+			(effects
+				(font
+					(size 1.27 1.27)
+				)
+			)
+		)
+		(property "Description" "Resistor"
+			(at 31.75 60.96 0)
+			(hide yes)
+			(show_name no)
+			(do_not_autoplace no)
+			(effects
+				(font
+					(size 1.27 1.27)
+				)
+			)
+		)
+		(pin "1"
+		)
+		(pin "2"
+		)
+		(instances
+			(project "PS-ChargerInterfacePCB"
+				(path "/894adbd2-6316-426a-afb4-88808e8ec51a/81e1c9b9-1f16-4620-9331-536fea3807a2"
+					(reference "R2")
 					(unit 1)
 				)
@@
 		)
 		(instances
+			(project "atempt_2"
+				(path "/86244622-fc6f-4400-a6c8-ba7d84e5ad42/81e1c9b9-1f16-4620-9331-536fea3807a2"
+					(reference "R1")
+					(unit 1)
+				)
+			)
 			(project "PS-ChargerInterfacePCB"
 				(path "/894adbd2-6316-426a-afb4-88808e8ec51a/81e1c9b9-1f16-4620-9331-536fea3807a2"
@@
 		)
 		(instances
+			(project "atempt_2"
+				(path "/86244622-fc6f-4400-a6c8-ba7d84e5ad42/81e1c9b9-1f16-4620-9331-536fea3807a2"
+					(reference "C1")
+					(unit 1)
+				)
+			)
 			(project "PS-ChargerInterfacePCB"
 				(path "/894adbd2-6316-426a-afb4-88808e8ec51a/81e1c9b9-1f16-4620-9331-536fea3807a2"
@@
 				(path "/c8207045-8aef-4538-bcc4-1e380c549c2c"
 					(reference "C1")
+					(unit 1)
+				)
+			)
+		)
+	)
+	(symbol
+		(lib_id "Device:R")
+		(at 31.75 68.58 0)
+		(unit 1)
+		(body_style 1)
+		(exclude_from_sim no)
+		(in_bom yes)
+		(on_board yes)
+		(in_pos_files yes)
+		(dnp no)
+		(property "Reference" "R3"
+			(at 33.02 67.31 0)
+			(show_name no)
+			(do_not_autoplace no)
+			(effects
+				(font
+					(size 1.27 1.27)
+				)
+				(justify left)
+			)
+		)
+		(property "Value" "4.7k"
+			(at 33.02 69.85 0)
+			(show_name no)
+			(do_not_autoplace no)
+			(effects
+				(font
+					(size 1.27 1.27)
+				)
+				(justify left)
+			)
+		)
+		(property "Footprint" ""
+			(at 29.972 68.58 90)
+			(hide yes)
+			(show_name no)
+			(do_not_autoplace no)
+			(effects
+				(font
+					(size 1.27 1.27)
+				)
+			)
+		)
+		(property "Datasheet" ""
+			(at 31.75 68.58 0)
+			(hide yes)
+			(show_name no)
+			(do_not_autoplace no)
+			(effects
+				(font
+					(size 1.27 1.27)
+				)
+			)
+		)
+		(property "Description" "Resistor"
+			(at 31.75 68.58 0)
+			(hide yes)
+			(show_name no)
+			(do_not_autoplace no)
+			(effects
+				(font
+					(size 1.27 1.27)
+				)
+			)
+		)
+		(pin "2"
+		)
+		(pin "1"
+		)
+		(instances
+			(project "PS-ChargerInterfacePCB"
+				(path "/894adbd2-6316-426a-afb4-88808e8ec51a/81e1c9b9-1f16-4620-9331-536fea3807a2"
+					(reference "R3")
 					(unit 1)
 				)
@@
 		)
 		(instances
+			(project "atempt_2"
+				(path "/86244622-fc6f-4400-a6c8-ba7d84e5ad42/81e1c9b9-1f16-4620-9331-536fea3807a2"
+					(reference "U1")
+					(unit 1)
+				)
+			)
 			(project "PS-ChargerInterfacePCB"
 				(path "/894adbd2-6316-426a-afb4-88808e8ec51a/81e1c9b9-1f16-4620-9331-536fea3807a2"
@@
 		)
 		(instances
+			(project "atempt_2"
+				(path "/86244622-fc6f-4400-a6c8-ba7d84e5ad42/81e1c9b9-1f16-4620-9331-536fea3807a2"
+					(reference "C3")
+					(unit 1)
+				)
+			)
 			(project "PS-ChargerInterfacePCB"
 				(path "/894adbd2-6316-426a-afb4-88808e8ec51a/81e1c9b9-1f16-4620-9331-536fea3807a2"
@@
 		)
 		(instances
+			(project "atempt_2"
+				(path "/86244622-fc6f-4400-a6c8-ba7d84e5ad42/81e1c9b9-1f16-4620-9331-536fea3807a2"
+					(reference "C2")
+					(unit 1)
+				)
+			)
 			(project "PS-ChargerInterfacePCB"
 				(path "/894adbd2-6316-426a-afb4-88808e8ec51a/81e1c9b9-1f16-4620-9331-536fea3807a2"

Commit message: i will fix the stupid pins on the mcu schem later
Parts:
- removed R2: 16k, Package_DIP:DIP-8_W7.62mm, symbol Device:R
- removed R3: 4.7k, symbol Device:R
Other:
- note added: "R1"
- note added: "R2"
- moved on the sheet: C1, C2, C3, C4, R1, U1

Commit message: updated from review
Parts:
- C1, C2, C3, C4: value 0.1uF -> 0.1u; Mfg MLASH168SB7104KTNA01 -> (none)
- U3: renamed from U1; MANUFACTURER Texas Instruments -> (none); MAXIMUM_PACKAGE_HEIGHT 0.6mm -> (none); PARTREV A -> (none); STANDARD IPC-7351B -> (none)
Other:
- moved on the sheet: C1, C2, C3, C4, R1, U3
