File: LEDS.kicad_sch (KiCad schematic)
At the start: 20 parts, among them Q15 IRLML0030TRPBF, Q16 IRLML0030TRPBF, Q17 IRLML0030TRPBF, Q18 IRLML0030TRPBF

Commit message: implemented some of new comments
Parts:
- renumbered D18 to D16, D19 to D17, D23 to D18, D20 to D19, D21 to D20, Q15 to Q2, Q16 to Q5, Q17 to Q6, Q18 to Q7, R46 to R36, R47 to R39, R48 to R40, R49 to R41, R50 to R42, R56 to R43, R51 to R44, R52 to R45, R42 to R46, R43 to R47, R44 to R48
Changed lines of the file:
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@@
 		(in_pos_files yes)
 		(dnp no)
-		(property "Reference" "Q17"
+		(property "Reference" "Q6"
 			(at 108.966 28.194 0)
 			(show_name no)
@@
 			)
 			(project "PS-ChargerInterfacePCB"
-				(path "/894adbd2-6316-426a-afb4-88808e8ec51a/f531d34f-a843-4846-a55a-2a1a0e6cd2bb"
-					(reference "Q17")
+				(path "/894adbd2-6316-426a-afb4-88808e8ec51a/bee5c61a-f058-4607-9a84-1edb0b41c252"
+					(reference "Q6")
 					(unit 1)
 				)
@@
 		(dnp no)
 		(fields_autoplaced yes)
-		(property "Reference" "D21"
+		(property "Reference" "D20"
 			(at 158.75 17.78 0)
 			(show_name no)
@@
 		(instances
 			(project "PS-ChargerInterfacePCB"
-				(path "/894adbd2-6316-426a-afb4-88808e8ec51a/f531d34f-a843-4846-a55a-2a1a0e6cd2bb"
-					(reference "D21")
+				(path "/894adbd2-6316-426a-afb4-88808e8ec51a/bee5c61a-f058-4607-9a84-1edb0b41c252"
+					(reference "D20")
 					(unit 1)
 				)
@@
 		(in_pos_files yes)
 		(dnp no)
-		(property "Reference" "Q15"
+		(property "Reference" "Q2"
 			(at 61.722 25.146 0)
 			(show_name no)
@@
 			)
 			(project "PS-ChargerInterfacePCB"
-				(path "/894adbd2-6316-426a-afb4-88808e8ec51a/f531d34f-a843-4846-a55a-2a1a0e6cd2bb"
-					(reference "Q15")
+				(path "/894adbd2-6316-426a-afb4-88808e8ec51a/bee5c61a-f058-4607-9a84-1edb0b41c252"
+					(reference "Q2")
 					(unit 1)
 				)
@@
 		(in_pos_files yes)
 		(dnp no)
-		(property "Reference" "R44"
+		(property "Reference" "R48"
 			(at 166.624 33.782 90)
 			(show_name no)
@@
 		(instances
 			(project "PS-ChargerInterfacePCB"
-				(path "/894adbd2-6316-426a-afb4-88808e8ec51a/f531d34f-a843-4846-a55a-2a1a0e6cd2bb"
-					(reference "R44")
+				(path "/894adbd2-6316-426a-afb4-88808e8ec51a/bee5c61a-f058-4607-9a84-1edb0b41c252"
+					(reference "R48")
 					(unit 1)
 				)
@@
 		(in_pos_files yes)
 		(dnp no)
-		(property "Reference" "R47"
+		(property "Reference" "R39"
 			(at 40.132 36.068 0)
 			(show_name no)
@@
 			)
 			(project "PS-ChargerInterfacePCB"
-				(path "/894adbd2-6316-426a-afb4-88808e8ec51a/f531d34f-a843-4846-a55a-2a1a0e6cd2bb"
-					(reference "R47")
+				(path "/894adbd2-6316-426a-afb4-88808e8ec51a/bee5c61a-f058-4607-9a84-1edb0b41c252"
+					(reference "R39")
 					(unit 1)
 				)
@@
 		(dnp no)
 		(fields_autoplaced yes)
-		(property "Reference" "R50"
+		(property "Reference" "R42"
 			(at 83.82 35.5599 0)
 			(show_name no)
@@
 			)
 			(project "PS-ChargerInterfacePCB"
-				(path "/894adbd2-6316-426a-afb4-88808e8ec51a/f531d34f-a843-4846-a55a-2a1a0e6cd2bb"
-					(reference "R50")
+				(path "/894adbd2-6316-426a-afb4-88808e8ec51a/bee5c61a-f058-4607-9a84-1edb0b41c252"
+					(reference "R42")
 					(unit 1)
 				)
@@
 		(in_pos_files yes)
 		(dnp no)
-		(property "Reference" "D19"
+		(property "Reference" "D17"
 			(at 53.086 69.088 90)
 			(show_name no)
@@
 			)
 			(project "PS-ChargerInterfacePCB"
-				(path "/894adbd2-6316-426a-afb4-88808e8ec51a/f531d34f-a843-4846-a55a-2a1a0e6cd2bb"
-					(reference "D19")
+				(path "/894adbd2-6316-426a-afb4-88808e8ec51a/bee5c61a-f058-4607-9a84-1edb0b41c252"
+					(reference "D17")
 					(unit 1)
 				)
@@
 		(in_pos_files yes)
 		(dnp no)
-		(property "Reference" "D18"
+		(property "Reference" "D16"
 			(at 40.386 44.958 90)
 			(show_name no)
@@
 			)
 			(project "PS-ChargerInterfacePCB"
-				(path "/894adbd2-6316-426a-afb4-88808e8ec51a/f531d34f-a843-4846-a55a-2a1a0e6cd2bb"
-					(reference "D18")
+				(path "/894adbd2-6316-426a-afb4-88808e8ec51a/bee5c61a-f058-4607-9a84-1edb0b41c252"
+					(reference "D16")
 					(unit 1)
 				)
@@
 		(dnp no)
 		(fields_autoplaced yes)
-		(property "Reference" "R48"
+		(property "Reference" "R40"
 			(at 43.18 62.2299 0)
 			(show_name no)
@@
 			)
 			(project "PS-ChargerInterfacePCB"
-				(path "/894adbd2-6316-426a-afb4-88808e8ec51a/f531d34f-a843-4846-a55a-2a1a0e6cd2bb"
-					(reference "R48")
+				(path "/894adbd2-6316-426a-afb4-88808e8ec51a/bee5c61a-f058-4607-9a84-1edb0b41c252"
+					(reference "R40")
 					(unit 1)
 				)
@@
 		(in_pos_files yes)
 		(dnp no)
-		(property "Reference" "R49"
+		(property "Reference" "R41"
 			(at 52.832 60.198 0)
 			(show_name no)
@@
 			)
 			(project "PS-ChargerInterfacePCB"
-				(path "/894adbd2-6316-426a-afb4-88808e8ec51a/f531d34f-a843-4846-a55a-2a1a0e6cd2bb"
-					(reference "R49")
+				(path "/894adbd2-6316-426a-afb4-88808e8ec51a/bee5c61a-f058-4607-9a84-1edb0b41c252"
+					(reference "R41")
 					(unit 1)
 				)
@@
 		(dnp no)
 		(fields_autoplaced yes)
-		(property "Reference" "R51"
+		(property "Reference" "R44"
 			(at 107.95 60.9599 0)
 			(show_name no)
@@
 			)
 			(project "PS-ChargerInterfacePCB"
-				(path "/894adbd2-6316-426a-afb4-88808e8ec51a/f531d34f-a843-4846-a55a-2a1a0e6cd2bb"
-					(reference "R51")
+				(path "/894adbd2-6316-426a-afb4-88808e8ec51a/bee5c61a-f058-4607-9a84-1edb0b41c252"
+					(reference "R44")
 					(unit 1)
 				)
@@
 		(dnp no)
 		(fields_autoplaced yes)
-		(property "Reference" "R46"
+		(property "Reference" "R36"
 			(at 29.21 35.5599 0)
 			(show_name no)
@@
 			)
 			(project "PS-ChargerInterfacePCB"
-				(path "/894adbd2-6316-426a-afb4-88808e8ec51a/f531d34f-a843-4846-a55a-2a1a0e6cd2bb"
-					(reference "R46")
+				(path "/894adbd2-6316-426a-afb4-88808e8ec51a/bee5c61a-f058-4607-9a84-1edb0b41c252"
+					(reference "R36")
 					(unit 1)
 				)
@@
 		(in_pos_files yes)
 		(dnp no)
-		(property "Reference" "R43"
+		(property "Reference" "R47"
 			(at 166.624 28.448 90)
 			(show_name no)
@@
 		(instances
 			(project "PS-ChargerInterfacePCB"
-				(path "/894adbd2-6316-426a-afb4-88808e8ec51a/f531d34f-a843-4846-a55a-2a1a0e6cd2bb"
-					(reference "R43")
+				(path "/894adbd2-6316-426a-afb4-88808e8ec51a/bee5c61a-f058-4607-9a84-1edb0b41c252"
+					(reference "R47")
 					(unit 1)
 				)
@@
 		(in_pos_files yes)
 		(dnp no)
-		(property "Reference" "Q16"
+		(property "Reference" "Q5"
 			(at 67.056 53.086 0)
 			(show_name no)
@@
 			)
 			(project "PS-ChargerInterfacePCB"
-				(path "/894adbd2-6316-426a-afb4-88808e8ec51a/f531d34f-a843-4846-a55a-2a1a0e6cd2bb"
-					(reference "Q16")
+				(path "/894adbd2-6316-426a-afb4-88808e8ec51a/bee5c61a-f058-4607-9a84-1edb0b41c252"
+					(reference "Q5")
 					(unit 1)
 				)
@@
 		(in_pos_files yes)
 		(dnp no)
-		(property "Reference" "R42"
+		(property "Reference" "R46"
 			(at 166.624 23.368 90)
 			(show_name no)
@@
 		(instances
 			(project "PS-ChargerInterfacePCB"
-				(path "/894adbd2-6316-426a-afb4-88808e8ec51a/f531d34f-a843-4846-a55a-2a1a0e6cd2bb"
-					(reference "R42")
+				(path "/894adbd2-6316-426a-afb4-88808e8ec51a/bee5c61a-f058-4607-9a84-1edb0b41c252"
+					(reference "R46")
 					(unit 1)
 				)
@@
 		(in_pos_files yes)
 		(dnp no)
-		(property "Reference" "R52"
+		(property "Reference" "R45"
 			(at 117.602 60.198 0)
 			(show_name no)
@@
 			)
 			(project "PS-ChargerInterfacePCB"
-				(path "/894adbd2-6316-426a-afb4-88808e8ec51a/f531d34f-a843-4846-a55a-2a1a0e6cd2bb"
-					(reference "R52")
+				(path "/894adbd2-6316-426a-afb4-88808e8ec51a/bee5c61a-f058-4607-9a84-1edb0b41c252"
+					(reference "R45")
 					(unit 1)
 				)
@@
 		(in_pos_files yes)
 		(dnp no)
-		(property "Reference" "D20"
+		(property "Reference" "D19"
 			(at 117.856 69.088 90)
 			(show_name no)
@@
 			)
 			(project "PS-ChargerInterfacePCB"
-				(path "/894adbd2-6316-426a-afb4-88808e8ec51a/f531d34f-a843-4846-a55a-2a1a0e6cd2bb"
-					(reference "D20")
+				(path "/894adbd2-6316-426a-afb4-88808e8ec51a/bee5c61a-f058-4607-9a84-1edb0b41c252"
+					(reference "D19")
 					(unit 1)
 				)
@@
 		(in_pos_files yes)
 		(dnp no)
-		(property "Reference" "R56"
+		(property "Reference" "R43"
 			(at 93.472 36.068 0)
 			(show_name no)
@@
 			)
 			(project "PS-ChargerInterfacePCB"
-				(path "/894adbd2-6316-426a-afb4-88808e8ec51a/f531d34f-a843-4846-a55a-2a1a0e6cd2bb"
-					(reference "R56")
+				(path "/894adbd2-6316-426a-afb4-88808e8ec51a/bee5c61a-f058-4607-9a84-1edb0b41c252"
+					(reference "R43")
 					(unit 1)
 				)
@@
 		(in_pos_files yes)
 		(dnp no)
-		(property "Reference" "Q18"
+		(property "Reference" "Q7"
 			(at 134.366 54.102 0)
 			(show_name no)
@@
 			)
 			(project "PS-ChargerInterfacePCB"
-				(path "/894adbd2-6316-426a-afb4-88808e8ec51a/f531d34f-a843-4846-a55a-2a1a0e6cd2bb"
-					(reference "Q18")
+				(path "/894adbd2-6316-426a-afb4-88808e8ec51a/bee5c61a-f058-4607-9a84-1edb0b41c252"
+					(reference "Q7")
 					(unit 1)
 				)
@@
 		(in_pos_files yes)
 		(dnp no)
-		(property "Reference" "D23"
+		(property "Reference" "D18"
 			(at 93.726 44.958 90)
 			(show_name no)
@@
 			)
 			(project "PS-ChargerInterfacePCB"
-				(path "/894adbd2-6316-426a-afb4-88808e8ec51a/f531d34f-a843-4846-a55a-2a1a0e6cd2bb"
-					(reference "D23")
-					(unit 1)
-				)
+				(path "/894adbd2-6316-426a-afb4-88808e8ec51a/bee5c61a-f058-4607-9a84-1edb0b41c252"
+					(reference "D18")
+					(unit 1)
+				)

Commit message: final schem is done
Parts:
- removed D20: LED_RGBA, LED_SMD:LED_Cree-XHP50_3V_HighDensity, symbol Device:LED_RGBA
- removed R46, R47: 100, symbol Device:R
- removed R48: 330, symbol Device:R
- added D20, D21, D23: LED, LED_SMD:LED_0603_1608Metric, symbol Device:LED
- added Q10, Q8, Q9: IRLML0030TRPBF, charger_parts:IRLML0030TRPBF, symbol IRLML0030TRPBF:IRLML0030TRPBF
- added R46, R48, R50: 100k, Resistor_SMD:R_0603_1608Metric, symbol Device:R_US
- added R47, R49: 30, Resistor_SMD:R_0603_1608Metric, symbol Device:R_US
- added R51: 150, Resistor_SMD:R_0603_1608Metric, symbol Device:R_US
- Q2, Q5, Q6, Q7: Height 1.12 -> (none); Manufacturer_Name Infineon -> (none); Manufacturer_Part_Number IRLML0030TRPBF -> (none); Mouser Part Number 942-IRLML0030TRPBF -> (none); Mouser Price/Stock https://www.mouser.co.uk/ProductDetail/Infineon-Technologie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 -> (none)
Connections:
- net ANODE_IN: now also Q10.3 (D), Q8.3 (D), Q9.3 (D)
- net GND: now also D20.1 (K), D21.1 (K), D23.1 (K), Q10.2 (S), Q8.2 (S), Q9.2 (S), R46.2, R48.2, R50.2
- net MCU_B: now also Q8.1 (G), R46.1, R47.1
- net MCU_G: now also Q9.1 (G), R48.1, R49.1
- net MCU_R: now also Q10.1 (G), R50.1, R51.1
- new net: D21.2 (A), R49.2
- new net: D20.2 (A), R47.2
- new net: D23.2 (A), R51.2
Other:
- note added: "External Leds"
- note added: "LEDS"

Commit message: shoupu review done
Changed lines of the file:
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@@
 	(text "LEDS"
 		(exclude_from_sim no)
-		(at 18.288 17.018 0)
+		(at 17.78 16.51 0)
 		(effects
 			(font
@@
 	(text "External Leds"
 		(exclude_from_sim no)
-		(at 23.368 95.25 0)
+		(at 22.86 95.25 0)
 		(effects
 			(font
@@
 	(wire
 		(pts
-			(xy 128.27 43.18) (xy 130.048 41.91)
+			(xy 128.27 43.18) (xy 129.54 41.91)
 		)
 		(stroke
@@
 	(hierarchical_label "CHARGE-"
 		(shape input)
-		(at 130.048 41.91 0)
-		(effects
-			(font
+		(at 129.54 41.91 0)
+		(effects
+			(font

Commit message: minor changes from comments
Other:
- note added: "RGB LED"
- note removed: "External Leds"
- moved on the sheet: D17, D18, D19, D20, D21, D23, Q10, Q5, Q6, Q7, Q8, Q9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
