File: PS-ChargerInterfacePCB.kicad_pcb (KiCad board)
At the start: 2 copper layers, 183 parts, among them IC1 TCAN3413DR, IC2 LM74502DDFR, IC3 TCAN3413DR, J10 ESTOP, J11 SHUTDOWN, J12 SWD, J13 LEDS, J14 Conn_01x08, J15 Buzzer, J2 ELCON_CAN, J3 CHARGER_CAN, J5 EVSE, J7 SPI_DEBUG, J8 SWD_Header, J9 BUZ_PWM, Q1 IRLML0030TRPBF, Q10 IRLML0030TRPBF, Q2 IRLML0030TRPBF, Q3 PSMN012-100YS, Q4 PSMN012-100YS, Q5 IRLML0030TRPBF, Q6 IRLML0030TRPBF, Q7 IRLML0030TRPBF, Q8 IRLML0030TRPBF, Q9 IRLML0030TRPBF, SW1 Reset, SW2 SW_SPDT, U1 LMR51635XDDCR, U2 STM32G473CETx, U3 TPS2117DRLR, U5 MCP1826S, Y1 Crystal

Commit message: nothing of importance
Parts:
- moved U3 107.2 mm to (247.6, 96.6)
- moved C1 107.2 mm to (243.1, 96.0)
- moved C3 107.2 mm to (243.1, 101.0)
- moved C4 107.2 mm to (243.1, 103.5)
- moved C2 107.2 mm to (243.1, 98.5)
- moved R1 107.2 mm to (243.1, 106.0)
- moved C20 95.9 mm to (223.5, 136.7)
- moved D10 95.9 mm to (218.9, 139.2)
- moved D9 95.9 mm to (224.0, 133.5)
- moved R21 95.9 mm to (218.9, 133.1)
- moved R22 95.9 mm to (218.9, 135.6)
- moved C39 84.4 mm to (223.2, 102.3)
- moved C40 84.4 mm to (227.0, 94.5)
- moved C41 84.4 mm to (222.8, 94.5)
- moved C42 84.4 mm to (217.8, 95.3)
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Changed lines of the file:
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@@
 	(footprint "Resistor_SMD:R_0603_1608Metric"
 		(layer "F.Cu")
-		(at 142.685 72.995)
+		(at 222.825 99.5)
 		(descr "Resistor SMD 0603 (1608 Metric), square (rectangular) end terminal, IPC-7351 nominal, (Body size source: IPC-SM-782 page 72, https://www.pcb-3d.com/wordpress/wp-content/uploads/ipc-sm-782a_amendment_1_and_2.pdf)")
 		(tags "resistor")
@@
 	(footprint "Resistor_SMD:R_0603_1608Metric_Pad0.98x0.95mm_HandSolder"
 		(layer "F.Cu")
-		(at 137.865 126.425)
+		(at 243.1375 106.04)
 		(descr "Resistor SMD 0603 (1608 Metric), square (rectangular) end terminal, IPC-7351 nominal with elongated pad for handsoldering. (Body size source: IPC-SM-782 page 72, https://www.pcb-3d.com/wordpress/wp-content/uploads/ipc-sm-782a_amendment_1_and_2.pdf)")
 		(tags "resistor handsolder")
@@
 	(footprint "Capacitor_SMD:C_0805_2012Metric_Pad1.18x1.45mm_HandSolder"
 		(layer "F.Cu")
-		(at 143.085 78.765)
+		(at 223.225 105.27)
 		(descr "Capacitor SMD 0805 (2012 Metric), square (rectangular) end terminal, IPC-7351 nominal with elongated pad for handsoldering. (Body size source: IPC-SM-782 page 76, https://www.pcb-3d.com/wordpress/wp-content/uploads/ipc-sm-782a_amendment_1_and_2.pdf, https://docs.google.com/spreadsheets/d/1BsfQQcO9C6DZCsRaXUlFlo91Tg2WpOkGARC1WS5S8t0/edit?usp=sharing)")
 		(tags "capacitor handsolder")
@@
 	(footprint "Capacitor_SMD:C_0603_1608Metric_Pad1.08x0.95mm_HandSolder"
 		(layer "F.Cu")
-		(at 137.865 123.915)
+		(at 243.1375 103.53)
 		(descr "Capacitor SMD 0603 (1608 Metric), square (rectangular) end terminal, IPC-7351 nominal with elongated pad for handsoldering. (Body size source: IPC-SM-782 page 76, https://www.pcb-3d.com/wordpress/wp-content/uploads/ipc-sm-782a_amendment_1_and_2.pdf)")
 		(tags "capacitor handsolder")
@@
 	(footprint "Resistor_SMD:R_0603_1608Metric"
 		(layer "F.Cu")
-		(at 142.685 70.485)
+		(at 222.825 96.99)
 		(descr "Resistor SMD 0603 (1608 Metric), square (rectangular) end terminal, IPC-7351 nominal, (Body size source: IPC-SM-782 page 72, https://www.pcb-3d.com/wordpress/wp-content/uploads/ipc-sm-782a_amendment_1_and_2.pdf)")
 		(tags "resistor")
@@
 	(footprint "Capacitor_SMD:C_1210_3225Metric_Pad1.33x2.70mm_HandSolder"
 		(layer "F.Cu")
-		(at 137.675 73.095)
+		(at 217.815 99.6)
 		(descr "Capacitor SMD 1210 (3225 Metric), square (rectangular) end terminal, IPC-7351 nominal with elongated pad for handsoldering. (Body size source: IPC-SM-782 page 76, https://www.pcb-3d.com/wordpress/wp-content/uploads/ipc-sm-782a_amendment_1_and_2.pdf)")
 		(tags "capacitor handsolder")
@@
 	(footprint "Capacitor_SMD:C_0603_1608Metric_Pad1.08x0.95mm_HandSolder"
 		(layer "F.Cu")
-		(at 137.865 121.405)
+		(at 243.1375 101.02)
 		(descr "Capacitor SMD 0603 (1608 Metric), square (rectangular) end terminal, IPC-7351 nominal with elongated pad for handsoldering. (Body size source: IPC-SM-782 page 76, https://www.pcb-3d.com/wordpress/wp-content/uploads/ipc-sm-782a_amendment_1_and_2.pdf)")
 		(tags "capacitor handsolder")
@@
 	(footprint "Capacitor_SMD:C_0603_1608Metric"
 		(layer "F.Cu")
-		(at 142.685 67.975)
+		(at 222.825 94.48)
 		(descr "Capacitor SMD 0603 (1608 Metric), square (rectangular) end terminal, IPC-7351 nominal, (Body size source: IPC-SM-782 page 76, https://www.pcb-3d.com/wordpress/wp-content/uploads/ipc-sm-782a_amendment_1_and_2.pdf)")
 		(tags "capacitor")
@@
 	(footprint "LHRS_ICs:DDC0006A-MFG"
 		(layer "F.Cu")
-		(at 137.870001 77.320001)
+		(at 218.010001 103.825001)
 		(tags "LMR51635XDDCR ")
 		(property "Reference" "U1"
@@
 	(footprint "Resistor_SMD:R_0603_1608Metric_Pad0.98x0.95mm_HandSolder"
 		(layer "F.Cu")
-		(at 136.845 83.525)
+		(at 218.905 133.08)
 		(descr "Resistor SMD 0603 (1608 Metric), square (rectangular) end terminal, IPC-7351 nominal with elongated pad for handsoldering. (Body size source: IPC-SM-782 page 72, https://www.pcb-3d.com/wordpress/wp-content/uploads/ipc-sm-782a_amendment_1_and_2.pdf)")
 		(tags "resistor handsolder")
@@
 	(footprint "Capacitor_SMD:C_0603_1608Metric_Pad1.08x0.95mm_HandSolder"
 		(layer "F.Cu")
-		(at 137.865 118.895)
+		(at 243.1375 98.51)
 		(descr "Capacitor SMD 0603 (1608 Metric), square (rectangular) end terminal, IPC-7351 nominal with elongated pad for handsoldering. (Body size source: IPC-SM-782 page 76, https://www.pcb-3d.com/wordpress/wp-content/uploads/ipc-sm-782a_amendment_1_and_2.pdf)")
 		(tags "capacitor handsolder")
@@
 	(footprint "Resistor_SMD:R_0603_1608Metric_Pad0.98x0.95mm_HandSolder"
 		(layer "F.Cu")
-		(at 136.845 86.035)
+		(at 218.905 135.59)
 		(descr "Resistor SMD 0603 (1608 Metric), square (rectangular) end terminal, IPC-7351 nominal with elongated pad for handsoldering. (Body size source: IPC-SM-782 page 72, https://www.pcb-3d.com/wordpress/wp-content/uploads/ipc-sm-782a_amendment_1_and_2.pdf)")
 		(tags "resistor handsolder")
@@
 	(footprint "Capacitor_SMD:C_0805_2012Metric_Pad1.18x1.45mm_HandSolder"
 		(layer "F.Cu")
-		(at 141.425 87.125)
+		(at 223.485 136.68)
 		(descr "Capacitor SMD 0805 (2012 Metric), square (rectangular) end terminal, IPC-7351 nominal with elongated pad for handsoldering. (Body size source: IPC-SM-782 page 76, https://www.pcb-3d.com/wordpress/wp-content/uploads/ipc-sm-782a_amendment_1_and_2.pdf, https://docs.google.com/spreadsheets/d/1BsfQQcO9C6DZCsRaXUlFlo91Tg2WpOkGARC1WS5S8t0/edit?usp=sharing)")
 		(tags "capacitor handsolder")
@@
 	(footprint "Package_TO_SOT_SMD:SOT-143"
 		(layer "F.Cu")
-		(at 136.795 89.69)
+		(at 218.855 139.245)
 		(descr "SOT-143 https://www.nxp.com/docs/en/package-information/SOT143B.pdf")
 		(tags "SOT-143")
@@
 	(footprint "Capacitor_SMD:C_1210_3225Metric_Pad1.33x2.70mm_HandSolder"
 		(layer "F.Cu")
-		(at 137.675 68.845)
+		(at 217.815 95.35)
 		(descr "Capacitor SMD 1210 (3225 Metric), square (rectangular) end terminal, IPC-7351 nominal with elongated pad for handsoldering. (Body size source: IPC-SM-782 page 76, https://www.pcb-3d.com/wordpress/wp-content/uploads/ipc-sm-782a_amendment_1_and_2.pdf)")
 		(tags "capacitor handsolder")
@@
 	(footprint "Capacitor_SMD:C_0603_1608Metric_Pad1.08x0.95mm_HandSolder"
 		(layer "F.Cu")
-		(at 137.865 116.385)
+		(at 243.1375 96)
 		(descr "Capacitor SMD 0603 (1608 Metric), square (rectangular) end terminal, IPC-7351 nominal with elongated pad for handsoldering. (Body size source: IPC-SM-782 page 76, https://www.pcb-3d.com/wordpress/wp-content/uploads/ipc-sm-782a_amendment_1_and_2.pdf)")
 		(tags "capacitor handsolder")
@@
 	(footprint "LHRS_Power:TPS2117DRLR"
 		(layer "F.Cu")
-		(at 142.34 116.955)
+		(at 247.6125 96.57)
 		(property "Reference" "U3"
 			(at 0.782 -1.9064 0)
@@
 	(footprint "Capacitor_SMD:C_0603_1608Metric_Pad1.08x0.95mm_HandSolder"
 		(layer "F.Cu")
-		(at 146.865 67.975)
+		(at 227.005 94.48)
 		(descr "Capacitor SMD 0603 (1608 Metric), square (rectangular) end terminal, IPC-7351 nominal with elongated pad for handsoldering. (Body size source: IPC-SM-782 page 76, https://www.pcb-3d.com/wordpress/wp-content/uploads/ipc-sm-782a_amendment_1_and_2.pdf)")
 		(tags "capacitor handsolder")
@@
 	(footprint "Capacitor_SMD:C_0805_2012Metric_Pad1.18x1.45mm_HandSolder"
 		(layer "F.Cu")
-		(at 143.085 75.755)
+		(at 223.225 102.26)
 		(descr "Capacitor SMD 0805 (2012 Metric), square (rectangular) end terminal, IPC-7351 nominal with elongated pad for handsoldering. (Body size source: IPC-SM-782 page 76, https://www.pcb-3d.com/wordpress/wp-content/uploads/ipc-sm-782a_amendment_1_and_2.pdf, https://docs.google.com/spreadsheets/d/1BsfQQcO9C6DZCsRaXUlFlo91Tg2WpOkGARC1WS5S8t0/edit?usp=sharing)")
 		(tags "capacitor handsolder")
@@
 	(footprint "Diode_SMD:D_SOD-123"
 		(layer "F.Cu")
-		(at 141.94 83.945)
+		(at 224 133.5)
 		(descr "SOD-123")
 		(tags "SOD-123")

Commit message: review council
Parts:
- moved U5 130.4 mm to (253.5, 103.0)
- moved C51 126.0 mm to (245.0, 99.9)
- moved C52 125.6 mm to (245.1, 105.3)
- moved D13 120.5 mm to (245.0, 102.8), turned to 180 degrees
- moved TP_3.3V2 116.6 mm to (247.8, 111.4)
- moved J2 79.7 mm to (167.6, 64.1)
- moved R9 79.7 mm to (189.3, 63.6)
- moved C20 58.0 mm to (212.2, 79.8)
- moved R21 58.0 mm to (207.6, 76.2)
- moved D10 58.0 mm to (207.6, 82.3)
- moved D9 58.0 mm to (212.7, 76.6)
- moved R22 58.0 mm to (207.6, 78.7)
- moved C2 54.2 mm to (232.3, 45.4)
- moved R1 54.2 mm to (232.3, 52.9)
- moved C1 54.2 mm to (232.3, 42.9)
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Routing:
- net GND: track 44.4 -> 0.00 mm
- net /Vin: track 42.6 -> 0.00 mm
- net Net-(D12-K): track 18.0 -> 0.00 mm
- net /PowerProtection/source: track 16.2 -> 0.00 mm
- net /PowerProtection/gate: track 12.9 -> 0.00 mm
- net /PowerProtection/OV: track 11.0 -> 0.00 mm
- net /PowerProtection/EN/UVLO: track 9.06 -> 0.00 mm
- net /PowerProtection/Vout: track 5.76 -> 0.00 mm
- net Net-(IC2-VCAP): track 2.34 -> 0.00 mm
- net Net-(C35-Pad1): track 2.19 -> 0.00 mm

Commit message: meh
Parts:
- added C12: 0.1uF, Capacitor_SMD:C_0603_1608Metric_Pad1.08x0.95mm_HandSolder, F.Cu at (46.1, 143.9)
- added C16: 0.1uF, Capacitor_SMD:C_0603_1608Metric_Pad1.08x0.95mm_HandSolder, F.Cu at (46.1, 146.4)
- added C19: 100nF, Capacitor_SMD:C_0603_1608Metric_Pad1.08x0.95mm_HandSolder, F.Cu at (46.1, 149.0)
- added C7: 0.1uF, Capacitor_SMD:C_0603_1608Metric_Pad1.08x0.95mm_HandSolder, F.Cu at (46.1, 138.9)
- added C9: 0.1uF, Capacitor_SMD:C_0603_1608Metric_Pad1.08x0.95mm_HandSolder, F.Cu at (46.1, 141.4)
- added D8: LED, LED_SMD:LED_0603_1608Metric, F.Cu at (50.3, 147.6)
- added FB2: FerriteBead, Capacitor_SMD:C_0603_1608Metric_Pad1.08x0.95mm_HandSolder, F.Cu at (46.1, 151.5)
- added J1: ELCON_CAN_DEBUG, LHRS_Connectors:Molex_Nano-Fit_105309-xx04_1x04_P2.50mm_Vertical, F.Cu at (100.3, 154.3)
- added J4: CHARGER_CAN_DEBUG0, LHRS_Connectors:Molex_Nano-Fit_105309-xx04_1x04_P2.50mm_Vertical, F.Cu at (108.7, 154.3)
- added J6: USB_C_Receptacle_USB2.0_16P, LHRS_Connectors:USB_C_Receptacle_GCT_USB4105-xx-A_16P_TopMnt_Horizontal, F.Cu at (210.7, 94.9)
- added J8: SWD_Header, LHRS_Connectors:SWD_Conn, F.Cu at (53.7, 142.0)
- added R14: 10k, Resistor_SMD:R_0603_1608Metric_Pad0.98x0.95mm_HandSolder, F.Cu at (46.1, 154.0)
- added R15: 1k, Resistor_SMD:R_0603_1608Metric_Pad0.98x0.95mm_HandSolder, F.Cu at (46.1, 156.5)
- added R19: 10k, Resistor_SMD:R_0603_1608Metric_Pad0.98x0.95mm_HandSolder, F.Cu at (46.1, 159.0)
- C41: footprint Capacitor_SMD:C_0603_1608Metric -> Capacitor_SMD:C_0603_1608Metric_Pad1.08x0.95mm_HandSolder
- C53, C54: footprint Capacitor_SMD:C_0201_0603Metric_Pad0.64x0.40mm_HandSolder -> Capacitor_SMD:C_0603_1608Metric_Pad1.08x0.95mm_HandSolder
- C72, C8: footprint Capacitor_SMD:C_0805_2012Metric -> Capacitor_SMD:C_0805_2012Metric_Pad1.18x1.45mm_HandSolder
- D2: value LED -> Fault
- D3: value LED -> 14V
- D4: value LED -> 5V
- D5: value LED -> 3V3
- R28: value 7.5k -> 7.32k
- R30: value 16k -> 15.8k
- TP1, TP10, TP11, TP12, TP13, TP14, TP15, TP16, TP17, TP18, TP2, TP3, TP4, TP9: footprint LHRS_Connectors:5754 -> TestPoint:TestPoint_Loop_D1.80mm_Drill1.0mm_Beaded
- moved C12 43.4 mm to (64.7, 138.5)
- moved C15 43.4 mm to (64.7, 146.0)
- moved C18 43.4 mm to (69.1, 138.5)
- moved C5 43.4 mm to (60.4, 138.5)
- moved C9 43.4 mm to (60.4, 146.0)
- moved FB2 43.4 mm to (69.1, 146.0)
- moved R15 43.4 mm to (73.4, 138.5)
- moved R18 43.4 mm to (73.4, 146.0)
- moved C10 43.4 mm to (60.4, 148.5)
- moved C13 43.4 mm to (64.7, 141.0)
- moved C16 43.4 mm to (64.7, 148.5)
- moved C19 43.4 mm to (69.1, 141.0)
- moved C6 43.4 mm to (60.4, 141.0)
- moved D7 43.4 mm to (60.4, 165.6)
- moved J12 43.4 mm to (84.5, 154.6)
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- renumbered C34 to C33, C35 to C34, C36 to C35, C37 to C36, C38 to C37
Connections:
- C1 pad 2: /Power_Mux/MX_GND -> GND
- C2 pad 2: /Power_Mux/MX_GND -> GND
- C3 pad 2: /Power_Mux/MX_GND -> GND
- C35 pad 1: /PowerProtection/Vout -> +14V
- C4 pad 2: /Power_Mux/MX_GND -> GND
- Q4 pad 5: /PowerProtection/Vout -> +14V
- R3 pad 2: /Power_Mux/MX_GND -> GND
- R9 pad 2: /PowerProtection/Vout -> +14V
- TP18 pad 1: /BUZ_DRAIN -> /BUZ-
- TP2 pad 1: /PowerProtection/Vout -> +14V
- U3 pad 1: /Power_Mux/MX_GND -> GND

Commit message: nothing big
Parts:
- moved D11 31.8 mm to (173.8, 26.0), turned to 0 degrees
- moved R9 29.7 mm to (189.7, 23.9)
- moved J6 20.4 mm to (197.3, 79.6), turned to -90 degrees
- moved R29 17.5 mm to (174.7, 35.9), turned to 0 degrees
- moved C22 17.1 mm to (170.3, 35.9), turned to 180 degrees
- moved R30 16.3 mm to (189.3, 57.1)
- moved C37 16.3 mm to (189.3, 54.9)
- moved R25 15.9 mm to (174.7, 37.9)
- moved D12 9.75 mm to (177.8, 42.0), turned to 180 degrees
- moved IC2 9.53 mm to (179.3, 36.4), turned to 0 degrees
- moved C33 9.25 mm to (179.3, 39.1)
- moved R27 8.79 mm to (170.3, 37.8), turned to 180 degrees
- moved R21 8.27 mm to (206.0, 84.3), turned to 90 degrees
- moved C36 8.07 mm to (173.8, 50.0)
- moved R28 8.07 mm to (173.8, 52.0)
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Routing:
- net /USB_D+: track 0.00 -> 6.89 mm
- net /USB_D-: track 0.00 -> 6.81 mm
- net /USB-C_Connector/VBUS_IN: track 0.00 -> 5.10 mm
- net /5V_USB: track 0.00 -> 2.98 mm

Commit message: usbc,ldo,buck
Parts:
- added D24: 5V, LED_SMD:LED_0603_1608Metric, F.Cu at (228.3, 24.1)
- added D25: 5V, LED_SMD:LED_0603_1608Metric, F.Cu at (63.8, 17.7)
- added L1: 8.2u, LHRS_Passives:74439369082, F.Cu at (54.8, 25.1)
- added R54: 2.2k, Resistor_SMD:R_0603_1608Metric_Pad0.98x0.95mm_HandSolder, F.Cu at (232.4, 24.1)
- added R55: 2.2k, Resistor_SMD:R_0603_1608Metric_Pad0.98x0.95mm_HandSolder, F.Cu at (61.5, 18.7)
- added TP1: PRE_PP, TestPoint:TestPoint_Loop_D1.80mm_Drill1.0mm_Beaded, F.Cu at (256.8, 34.9)
- C42, C43: footprint Capacitor_SMD:C_1210_3225Metric_Pad1.33x2.70mm_HandSolder -> Capacitor_SMD:C_1206_3216Metric_Pad1.33x1.80mm_HandSolder
- R2: footprint Resistor_SMD:R_0603_1608Metric -> Resistor_SMD:R_0603_1608Metric_Pad0.98x0.95mm_HandSolder
- R21, R22: moved to B.Cu
- R3, R5, R7, R8: footprint Package_DIP:DIP-8_W7.62mm -> Resistor_SMD:R_0603_1608Metric_Pad0.98x0.95mm_HandSolder
- moved R21 184.1 mm to (34.0, 18.6), turned to -90 degrees
- moved R22 182.9 mm to (35.8, 24.2), turned to 180 degrees
- moved C20 180.8 mm to (38.7, 22.1)
- moved D9 178.4 mm to (37.3, 18.9)
- moved J6 178.4 mm to (28.3, 22.6)
- moved D10 178.2 mm to (35.5, 22.1)
- moved C39 177.6 mm to (41.6, 21.4), turned to 180 degrees
- moved R34 177.0 mm to (41.9, 17.8), turned to 180 degrees
- moved C40 175.7 mm to (41.8, 19.5), turned to 180 degrees
- moved R31 173.3 mm to (45.2, 17.8), turned to 180 degrees
- moved D4 168.3 mm to (247.9, 42.4), turned to 90 degrees
- moved C41 166.4 mm to (48.5, 17.8)
- moved U1 163.9 mm to (46.2, 20.1)
- moved C44 156.2 mm to (62.5, 28.8)
- moved C43 145.5 mm to (63.0, 25.1)
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Connections:
- C22 pad 1: /Vin -> /PowerProtection/Vin
- D11 pad 2: /Vin -> /PowerProtection/Vin
- Q3 pad 5: /Vin -> /PowerProtection/Vin
- R25 pad 2: /Vin -> /PowerProtection/Vin
- R27 pad 1: /Vin -> /PowerProtection/Vin
- R29 pad 1: /Vin -> /PowerProtection/Vin
- R9 pad 1: /Vin -> /PowerProtection/Vin
Routing:
- net GND: track 0.00 -> 9.15 mm, vias 0 -> 4
- net /USB-C_Connector/VBUS_IN: track 5.10 -> 11.8 mm
- net /USB-C_Connector/CC1: track 0.00 -> 3.37 mm, vias 0 -> 1
- net /12VBuck/FB: track 0.00 -> 3.27 mm
- net /USB-C_Connector/CC2: track 0.00 -> 2.93 mm, vias 0 -> 1
- net Net-(D25-A): track 0.00 -> 1.52 mm
- net /5V_USB: track 2.98 -> 2.24 mm
- net /USB_D-: track 6.81 -> 7.49 mm
- net /USB_D+: track 6.89 -> 7.42 mm
- added copper zone on F.Cu, net +14V
- added copper zone on F.Cu, net /12VBuck/SW
- added copper zone on F.Cu, net /12VBuck/V_out_5V

Commit message: add layout/routing for pp, mux, usb pd, LDO, and Buck
Parts:
- removed the TP1 at (256.8, 34.9)
- moved TP1 216.3 mm to (249.7, 21.0)
- moved J1 192.8 mm to (265.6, 114.6)
- moved J4 192.8 mm to (274.0, 114.6)
- moved R54 192.0 mm to (40.5, 23.8), turned to -90 degrees
- moved D24 188.8 mm to (39.5, 26.5)
- moved J10 178.9 mm to (235.0, 122.8)
- moved J11 178.9 mm to (243.4, 122.8)
- moved J13 178.9 mm to (235.0, 134.1)
- moved J15 178.9 mm to (251.8, 122.8)
- moved J3 178.9 mm to (254.3, 133.8)
- moved J5 178.9 mm to (262.7, 133.8)
- moved J7 178.9 mm to (246.6, 150.3)
- moved D4 176.9 mm to (72.7, 18.0), turned to 180 degrees
- moved R11 176.8 mm to (70.3, 18.9)
- moved U3 176.5 mm to (61.1, 25.8), turned to 180 degrees
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Routing:
- net GND: track 9.15 -> 92.4 mm, vias 4 -> 13
- net +3V3: track 0.00 -> 22.4 mm
- net /PowerProtection/gate: track 0.00 -> 13.2 mm, vias 0 -> 2
- net /PowerProtection/OV: track 0.00 -> 12.6 mm, vias 0 -> 2
- net /12VBuck/SW: track 0.00 -> 12.5 mm
- net /12VBuck/V_out_5V: track 0.00 -> 11.3 mm, vias 0 -> 2
- net Net-(D12-K): track 0.00 -> 11.2 mm
- net /Elcon_CAN_L: track 0.00 -> 8.87 mm
- net +5V: track 0.00 -> 8.17 mm
- net Net-(D13-K): track 0.00 -> 6.33 mm
- net Net-(C30-Pad2): track 0.00 -> 6.09 mm
- net /PowerProtection/EN/UVLO: track 0.00 -> 5.80 mm
- net /5V_USB: track 2.24 -> 7.82 mm
- net /Power_Mux/PR1: track 0.00 -> 5.38 mm
- net /LED_CHARGE: track 0.00 -> 3.81 mm
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- added copper zone on F.Cu, net /PowerProtection/Vin
- added copper zone on F.Cu, net /PowerProtection/source
- removed copper zone on F.Cu, net /12VBuck/SW
