File: EVSE.kicad_sch (KiCad schematic)
At the start: 14 parts

Commit message: org stuf
Parts:
- TP10: value TestPoint -> CP_V
- TP11: value TestPoint -> MCU_CP
- TP12: value TestPoint -> EVSE_PP
- TP9: value TestPoint -> EVSE_CP

Commit message: final schem is done
Parts:
- C72: Distrbutor Link https://www.mouser.com/ProductDetail/KYOCERA-AVX/08055D475K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 -> (none)
- D22: Height 1.45 -> (none); Manufacturer_Name Diodes Incorporated -> (none); Manufacturer_Part_Number 1N5819HW-7-F -> (none); Mouser Part Number 621-1N5819HW-F -> (none); Mouser Price/Stock https://www.mouser.co.uk/ProductDetail/Diodes-Incorporated/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 -> (none)
- TP10, TP11, TP12, TP9: footprint TestPoint:TestPoint_THTPad_D1.5mm_Drill0.7mm -> LHRS_Connectors:5754

Commit message: shoupu review done
Changed lines of the file:
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@@
 	(text "Vout = Vin* ((R13+R21)/(R13+R21+R12))\nVout/Vin = 3/12 = 0.25\nVin = 12V\nVout = 3V\n\n\nR12 = \n0.25(R12+R13+R21)=R13+R21\nR12 = 3(R13+R21)\nR13 + R21 = 15.1k ohms, R12 = 45.3\n\nVout = 12*(15.1k/45.3k+15.1k) = 3V"
 		(exclude_from_sim no)
-		(at 39.878 67.31 0)
+		(at 39.37 67.31 0)
 		(effects
 			(font
@@
 	(text "12V"
 		(exclude_from_sim no)
-		(at 53.848 28.702 0)
+		(at 53.34 29.21 0)
 		(effects
 			(font
@@
 	(text "Current draw (worst case)\nI = 3.3/2.2k+220 = 1mA"
 		(exclude_from_sim no)
-		(at 159.512 60.452 0)
+		(at 160.02 60.96 0)
 		(effects
 			(font
@@
 	(text "VPP MCU reading: \n32A cable: ~220Ω \n\nVpp = 3.3 (Rcabel/Rpull up + Rcabel)\nVpp = 3.3 (220/2.2k+220)\nVpp = 0.3V"
 		(exclude_from_sim no)
-		(at 160.02 51.054 0)
+		(at 160.02 50.8 0)
 		(effects
 			(font
@@
 	(text "State A = no EV (12V)\nState C  = ready to charge (3V)\n"
 		(exclude_from_sim no)
-		(at 58.674 18.288 0)
+		(at 58.42 17.78 0)
 		(effects
 			(font
@@
 	(text "3V"
 		(exclude_from_sim no)
-		(at 80.01 40.894 0)
+		(at 80.01 40.64 0)
 		(effects
 			(font

Commit message: review council
Parts:
- C72: footprint Capacitor_SMD:C_0805_2012Metric -> Capacitor_SMD:C_0805_2012Metric_Pad1.18x1.45mm_HandSolder
- TP10, TP11, TP12, TP9: footprint LHRS_Connectors:5754 -> TestPoint:TestPoint_Loop_D1.80mm_Drill1.0mm_Beaded
Changed lines of the file:
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@@
 			)
 		)
-		(property "Footprint" "Capacitor_SMD:C_0805_2012Metric"
+		(property "Footprint" "Capacitor_SMD:C_0805_2012Metric_Pad1.18x1.45mm_HandSolder"
 			(at 89.8652 50.8 0)
 			(hide yes)
@@
 			)
 		)
-		(property "Footprint" "LHRS_Connectors:5754"
+		(property "Footprint" "TestPoint:TestPoint_Loop_D1.80mm_Drill1.0mm_Beaded"
 			(at 43.18 30.48 0)
 			(hide yes)
@@
 			)
 		)
-		(property "Footprint" "LHRS_Connectors:5754"
+		(property "Footprint" "TestPoint:TestPoint_Loop_D1.80mm_Drill1.0mm_Beaded"
 			(at 127 39.37 0)
 			(hide yes)
@@
 			)
 		)
-		(property "Footprint" "LHRS_Connectors:5754"
+		(property "Footprint" "TestPoint:TestPoint_Loop_D1.80mm_Drill1.0mm_Beaded"
 			(at 22.86 30.48 0)
 			(hide yes)
@@
 			)
 		)
-		(property "Footprint" "LHRS_Connectors:5754"
+		(property "Footprint" "TestPoint:TestPoint_Loop_D1.80mm_Drill1.0mm_Beaded"
 			(at 88.9 41.91 0)
 			(hide yes)

Commit message: revised ish
Connections:
- net +3.3V renamed +3v3
Changed lines of the file:
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@@
 			)
 		)
-		(property "Value" "+3.3V"
-			(at 144.78 16.51 0)
+		(property "Value" "+3v3"
+			(at 147.32 20.3199 0)
 			(show_name no)
 			(do_not_autoplace no)
@@
 					(size 1.27 1.27)
 				)
+				(justify left)
 			)
 		)

Commit message: everything is routed, need to do DRC
Connections:
- net +3v3 renamed +3V3
Changed lines of the file:
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@@
 			)
 		)
-		(property "Value" "+3v3"
+		(property "Value" "+3V3"
 			(at 147.32 20.3199 0)
 			(show_name no)
