File: External Sch/12V-24VBoostConverter.kicad_sch (KiCad schematic)
At the start: 16 parts, among them IC2 TPS613771RYHR

Commit message: small rev3 changes
Parts:
- added C22, C23: 22u, symbol Device:C
- C12: value 56u -> 22u
Connections:
- net GND: now also C22.2, C23.2
- net at C12.1, C41.1, F3.1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: now also C22.1, C23.1
Other:
- moved on the sheet: C41
