File: External Sch/Input_PP.kicad_sch (KiCad schematic)
At the start: 19 parts, among them IC1 LM74502HDDFR, Q1 PSMN8R5-40MSDX

Commit message: small rev3 changes
Connections:
- net LV+ is gone; now on net 12V_IN: R28.1
Changed lines of the file:
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@@
 	(text "Resistor 1"
 		(exclude_from_sim no)
-		(at 122.174 68.58 0)
+		(at 110.744 69.342 0)
 		(effects
 			(font
@@
 	(text "Resistor 2"
 		(exclude_from_sim no)
-		(at 132.08 72.644 0)
+		(at 132.08 74.676 0)
 		(effects
 			(font
@@
 		)
 	)
-	(label "LV+"
-		(at 115.57 67.31 0)
-		(effects
-			(font
-				(size 1.27 1.27)
-			)
-			(justify left bottom)
-		)
-	)
 	(label "RPP_EN"
 		(at 75.565 73.025 0)
@@
 		(effects
 			(font
+				(size 1.27 1.27)
+			)
+			(justify left)
+		)
+	)
+	(hierarchical_label "12V_IN"
+		(shape input)
+		(at 115.57 67.31 0)
+		(effects
+			(font
