File: External Parts/Output_PP.kicad_sch (KiCad schematic)
At the start: 19 parts, among them IC3 LM74502HDDFR, Q2 PSMN8R5-40MSDX

Commit message: RevA5
Other:
- note added: "Overvoltage Protection: 29.03V Vovr = (R2 * Vov)/(R1 + R2) Vov = Vovr * (R1 + R2) / R2 29.03 = 1.25 * (200k + 9k) / 9k"
Changed lines of the file:
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@@
+		)
+	)
+	(text "Overvoltage Protection: 29.03V\nVovr = (R2 * Vov)/(R1 + R2)\nVov = Vovr * (R1 + R2) / R2\n29.03 = 1.25 * (200k + 9k) / 9k"
+		(exclude_from_sim no)
+		(at 184.404 96.52 0)
+		(effects
+			(font
+				(size 1.27 1.27)
+			)
 		)
 	)
