File: Hardware/PS-ChargerInterfacePCB.kicad_pcb (KiCad board)
At the start: 2 copper layers, 74.2 x 75.5 mm, 84 parts, among them IC1 TPS613771RYHR, IC2 LM74502HDDFR, IC3 LM74502HDDFR, J1 LV_Elcon_Connector, J2 SFH11-PBPC-D05-ST-BK, J3 BPSConn, J4 SFH11-PBPC-D05-ST-BK, J5 Estop 3, J6 BuzzConn, Q1 PSMN8R5-40MSDX, Q2 PSMN8R5-40MSDX, Q3 PSMN8R5-40MSDX, U1 LeaderSOM, U2 3568

Commit message: saving changes
Parts:
- removed C15, C20, C21: 0.1u, Capacitor_SMD:C_0603_1608Metric
- removed U1: LeaderSOM, UTSVT_Special:LeaderSOM
- removed U2: 3568, 3568:3568
- removed Z2: SMAF4744A, UTSVT_Passives:SODFL5026X125N
- added CR1: V8PAM10S-M3/I, V8PAM10S-M3-I:CR_10S-M3&slash_I_VIS, F.Cu at (74.2, 85.1)
- added D10: LED, LED_SMD:LED_0603_1608Metric, F.Cu at (109.0, 46.7)
- added D7: LED, LED_SMD:LED_0603_1608Metric, F.Cu at (109.0, 54.5)
- added D8: LED, LED_SMD:LED_0603_1608Metric, F.Cu at (109.0, 51.9)
- added D9: LED, LED_SMD:LED_0603_1608Metric, F.Cu at (109.0, 49.3)
- added J7: 105314-1110, 105314-1110:CONN_SD-105314-100_10_MOL, F.Cu at (73.2, 61.1)
- added J8: EVSE Conn, 1053091303:CONN_SD-105309-100_03_MOL, F.Cu at (64.8, 70.3)
- added J9: CarCANConnector, UTSVT_Connectors:Molex_Nano-Fit_105309-xx02_1x02_P2.50mm_Vertical, F.Cu at (132.9, 71.2)
- added Q13: IRLML0030TRPBF, IRLML0030TRPBF:SOT95P237X112-3N, F.Cu at (84.1, 63.2)
- added Q4: IRLML0030TRPBF, IRLML0030TRPBF:SOT95P237X112-3N, F.Cu at (84.1, 44.9)
- added Q5: IRLML0030TRPBF, IRLML0030TRPBF:SOT95P237X112-3N, F.Cu at (84.1, 49.4)
- added Q6: IRLML0030TRPBF, IRLML0030TRPBF:SOT95P237X112-3N, F.Cu at (84.1, 54.0)
- added Q7: IRLML0030TRPBF, IRLML0030TRPBF:SOT95P237X112-3N, F.Cu at (84.1, 58.6)
- added Q8: IRLML0030TRPBF, IRLML0030TRPBF:SOT95P237X112-3N, F.Cu at (133.6, 91.9)
- added Q9: NVMFWS1D7N04XMT1G, NVMFWS1D7N04XMT1G:NVMFWS3D0P04M8LT1G, F.Cu at (104.3, 85.5)
- added R19: 100k, Resistor_SMD:R_0603_1608Metric, F.Cu at (89.4, 47.8)
- added R20: 0, Resistor_SMD:R_0603_1608Metric, F.Cu at (71.0, 70.4)
- added R21: 5.1k, Resistor_SMD:R_0603_1608Metric, F.Cu at (77.0, 90.2)
- added R22: 150, Resistor_SMD:R_0603_1608Metric, F.Cu at (87.3, 87.4)
- added R23: 5.1k, Resistor_SMD:R_0603_1608Metric, F.Cu at (86.6, 91.3)
- added R24: 5.1k, Resistor_SMD:R_0603_1608Metric, F.Cu at (86.5, 89.6)
- added R25: 150, Resistor_SMD:R_0603_1608Metric, F.Cu at (89.1, 87.3)
- added R26: 10k, Resistor_SMD:R_0603_1608Metric, F.Cu at (119.5, 106.8)
- added R27: 2.2k, Resistor_SMD:R_0603_1608Metric, F.Cu at (130.0, 53.5)
- added R28: 22k, Resistor_SMD:R_0603_1608Metric, F.Cu at (119.7, 69.0)
- added R29: 0, Resistor_SMD:R_2512_6332Metric, F.Cu at (104.8, 107.3)
- added R30: 10k, Resistor_SMD:R_0603_1608Metric, F.Cu at (134.6, 97.2)
- added R31: 22k, Resistor_SMD:R_0603_1608Metric, F.Cu at (132.1, 78.4)
- added R32: 470, Resistor_SMD:R_0603_1608Metric, F.Cu at (105.0, 57.1)
- added R33: 470, Resistor_SMD:R_0603_1608Metric, F.Cu at (105.0, 54.6)
- added R34: 470, Resistor_SMD:R_0603_1608Metric, F.Cu at (105.0, 52.1)
- added R35: 470, Resistor_SMD:R_0603_1608Metric, F.Cu at (105.0, 49.6)
- added R36: 470, Resistor_SMD:R_0603_1608Metric, F.Cu at (105.0, 47.1)
- added TH1: Through hole TP, MountingHole:MountingHole_2.2mm_M2, F.Cu at (193.5, 89.3)
- added TH2: Through hole TP, MountingHole:MountingHole_2.2mm_M2, F.Cu at (193.5, 95.2)
- added TH3: Through hole TP, MountingHole:MountingHole_2.2mm_M2, F.Cu at (193.5, 101.2)
- added TP_+14V1: TestPoint, UTSVT_Special:TestPoint_HEX_3mmID, F.Cu at (106.2, 95.3)
- added TP_+24V1: TestPoint, UTSVT_Special:TestPoint_HEX_3mmID, F.Cu at (97.1, 84.4)
- added TP_24VOUT1: TestPoint, UTSVT_Special:TestPoint_HEX_3mmID, F.Cu at (132.6, 81.6)
- added TP_BOOT1: TestPoint, UTSVT_Special:TestPoint_HEX_3mmID, F.Cu at (84.2, 107.8)
- added TP_COMP1: TestPoint, UTSVT_Special:TestPoint_HEX_3mmID, F.Cu at (78.0, 113.8)
- added TP_Drain1: TestPoint, UTSVT_Special:TestPoint_HEX_3mmID, F.Cu at (104.7, 113.7)
- added TP_Drain3: TestPoint, UTSVT_Special:TestPoint_HEX_3mmID, F.Cu at (113.0, 113.8)
- added TP_FB1: TestPoint, UTSVT_Special:TestPoint_HEX_3mmID, F.Cu at (73.8, 110.1)
- added TP_Gate1: TP_Gate, UTSVT_Special:TestPoint_HEX_3mmID, F.Cu at (110.9, 95.2)
- added TP_Gate2: TP_Gate, UTSVT_Special:TestPoint_HEX_3mmID, F.Cu at (119.3, 92.8)
- added TP_ILIM1: TestPoint, UTSVT_Special:TestPoint_HEX_3mmID, F.Cu at (73.9, 113.8)
- added TP_IN1: TestPoint, UTSVT_Special:TestPoint_HEX_3mmID, F.Cu at (96.3, 114.0)
- added TP_OUT1: TestPoint, UTSVT_Special:TestPoint_HEX_3mmID, F.Cu at (132.8, 87.2)
- added TP_OV1: TestPoint, UTSVT_Special:TestPoint_HEX_3mmID, F.Cu at (100.4, 113.8)
- added TP_OV2: TestPoint, UTSVT_Special:TestPoint_HEX_3mmID, F.Cu at (115.3, 93.0)
- added TP_SD1: TestPoint, UTSVT_Special:TestPoint_HEX_3mmID, F.Cu at (106.1, 90.9)
- added TP_SW1: TestPoint, UTSVT_Special:TestPoint_HEX_3mmID, F.Cu at (92.4, 113.9)
- added TP_SW2: TestPoint, UTSVT_Special:TestPoint_HEX_3mmID, F.Cu at (88.0, 113.9)
- added TP_VCC1: TestPoint, UTSVT_Special:TestPoint_HEX_3mmID, F.Cu at (83.8, 114.0)
- added TP_VS1: TestPoint, UTSVT_Special:TestPoint_HEX_3mmID, F.Cu at (122.3, 106.3)
- added TP_VS2: TestPoint, UTSVT_Special:TestPoint_HEX_3mmID, F.Cu at (154.3, 106.6)
- added TP_Vcap1: TestPoint, UTSVT_Special:TestPoint_HEX_3mmID, F.Cu at (109.0, 113.7)
- added TP_Vcap2: TestPoint, UTSVT_Special:TestPoint_HEX_3mmID, F.Cu at (110.8, 90.9)
- added Z4: SMAF4744A, UTSVT_Passives:SODFL5026X125N, F.Cu at (132.5, 106.6)
- C11, C17: value 0.22u -> 220n
- C13: value 10u -> 4.7u
- C19: value 10u -> 0.1u; footprint Capacitor_SMD:C_0805_2012Metric -> Capacitor_SMD:C_0603_1608Metric
- D1: value D_Schottky -> LED; footprint SK32A_LTP:SDO_DO-214AC-SMA_MCE -> LED_SMD:LED_0603_1608Metric
- DS1: moved to B.Cu
- J1: value LV_Elcon_Connector -> ElconConn
- J4: value SFH11-PBPC-D05-ST-BK -> PWM TP; footprint UTSVT_Connectors:CONN_SFH11-xxxC-D05-ST-XX_SUL -> 22284030:CONN_SD-42375-001_M240_03_MOL
- Q1, Q2, Q3: value PSMN8R5-40MSDX -> NVMFWS1D7N04XMT1G; footprint UTSVT_Power:PSMN8R5-40MSDX -> NVMFWS1D7N04XMT1G:NVMFWS3D0P04M8LT1G
- R1: value 100k -> 45.3k
- R12: value 10k -> 45.3k
- R15, R16, R17, R18: value 590R -> 100k
- R2, R5: value 4.3k -> 2k
- R3: value 0 -> 1k
- R4: value 47k -> 22k
- moved J4 127.3 mm to (193.7, 77.8), turned to 0 degrees
- moved TP_GND1 53.0 mm to (117.3, 53.2)
- moved R3 50.3 mm to (82.2, 84.9), turned to 90 degrees
- moved R15 46.1 mm to (89.4, 57.8), turned to 180 degrees
- moved R16 43.8 mm to (89.4, 53.5), turned to 180 degrees
- moved R12 43.0 mm to (78.6, 85.4), turned to -90 degrees
- moved R17 42.0 mm to (89.4, 55.8), turned to 180 degrees
- moved D4 41.3 mm to (134.7, 94.5), turned to 180 degrees
- moved R18 39.7 mm to (89.4, 50.3), turned to 180 degrees
- moved R13 32.6 mm to (77.8, 87.8), turned to 180 degrees
- moved C25 29.7 mm to (105.2, 69.6), turned to 90 degrees
- moved C13 28.9 mm to (79.6, 89.7), turned to 0 degrees
- moved C35 28.3 mm to (106.9, 64.5), turned to -90 degrees
- moved DS1 27.3 mm to (108.2, 66.8), turned to 180 degrees
- moved D1 26.5 mm to (122.5, 115.2)
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Connections:
- net /Power12V/OV renamed /Power14V/OV
- net Net-(IC1-BOOT) renamed /14V-24V Boost Converter/BOOT
- net Net-(IC1-COMP) renamed /14V-24V Boost Converter/COMP
- net Net-(IC1-EN/UVLO) renamed /14V-24V Boost Converter/EN/UVLO
- net Net-(IC1-FB_1) renamed /14V-24V Boost Converter/FB
- net Net-(IC1-ILIM) renamed /14V-24V Boost Converter/ILIM
- net Net-(IC1-SW) renamed /14V-24V Boost Converter/PostL1
- net Net-(IC1-VCC_1) renamed /14V-24V Boost Converter/VCC
- net Net-(IC2-VCAP) renamed /Power14V/Vcap
- net Net-(IC3-VCAP) renamed /Power24V/Vcap
- C1 pad 1: +12V -> +14V
- C10 pad 2: /Power12V/RPP_EN -> /14V_IN
- C11 pad 1: /Power12V/RPP_EN -> /14V_IN
- C12 pad 1: +12V -> +14V
- C13 pad 1: +12V -> /MCU_CP
- C14 pad 1: +12V -> /14V_IN
- C16 pad 2: /Power24V/RPP_EN -> /24V_OUT
- C17 pad 1: /Power24V/RPP_EN -> /24V_OUT
- C19 pad 1: +24V -> /24V_OUT
- C22 pad 1: +12V -> +14V
- C23 pad 1: +12V -> +14V
- C6 pad 1: /12V-24V Boost Converter/24VOut_B4Diodes -> /14V-24V Boost Converter/24V_Out_Fuse
- C7 pad 1: /12V-24V Boost Converter/24VOut_B4Diodes -> /14V-24V Boost Converter/24V_Out_Fuse
- C8 pad 1: /12V-24V Boost Converter/24VOut_B4Diodes -> /14V-24V Boost Converter/24V_Out_Fuse
- C9 pad 1: /12V-24V Boost Converter/24VOut_B4Diodes -> /14V-24V Boost Converter/24V_Out_Fuse
- D1 pad 1: /12V-24V Boost Converter/24V_Out_Fuse -> GND
- D1 pad 2: /12V-24V Boost Converter/24VOut_B4Diodes -> Net-(D1-A)
- D2 pad 1: +12V -> +14V
- D2 pad 2: /Buzzer/Buzz_Post_Diodes -> /Buzzer/Buzz_Drain
- D3 pad 1: Net-(D3-K) -> GND
- D3 pad 2: /LED_HV -> Net-(D3-A)
- D4 pad 1: Net-(D4-K) -> GND
- D4 pad 2: /LED_FAULT -> Net-(D4-A)
- D5 pad 1: Net-(D5-K) -> GND
- D5 pad 2: /LED_CHARGE -> Net-(D5-A)
- D6 pad 1: Net-(D6-K) -> GND
- D6 pad 2: /LED_HEART -> Net-(D6-A)
- IC1 pad 1: +12V -> +14V
- IC1 pad 4: /12V-24V Boost Converter/24VOut_B4Diodes -> /14V-24V Boost Converter/24V_Out_Fuse
- IC1 pad 5: /12V-24V Boost Converter/24VOut_B4Diodes -> /14V-24V Boost Converter/24V_Out_Fuse
- IC2 pad 1: /Power12V/RPP_EN -> /14V_IN
- IC2 pad 5: /Power12V/RPP_EN -> /14V_IN
- IC2 pad 6: Net-(IC2-GATE) -> /Power14V/OV/RPP Gate
- IC2 pad 8: +12V -> /Power14V/FETConn
- IC3 pad 1: /Power24V/RPP_EN -> /24V_OUT
- IC3 pad 5: /Power24V/RPP_EN -> /24V_OUT
- IC3 pad 6: Net-(IC3-GATE) -> /Power24V/OV/RPP Gate
- IC3 pad 8: +24V -> /Power24V/FETConn
- J1 pad 1: /12V_IN -> /14V_IN
- J1 pad 2: /CAN_Elcon_+ -> GND
- J1 pad 3: /CAN_Elcon_- -> /ElconCAN_H
- J1 pad 4: GND -> /ElconCAN_L
- J2 pad 7: unconnected-(J2-CH3-Pad7) -> /BuzzPWM
- J3 pad 3: /CAN_Car_+ -> /CarCAN_H
- J3 pad 4: /CAN_Car_- -> /CarCAN_L
- J4 pad 2: GND -> /Buzzer/Buzz_Drain
- J4 pad 3: /LED_CHARGE -> /BuzzPWM
- J6 pad 1: +12V -> +14V
- J6 pad 2: /Buzzer/Buzz_Post_Diodes -> /Buzzer/Buzz_Drain
- L1 pad 1: +12V -> +14V
- Q1 pad 1: +12V -> /Power14V/FETConn
- Q1 pad 2: Net-(IC2-GATE) -> /Power14V/FETConn
- Q1 pad 3: /12V_IN -> /Power14V/FETConn
- Q2 pad 1: +24V -> /Power24V/FETConn
- Q2 pad 2: Net-(IC3-GATE) -> /Power24V/FETConn
- Q2 pad 3: /24V_OUT -> /Power24V/FETConn
- Q3 pad 1: GND -> +14V
- Q3 pad 2: /BuzzPWM -> +14V
- Q3 pad 3: /Buzzer/Buzz_Post_Diodes -> +14V
- R10 pad 1: /12V-24V Boost Converter/24VOut_B4Diodes -> /14V-24V Boost Converter/24V_Out_Fuse
- R12 pad 1: /12V_IN -> Net-(CR1-Pad1)
- R12 pad 2: /Power12V/RPP_EN -> /MCU_CP
- R13 pad 1: /24V_OUT -> /MCU_CP
- R13 pad 2: /Power24V/RPP_EN -> Net-(R13-Pad2)
- R15 pad 1: GND -> /LED_HV
- R15 pad 2: Net-(D3-K) -> GND
- R16 pad 1: GND -> /LED_FAULT
- R16 pad 2: Net-(D4-K) -> GND
- R17 pad 1: GND -> /LED_HEART
- R17 pad 2: Net-(D5-K) -> GND
- R18 pad 1: GND -> /LED_CHARGE
- R18 pad 2: Net-(D6-K) -> GND
- R3 pad 1: +3.3V -> Net-(CR1-Pad1)
- R3 pad 2: /Estop -> GND
- R4 pad 1: /12V_IN -> /14V_IN
- R6 pad 1: +12V -> +14V
- TP_12V1 pad 1: +12V -> +14V
Routing:
- net /CAN_Elcon_+: track 121.7 -> 0.00 mm, vias 2 -> 0
- net /CAN_Elcon_-: track 116.7 -> 0.00 mm, vias 3 -> 0
- net /LED_FAULT: track 97.8 -> 0.00 mm, vias 4 -> 0
- net /LED_HEART: track 97.1 -> 0.00 mm, vias 4 -> 0
- net /LED_HV: track 93.8 -> 0.00 mm, vias 2 -> 0
- net /LED_CHARGE: track 93.0 -> 0.00 mm, vias 4 -> 0
- net +3.3V: track 83.6 -> 0.00 mm
- net /Estop: track 80.0 -> 0.00 mm, vias 2 -> 0
- net /CAN_Car_-: track 76.5 -> 0.00 mm, vias 2 -> 0
- net /CAN_Car_+: track 73.8 -> 0.00 mm, vias 2 -> 0
- net /BuzzPWM: track 43.3 -> 0.00 mm, vias 2 -> 0
- net /Display_NSS: track 40.9 -> 0.00 mm, vias 2 -> 0
- net /Power24V/RPP_EN: track 40.7 -> 0.00 mm, vias 3 -> 0
- net /Display_MOSI: track 40.0 -> 0.00 mm
- net /Display_RES: track 39.9 -> 0.00 mm, vias 2 -> 0
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- removed copper zone on F.Cu, net +12V
- removed copper zone on F.Cu, net +24V
- removed copper zone on F.Cu, net /12V-24V Boost Converter/24VOut_B4Diodes
- removed copper zone on F.Cu, net /12V-24V Boost Converter/24V_Out_Fuse
- removed copper zone on F.Cu, net /12V_IN
- removed copper zone on F.Cu, net /24V_OUT
- removed copper zone on F.Cu, net /Buzzer/Buzz_Post_Diodes
Other:
- board text added: "Priority Levels: - GND: 0 - PWR: 1/2"

Commit message: layout ready
Parts:
- removed J4: PWM TP, 22284030:CONN_SD-42375-001_M240_03_MOL
- removed TH1, TH2, TH3: Through hole TP, MountingHole:MountingHole_2.2mm_M2
- removed TP_+14V1, TP_+24V1, TP_VS1, TP_VS2: TestPoint, UTSVT_Special:TestPoint_HEX_3mmID
- added TP1: TestPoint, TestPoint:TestPoint_Pad_D1.5mm, F.Cu at (71.0, 67.5)
- added TP2: TestPoint, TestPoint:TestPoint_Pad_D1.5mm, F.Cu at (71.2, 71.0)
- added TP3: TestPoint, TestPoint:TestPoint_Pad_D1.5mm, F.Cu at (74.2, 71.0)
- added TP4: TestPoint, TestPoint:TestPoint_Pad_D1.5mm, F.Cu at (74.0, 67.5)
- added U1: LeaderSOM, UTSVT_Special:LeaderSOM, F.Cu at (92.1, 71.6)
- added U2: 4A, 3568:3568, F.Cu at (124.4, 80.3)
- TP_BOOT1, TP_COMP1, TP_Drain3, TP_FB1, TP_Gate1, TP_Gate2, TP_ILIM1, TP_OV1, TP_OV2, TP_SD1, TP_SW1, TP_SW2, TP_VCC1, TP_Vcap1, TP_Vcap2: footprint UTSVT_Special:TestPoint_HEX_3mmID -> TestPoint:TestPoint_Pad_D1.5mm
- moved TP_Gate1 23.6 mm to (102.5, 117.3), turned to 180 degrees
- moved D10 22.4 mm to (92.3, 61.6), turned to 90 degrees
- moved R36 21.1 mm to (89.7, 61.6), turned to 90 degrees
- moved D6 20.0 mm to (92.2, 46.2), turned to 90 degrees
- moved TP_OV1 18.9 mm to (118.9, 117.6), turned to 180 degrees
- moved R32 18.8 mm to (89.7, 46.2), turned to 90 degrees
- moved D9 18.7 mm to (92.3, 57.7), turned to 90 degrees
- moved R35 17.2 mm to (89.9, 57.7), turned to 90 degrees
- moved D8 17.1 mm to (92.0, 50.1), turned to 90 degrees
- moved D7 16.9 mm to (92.1, 53.8), turned to 90 degrees
- moved TP_GND1 16.3 mm to (133.6, 52.5)
- moved R34 15.6 mm to (89.6, 50.1), turned to 90 degrees
- moved R33 15.3 mm to (89.7, 53.8), turned to 90 degrees
- moved R19 14.0 mm to (87.1, 61.6), turned to 90 degrees
- moved TP_Vcap2 13.9 mm to (97.5, 86.9), turned to 180 degrees
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Connections:
- J2 pad 10: /Display_NSS -> /Display_MOSI
- J2 pad 3: /Display_MOSI -> /Display_NSS
- J2 pad 4: /Display_SCLK -> /Display_RES
- J2 pad 7: /BuzzPWM -> unconnected-(J2-CH3-Pad7)
- J2 pad 8: /Display_RES -> /Display_SCLK
- J2 pad 9: unconnected-(J2-CH1-Pad9) -> /BuzzPWM
- J8 pad 2: /EVSE_PP -> /EVSE_CP
- J8 pad 3: /EVSE_CP -> /EVSE_PP
Routing:
- net /BuzzPWM: track 0.00 -> 114.7 mm, vias 0 -> 2
- net +14V: track 1.87 -> 110.8 mm, vias 0 -> 1
- net /ElconCAN_L: track 0.00 -> 94.5 mm, vias 0 -> 2
- net /ElconCAN_H: track 0.00 -> 92.1 mm, vias 0 -> 2
- net +3.3V: track 0.00 -> 64.5 mm
- net /Display_MOSI: track 0.00 -> 54.5 mm
- net /Display_NSS: track 0.00 -> 54.3 mm, vias 0 -> 2
- net /Display_SCLK: track 0.00 -> 52.6 mm, vias 0 -> 2
- net /Display_MISO: track 0.00 -> 51.8 mm
- net /CarCAN_L: track 0.00 -> 51.1 mm, vias 0 -> 1
- net /Display_RES: track 0.00 -> 50.8 mm
- net /CarCAN_H: track 0.00 -> 50.3 mm, vias 0 -> 1
- net /EVSE_PP: track 0.00 -> 46.8 mm, vias 0 -> 2
- net /LED_HV: track 0.00 -> 45.3 mm, vias 0 -> 2
- net /Estop: track 0.00 -> 44.4 mm
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- added copper zone on F.Cu, net +14V
- added copper zone on F.Cu, net +24V
- added copper zone on F.Cu, net /14V-24V Boost Converter/24V_Out_Fuse
- added copper zone on F.Cu, net /14V_IN
- added copper zone on F.Cu, net /24V_OUT
- added copper zone on F.Cu, net /Power14V/FETConn
- added copper zone on F.Cu, net /Power24V/FETConn
Other:
- board size 74.2 x 75.5 mm -> 74.2 x 79.4 mm
- board text removed: "R15-R18"

Commit message: Review council
Parts:
- removed Q3, Q9: NVMFWS1D7N04XMT1G, NVMFWS1D7N04XMT1G:NVMFWS3D0P04M8LT1G
- removed TP_Drain3, TP_SD1: TestPoint, TestPoint:TestPoint_Pad_D1.5mm
- removed Z1: SMAF4751A-TP, UTSVT_Passives:SODFL5026X125N
- removed Z4: SMAF4744A, UTSVT_Passives:SODFL5026X125N
- added Q10: NVMFWS1D7N04XMT1G, UTSVT_Power:NVMFWS3D0P04M8LT1G, F.Cu at (116.3, 101.3)
- added Q11: NVMFWS1D7N04XMT1G, UTSVT_Power:NVMFWS3D0P04M8LT1G, F.Cu at (117.0, 86.6)
- added TP_FETConn1: TestPoint, TestPoint:TestPoint_Pad_D1.5mm, F.Cu at (111.0, 117.3)
- added TP_FETConn2: TestPoint, TestPoint:TestPoint_Pad_D1.5mm, F.Cu at (105.1, 91.6)
- added Z2: SMAF4758A-TP, UTSVT_Passives:SODFL5026X125N, F.Cu at (133.0, 104.9)
- added Z3: SMAF4758A-TP, UTSVT_Passives:SODFL5026X125N, F.Cu at (124.9, 75.7)
- J9: value CarCANConnector -> ElconConn
- Q1, Q2: footprint NVMFWS1D7N04XMT1G:NVMFWS3D0P04M8LT1G -> UTSVT_Power:NVMFWS3D0P04M8LT1G
- moved Q2 13.1 mm to (104.0, 85.6), turned to 90 degrees
- moved TP_3V1 12.9 mm to (130.0, 50.6)
- moved Q1 8.97 mm to (107.6, 100.4), turned to 90 degrees
- moved R27 6.33 mm to (123.7, 52.9), turned to 0 degrees
- moved C30 5.82 mm to (94.5, 64.1), turned to -90 degrees
- moved TP_14V1 2.36 mm to (133.1, 99.7)
- moved D1 2.02 mm to (122.6, 117.2)
- moved TP_GND1 1.82 mm to (134.1, 50.7)
- moved J1 1.79 mm to (126.5, 112.0)
- moved U2 1.45 mm to (124.4, 81.8)
- moved J6 1.41 mm to (127.7, 99.9)
- moved J9 1.34 mm to (133.4, 72.4)
- moved R31 1.18 mm to (132.2, 79.6)
- moved TP_24VOUT1 1.18 mm to (132.2, 82.8)
- moved D5 1.18 mm to (134.7, 80.3)
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- renumbered TP_12V1 to TP_14V1
Connections:
- net /Power14V/FETConn renamed Net-(IC2-SRC)
- net /Power24V/FETConn renamed Net-(IC3-SRC)
- Q1 pad 5: /14V_IN -> +14V
- Q2 pad 5: /24V_OUT -> +24V
- R5 pad 1: /Power14V/OV -> GND
- R5 pad 2: GND -> /Power14V/OV
Routing:
- net /Power14V/OV/RPP Gate: track 28.1 -> 35.4 mm
- net /Power24V/OV/RPP Gate: track 29.7 -> 34.5 mm, vias 4 -> 2
- net +3.3V: track 64.5 -> 59.8 mm
- net /Buzzer/Buzz_Drain: track 41.8 -> 46.3 mm
- net Net-(IC2-SRC): track 20.2 -> 17.8 mm
- net +14V: track 110.8 -> 108.4 mm
- net Net-(D1-A): track 8.47 -> 10.5 mm
- net /Estop: track 44.4 -> 42.8 mm
- net /CarCAN_L: track 51.1 -> 52.2 mm
- net /BuzzPWM: track 114.7 -> 115.7 mm
- net +24V: track 15.4 -> 16.4 mm
- net Net-(DS1-VOUT): track 2.68 -> 1.75 mm
- net GND: track 18.6 -> 17.7 mm, vias 8 -> 11
- net /Display_MISO: track 51.8 -> 52.7 mm
- net /Display_SCLK: track 52.6 -> 53.4 mm
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