File: Hardware/PS-ChargerInterfacePCB.kicad_sch (KiCad schematic)
At the start: 23 parts, among them J1 ElconConn, J2 SFH11-PBPC-D05-ST-BK, J3 BPSConn, J5 Estop 3, J8 EVSE Conn, U1 LeaderSOM

Commit message: saving changes
Parts:
- added D1, D3, D4, D5: LED, LED_SMD:LED_0603_1608Metric, symbol Device:LED
- added J9: CarCANConnector, UTSVT_Connectors:Molex_Nano-Fit_105309-xx02_1x02_P2.50mm_Vertical, symbol utsvt_connectors2:CarCANConnector
- added R26, R30: 10k, Resistor_SMD:R_0603_1608Metric, symbol Device:R_US
- added R27: 2.2k, Resistor_SMD:R_0603_1608Metric, symbol Device:R_US
- added R28, R31: 22k, Resistor_SMD:R_0603_1608Metric, symbol Device:R_US
- added R29: 0, Resistor_SMD:R_2512_6332Metric, symbol Device:R_US
- J5: P/N 1053091202 -> 105309-1202
- J8: footprint CONN_SD-105309-100_03_MOL -> 1053091303:CONN_SD-105309-100_03_MOL; symbol 1053091303:1053091303 -> Connector_Generic:Conn_01x03; P/N (none) -> 105309-1303
- R20: footprint (none) -> Resistor_SMD:R_0603_1608Metric; P/N (none) -> CRCW06030000Z0EE
- R4: P/N CRCW060347K0FKECC -> CRCW060322K0FKEAHP
- TH1, TH2, TH3: footprint (none) -> MountingHole:MountingHole_2.2mm_M2
- U1: now in the parts list
- Z1: P/N (none) -> SMAF4751A-TP
- Z4: P/N (none) -> SMAF4744A
Connections:
- net +14V: now also R29.2, R30.2
- net +24V: now also R28.2
- net BuzzPWM: now also J2.7 (CH3)
- net Display_MISO: now also U1.42 (SPI3_MISO); no longer U1.14 (SPI2_MISO)
- net Display_MOSI: now also U1.46 (SPI3_MOSI); no longer U1.18 (SPI2_MOSI)
- net Display_NSS: now also U1.44 (SPI3_NSS); no longer U1.16 (SPI2_NSS)
- net Display_SCLK: now also U1.48 (SPI3_SCK); no longer U1.20 (SPI2_SCK)
- net EVSE_CP: now also J8.3 (Pin_3); no longer J8.1
- net Earth_Protective: now also J8.1 (Pin_1); no longer J8.3
- net GND: now also D1.1 (K), D3.1 (K), D4.1 (K), D5.1 (K), R27.1; no longer J1.1 (14V), J2.5 (CH5), J5.2 (Pin_2), R1.1, R4.1, TH1.1, U1.41 (ADC1_IN2)
- net LED_CHARGE: now also U1.18 (SPI2_MOSI); no longer U1.46 (SPI3_MOSI)
- net LED_FAULT: now also U1.16 (SPI2_NSS); no longer U1.44 (SPI3_NSS)
- net LED_HEART: now also U1.20 (SPI2_SCK); no longer U1.48 (SPI3_SCK)
- net LED_HV: now also U1.14 (SPI2_MISO); no longer U1.42 (SPI3_MISO)
- net CAN_Car_+ renamed CarCAN_H
- net CAN_Car_- renamed CarCAN_L
- net CAN_Elcon_+ renamed ElconCAN_H
- net ElconCAN_H: now also J9.1 (CAN_H); no longer J2.7 (CH3)
- net CAN_Elcon_- renamed ElconCAN_L
- net ElconCAN_L: now also J9.2 (CAN_L); no longer J2.9 (CH1)
- new net: D3.2 (A), R28.1
- new net: D4.2 (A), R30.1
- new net: D5.2 (A), R31.1
- new net: D1.2 (A), R26.1
- new net 14V_IN: J1.1 (14V), R26.2, R29.1, R4.1
- new net 24V_OUT: R1.1, R31.2, TH1.1
- new net Estop: J2.5 (CH5), J5.2 (Pin_2), R27.2, U1.41 (ADC1_IN2)
Other:
- sheet Power12V renamed Power14V
- note added: "Power LEDs"
- note removed: "Net Class for Diff Pair: CAN_H_Elcon = CAN_Elcon_+ CAN_L_Elcon = CAN_Elcon_- CAN_H_Car = CAN_Car_+ CAN_L_Car = CAN_Car_-"
- moved on the sheet: H1, H2, H3, J1, J2, J3, R1, R2, R20, TH1, TH2, TH3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

Commit message: layout ready
Parts:
- removed TH1, TH2, TH3: Through hole TP, MountingHole:MountingHole_2.2mm_M2, symbol Connector:TestPoint
Connections:
- net BuzzPWM: now also J2.9 (CH1); no longer J2.7 (CH3)
- net Display_MOSI: now also J2.10 (CH0); no longer J2.3 (CH7)
- net Display_NSS: now also J2.3 (CH7); no longer J2.10 (CH0)
- net Display_RES: now also J2.4 (CH6), U1.40 (ADC1_IN7); no longer J2.8 (CH2), U1.12 (ADC1_IN11)
- net Display_SCLK: now also J2.8 (CH2); no longer J2.4 (CH6)
- net EVSE_CP: now also J8.2 (Pin_2); no longer J8.3 (Pin_3)
- net EVSE_PP: now also J8.3 (Pin_3); no longer J8.2 (Pin_2)
- net Estop: now also U1.20 (SPI2_SCK); no longer U1.41 (ADC1_IN2)
- net LED_CHARGE: now also U1.41 (ADC1_IN2); no longer U1.18 (SPI2_MOSI)
- net LED_FAULT: now also U1.33 (ADC1_IN15); no longer U1.16 (SPI2_NSS)
- net LED_HEART: now also U1.39 (ADC1_IN3); no longer U1.20 (SPI2_SCK)
- net LED_HV: now also U1.31 (ADC1_IN12); no longer U1.14 (SPI2_MISO)
- no-connect marks 17 -> 18
Other:
- note removed: "Throughole Test Points"

Commit message: Review council
Parts:
- removed Z1: SMAF4751A-TP, UTSVT_Passives:SODFL5026X125N, symbol UTSVT_Power:SMAF4749A-TP
- removed Z4: SMAF4744A, UTSVT_Passives:SODFL5026X125N, symbol UTSVT_Power:SMAF4749A-TP
- J9: value CarCANConnector -> ElconConn
- renumbered TP_12V1 to TP_14V1
Connections:
- net GND: now also R5.1; no longer R5.2
- net Power14V/OV: now also R5.2; no longer R5.1
Other:
- sheet Power14V ports: added none; removed Fuse
- sheet Power24V ports: added none; removed Fuse
- note added: "12 to 24V Boost w RPP/OV"
- note removed: "Boost Converter"
- note removed: "Connectors"
- note removed: "Power Protection"
- moved on the sheet: D1, D3, D4, D5, H1, H2, H3, J1, J2, J3, J5, J8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

Commit message: Layout again
Parts:
- removed J5: Estop 3, 153091202:1053091202, symbol Connector_Generic:Conn_01x02
- added Estop1: EStop Conn, UTSVT_Connectors:Molex_Nano-Fit_105309-xx02_1x02_P2.50mm_Vertical, symbol utsvt_connectors2:CarCANConnector
- renumbered TP_14V1 to +14V1, TP_24V1 to +24V1, TP_3V1 to +3V3, J8 to EVSE1, J1 to Elcon1, J3 to Elcon2, TP_GND1 to GND1, J2 to Logic_Analyzer1
Connections:
- net +3.3V: now also Estop1.1 (+3V3)
- net Estop: now also Estop1.2 (MCU)
Other:
- moved on the sheet: R27

Commit message: Geber + BOM
Parts:
- +14V1, +24V1, +3V3, GND1: footprint UTSVT_Special:TestPoint_HEX_3mmID -> TestPoint:TestPoint_THTPad_D3.0mm_Drill1.5mm
- D1, D4: P/N LS Q976.01-N1Q2-1 -> NCD0603R1
- D3, D5: P/N LTST-C193TBKT-5A -> XL-1608UBC-06A
- J9: value ElconConn -> ElconCANConn
- R26, R30: value 10k -> 4.3k
- R27: value 2.2k -> 10k
- R28, R31: value 22k -> 10k
Changed lines of the file:
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@@
 			)
 		)
-		(property "Footprint" "UTSVT_Special:TestPoint_HEX_3mmID"
+		(property "Footprint" "TestPoint:TestPoint_THTPad_D3.0mm_Drill1.5mm"
 			(at 189.23 110.49 0)
 			(effects
@@
 			)
 		)
-		(property "Value" "22k"
+		(property "Value" "10k"
 			(at 187.198 141.986 0)
 			(effects
@@
 			)
 		)
-		(property "P/N" "LTST-C193TBKT-5A"
+		(property "P/N" "XL-1608UBC-06A"
 			(at 184.15 149.86 90)
 			(effects
@@
 			)
 		)
-		(property "Footprint" "UTSVT_Special:TestPoint_HEX_3mmID"
+		(property "Footprint" "TestPoint:TestPoint_THTPad_D3.0mm_Drill1.5mm"
 			(at 208.28 110.49 0)
 			(effects
@@
 			)
 		)
-		(property "Value" "10k"
+		(property "Value" "4.3k"
 			(at 212.598 141.986 0)
 			(effects
@@
 			)
 		)
-		(property "P/N" "LTST-C193TBKT-5A"
+		(property "P/N" "XL-1608UBC-06A"
 			(at 193.04 149.86 90)
 			(effects
@@
 			)
 		)
-		(property "Value" "10k"
+		(property "Value" "4.3k"
 			(at 203.708 141.986 0)
 			(effects
@@
 			)
 		)
-		(property "Value" "22k"
+		(property "Value" "10k"
 			(at 196.088 141.986 0)
 			(effects
@@
 			)
 		)
-		(property "Footprint" "UTSVT_Special:TestPoint_HEX_3mmID"
+		(property "Footprint" "TestPoint:TestPoint_THTPad_D3.0mm_Drill1.5mm"
 			(at 195.58 110.49 0)
 			(effects
@@
 			)
 		)
-		(property "P/N" "LS Q976.01-N1Q2-1"
+		(property "P/N" "NCD0603R1"
 			(at 200.66 149.86 90)
 			(effects
@@
 			)
 		)
-		(property "Value" "2.2k"
+		(property "Value" "10k"
 			(at 252.73 68.326 0)
 			(effects
@@
 			)
 		)
-		(property "Footprint" "UTSVT_Special:TestPoint_HEX_3mmID"
+		(property "Footprint" "TestPoint:TestPoint_THTPad_D3.0mm_Drill1.5mm"
 			(at 201.93 110.49 0)
 			(effects
@@
 			)
 		)
-		(property "Value" "ElconConn"
+		(property "Value" "ElconCANConn"
 			(at 95.25 77.47 0)
 			(effects
@@
 			)
 		)
-		(property "P/N" "LS Q976.01-N1Q2-1"
+		(property "P/N" "NCD0603R1"
 			(at 209.55 149.86 90)
 			(effects
