File: Hardware/PS-ChargerInterfacePCB.kicad_sch (KiCad schematic)
At the start: 29 parts, among them J9 ElconCANConn, U1 LeaderSOM

Commit message: last changes + silkscreen
Parts:
- added H4: MountingHole, MountingHole:MountingHole_3mm_Pad_TopBottom, symbol Mechanical:MountingHole
Connections:
- net BuzzPWM: now also Logic_Analyzer1.5 (CH5); no longer Logic_Analyzer1.9 (CH1)
- net Estop: now also Logic_Analyzer1.9 (CH1); no longer Logic_Analyzer1.5 (CH5)
Changed lines of the file:
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@@
 		)
 	)
+	(label "BuzzPWM"
+		(at 170.18 140.97 180)
+		(effects
+			(font
+				(size 1.016 1.016)
+			)
+			(justify right bottom)
+		)
+	)
 	(label "LED_CHARGE"
 		(at 229.87 101.6 0)
@@
 		)
 	)
-	(label "BuzzPWM"
-		(at 170.18 151.13 180)
-		(effects
-			(font
-				(size 1.016 1.016)
-			)
-			(justify right bottom)
-		)
-	)
 	(label "Display_NSS"
 		(at 134.62 149.86 180)
@@
 		)
 	)
+	(label "Estop"
+		(at 170.18 151.13 180)
+		(effects
+			(font
+				(size 1.016 1.016)
+			)
+			(justify right bottom)
+		)
+	)
 	(label "24V_OUT"
 		(at 193.04 125.73 270)
@@
 		)
 	)
-	(label "Estop"
-		(at 170.18 140.97 180)
-		(effects
-			(font
-				(size 1.016 1.016)
-			)
-			(justify right bottom)
-		)
-	)
 	(label "Display_SCLK"
 		(at 231.14 140.97 0)
@@
 					(unit 1)
 				)
+			)
+		)
+	)
+	(symbol
+		(lib_id "Mechanical:MountingHole")
+		(at 153.67 113.03 0)
+		(unit 1)
+		(exclude_from_sim no)
+		(in_bom no)
+		(on_board yes)
+		(dnp no)
+		(fields_autoplaced yes)
+		(property "Reference" "H4"
+			(at 156.21 111.7599 0)
+			(effects
+				(font
+					(size 1.27 1.27)
+				)
+				(justify left)
+			)
+		)
+		(property "Value" "MountingHole"
+			(at 156.21 114.2999 0)
+			(effects
+				(font
+					(size 1.27 1.27)
+				)
+				(justify left)
+			)
+		)
+		(property "Footprint" "MountingHole:MountingHole_3mm_Pad_TopBottom"
+			(at 153.67 113.03 0)
+			(effects
+				(font
+					(size 1.27 1.27)
+				)
+				(hide yes)
+			)
+		)
+		(property "Datasheet" "~"
+			(at 153.67 113.03 0)
+			(effects
+				(font
+					(size 1.27 1.27)
+				)
+				(hide yes)
+			)
+		)
+		(property "Description" "Mounting Hole without connection"
+			(at 153.67 113.03 0)
+			(effects
+				(font
+					(size 1.27 1.27)
+				)
+				(hide yes)
+			)
+		)
+		(property "Part #" ""
+			(at 153.67 113.03 0)
+			(effects
+				(font
+					(size 1.27 1.27)
+				)
+				(hide yes)
+			)
+		)
+		(property "Sim.Pins" ""
+			(at 153.67 113.03 0)
+			(effects
+				(font
+					(size 1.27 1.27)
+				)
+				(hide yes)
+			)
+		)
+		(instances
+			(project "PS-ChargerInterfacePCB"
+				(path "/d45494af-ff47-4110-bed2-dd613b557244"
+					(reference "H4")
+					(unit 1)
+				)

Commit message: Cleaned up Branch
Parts:
- EVSE1: footprint 1053091303:CONN_SD-105309-100_03_MOL -> External Parts Mod:105309-1303
- R29: P/N CRCW06030000Z0EE -> (none)
Changed lines of the file:
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@@
 			)
 		)
-		(property "Footprint" "1053091303:CONN_SD-105309-100_03_MOL"
+		(property "Footprint" "External Parts Mod:105309-1303"
 			(at 20.32 81.28 0)
 			(effects
@@
 			)
 		)
-		(property "P/N" "CRCW06030000Z0EE"
+		(property "P/N" ""
 			(at 68.58 17.78 90)
 			(effects

Commit message: Updated sym/mod folder names
Parts:
- EVSE1: footprint External Parts Mod:105309-1303 -> charger_parts:105309-1303
Changed lines of the file:
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@@
 			)
 		)
-		(property "Footprint" "External Parts Mod:105309-1303"
+		(property "Footprint" "charger_parts:105309-1303"
 			(at 20.32 81.28 0)
 			(effects
