File: Hardware/Power.kicad_sch (KiCad schematic)
At the start: 14 parts, among them IC2 LM74502HDDFR, Q1 NVMFWS1D7N04XMT1G, Q3 NVMFWS1D7N04XMT1G

Commit message: saving changes
Parts:
- Q1, Q3: footprint NVMFWS3D0P04M8LT1G -> NVMFWS1D7N04XMT1G:NVMFWS3D0P04M8LT1G; P/N (none) -> NVMFWS1D7N04XMT1G
- TP_Gate1: value TestPoint -> TP_Gate
- renumbered TP_Source1 to TP_+14V1, TP_OV to TP_OV1, TP_VS to TP_VS1, TP_Vcap to TP_Vcap1
Connections:
- net FETConn: now reaches IC2.8 (SRC), Q1.1 (S), Q1.2 (S), Q1.3 (S), Q3.5 (D), TP_Drain3.1

Commit message: layout ready
Parts:
- removed TP_+14V1, TP_VS1: TestPoint, UTSVT_Special:TestPoint_HEX_3mmID, symbol Connector:TestPoint
- TP_Drain3, TP_Gate1, TP_OV1, TP_Vcap1: footprint UTSVT_Special:TestPoint_HEX_3mmID -> TestPoint:TestPoint_Pad_D1.5mm

Commit message: Review council
Parts:
- removed Q1, Q3: NVMFWS1D7N04XMT1G, NVMFWS1D7N04XMT1G:NVMFWS3D0P04M8LT1G, symbol Transistor_FET:CSD18509Q5B
- removed TP_Drain3: TestPoint, TestPoint:TestPoint_Pad_D1.5mm, symbol Connector:TestPoint
- added Q1, Q10: NVMFWS1D7N04XMT1G, UTSVT_Power:NVMFWS3D0P04M8LT1G, symbol utsvt_misc:NVMFWS1D7N04XMT1G
- added TP_FETConn1: TestPoint, TestPoint:TestPoint_Pad_D1.5mm, symbol Connector:TestPoint
- added Z2: SMAF4758A-TP, SODFL5026X125N, symbol Device:D_Zener
Connections:
- net GND: now also Z2.2 (A)
- net OV/RPP Gate: now also Q1.4, Q10.4
- net V_OUT: now also Q1.5, Q1.6, Q1.7, Q1.8, Q1.9
- net FETConn: no longer names the net of IC2.8 (SRC)
- net FETConn: now also Q1.1, Q1.2, Q1.3, Q10.1, Q10.2, Q10.3, TP_FETConn1.1
- net Fuse renamed VIN
- net VIN: now also Q10.5, Q10.6, Q10.7, Q10.8, Q10.9, Z2.1 (K)

Commit message: Layout again
Parts:
- renumbered TP_Gate1 to Gate1, TP_OV1 to OV1, TP_Drain1 to RPP_EN1, TP_Vcap1 to Vcap1
Changed lines of the file:
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@@
 		(on_board yes)
 		(dnp no)
-		(property "Reference" "TP_Gate1"
-			(at 28.448 104.902 0)
+		(property "Reference" "Gate1"
+			(at 27.432 104.902 0)
 			(effects
 				(font
@@
 			(project "PS-ChargerInterfacePCB"
 				(path "/d45494af-ff47-4110-bed2-dd613b557244/ac7656e7-8ca1-4189-8850-b703de13aef3"
-					(reference "TP_Gate2")
+					(reference "Gate2")
 					(unit 1)
 				)
 				(path "/d45494af-ff47-4110-bed2-dd613b557244/f4ec1410-3a5f-45f2-a31b-30d8be6fbeab"
-					(reference "TP_Gate1")
+					(reference "Gate1")
 					(unit 1)
 				)
@@
 		(on_board yes)
 		(dnp no)
-		(property "Reference" "TP_OV1"
-			(at 41.148 120.142 0)
+		(property "Reference" "OV1"
+			(at 38.862 119.888 0)
 			(effects
 				(font
@@
 			(project "PS-ChargerInterfacePCB"
 				(path "/d45494af-ff47-4110-bed2-dd613b557244/ac7656e7-8ca1-4189-8850-b703de13aef3"
-					(reference "TP_OV2")
+					(reference "OV2")
 					(unit 1)
 				)
 				(path "/d45494af-ff47-4110-bed2-dd613b557244/f4ec1410-3a5f-45f2-a31b-30d8be6fbeab"
-					(reference "TP_OV1")
+					(reference "OV1")
 					(unit 1)
 				)
@@
 		(on_board yes)
 		(dnp no)
-		(property "Reference" "TP_Drain1"
-			(at 38.608 104.902 0)
+		(property "Reference" "RPP_EN1"
+			(at 38.862 104.394 0)
 			(effects
 				(font
@@
 			(project "PS-ChargerInterfacePCB"
 				(path "/d45494af-ff47-4110-bed2-dd613b557244/ac7656e7-8ca1-4189-8850-b703de13aef3"
-					(reference "TP_24VOUT1")
+					(reference "+24V_IN1")
 					(unit 1)
 				)
 				(path "/d45494af-ff47-4110-bed2-dd613b557244/f4ec1410-3a5f-45f2-a31b-30d8be6fbeab"
-					(reference "TP_Drain1")
+					(reference "RPP_EN1")
 					(unit 1)
 				)
@@
 		(on_board yes)
 		(dnp no)
-		(property "Reference" "TP_Vcap1"
+		(property "Reference" "Vcap1"
 			(at 28.448 120.142 0)
 			(effects
@@
 			(project "PS-ChargerInterfacePCB"
 				(path "/d45494af-ff47-4110-bed2-dd613b557244/ac7656e7-8ca1-4189-8850-b703de13aef3"
-					(reference "TP_Vcap2")
+					(reference "Vcap2")
 					(unit 1)
 				)
 				(path "/d45494af-ff47-4110-bed2-dd613b557244/f4ec1410-3a5f-45f2-a31b-30d8be6fbeab"
-					(reference "TP_Vcap1")
-					(unit 1)
-				)
+					(reference "Vcap1")
+					(unit 1)
+				)

Commit message: Layout again yes
Parts:
- Z2: P/N (none) -> SMAF4758A-TP
Changed lines of the file:
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@@
+			)
+		)
+		(property "P/N" "SMAF4758A-TP"
+			(at 33.02 69.85 90)
+			(effects
+				(font
+					(size 1.27 1.27)
+				)
+				(hide yes)
 			)
 		)

Commit message: Geber + BOM
Parts:
- Gate1, OV1, TP_FETConn1, Vcap1: footprint TestPoint:TestPoint_Pad_D1.5mm -> TestPoint:TestPoint_THTPad_D1.5mm_Drill0.7mm
- RPP_EN1: footprint UTSVT_Special:TestPoint_HEX_3mmID -> TestPoint:TestPoint_THTPad_D3.0mm_Drill1.5mm
- Z2: footprint SODFL5026X125N -> UTSVT_Passives:SODFL5026X125N
Changed lines of the file:
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@@
 			)
 		)
-		(property "Footprint" "TestPoint:TestPoint_Pad_D1.5mm"
+		(property "Footprint" "TestPoint:TestPoint_THTPad_D1.5mm_Drill0.7mm"
 			(at 20.32 99.06 0)
 			(effects
@@
 			)
 		)
-		(property "Footprint" "TestPoint:TestPoint_Pad_D1.5mm"
+		(property "Footprint" "TestPoint:TestPoint_THTPad_D1.5mm_Drill0.7mm"
 			(at 71.12 50.8 0)
 			(effects
@@
 			)
 		)
-		(property "Footprint" "TestPoint:TestPoint_Pad_D1.5mm"
+		(property "Footprint" "TestPoint:TestPoint_THTPad_D1.5mm_Drill0.7mm"
 			(at 33.02 114.3 0)
 			(effects
@@
 			)
 		)
-		(property "Footprint" "UTSVT_Special:TestPoint_HEX_3mmID"
+		(property "Footprint" "TestPoint:TestPoint_THTPad_D3.0mm_Drill1.5mm"
 			(at 30.48 99.06 0)
 			(effects
@@
 			)
 		)
-		(property "Footprint" "TestPoint:TestPoint_Pad_D1.5mm"
+		(property "Footprint" "TestPoint:TestPoint_THTPad_D1.5mm_Drill0.7mm"
 			(at 20.32 114.3 0)
 			(effects
@@
 			)
 		)
-		(property "Footprint" "SODFL5026X125N"
+		(property "Footprint" "UTSVT_Passives:SODFL5026X125N"
 			(at -60.63 80.01 0)
 			(effects
