File: Hardware/12V-24VBoostConverter.kicad_sch (KiCad schematic)
At the start: 26 parts, among them IC1 TPS613771RYHR, U2 3568

Commit message: saving changes
Parts:
- added TP_BOOT1: TestPoint, UTSVT_Special:TestPoint_HEX_3mmID, symbol Connector:TestPoint
- R6: P/N CRCW060310K0FKEI -> CRCW060310K0FKEI
- U2: value 3568 -> 4A; footprint 3568 -> 3568:3568
- renumbered TP_FB to TP_FB1, TP_ILIM to TP_ILIM1, TP_IN to TP_IN1, TP_OUT to TP_OUT1, TP_SW to TP_SW2, TP_VCC to TP_VCC1
Connections:
- net BOOT: now reaches C5.2, IC1.13 (BOOT)
- net BOOT: now also TP_BOOT1.1

Commit message: layout ready
Parts:
- TP_BOOT1, TP_COMP1, TP_FB1, TP_ILIM1, TP_SW1, TP_SW2, TP_VCC1: footprint UTSVT_Special:TestPoint_HEX_3mmID -> TestPoint:TestPoint_Pad_D1.5mm
Changed lines of the file:
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@@
 			)
 		)
-		(property "Footprint" "UTSVT_Special:TestPoint_HEX_3mmID"
+		(property "Footprint" "TestPoint:TestPoint_Pad_D1.5mm"
 			(at 33.02 78.74 0)
 			(effects
@@
 			)
 		)
-		(property "Footprint" "UTSVT_Special:TestPoint_HEX_3mmID"
+		(property "Footprint" "TestPoint:TestPoint_Pad_D1.5mm"
 			(at 34.29 93.98 0)
 			(effects
@@
 			)
 		)
-		(property "Footprint" "UTSVT_Special:TestPoint_HEX_3mmID"
+		(property "Footprint" "TestPoint:TestPoint_Pad_D1.5mm"
 			(at 22.86 127 0)
 			(effects
@@
 			)
 		)
-		(property "Footprint" "UTSVT_Special:TestPoint_HEX_3mmID"
+		(property "Footprint" "TestPoint:TestPoint_Pad_D1.5mm"
 			(at 44.45 78.74 0)
 			(effects
@@
 			)
 		)
-		(property "Footprint" "UTSVT_Special:TestPoint_HEX_3mmID"
+		(property "Footprint" "TestPoint:TestPoint_Pad_D1.5mm"
 			(at 22.86 93.98 0)
 			(effects
@@
 			)
 		)
-		(property "Footprint" "UTSVT_Special:TestPoint_HEX_3mmID"
+		(property "Footprint" "TestPoint:TestPoint_Pad_D1.5mm"
 			(at 21.59 110.49 0)
 			(effects
@@
 			)
 		)
-		(property "Footprint" "UTSVT_Special:TestPoint_HEX_3mmID"
+		(property "Footprint" "TestPoint:TestPoint_Pad_D1.5mm"
 			(at 45.72 93.98 0)
 			(effects

Commit message: Layout again
Parts:
- renumbered TP_IN1 to +14V2, TP_OUT1 to 24V_OUT1, TP_BOOT1 to BOOT1, TP_COMP1 to COMP1, TP_SW1 to EN/UVLO1, TP_FB1 to FB1, TP_ILIM1 to ILIM1, TP_SW2 to SW1, TP_VCC1 to VCC1
Connections:
- net PostL1 renamed SW
Changed lines of the file:
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@@
 		)
 	)
-	(label "PostL1"
+	(label "SW"
 		(at 38.1 72.39 180)
 		(effects
@@
 		)
 	)
-	(label "PostL1"
+	(label "SW"
 		(at 95.25 29.21 90)
 		(effects
@@
 		(on_board yes)
 		(dnp no)
-		(property "Reference" "TP_SW2"
-			(at 40.132 84.582 0)
+		(property "Reference" "SW1"
+			(at 39.116 84.582 0)
 			(effects
 				(font
@@
 			(project "PS-ChargerInterfacePCB"
 				(path "/d45494af-ff47-4110-bed2-dd613b557244/a5946dd4-2cac-491d-9b85-f213ab9011e7"
-					(reference "TP_SW2")
+					(reference "SW1")
 					(unit 1)
 				)
@@
 		(on_board yes)
 		(dnp no)
-		(property "Reference" "TP_ILIM1"
-			(at 43.18 99.822 0)
+		(property "Reference" "ILIM1"
+			(at 41.402 99.568 0)
 			(effects
 				(font
@@
 			(project "PS-ChargerInterfacePCB"
 				(path "/d45494af-ff47-4110-bed2-dd613b557244/a5946dd4-2cac-491d-9b85-f213ab9011e7"
-					(reference "TP_ILIM1")
+					(reference "ILIM1")
 					(unit 1)
 				)
@@
 		(on_board yes)
 		(dnp no)
-		(property "Reference" "TP_BOOT1"
+		(property "Reference" "BOOT1"
 			(at 29.972 132.842 0)
 			(effects
@@
 			(project "PS-ChargerInterfacePCB"
 				(path "/d45494af-ff47-4110-bed2-dd613b557244/a5946dd4-2cac-491d-9b85-f213ab9011e7"
-					(reference "TP_BOOT1")
+					(reference "BOOT1")
 					(unit 1)
 				)
@@
 		(on_board yes)
 		(dnp no)
-		(property "Reference" "TP_OUT1"
+		(property "Reference" "24V_OUT1"
 			(at 43.18 116.332 0)
 			(effects
@@
 			(project "PS-ChargerInterfacePCB"
 				(path "/d45494af-ff47-4110-bed2-dd613b557244/a5946dd4-2cac-491d-9b85-f213ab9011e7"
-					(reference "TP_OUT1")
+					(reference "24V_OUT1")
 					(unit 1)
 				)
@@
 		(on_board yes)
 		(dnp no)
-		(property "Reference" "TP_IN1"
-			(at 30.988 84.582 0)
+		(property "Reference" "+14V2"
+			(at 28.702 84.582 0)
 			(effects
 				(font
@@
 			(project "PS-ChargerInterfacePCB"
 				(path "/d45494af-ff47-4110-bed2-dd613b557244/a5946dd4-2cac-491d-9b85-f213ab9011e7"
-					(reference "TP_IN1")
+					(reference "+14V2")
 					(unit 1)
 				)
@@
 		(on_board yes)
 		(dnp no)
-		(property "Reference" "TP_SW1"
+		(property "Reference" "EN/UVLO1"
 			(at 51.562 84.582 0)
 			(effects
@@
 			(project "PS-ChargerInterfacePCB"
 				(path "/d45494af-ff47-4110-bed2-dd613b557244/a5946dd4-2cac-491d-9b85-f213ab9011e7"
-					(reference "TP_SW1")
+					(reference "EN/UVLO1")
 					(unit 1)
 				)
@@
 		(on_board yes)
 		(dnp no)
-		(property "Reference" "TP_COMP1"
-			(at 31.75 99.822 0)
+		(property "Reference" "COMP1"
+			(at 30.226 100.076 0)
 			(effects
 				(font
@@
 			(project "PS-ChargerInterfacePCB"
 				(path "/d45494af-ff47-4110-bed2-dd613b557244/a5946dd4-2cac-491d-9b85-f213ab9011e7"
-					(reference "TP_COMP1")
+					(reference "COMP1")
 					(unit 1)
 				)
@@
 		(on_board yes)
 		(dnp no)
-		(property "Reference" "TP_FB1"
-			(at 30.48 116.332 0)
+		(property "Reference" "FB1"
+			(at 27.432 116.078 0)
 			(effects
 				(font
@@
 			(project "PS-ChargerInterfacePCB"
 				(path "/d45494af-ff47-4110-bed2-dd613b557244/a5946dd4-2cac-491d-9b85-f213ab9011e7"
-					(reference "TP_FB1")
+					(reference "FB1")
 					(unit 1)
 				)
@@
 		(on_board yes)
 		(dnp no)
-		(property "Reference" "TP_VCC1"
-			(at 54.61 99.822 0)
+		(property "Reference" "VCC1"
+			(at 52.578 99.822 0)
 			(effects
 				(font
@@
 			(project "PS-ChargerInterfacePCB"
 				(path "/d45494af-ff47-4110-bed2-dd613b557244/a5946dd4-2cac-491d-9b85-f213ab9011e7"
-					(reference "TP_VCC1")
+					(reference "VCC1")
 					(unit 1)
 				)

Commit message: Geber + BOM
Parts:
- +14V2, 24V_OUT1: footprint UTSVT_Special:TestPoint_HEX_3mmID -> TestPoint:TestPoint_THTPad_D3.0mm_Drill1.5mm
- BOOT1, COMP1, EN/UVLO1, FB1, ILIM1, SW1, VCC1: footprint TestPoint:TestPoint_Pad_D1.5mm -> TestPoint:TestPoint_THTPad_D1.5mm_Drill0.7mm
- C4: P/N GCJ188R71E222KA01D -> 0603B222K500NT
Changed lines of the file:
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@@
 			)
 		)
-		(property "P/N" "GCJ188R71E222KA01D"
+		(property "P/N" "0603B222K500NT"
 			(at 97.79 82.55 0)
 			(effects
@@
 			)
 		)
-		(property "Footprint" "TestPoint:TestPoint_Pad_D1.5mm"
+		(property "Footprint" "TestPoint:TestPoint_THTPad_D1.5mm_Drill0.7mm"
 			(at 33.02 78.74 0)
 			(effects
@@
 			)
 		)
-		(property "Footprint" "TestPoint:TestPoint_Pad_D1.5mm"
+		(property "Footprint" "TestPoint:TestPoint_THTPad_D1.5mm_Drill0.7mm"
 			(at 34.29 93.98 0)
 			(effects
@@
 			)
 		)
-		(property "Footprint" "TestPoint:TestPoint_Pad_D1.5mm"
+		(property "Footprint" "TestPoint:TestPoint_THTPad_D1.5mm_Drill0.7mm"
 			(at 22.86 127 0)
 			(effects
@@
 			)
 		)
-		(property "Footprint" "UTSVT_Special:TestPoint_HEX_3mmID"
+		(property "Footprint" "TestPoint:TestPoint_THTPad_D3.0mm_Drill1.5mm"
 			(at 34.29 110.49 0)
 			(effects
@@
 			)
 		)
-		(property "Footprint" "UTSVT_Special:TestPoint_HEX_3mmID"
+		(property "Footprint" "TestPoint:TestPoint_THTPad_D3.0mm_Drill1.5mm"
 			(at 22.86 78.74 0)
 			(effects
@@
 			)
 		)
-		(property "Footprint" "TestPoint:TestPoint_Pad_D1.5mm"
+		(property "Footprint" "TestPoint:TestPoint_THTPad_D1.5mm_Drill0.7mm"
 			(at 44.45 78.74 0)
 			(effects
@@
 			)
 		)
-		(property "Footprint" "TestPoint:TestPoint_Pad_D1.5mm"
+		(property "Footprint" "TestPoint:TestPoint_THTPad_D1.5mm_Drill0.7mm"
 			(at 22.86 93.98 0)
 			(effects
@@
 			)
 		)
-		(property "Footprint" "TestPoint:TestPoint_Pad_D1.5mm"
+		(property "Footprint" "TestPoint:TestPoint_THTPad_D1.5mm_Drill0.7mm"
 			(at 21.59 110.49 0)
 			(effects
@@
 			)
 		)
-		(property "Footprint" "TestPoint:TestPoint_Pad_D1.5mm"
+		(property "Footprint" "TestPoint:TestPoint_THTPad_D1.5mm_Drill0.7mm"
 			(at 45.72 93.98 0)
 			(effects

Commit message: Cleaned up Branch
Parts:
- L1: footprint XGL4020-472MEC:IND_XGL4020_COC -> External Parts Mod:XGL4020_COC
Changed lines of the file:
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@@
 			)
 		)
-		(property "Footprint" "XGL4020-472MEC:IND_XGL4020_COC"
+		(property "Footprint" "External Parts Mod:XGL4020_COC"
 			(at 90.17 29.21 0)
 			(effects

Commit message: Updated sym/mod folder names
Parts:
- L1: footprint External Parts Mod:XGL4020_COC -> charger_parts:XGL4020_COC
Changed lines of the file:
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@@
 			)
 		)
-		(property "Footprint" "External Parts Mod:XGL4020_COC"
+		(property "Footprint" "charger_parts:XGL4020_COC"
 			(at 90.17 29.21 0)
 			(effects
