File: Hardware/Buzzer.kicad_sch (KiCad schematic)
At the start: 7 parts, among them J4 PWM TP, J6 BuzzConn, Q8 IRLML0030TRPBF

Commit message: saving changes
Parts:
- J4: footprint CONN_SD-42375-001_M240_03_MOL -> 22284030:CONN_SD-42375-001_M240_03_MOL; P/N (none) -> 22-28-4030
- J6: P/N 1053091202 -> 105309-1202
- Q8: footprint SOT95P237X112-3N -> IRLML0030TRPBF:SOT95P237X112-3N; P/N (none) -> IRLML0030TRPBF:SOT95P237X112-3N
Changed lines of the file:
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@@
+			)
+		)
+		(property "Part #" ""
+			(at 53.34 64.77 0)
+			(effects
+				(font
+					(size 1.27 1.27)
+				)
+				(hide yes)
+			)
+		)
+		(property "Sim.Pins" ""
+			(at 53.34 64.77 0)
+			(effects
+				(font
+					(size 1.27 1.27)
+				)
+				(hide yes)
 			)
 		)
@@
 			)
 		)
+		(property "Part #" ""
+			(at 92.71 35.56 0)
+			(effects
+				(font
+					(size 1.27 1.27)
+				)
+				(hide yes)
+			)
+		)
+		(property "Sim.Pins" ""
+			(at 92.71 35.56 0)
+			(effects
+				(font
+					(size 1.27 1.27)
+				)
+				(hide yes)
+			)
+		)
 		(pin "2"
 		)
@@
 			)
 		)
-		(property "Footprint" "CONN_SD-42375-001_M240_03_MOL"
+		(property "Footprint" "22284030:CONN_SD-42375-001_M240_03_MOL"
 			(at 38.1 26.67 0)
 			(effects
@@
 		)
 		(property "Description" ""
+			(at 38.1 26.67 0)
+			(effects
+				(font
+					(size 1.27 1.27)
+				)
+				(hide yes)
+			)
+		)
+		(property "Part #" ""
+			(at 38.1 26.67 0)
+			(effects
+				(font
+					(size 1.27 1.27)
+				)
+				(hide yes)
+			)
+		)
+		(property "Sim.Pins" ""
+			(at 38.1 26.67 0)
+			(effects
+				(font
+					(size 1.27 1.27)
+				)
+				(hide yes)
+			)
+		)
+		(property "P/N" "22-28-4030"
 			(at 38.1 26.67 0)
 			(effects
@@
 			)
 		)
+		(property "Part #" ""
+			(at 105.41 35.56 0)
+			(effects
+				(font
+					(size 1.27 1.27)
+				)
+				(hide yes)
+			)
+		)
+		(property "Sim.Pins" ""
+			(at 105.41 35.56 0)
+			(effects
+				(font
+					(size 1.27 1.27)
+				)
+				(hide yes)
+			)
+		)
 		(pin "2"
 		)
@@
 			)
 		)
+		(property "Part #" ""
+			(at 121.92 49.53 90)
+			(effects
+				(font
+					(size 1.27 1.27)
+				)
+				(hide yes)
+			)
+		)
+		(property "Sim.Pins" ""
+			(at 121.92 49.53 90)
+			(effects
+				(font
+					(size 1.27 1.27)
+				)
+				(hide yes)
+			)
+		)
 		(pin "1"
 		)
@@
 			)
 		)
-		(property "P/N" "1053091202"
+		(property "P/N" "105309-1202"
+			(at 135.89 49.53 0)
+			(effects
+				(font
+					(size 1.27 1.27)
+				)
+				(hide yes)
+			)
+		)
+		(property "Part #" ""
+			(at 135.89 49.53 0)
+			(effects
+				(font
+					(size 1.27 1.27)
+				)
+				(hide yes)
+			)
+		)
+		(property "Sim.Pins" ""
 			(at 135.89 49.53 0)
 			(effects
@@
 			)
 		)
-		(property "Footprint" "SOT95P237X112-3N"
+		(property "Footprint" "IRLML0030TRPBF:SOT95P237X112-3N"
 			(at 95.25 148.26 0)
 			(effects
@@
 				(hide yes)
 			)
+		)
+		(property "Part #" ""
+			(at 78.74 53.34 0)
+			(effects
+				(font
+					(size 1.27 1.27)
+				)
+				(hide yes)
+			)
+		)
+		(property "Sim.Pins" ""
+			(at 78.74 53.34 0)
+			(effects
+				(font
+					(size 1.27 1.27)
+				)
+				(hide yes)
+			)
+		)
+		(property "P/N" "IRLML0030TRPBF:SOT95P237X112-3N"
+			(at 78.74 53.34 0)
+			(effects
+				(font
+					(size 1.27 1.27)
+				)
+				(hide yes)
+			)

Commit message: layout ready
Parts:
- removed J4: PWM TP, 22284030:CONN_SD-42375-001_M240_03_MOL, symbol 0022284030:22284030
Changed lines of the file:
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@@
-	(wire
-		(pts
-			(xy 25.4 29.21) (xy 38.1 29.21)
-		)
-		(stroke
-			(width 0)
-			(type default)
-		)
-	)
 	(wire
 		(pts
@@
 	(wire
 		(pts
-			(xy 35.56 31.75) (xy 38.1 31.75)
-		)
-		(stroke
-			(width 0)
-			(type default)
-		)
-	)
-	(wire
-		(pts
 			(xy 121.92 45.72) (xy 125.73 45.72)
 		)
@@
 		(pts
 			(xy 106.68 53.34) (xy 121.92 53.34)
-		)
-		(stroke
-			(width 0)
-			(type default)
-		)
-	)
-	(wire
-		(pts
-			(xy 25.4 26.67) (xy 38.1 26.67)
 		)
 		(stroke
@@
 		)
 	)
-	(label "Buzz_Source"
-		(at 25.4 26.67 0)
-		(effects
-			(font
-				(size 1.27 1.27)
-			)
-			(justify left bottom)
-		)
-	)
-	(label "Buzz_Drain"
-		(at 25.4 29.21 0)
-		(effects
-			(font
-				(size 1.27 1.27)
-			)
-			(justify left bottom)
-		)
-	)
 	(hierarchical_label "BuzzPWM"
 		(shape input)
 		(at 39.37 57.15 180)
-		(effects
-			(font
-				(size 1.27 1.27)
-			)
-			(justify right)
-		)
-	)
-	(hierarchical_label "BuzzPWM"
-		(shape input)
-		(at 35.56 31.75 180)
 		(effects
 			(font
@@
 					(unit 1)
 				)
-			)
-		)
-	)
-	(symbol
-		(lib_id "0022284030:22284030")
-		(at 38.1 26.67 0)
-		(unit 1)
-		(exclude_from_sim no)
-		(in_bom yes)
-		(on_board yes)
-		(dnp no)
-		(fields_autoplaced yes)
-		(property "Reference" "J4"
-			(at 52.07 27.9399 0)
-			(effects
-				(font
-					(size 1.524 1.524)
-				)
-				(justify left)
-			)
-		)
-		(property "Value" "PWM TP"
-			(at 52.07 30.4799 0)
-			(effects
-				(font
-					(size 1.524 1.524)
-				)
-				(justify left)
-			)
-		)
-		(property "Footprint" "22284030:CONN_SD-42375-001_M240_03_MOL"
-			(at 38.1 26.67 0)
-			(effects
-				(font
-					(size 1.27 1.27)
-					(italic yes)
-				)
-				(hide yes)
-			)
-		)
-		(property "Datasheet" "https://www.molex.com/en-us/products/part-detail-pdf/22284030?display=pdf"
-			(at 38.1 26.67 0)
-			(effects
-				(font
-					(size 1.27 1.27)
-					(italic yes)
-				)
-				(hide yes)
-			)
-		)
-		(property "Description" ""
-			(at 38.1 26.67 0)
-			(effects
-				(font
-					(size 1.27 1.27)
-				)
-				(hide yes)
-			)
-		)
-		(property "Part #" ""
-			(at 38.1 26.67 0)
-			(effects
-				(font
-					(size 1.27 1.27)
-				)
-				(hide yes)
-			)
-		)
-		(property "Sim.Pins" ""
-			(at 38.1 26.67 0)
-			(effects
-				(font
-					(size 1.27 1.27)
-				)
-				(hide yes)
-			)
-		)
-		(property "P/N" "22-28-4030"
-			(at 38.1 26.67 0)
-			(effects
-				(font
-					(size 1.27 1.27)
-				)
-				(hide yes)
-			)
-		)
-		(pin "1"
-		)
-		(pin "2"
-		)
-		(pin "3"
-		)
-		(instances
-			(project ""
-				(path "/d45494af-ff47-4110-bed2-dd613b557244/5a3494bd-2769-4cc7-96c1-4c8c29abb5e6"
-					(reference "J4")
-					(unit 1)
-				)

Commit message: Layout again
Parts:
- removed D2: D_Schottky, SK32A_LTP:SDO_DO-214AC-SMA_MCE, symbol Device:D_Schottky
- added D11: 1N5819HW-7-F, SOD3716X145N, symbol Device:D_Schottky
- renumbered J6 to Buzzer1
Connections:
- net +14V: now also D11.1 (K)
- net Buzz_Drain: now also D11.2 (A)
Changed lines of the file:
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@@
 	)
 	(junction
-		(at 121.92 53.34)
+		(at 120.65 53.34)
+		(diameter 0)
+		(color 0 0 0 0)
+	)
+	(junction
+		(at 120.65 45.72)
 		(diameter 0)
 		(color 0 0 0 0)
@@
 	)
 	(junction
-		(at 121.92 45.72)
-		(diameter 0)
-		(color 0 0 0 0)
-	)
-	(junction
 		(at 92.71 39.37)
 		(diameter 0)
@@
 	(wire
 		(pts
-			(xy 121.92 53.34) (xy 125.73 53.34)
-		)
-		(stroke
-			(width 0)
-			(type default)
-		)
-	)
-	(wire
-		(pts
 			(xy 125.73 45.72) (xy 125.73 49.53)
 		)
@@
 	(wire
 		(pts
+			(xy 120.65 45.72) (xy 125.73 45.72)
+		)
+		(stroke
+			(width 0)
+			(type default)
+		)
+	)
+	(wire
+		(pts
 			(xy 105.41 31.75) (xy 92.71 31.75)
 		)
@@
 	(wire
 		(pts
-			(xy 121.92 45.72) (xy 125.73 45.72)
-		)
-		(stroke
-			(width 0)
-			(type default)
-		)
-	)
-	(wire
-		(pts
-			(xy 106.68 53.34) (xy 121.92 53.34)
-		)
-		(stroke
-			(width 0)
-			(type default)
-		)
-	)
-	(wire
-		(pts
-			(xy 115.57 45.72) (xy 121.92 45.72)
+			(xy 115.57 45.72) (xy 120.65 45.72)
+		)
+		(stroke
+			(width 0)
+			(type default)
+		)
+	)
+	(wire
+		(pts
+			(xy 106.68 53.34) (xy 120.65 53.34)
 		)
 		(stroke
@@
 		(pts
 			(xy 92.71 39.37) (xy 92.71 40.64)
+		)
+		(stroke
+			(width 0)
+			(type default)
+		)
+	)
+	(wire
+		(pts
+			(xy 120.65 53.34) (xy 125.73 53.34)
 		)
 		(stroke
@@
 	)
 	(symbol
+		(lib_name "D_Schottky_1")
+		(lib_id "Device:D_Schottky")
+		(at 120.65 49.53 270)
+		(unit 1)
+		(exclude_from_sim no)
+		(in_bom yes)
+		(on_board yes)
+		(dnp no)
+		(property "Reference" "D11"
+			(at 119.126 55.118 90)
+			(effects
+				(font
+					(size 1.27 1.27)
+				)
+				(justify left)
+			)
+		)
+		(property "Value" "1N5819HW-7-F"
+			(at 119.126 57.404 90)
+			(effects
+				(font
+					(size 1.27 1.27)
+				)
+				(justify left)
+			)
+		)
+		(property "Footprint" "SOD3716X145N"
+			(at 23.19 60.96 0)
+			(effects
+				(font
+					(size 1.27 1.27)
+				)
+				(justify left top)
+				(hide yes)
+			)
+		)
+		(property "Datasheet" "https://www.diodes.com//assets/Datasheets/1N5819HW.pdf"
+			(at -76.81 60.96 0)
+			(effects
+				(font
+					(size 1.27 1.27)
+				)
+				(justify left top)
+				(hide yes)
+			)
+		)
+		(property "Description" "Diode Schottky 1A 40V SOD123 Diodes Inc 1N5819HW-7-F, SMT Schottky Diode, 40V 1A, 2-Pin SOD-123"
+			(at 120.65 49.53 0)
+			(effects
+				(font
+					(size 1.27 1.27)
+				)
+				(hide yes)
+			)
+		)
+		(property "Height" "1.45"
+			(at -276.81 60.96 0)
+			(effects
+				(font
+					(size 1.27 1.27)
+				)
+				(justify left top)
+				(hide yes)
+			)
+		)
+		(property "Mouser Part Number" "621-1N5819HW-F"
+			(at -376.81 60.96 0)
+			(effects
+				(font
+					(size 1.27 1.27)
+				)
+				(justify left top)
+				(hide yes)
+			)
+		)
+		(property "Mouser Price/Stock" "https://www.mouser.co.uk/ProductDetail/Diodes-Incorporated/1N5819HW-7-F?qs=NQ47qNm99eDyWTEd07miYA%3D%3D"
+			(at -476.81 60.96 0)
+			(effects
+				(font
+					(size 1.27 1.27)
+				)
+				(justify left top)
+				(hide yes)
+			)
+		)
+		(property "Manufacturer_Name" "Diodes Incorporated"
+			(at -576.81 60.96 0)
+			(effects
+				(font
+					(size 1.27 1.27)
+				)
+				(justify left top)
+				(hide yes)
+			)
+		)
+		(property "Manufacturer_Part_Number" "1N5819HW-7-F"
+			(at -676.81 60.96 0)
+			(effects
+				(font
+					(size 1.27 1.27)
+				)
+				(justify left top)
+				(hide yes)
+			)
+		)
+		(pin "2"
+		)
+		(pin "1"
+		)
+		(instances
+			(project ""
+				(path "/d45494af-ff47-4110-bed2-dd613b557244/5a3494bd-2769-4cc7-96c1-4c8c29abb5e6"
+					(reference "D11")
+					(unit 1)
+				)
+			)
+		)
+	)
+	(symbol
 		(lib_id "Device:C")
 		(at 92.71 35.56 0)
@@
 	)
 	(symbol
-		(lib_id "Device:D_Schottky")
-		(at 121.92 49.53 90)
-		(mirror x)
-		(unit 1)
-		(exclude_from_sim no)
-		(in_bom yes)
-		(on_board yes)
-		(dnp no)
-		(property "Reference" "D2"
-			(at 121.92 41.91 90)
-			(effects
-				(font
-					(size 1.27 1.27)
-				)
-			)
-		)
-		(property "Value" "D_Schottky"
-			(at 121.92 43.688 90)
-			(effects
-				(font
-					(size 1.27 1.27)
-				)
-			)
-		)
-		(property "Footprint" "SK32A_LTP:SDO_DO-214AC-SMA_MCE"
-			(at 121.92 49.53 0)
-			(effects
-				(font
-					(size 1.27 1.27)
-				)
-				(hide yes)
-			)
-		)
-		(property "Datasheet" "https://www.mouser.com/datasheet/3/225/1/SK32A-L-SK310A-L(SMA).pdf"
-			(at 121.92 49.53 0)
-			(effects
-				(font
-					(size 1.27 1.27)
-				)
-				(hide yes)
-			)
-		)
-		(property "Description" "Schottky diode"
-			(at 121.92 49.53 0)
-			(effects
-				(font
-					(size 1.27 1.27)
-				)
-				(hide yes)
-			)
-		)
-		(property "MANUFACTURER" ""
-			(at 121.92 49.53 0)
-			(effects
-				(font
-					(size 1.27 1.27)
-				)
-				(hide yes)
-			)
-		)
-		(property "PARTREV" ""
-			(at 121.92 49.53 0)
-			(effects
-				(font
-					(size 1.27 1.27)
-				)
-				(hide yes)
-			)
-		)
-		(property "STANDARD" ""
-			(at 121.92 49.53 0)
-			(effects
-				(font
-					(size 1.27 1.27)
-				)
-				(hide yes)
-			)
-		)
-		(property "Distrbutor Link" "https://www.mouser.com/ProductDetail/Micro-Commercial-Components-MCC/SK32A-LTP?qs=JeAkOuORR2U5XhGW5SLK2g%3D%3D&srsltid=AfmBOoqFiyx6irMBt28Q3Vo65pAmn7yAO98wOsjACKNj2Ab_fSU83u8p"
-			(at 121.92 49.53 90)
-			(effects
-				(font
-					(size 1.27 1.27)
-				)
-				(hide yes)
-			)
-		)
-		(property "Manufacturer" "Micro Commercial Components (MCC)"
-			(at 121.92 49.53 90)
-			(effects
-				(font
-					(size 1.27 1.27)
-				)
-				(hide yes)
-			)
-		)
-		(property "P/N" "SK32A-LTP"
-			(at 121.92 49.53 90)
-			(effects
-				(font
-					(size 1.27 1.27)
-				)
-				(hide yes)
-			)
-		)
-		(property "Part #" ""
-			(at 121.92 49.53 90)
-			(effects
-				(font
-					(size 1.27 1.27)
-				)
-				(hide yes)
-			)
-		)
-		(property "Sim.Pins" ""
-			(at 121.92 49.53 90)
-			(effects
-				(font
-					(size 1.27 1.27)
-				)
-				(hide yes)
-			)
-		)
-		(pin "1"
-		)
-		(pin "2"
-		)
-		(instances
-			(project "PS-ChargerInterfacePCB"
-				(path "/d45494af-ff47-4110-bed2-dd613b557244/5a3494bd-2769-4cc7-96c1-4c8c29abb5e6"
-					(reference "D2")
-					(unit 1)
-				)
-			)
-		)
-	)
-	(symbol
 		(lib_id "Connector_Generic:Conn_01x02")
 		(at 135.89 49.53 0)
@@
 		(on_board yes)
 		(dnp no)
-		(property "Reference" "J6"
+		(property "Reference" "Buzzer1"
 			(at 135.89 43.18 0)
 			(effects
@@
 			(project "PS-ChargerInterfacePCB"
 				(path "/d45494af-ff47-4110-bed2-dd613b557244/5a3494bd-2769-4cc7-96c1-4c8c29abb5e6"
-					(reference "J6")
+					(reference "Buzzer1")
 					(unit 1)
 				)

Commit message: Layout again yes
Parts:
- D11: P/N (none) -> 1N5819HW-7-F
Changed lines of the file:
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@@
+			)
+		)
+		(property "P/N" "1N5819HW-7-F"
+			(at 120.65 49.53 90)
+			(effects
+				(font
+					(size 1.27 1.27)
+				)
+				(hide yes)
 			)
 		)

Commit message: last changes + silkscreen
Parts:
- Buzzer1: footprint 153091202:1053091202 -> UTSVT_Connectors:Molex_Nano-Fit_105309-xx02_1x02_P2.50mm_Vertical
Changed lines of the file:
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@@
 			)
 		)
-		(property "Footprint" "153091202:1053091202"
+		(property "Footprint" "UTSVT_Connectors:Molex_Nano-Fit_105309-xx02_1x02_P2.50mm_Vertical"
 			(at 135.89 49.53 0)
 			(effects

Commit message: Cleaned up Branch
Parts:
- D11: footprint SOD3716X145N -> External Parts Mod:1N5819HW-7-F
- Q8: footprint IRLML0030TRPBF:SOT95P237X112-3N -> External Parts Mod:IRLML0030TRPBF
Changed lines of the file:
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@@
 			)
 		)
-		(property "Footprint" "SOD3716X145N"
+		(property "Footprint" "External Parts Mod:1N5819HW-7-F"
 			(at 23.19 60.96 0)
 			(effects
@@
 			)
 		)
-		(property "Footprint" "IRLML0030TRPBF:SOT95P237X112-3N"
+		(property "Footprint" "External Parts Mod:IRLML0030TRPBF"
 			(at 95.25 148.26 0)
 			(effects

Commit message: Updated sym/mod folder names
Parts:
- D11: footprint External Parts Mod:1N5819HW-7-F -> charger_parts:1N5819HW-7-F
- Q8: footprint External Parts Mod:IRLML0030TRPBF -> charger_parts:IRLML0030TRPBF
Changed lines of the file:
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@@
 			)
 		)
-		(property "Footprint" "External Parts Mod:1N5819HW-7-F"
+		(property "Footprint" "charger_parts:1N5819HW-7-F"
 			(at 23.19 60.96 0)
 			(effects
@@
 			)
 		)
-		(property "Footprint" "External Parts Mod:IRLML0030TRPBF"
+		(property "Footprint" "charger_parts:IRLML0030TRPBF"
 			(at 95.25 148.26 0)
 			(effects
