File: Hardware/EVCharger.kicad_sch (KiCad schematic)
At the start: 11 parts

Commit message: saving changes
Parts:
- removed JP1: SolderJumper_2_Open, symbol Jumper:SolderJumper_2_Open
- C13: footprint (none) -> Capacitor_SMD:C_0805_2012Metric; Distrbutor Link (none) -> https://www.mouser.com/ProductDetail/KYOCERA-AVX/08055D475K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; P/N (none) -> 08055D475KAT4A
- CR1: footprint CR_10S-M3/I_VIS -> V8PAM10S-M3-I:CR_10S-M3&slash_I_VIS; Distrbutor Link (none) -> https://www.mouser.com/ProductDetail/Vishay-General-Semicon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; P/N (none) -> V8PAM10S-M3/I
- R12: footprint (none) -> Resistor_SMD:R_0603_1608Metric; P/N (none) -> CRCW0603100KFKEE
- R13: footprint (none) -> Resistor_SMD:R_0603_1608Metric; P/N (none) -> CRCW060310K0FKEI
- R21, R23, R24: footprint (none) -> Resistor_SMD:R_0603_1608Metric; P/N (none) -> CRCW06035K10FKEC
- R22, R25: footprint (none) -> Resistor_SMD:R_0603_1608Metric; P/N (none) -> CRCW0603150RFKEC
- R3: footprint (none) -> Resistor_SMD:R_0603_1608Metric; P/N (none) -> CRCW06031K00FKEI
Connections:
- net PP is gone; now on net MCU_PP: R22.2, R23.1, R24.1
- net +3V3 renamed +3.3V

Commit message: layout ready
Parts:
- added TP1, TP2, TP3, TP4: TestPoint, TestPoint:TestPoint_Pad_D1.5mm, symbol Connector:TestPoint
Connections:
- net CP: now also TP1.1
- net MCU_CP: now also TP3.1
- net MCU_PP: now also TP4.1
- net at CR1.1, R12.1, R3.1: now also TP2.1

Commit message: Layout again
Parts:
- removed CR1: V8PAM10S-M3/I, V8PAM10S-M3-I:CR_10S-M3&slash_I_VIS, symbol V8PAM10S-M3-I:V8PAM10S-M3_I
- added D2: 1N5819HW-7-F, SOD3716X145N, symbol Device:D_Schottky
Connections:
- net CP: now also D2.2 (A)
- net at R12.1, R3.1, TP2.1: now also D2.1 (K)
Changed lines of the file:
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@@
+	(wire
+		(pts
+			(xy 44.45 29.21) (xy 49.53 29.21)
+		)
+		(stroke
+			(width 0)
+			(type default)
+		)
+	)
 	(wire
 		(pts
@@
 		(pts
 			(xy 49.53 29.21) (xy 58.42 29.21)
-		)
-		(stroke
-			(width 0)
-			(type default)
-		)
-	)
-	(wire
-		(pts
-			(xy 46.99 29.21) (xy 49.53 29.21)
 		)
 		(stroke
@@
 	)
 	(symbol
+		(lib_id "Device:D_Schottky")
+		(at 40.64 29.21 180)
+		(unit 1)
+		(exclude_from_sim no)
+		(in_bom yes)
+		(on_board yes)
+		(dnp no)
+		(fields_autoplaced yes)
+		(property "Reference" "D2"
+			(at 40.9575 22.86 0)
+			(effects
+				(font
+					(size 1.27 1.27)
+				)
+			)
+		)
+		(property "Value" "1N5819HW-7-F"
+			(at 40.9575 25.4 0)
+			(effects
+				(font
+					(size 1.27 1.27)
+				)
+			)
+		)
+		(property "Footprint" "SOD3716X145N"
+			(at 29.21 -68.25 0)
+			(effects
+				(font
+					(size 1.27 1.27)
+				)
+				(justify left top)
+				(hide yes)
+			)
+		)
+		(property "Datasheet" "https://www.diodes.com//assets/Datasheets/1N5819HW.pdf"
+			(at 29.21 -168.25 0)
+			(effects
+				(font
+					(size 1.27 1.27)
+				)
+				(justify left top)
+				(hide yes)
+			)
+		)
+		(property "Description" "Diode Schottky 1A 40V SOD123 Diodes Inc 1N5819HW-7-F, SMT Schottky Diode, 40V 1A, 2-Pin SOD-123"
+			(at 40.64 29.21 0)
+			(effects
+				(font
+					(size 1.27 1.27)
+				)
+				(hide yes)
+			)
+		)
+		(property "Height" "1.45"
+			(at 29.21 -368.25 0)
+			(effects
+				(font
+					(size 1.27 1.27)
+				)
+				(justify left top)
+				(hide yes)
+			)
+		)
+		(property "Mouser Part Number" "621-1N5819HW-F"
+			(at 29.21 -468.25 0)
+			(effects
+				(font
+					(size 1.27 1.27)
+				)
+				(justify left top)
+				(hide yes)
+			)
+		)
+		(property "Mouser Price/Stock" "https://www.mouser.co.uk/ProductDetail/Diodes-Incorporated/1N5819HW-7-F?qs=NQ47qNm99eDyWTEd07miYA%3D%3D"
+			(at 29.21 -568.25 0)
+			(effects
+				(font
+					(size 1.27 1.27)
+				)
+				(justify left top)
+				(hide yes)
+			)
+		)
+		(property "Manufacturer_Name" "Diodes Incorporated"
+			(at 29.21 -668.25 0)
+			(effects
+				(font
+					(size 1.27 1.27)
+				)
+				(justify left top)
+				(hide yes)
+			)
+		)
+		(property "Manufacturer_Part_Number" "1N5819HW-7-F"
+			(at 29.21 -768.25 0)
+			(effects
+				(font
+					(size 1.27 1.27)
+				)
+				(justify left top)
+				(hide yes)
+			)
+		)
+		(pin "1"
+		)
+		(pin "2"
+		)
+		(instances
+			(project ""
+				(path "/d45494af-ff47-4110-bed2-dd613b557244/ebfb1e9b-212e-4bda-bede-5250a5b1aee3"
+					(reference "D2")
+					(unit 1)
+				)
+			)
+		)
+	)
+	(symbol
 		(lib_id "Connector:TestPoint")
 		(at 29.21 29.21 180)
@@
 					(unit 1)
 				)
-			)
-		)
-	)
-	(symbol
-		(lib_id "V8PAM10S-M3-I:V8PAM10S-M3_I")
-		(at 36.83 29.21 0)
-		(unit 1)
-		(exclude_from_sim no)
-		(in_bom yes)
-		(on_board yes)
-		(dnp no)
-		(fields_autoplaced yes)
-		(property "Reference" "CR1"
-			(at 41.91 22.86 0)
-			(effects
-				(font
-					(size 1.524 1.524)
-				)
-			)
-		)
-		(property "Value" "V8PAM10S-M3/I"
-			(at 41.91 25.4 0)
-			(effects
-				(font
-					(size 1.524 1.524)
-				)
-			)
-		)
-		(property "Footprint" "V8PAM10S-M3-I:CR_10S-M3&slash_I_VIS"
-			(at 36.83 29.21 0)
-			(effects
-				(font
-					(size 1.27 1.27)
-					(italic yes)
-				)
-				(hide yes)
-			)
-		)
-		(property "Datasheet" "https://www.vishay.com/doc?87013"
-			(at 36.83 29.21 0)
-			(effects
-				(font
-					(size 1.27 1.27)
-					(italic yes)
-				)
-				(hide yes)
-			)
-		)
-		(property "Description" ""
-			(at 36.83 29.21 0)
-			(effects
-				(font
-					(size 1.27 1.27)
-				)
-				(hide yes)
-			)
-		)
-		(property "Part #" ""
-			(at 36.83 29.21 0)
-			(effects
-				(font
-					(size 1.27 1.27)
-				)
-				(hide yes)
-			)
-		)
-		(property "Sim.Pins" ""
-			(at 36.83 29.21 0)
-			(effects
-				(font
-					(size 1.27 1.27)
-				)
-				(hide yes)
-			)
-		)
-		(property "P/N" "V8PAM10S-M3/I"
-			(at 36.83 29.21 0)
-			(effects
-				(font
-					(size 1.27 1.27)
-				)
-				(hide yes)
-			)
-		)
-		(property "Distrbutor Link" "https://www.mouser.com/ProductDetail/Vishay-General-Semiconductor/V8PAM10S-M3-I?qs=7MVldsJ5UaxN9yrxRnd0cA%3D%3D"
-			(at 36.83 29.21 0)
-			(effects
-				(font
-					(size 1.27 1.27)
-				)
-				(hide yes)
-			)
-		)
-		(pin "1"
-		)
-		(pin "2"
-		)
-		(instances
-			(project ""
-				(path "/d45494af-ff47-4110-bed2-dd613b557244/ebfb1e9b-212e-4bda-bede-5250a5b1aee3"
-					(reference "CR1")
-					(unit 1)
-				)

Commit message: Layout again yes
Parts:
- D2: P/N (none) -> 1N5819HW-7-F
Changed lines of the file:
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@@
+			)
+		)
+		(property "P/N" "1N5819HW-7-F"
+			(at 40.64 29.21 0)
+			(effects
+				(font
+					(size 1.27 1.27)
+				)
+				(hide yes)
 			)
 		)

Commit message: Geber + BOM
Parts:
- TP1, TP2, TP3, TP4: footprint TestPoint:TestPoint_Pad_D1.5mm -> TestPoint:TestPoint_THTPad_D1.5mm_Drill0.7mm; now left out of the parts list
Changed lines of the file:
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@@
 		(unit 1)
 		(exclude_from_sim no)
-		(in_bom yes)
+		(in_bom no)
 		(on_board yes)
 		(dnp no)
@@
 			)
 		)
-		(property "Footprint" "TestPoint:TestPoint_Pad_D1.5mm"
+		(property "Footprint" "TestPoint:TestPoint_THTPad_D1.5mm_Drill0.7mm"
 			(at 90.17 40.64 0)
 			(effects
@@
 		(unit 1)
 		(exclude_from_sim no)
-		(in_bom yes)
+		(in_bom no)
 		(on_board yes)
 		(dnp no)
@@
 			)
 		)
-		(property "Footprint" "TestPoint:TestPoint_Pad_D1.5mm"
+		(property "Footprint" "TestPoint:TestPoint_THTPad_D1.5mm_Drill0.7mm"
 			(at 44.45 29.21 0)
 			(effects
@@
 		(unit 1)
 		(exclude_from_sim no)
-		(in_bom yes)
+		(in_bom no)
 		(on_board yes)
 		(dnp no)
@@
 			)
 		)
-		(property "Footprint" "TestPoint:TestPoint_Pad_D1.5mm"
+		(property "Footprint" "TestPoint:TestPoint_THTPad_D1.5mm_Drill0.7mm"
 			(at 128.27 38.1 0)
 			(effects
@@
 		(unit 1)
 		(exclude_from_sim no)
-		(in_bom yes)
+		(in_bom no)
 		(on_board yes)
 		(dnp no)
@@
 			)
 		)
-		(property "Footprint" "TestPoint:TestPoint_Pad_D1.5mm"
+		(property "Footprint" "TestPoint:TestPoint_THTPad_D1.5mm_Drill0.7mm"
 			(at 24.13 29.21 0)
 			(effects

Commit message: Cleaned up Branch
Parts:
- D2: footprint SOD3716X145N -> 1N5819HW-7-F:1N5819HW-7-F
Changed lines of the file:
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@@
 			)
 		)
-		(property "Footprint" "SOD3716X145N"
+		(property "Footprint" "1N5819HW-7-F:1N5819HW-7-F"
 			(at 29.21 -68.25 0)
 			(effects

Commit message: Updated sym/mod folder names
Parts:
- D2: footprint 1N5819HW-7-F:1N5819HW-7-F -> charger_parts:1N5819HW-7-F
Changed lines of the file:
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@@
 			)
 		)
-		(property "Footprint" "1N5819HW-7-F:1N5819HW-7-F"
+		(property "Footprint" "charger_parts:1N5819HW-7-F"
 			(at 29.21 -68.25 0)
 			(effects
