File: Hardware/EVCharger.kicad_sch (KiCad schematic)
At the start: 14 parts

Commit message: stuff
Changed lines of the file:
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@@
 	(text "Current draw (worst case)\nI = 3.3/2.2k+220 = 1mA"
 		(exclude_from_sim no)
-		(at 161.798 58.674 0)
+		(at 160.782 59.182 0)
 		(effects
 			(font
@@
 	(text "VPP MCU reading: \n32A cable: ~220Ω \n\nVpp = 3.3 (Rcabel/Rpull up + Rcabel)\nVpp = 3.3 (220/2.2k+220)\nVpp = 0.3V"
 		(exclude_from_sim no)
-		(at 162.306 49.276 0)
+		(at 161.29 49.784 0)
 		(effects
 			(font
