File: Hardware/SPI_display.kicad_sch (KiCad schematic)
At the start: 13 parts

Commit message: Cleaned up Branch
Parts:
- DS1: footprint NHD-C12832A1Z-FSB-FBW-3V3:NHDC12832A1ZFSBFBW3V3 -> External Parts Mod:NHD-C12832A1ZFSBFBW3V3
Changed lines of the file:
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@@
 			)
 		)
-		(property "Footprint" "NHD-C12832A1Z-FSB-FBW-3V3:NHDC12832A1ZFSBFBW3V3"
+		(property "Footprint" "External Parts Mod:NHD-C12832A1ZFSBFBW3V3"
 			(at 95.25 124.13 0)
 			(effects

Commit message: Updated sym/mod folder names
Parts:
- DS1: footprint External Parts Mod:NHD-C12832A1ZFSBFBW3V3 -> charger_parts:NHD-C12832A1ZFSBFBW3V3
Changed lines of the file:
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@@
 			)
 		)
-		(property "Footprint" "External Parts Mod:NHD-C12832A1ZFSBFBW3V3"
+		(property "Footprint" "charger_parts:NHD-C12832A1ZFSBFBW3V3"
 			(at 95.25 124.13 0)
 			(effects
